Commit message: VLP-16 Lidar(not working)

File: urc_gazebo/urdf/walli_prop.xacro (robot description, xacro)
@@ -46,3 +46,12 @@
     <color rgba="0 0 0 1"/>
   </material>
+   <!-- Lidar -->
+    <xacro:property name="lidar_pitch" value="0.0"/>
+    <xacro:property name="lidar_x" value="0.127"/>
+    <xacro:property name="lidar_z" value="0.8486"/>
+    <xacro:property name="lidar_hz" value="10"/>
+    <xacro:property name="lidar_samples" value="500"/>
+    <xacro:property name="lidar_support_x_dim" value="0.2"/>
+    <xacro:property name="lidar_support_y_dim" value="0.08"/>
+    <xacro:property name="lidar_support_z_dim" value="0.01"/>
 </robot>

File: urc_gazebo/urdf/wallii.xacro (robot description, xacro)
@@ -3,4 +3,5 @@
   <xacro:include filename="walli_prop.xacro"/>
   <xacro:include filename="walli_inertials.xacro"/>
+  <xacro:include filename="$(find velodyne_description)/urdf/VLP-16.urdf.xacro"/>
   <!-- The "wheel" macro defines an axle carrier, axle, and wheel. -->
   <xacro:macro name="wheel" params="lr_prefix fr_prefix lr_pos fr_pos">
@@ -176,79 +177,28 @@
             <remapping>~/out:=data</remapping>
           </ros>
-          <initial_orientation_as_reference>false</initial_orientation_as_reference>
+          <frame_name>gps</frame_name>
         </plugin>
         <always_on>true</always_on>
-        <updateRate>100000.0</updateRate>
-        <bodyName>base_link</bodyName>
-        <frameId>gps</frameId>
-        <topicName>/fix</topicName>
-        <velocityTopicName>/fix_velocity</velocityTopicName>
-        <referenceLatitude>33.774497</referenceLatitude>
-        <referenceLongitude>-84.405001</referenceLongitude>
-        <referenceHeading>90</referenceHeading>
-        <referenceAltitude>309.0</referenceAltitude>
-        <drift>0.001 0.001 0.001</drift>
-        <gaussianNoise>0.0001 0.0001 0.0001</gaussianNoise>
-        <velocityDrift>0 0 0</velocityDrift>
-        <velocityGaussianNoise>0.005 0.005 0.05</velocityGaussianNoise>
-    </sensor>
-  </gazebo>
-  <!-- Lidar -->
- <link name="lidar">
-    <visual>
-      <geometry>
-        <box size="0.1 0.1 0.1"/>
-      </geometry>
-    </visual>
-    <collision>
-      <geometry>
-        <box size="0.1 0.1 0.1"/>
-      </geometry>
-    </collision>
-    <xacro:box_inertia m="0.1" w="0.1" d="0.1" h="0.1"/>
-  </link>
-  <joint name="lidar_joint" type="fixed">
-		<axis xyz="1 0 0"/>
-		<origin xyz="0 0 0.05"/>
-		<parent link="base_link"/>
-		<child link="lidar"/>
-	</joint>
-  <gazebo reference="lidar">
-    <sensor name="lidar" type="ray">
-        <always_on>true</always_on>
-        <visualize>false</visualize>
-        <pose>0.0 0 0.0 0 0 0</pose>
-        <update_rate>15</update_rate>
-        <ray>
-          <scan>
-            <horizontal>
-              <samples>667</samples>
-              <resolution>0.54</resolution>
-              <min_angle>0.000000</min_angle>
-              <max_angle>6.280000</max_angle>
-            </horizontal>
-          </scan>
-          <range>
-            <min>0.120000</min>
-            <max>20</max>
-            <resolution>0.54</resolution>
-          </range>
-          <noise>
-            <type>gaussian</type>
-            <mean>0.0</mean>
-            <stddev>0.01</stddev>
-          </noise>
-        </ray>
-        <plugin name="bytes_laserscan" filename="libgazebo_ros_ray_sensor.so">
-          <ros>
-              <namespace>lidar</namespace>
-            <remapping>~/out:=scan</remapping>
-          </ros>
-          <output_type>sensor_msgs/LaserScan</output_type>
-          <frame_name>lidar</frame_name>
-        </plugin>
-    </sensor>
-    <material>Gazebo/Purple</material>
-</gazebo>
+        <updateRate>30</updateRate>
+    </sensor>
+  </gazebo>
+   <!-- LIDAR -->
+   <link name="lidar_support">
+        <visual>
+            <geometry>
+                <box size="${lidar_support_x_dim} ${lidar_support_y_dim} ${lidar_support_z_dim}"/>
+            </geometry>
+        </visual>
+    </link>
+    <joint name="base_link_to_lidar_support" type="fixed">
+        <parent link="base_link"/>
+        <child link="lidar_support"/>
+        <origin xyz="${lidar_x/2} 0.0 ${lidar_z-lidar_support_z_dim/2}" rpy="0.0 0.0 0.0"/>
+    </joint>
+    <!-- collision range = min sensing distance -->
+    <!-- gpu does gpu acceleration -->
+    <xacro:VLP-16 parent="lidar_support" name="lidar" topic="/velodyne_points" hz="${lidar_hz}" samples="${lidar_samples}" gpu="false">
+        <origin xyz="${lidar_x} 0.0 ${lidar_z}" rpy="0 ${lidar_pitch} 0" />
+    </xacro:VLP-16>
   <!-- cameras -->
   <link name="cam/center">
