Commit message: Load broken arm URDF

File: urc_gazebo/urdf/arm_urdf.urdf (robot description, URDF)
Before this commit: robot urc_gazebo, 7 links, 6 joints
Links:
- link bicep: geometry collision mesh filename=$(find urc_gazebo)/meshes/bicep.STL; visual mesh filename=$(find urc_gazebo)/meshes/bicep.STL
- link elbow: geometry collision mesh filename=$(find urc_gazebo)/meshes/elbow.STL; visual mesh filename=$(find urc_gazebo)/meshes/elbow.STL
- link end_effector: geometry collision mesh filename=$(find urc_gazebo)/meshes/end_effector.STL; visual mesh filename=$(find urc_gazebo)/meshes/end_effector.STL
- link forearm: geometry collision mesh filename=$(find urc_gazebo)/meshes/forearm.STL; visual mesh filename=$(find urc_gazebo)/meshes/forearm.STL
- link shoulder: geometry collision mesh filename=$(find urc_gazebo)/meshes/shoulder.STL; visual mesh filename=$(find urc_gazebo)/meshes/shoulder.STL
- link spine: geometry collision mesh filename=$(find urc_gazebo)/meshes/spine.STL; visual mesh filename=$(find urc_gazebo)/meshes/spine.STL
- link wrist: geometry collision mesh filename=$(find urc_gazebo)/meshes/wrist.STL; visual mesh filename=$(find urc_gazebo)/meshes/wrist.STL
