Commit message: ARM WORKING HOOOLY

File: urc_gazebo/urdf/RoboticArm.urdf (robot description, URDF)
Before this commit: robot RoboArm, 8 links, 7 joints
Links:
- link clawbase: mass 1.5984 -> 1.1594
- link endeffector: mass 1.8205 -> 2.2712
Joints:
- joint bicepjoint: axis 0.9991 0 0.042395 -> -1 0 0; origin xyz=0 0 0 rpy=-1.5708 0 -0.35187 -> xyz=0.068308 0.033227 0.041262 rpy=1.5708 0 2.9385; type fixed -> continuous
- joint clawbasejoint: axis 0 0 1 -> 1 0 0; origin xyz=0.059627 0.0042582 0.43251 rpy=1.9117 0 0.4234 -> xyz=0.049891 0.041686 -0.2346 rpy=1.2733 -1.2512 -1.5708
- joint clawjoint: axis 0 1 0 -> 1 0 0; origin xyz=-0.041275 0.0094698 -0.10395 rpy=-1.5708 0 -0.38633 -> xyz=0.51169 -2.7356E-05 2.9513E-05 rpy=0 0 0
- joint elbowjoint: axis 0 1 0 -> 1 0 0; origin xyz=0 0 0 rpy=-0.11095 1.1779 1.4682 -> xyz=0.1204 -0.12377 0.32658 rpy=0 0 0; type fixed -> continuous
- joint endeffectorjoint: axis 0.9117 0.41086 0 -> -1 0 0; origin xyz=0.33807 0.046323 0.048129 rpy=1.5708 1.0472 -1.5708 -> xyz=-0.63096 -0.034252 -0.036275 rpy=-0.3134 -0.81406 1.5708; type fixed -> continuous
- joint forearmjoint: origin xyz=-0.53446 -0.022729 0.034943 rpy=-1.5708 -0.6694 0 -> xyz=-0.060202 -0.19694 -0.1385 rpy=-1.5708 0.41929 -1.5708; type fixed -> continuous

Commit message: the robot got a little excited

File: urc_gazebo/urdf/RoboticArm.urdf (robot description, URDF)
Before this commit: robot RoboticArm, 9 links, 8 joints
Links:
- removed link base_link
- added link arm_base_link, mass 0.523; collision mesh filename=$(find urc_gazebo)/urdf/meshes/base_link.STL; visual mesh filename=$(find urc_gazebo)/urdf/meshes/base_link.STL
Joints:
- added joint arm_joint: type fixed, parent base_link, child arm_base_link, origin xyz=0.043 0 -0.001
- joint shoulderjoint: parent base_link -> arm_base_link

File: urc_gazebo/urdf/wallii.xacro (robot description, xacro)
@@ -4,4 +4,5 @@
   <xacro:include filename="walli_inertials.xacro"/>
   <xacro:include filename="$(find velodyne_description)/urdf/VLP-16.urdf.xacro"/>
+  <xacro:include filename="RoboticArm.urdf"/>
   <!-- The "wheel" macro defines an axle carrier, axle, and wheel. -->
   <xacro:macro name="wheel" params="lr_prefix fr_prefix lr_pos fr_pos">

Commit message: mounted properly but front camera is mounted up for some reason

File: urc_gazebo/urdf/RoboticArm.urdf (robot description, URDF)
Before this commit: robot RoboticArm, 9 links, 9 joints
Joints:
- joint arm_joint: origin xyz=0.043 0 -0.001 -> xyz=0 0 0.6

File: urc_gazebo/urdf/wallii.xacro (robot description, xacro)
@@ -79,5 +79,5 @@
   <joint name="imu_joint" type="fixed">
 		<axis xyz="1 0 0"/>
-		<origin xyz="0 0 0.05"/>
+		<origin xyz="0 0 .4"/>
 		<parent link="base_link"/>
 		<child link="imu"/>

Commit message: Arm copy to test ros2 control on arm only

File: urc_gazebo/urdf/RoboticArm.urdf (robot description, URDF)
Before this commit: robot RoboticArm, 9 links, 9 joints
Links:
- removed link bicep
- removed link clawbase
- removed link elbow
- removed link endeffector
- removed link forearm
- removed link leftgripper
- removed link rightgripper
Joints:
- removed joint bicepjoint
- removed joint clawbasejoint
- removed joint elbowjoint
- removed joint endeffectorjoint
- removed joint forearmjoint
- removed joint leftgripperjoint
- removed joint rightgripperjoint
