Commit message: unexpected behavior between active joints

File: urc_gazebo/urdf/ArmCopy.urdf (robot description, URDF)
Before this commit: robot RoboticArm, 10 links, 9 joints
Links:
- removed link clawbase
- removed link endeffector
- removed link leftgripper
- removed link rightgripper
- added link world
Joints:
- removed joint clawbasejoint
- removed joint endeffectorjoint
- removed joint leftgripperjoint
- removed joint rightgripperjoint
- added joint world_to_base: type fixed, parent world, child base_link, origin xyz=0 0 1 rpy=0 0 0
- joint arm_joint: limit (none) -> effort=100 velocity=5.0
- joint bicepjoint: limit (none) -> effort=100 velocity=5.0
- joint elbowjoint: limit (none) -> effort=100 velocity=5.0
- joint forearmjoint: limit (none) -> effort=100 velocity=5.0
- joint shoulderjoint: limit (none) -> effort=100 velocity=5.0
