Commit message: clean up before PR

File: urc_gazebo/urdf/WalliiArmV3.urdf (robot description, URDF)
Before this commit: robot WalliiArmV3, 9 links, 8 joints
Joints:
- joint clawjoint: limit lower=-3.14 upper=3.14 effort=0 velocity=0 -> (none); type revolute -> continuous
- joint forearmjoint: limit lower=-3.14 upper=3.14 effort=0 velocity=0 -> (none); type revolute -> continuous
- joint shoulderjoint: limit lower=-3.14 upper=3.14 effort=0 velocity=0 -> (none); type revolute -> continuous

File: urc_gazebo/urdf/wallii.xacro (robot description, xacro)
@@ -4,4 +4,5 @@
   <xacro:include filename="walli_inertials.xacro"/>
   <xacro:include filename="$(find velodyne_description)/urdf/VLP-16.urdf.xacro"/>
+  <!-- Import wallii arm urdf to walli's urdf. -->
   <xacro:include filename="WalliiArmV3.urdf"/>
   <!--- Something about this macro breaks the urdf parser. -->
@@ -35,4 +36,7 @@
       <axis xyz="0 0 -1"/>
       <limit effort="${axle_eff_limit}" velocity="${axle_vel_limit}"/>
+      <dynamics
+      damping="0"
+      friction="4.0" />
     </joint>
     <gazebo reference="${lr_prefix}_${fr_prefix}_wheel">
@@ -81,5 +85,4 @@
     <child link="body"/>
   </joint>
-    <!-- breaking urdf parser -->
   <!-- Wheels    -->
   <xacro:wheel lr_prefix="left_bogie" fr_prefix="front"
@@ -114,4 +117,9 @@
     <dynamics damping="60.0" friction="4.0"/>
   </joint>
+    <!--
+    Mock/Untested ros2 control scheme for operating the rover with ros2 control.
+    This matches how the control is supposed to be set up, but is commented out
+    because the way the urdf is designed, it interferes with the arm control.
+    -->
     <!--
     <ros2_control name="rover_control" type="system">
@@ -319,7 +327,7 @@
     <!-- collision range = min sensing distance -->
     <!-- gpu does gpu acceleration -->
-    <!-- <xacro:VLP-16 parent="lidar_support" name="lidar" topic="/scan" hz="${lidar_hz}" samples="${lidar_samples}" gpu="false">
+    <xacro:VLP-16 parent="lidar_support" name="lidar" topic="/scan" hz="${lidar_hz}" samples="${lidar_samples}" gpu="false">
         <origin xyz="${lidar_x} 0.0 ${lidar_z}" rpy="0 ${lidar_pitch} 0" />
-    </xacro:VLP-16> -->
+    </xacro:VLP-16>
   <!-- cameras -->
   <link name="cam/center">
@@ -339,5 +347,5 @@
 	<axis xyz="1 0 0"/>
 	<!-- Edit these parameters to change camera orientation -->
-	<origin xyz="0 0 0.05" rpy = "0 0 -.14"/>
+	<origin xyz="0.15 0 -0.1" rpy = "0 0 -.14"/>
 	<parent link="imu"/>
 	<child link="cam/center"/>
@@ -391,5 +399,5 @@
 	<axis xyz="1 0 0"/>
 	<!-- Edit these parameters to change camera orientation -->
-	<origin xyz="0 0 0.05" rpy = "0 0 1.5"/>
+	<origin xyz="0 0.1 0.0" rpy = "0 0 1.5"/>
 	<parent link="base_link"/>
 	<child link="cam/left"/>
@@ -443,5 +451,5 @@
 	<axis xyz="1 0 0"/>
 	<!-- Edit these parameters to change camera orientation -->
-	<origin xyz="0 0 0.05" rpy = "0 0 -1.5"/>
+	<origin xyz="0 -0.1 0.0" rpy = "0 0 -1.5"/>
 	<parent link="base_link"/>
 	<child link="cam/right"/>
