Commit message: Added IMU sensor and rocker bogie model

File: urc_gazebo/urdf/wallii.xacro (robot description, xacro)
@@ -1,51 +1,224 @@
 <?xml version='1.0'?>
 <robot name="wallii" xmlns:xacro="http://www.ros.org/wiki/xacro">
-  <link name='chassis'>
-    <pose>0 0 0.1 0 0 0</pose>
-    <inertial>
-      <mass value="15.0"/>
-      <origin xyz="0.0 0 0" rpy=" 0 0 0"/>
-      <inertia
-          ixx="0.1" ixy="0" ixz="0"
-          iyy="0.1" iyz="0"
-          izz="0.1"
-      />
-    </inertial>
-    <collision name='collision'>
-      <origin xyz="0 0 0.05" rpy=" 0 0 0"/>
-      <geometry>
-        <cylinder length="0.2" radius="0.25"/>
-      </geometry>
-    </collision>
-    <visual name='chassis_visual'>
-      <origin xyz="0 0 0.05" rpy=" 0 0 0"/>
-      <geometry>
-       <cylinder length="0.2" radius="0.25"/>
-      </geometry>
-    </visual>
-    <collision name='back_caster_collision'>
-      <origin xyz="-0.15 0 -0.05" rpy=" 0 0 0"/>
-      <geometry>
-        <sphere radius="0.0499"/>
-      </geometry>
-    </collision>
-    <visual name='back_caster_visual'>
-      <origin xyz="-0.15 0 -0.05" rpy=" 0 0 0"/>
-      <geometry>
-        <sphere radius="0.05"/>
-      </geometry>
-    </visual>
-    <collision name='front_caster_collision'>
-      <origin xyz="0.15 0 -0.05" rpy=" 0 0 0"/>
-      <geometry>
-        <sphere radius="0.0499"/>
-      </geometry>
-    </collision>
-    <visual name='front_caster_visual'>
-      <origin xyz="0.15 0 -0.05" rpy=" 0 0 0"/>
-      <geometry>
-        <sphere radius="0.05"/>
-      </geometry>
+  <xacro:include filename="walli_prop.xacro"/>
+  <xacro:include filename="walli_inertials.xacro"/>
+  <!-- The "wheel" macro defines an axle carrier, axle, and wheel. -->
+  <xacro:macro name="wheel" params="lr_prefix fr_prefix lr_pos fr_pos">
+    <joint name="${lr_prefix}_${fr_prefix}_axle" type="continuous">
+      <parent link="base_link"/>
+      <child link="${lr_prefix}_${fr_prefix}_wheel"/>
+      <origin xyz="${fr_pos}
+                   ${lr_pos}
+                   ${- body_clearance}"
+              rpy="${degrees_90} 0 0"/>
+      <axis xyz="0 0 -1"/>
+      <limit effort="${axle_eff_limit}" velocity="${axle_vel_limit}"/>
+    </joint>
+    <ros2_control name="GazeboSystem" type="system">
+      <transmission name="${lr_prefix}_${fr_prefix}_axle_trans">
+        <type>transmission_interface/SimpleTransmission</type>
+        <joint name="${lr_prefix}_${fr_prefix}_axle">
+          <hardwareInterface>VelocityJointInterface</hardwareInterface>
+        </joint>
+        <actuator name="${lr_prefix}_${fr_prefix}_axle_act">
+          <hardwareInterface>VelocityJointInterface</hardwareInterface>
+          <mechanicalReduction>1</mechanicalReduction>
+        </actuator>
+      </transmission>
+    </ros2_control>
+    <link name="${lr_prefix}_${fr_prefix}_wheel">
+      <visual>
+        <origin xyz="0 0 0"/>
+        <geometry>
+          <cylinder radius="${tire_dia / 2}" length="${tire_width}"/>
+        </geometry>
+        <material name="tire_mat"/>
+      </visual>
+      <collision>
+        <origin xyz="0 0 0"/>
+        <geometry>
+          <cylinder radius="${tire_dia / 2}" length="${tire_width}"/>
+        </geometry>
+      </collision>
+      <xacro:thick_walled_tube_inertial
+          inner_rad="${hub_dia / 2}" outer_rad="${tire_dia / 2}"
+          height="${tire_width}" mass="${wheel_mass}"/>
+    </link>
+    <gazebo reference="${lr_prefix}_${fr_prefix}_wheel">
+      <material>Gazebo/Black</material>
+    </gazebo>
+  </xacro:macro>
+  <!-- base_link must have geometry so that its axes can be displayed in
+       rviz. -->
+  <link name="base_link">
+    <visual>
+      <geometry>
+        <box size="0.05 0.05 0.01"/>
+      </geometry>
+      <material name="body_mat"/>
     </visual>
   </link>
+  <gazebo reference="base_link">
+    <material>Gazebo/Green</material>
+  </gazebo>
+  <link name="imu">
+    <visual>
+      <geometry>
+        <box size="0.1 0.1 0.1"/>
+      </geometry>
+    </visual>
+    <collision>
+      <geometry>
+        <box size="0.1 0.1 0.1"/>
+      </geometry>
+    </collision>
+    <xacro:box_inertia m="0.1" w="0.1" d="0.1" h="0.1"/>
+  </link>
+  <joint name="imu_joint" type="fixed">
+		<axis xyz="1 0 0"/>
+		<origin xyz="0 0 0.05"/>
+		<parent link="base_link"/>
+		<child link="imu"/>
+	</joint>
+	<gazebo reference="imu">
+    <sensor name="imu_sensor" type="imu">
+      <plugin filename="libgazebo_ros_imu_sensor.so" name="imu_plugin">
+        <ros>
+          <namespace>/imu</namespace>
+          <remapping>~/out:=data</remapping>
+        </ros>
+        <initial_orientation_as_reference>false</initial_orientation_as_reference>
+      </plugin>
+      <always_on>true</always_on>
+      <update_rate>100</update_rate>
+      <visualize>true</visualize>
+     <imu>
+     	<angular_velocity>
+     	  <x>
+     	    <noise type="gaussian">
+              <mean>0.0</mean>
+              <stddev>2e-4</stddev>
+              <bias_mean>0.0000075</bias_mean>
+              <bias_stddev>0.0000008</bias_stddev>
+            </noise>
+          </x>
+          <y>
+            <noise type="gaussian">
+              <mean>0.0</mean>
+              <stddev>2e-4</stddev>
+              <bias_mean>0.0000075</bias_mean>
+              <bias_stddev>0.0000008</bias_stddev>
+            </noise>
+          </y>
+          <z>
+            <noise type="gaussian">
+              <mean>0.0</mean>
+              <stddev>2e-4</stddev>
+              <bias_mean>0.0000075</bias_mean>
+              <bias_stddev>0.0000008</bias_stddev>
+            </noise>
+          </z>
+        </angular_velocity>
+        <linear_acceleration>
+          <x>
+            <noise type="gaussian">
+              <mean>0.0</mean>
+              <stddev>1.7e-2</stddev>
+              <bias_mean>0.1</bias_mean>
+              <bias_stddev>0.001</bias_stddev>
+            </noise>
+          </x>
+          <y>
+            <noise type="gaussian">
+              <mean>0.0</mean>
+              <stddev>1.7e-2</stddev>
+              <bias_mean>0.1</bias_mean>
+              <bias_stddev>0.001</bias_stddev>
+            </noise>
+          </y>
+          <z>
+            <noise type="gaussian">
+              <mean>0.0</mean>
+              <stddev>1.7e-2</stddev>
+              <bias_mean>0.1</bias_mean>
+              <bias_stddev>0.001</bias_stddev>
+            </noise>
+          </z>
+        </linear_acceleration>
+      </imu>
+    </sensor>
+  </gazebo>
+  <!-- body -->
+  <link name="body">
+    <visual>
+      <origin xyz="0 0 ${-body_height / 2}"/>
+      <geometry>
+        <box size="${body_length} ${body_width} ${body_height}"/>
+      </geometry>
+      <material name="body_mat"/>
+    </visual>
+    <collision>
+      <origin xyz="0 0 ${-body_height / 2}"/>
+      <geometry>
+        <box size="${body_length} ${body_width} ${body_height}"/>
+      </geometry>
+    </collision>
+    <xacro:solid_cuboid_inertial
+        width="${body_length}" depth="${body_width}"
+        height="${body_height}" mass="${body_mass}">
+      <origin xyz="0 0 ${-body_height / 2}"/>
+    </xacro:solid_cuboid_inertial>
+  </link>
+  <gazebo reference="body">
+    <material>Gazebo/Grey</material>
+  </gazebo>
+  <joint name="base_link_to_chasis" type="fixed">
+    <parent link="base_link"/>
+    <child link="body"/>
+  </joint>
+  <!-- Wheels -->
+  <xacro:wheel lr_prefix="left_bogie" fr_prefix="front"
+               lr_pos="${track / 2}"
+               fr_pos="${x_center_bogie + wheelbase_bogie / 2}"
+               />
+  <xacro:wheel lr_prefix="left_bogie" fr_prefix="rear"
+               lr_pos="${track / 2}"
+               fr_pos="${x_center_bogie - wheelbase_bogie / 2}"
+               />
+  <xacro:wheel lr_prefix="left_rocker" fr_prefix="rear"
+               lr_pos="${track / 2}"
+               fr_pos="${x_center_rocker - wheelbase_rocker / 2}"
+               />
+  <xacro:wheel lr_prefix="right_bogie" fr_prefix="front"
+               lr_pos="${- track / 2}"
+               fr_pos="${x_center_bogie + wheelbase_bogie / 2}"
+               />
+  <xacro:wheel lr_prefix="right_bogie" fr_prefix="rear"
+               lr_pos="${- track / 2}"
+               fr_pos="${x_center_bogie - wheelbase_bogie / 2}"
+               />
+  <xacro:wheel lr_prefix="right_rocker" fr_prefix="rear"
+               lr_pos="${- track / 2}"
+               fr_pos="${x_center_rocker - wheelbase_rocker / 2}"
+               />
+  <gazebo>
+    <sensor name="imu" type="imu">
+      <always_on>true</always_on>
+      <!-- Publish at 30 hz -->
+      <update_rate>30</update_rate>
+      <plugin name="imu" filename="libgazebo_ros_imu_sensor.so">
+        <ros>
+          <!-- Will publish to /imu/data -->
+          <namespace>/imu</namespace>
+          <argument>~/out:=data</argument>
+        </ros>
+        <frame_name>imu</frame_name>
+      </plugin>
+    </sensor>
+  </gazebo>
+  <ros2_control name="GazeboSystem" type="system">
+    <hardware>
+      <plugin>gazebo_ros2_control/GazeboSystem</plugin>
+    </hardware>
+  </ros2_control>
 </robot>

Commit message: Left right and center camera integration

File: urc_gazebo/urdf/wallii.xacro (robot description, xacro)
@@ -149,4 +149,139 @@
     </sensor>
   </gazebo>
+  <link name="cam/center">
+    <visual>
+      <geometry>
+        <box size="0.1 0.1 0.1"/>
+      </geometry>
+    </visual>
+    <collision>
+      <geometry>
+        <box size="0.1 0.1 0.1"/>
+      </geometry>
+    </collision>
+    <xacro:box_inertia m="0.1" w="0.1" d="0.1" h="0.1"/>
+  </link>
+  <joint name="center_cam_joint" type="fixed">
+	<axis xyz="1 0 0"/>
+	<!-- Edit these parameters to change camera orientation -->
+	<origin xyz="0 0 0.05" rpy = "0 0 -.14"/>
+	<parent link="imu"/>
+	<child link="cam/center"/>
+   </joint>
+   <gazebo reference="cam/center">
+    <sensor name="center_sensor" type="camera">
+        <plugin name="plugin_name" filename="libgazebo_ros_camera.so">
+        <ros>
+          <namespace>/image</namespace>
+          <remapping>~/image_raw:=center_img</remapping>
+          <remapping>~/camera_info:=center_info</remapping>
+        </ros>
+        <initial_orientation_as_reference>false</initial_orientation_as_reference>
+      </plugin>
+      <always_on>true</always_on>
+      <update_rate>100</update_rate>
+      <visualize>true</visualize>
+      <camera name="cam/center">
+          <distortion>
+            <k1>0.1</k1>
+            <k2>0.2</k2>
+            <k3>0.3</k3>
+            <p1>0.4</p1>
+            <p2>0.5</p2>
+            <center>0.5 0.5</center>
+          </distortion>
+       </camera>
+    </sensor>
+  </gazebo>
+  <link name="cam/left">
+    <visual>
+      <geometry>
+        <box size="0.1 0.1 0.1"/>
+      </geometry>
+    </visual>
+    <collision>
+      <geometry>
+        <box size="0.1 0.1 0.1"/>
+      </geometry>
+    </collision>
+    <xacro:box_inertia m="0.1" w="0.1" d="0.1" h="0.1"/>
+  </link>
+  <joint name="left_cam_joint" type="fixed">
+	<axis xyz="1 0 0"/>
+	<!-- Edit these parameters to change camera orientation -->
+	<origin xyz="0 0 0.05" rpy = "0 0 1.5"/>
+	<parent link="base_link"/>
+	<child link="cam/left"/>
+   </joint>
+   <gazebo reference="cam/left">
+    <sensor name="left_sensor" type="camera">
+        <plugin name="plugin_name" filename="libgazebo_ros_camera.so">
+        <ros>
+          <namespace>/image</namespace>
+          <remapping>~/image_raw:=left_img</remapping>
+          <remapping>~/camera_info:=left_info</remapping>
+        </ros>
+        <initial_orientation_as_reference>false</initial_orientation_as_reference>
+      </plugin>
+      <always_on>true</always_on>
+      <update_rate>100</update_rate>
+      <visualize>true</visualize>
+      <camera name="cam/left">
+          <distortion>
+            <k1>0.1</k1>
+            <k2>0.2</k2>
+            <k3>0.3</k3>
+            <p1>0.4</p1>
+            <p2>0.5</p2>
+            <center>0.5 0.5</center>
+          </distortion>
+       </camera>
+    </sensor>
+  </gazebo>
+  <link name="cam/right">
+    <visual>
+      <geometry>
+        <box size="0.1 0.1 0.1"/>
+      </geometry>
+    </visual>
+    <collision>
+      <geometry>
+        <box size="0.1 0.1 0.1"/>
+      </geometry>
+    </collision>
+    <xacro:box_inertia m="0.1" w="0.1" d="0.1" h="0.1"/>
+  </link>
+  <joint name="right_cam_joint" type="fixed">
+	<axis xyz="1 0 0"/>
+	<!-- Edit these parameters to change camera orientation -->
+	<origin xyz="0 0 0.05" rpy = "0 0 -1.5"/>
+	<parent link="base_link"/>
+	<child link="cam/right"/>
+   </joint>
+   <gazebo reference="cam/right">
+    <sensor name="right_sensor" type="camera">
+        <plugin name="plugin_name" filename="libgazebo_ros_camera.so">
+        <ros>
+          <namespace>/image</namespace>
+          <remapping>~/image_raw:=right_img</remapping>
+          <remapping>~/camera_info:=right_info</remapping>
+        </ros>
+        <initial_orientation_as_reference>false</initial_orientation_as_reference>
+      </plugin>
+      <always_on>true</always_on>
+      <update_rate>100</update_rate>
+      <visualize>true</visualize>
+      <camera name="cam/right">
+          <distortion>
+            <k1>0.1</k1>
+            <k2>0.2</k2>
+            <k3>0.3</k3>
+            <p1>0.4</p1>
+            <p2>0.5</p2>
+            <center>0.5 0.5</center>
+          </distortion>
+       </camera>
+    </sensor>
+  </gazebo>
   <!-- body -->
   <link name="body">
@@ -216,4 +351,76 @@
       </plugin>
     </sensor>
+    <sensor type="camera" name="center_sensor">
+          <!-- Set always_on only sensor, not on plugin -->
+          <always_on>0</always_on>
+          <!-- Set update_rate only sensor, not on plugin -->
+          <update_rate>1</update_rate>
+          <!-- Use camera, not camera_triggered -->
+          <plugin name="plugin_name" filename="libgazebo_ros_camera.so">
+            <!-- Change namespace, camera name and topics so:
+                 * Images are published to: /custom_ns/custom_camera/custom_image
+                 * Camera info is published to: /custom_ns/custom_camera/custom_info
+            -->
+            <ros>
+              <namespace>/image</namespace>
+              <argument>~/image_raw:=center_img</argument>
+              <argument>~/camera_info:=center_info</argument>
+            </ros>
+            <!-- Set camera name. If empty, defaults to sensor name (i.e. "sensor_name") -->
+            <camera_name>center_camera</camera_name>
+            <!-- Set TF frame name. If empty, defaults to link name (i.e. "link_name") -->
+            <frame_name>center_tf</frame_name>
+            <hack_baseline>0.07</hack_baseline>
+            <!-- No need to repeat distortion parameters or to set autoDistortion -->
+          </plugin>
+        </sensor>
+     <sensor type="camera" name="left_sensor">
+          <!-- Set always_on only sensor, not on plugin -->
+          <always_on>0</always_on>
+          <!-- Set update_rate only sensor, not on plugin -->
+          <update_rate>1</update_rate>
+          <!-- Use camera, not camera_triggered -->
+          <plugin name="plugin_name" filename="libgazebo_ros_camera.so">
+            <!-- Change namespace, camera name and topics so:
+                 * Images are published to: /custom_ns/custom_camera/custom_image
+                 * Camera info is published to: /custom_ns/custom_camera/custom_info
+            -->
+            <ros>
+              <namespace>/image</namespace>
+              <argument>~/image_raw:=left_img</argument>
+              <argument>~/camera_info:=left_info</argument>
+            </ros>
+            <!-- Set camera name. If empty, defaults to sensor name (i.e. "sensor_name") -->
+            <camera_name>left_camera</camera_name>
+            <!-- Set TF frame name. If empty, defaults to link name (i.e. "link_name") -->
+            <frame_name>left_tf</frame_name>
+            <hack_baseline>0.07</hack_baseline>
+            <!-- No need to repeat distortion parameters or to set autoDistortion -->
+          </plugin>
+        </sensor>
+      <sensor type="camera" name="right_sensor">
+          <!-- Set always_on only sensor, not on plugin -->
+          <always_on>0</always_on>
+          <!-- Set update_rate only sensor, not on plugin -->
+          <update_rate>1</update_rate>
+          <!-- Use camera, not camera_triggered -->
+          <plugin name="plugin_name" filename="libgazebo_ros_camera.so">
+            <!-- Change namespace, camera name and topics so:
+                 * Images are published to: /custom_ns/custom_camera/custom_image
+                 * Camera info is published to: /custom_ns/custom_camera/custom_info
+            -->
+            <ros>
+              <namespace>/image</namespace>
+              <argument>~/image_raw:=right_img</argument>
+              <argument>~/camera_info:=right_info</argument>
+            </ros>
+            <!-- Set camera name. If empty, defaults to sensor name (i.e. "sensor_name") -->
+            <camera_name>right_camera</camera_name>
+            <!-- Set TF frame name. If empty, defaults to link name (i.e. "link_name") -->
+            <frame_name>right_tf</frame_name>
+            <hack_baseline>0.07</hack_baseline>
+            <!-- No need to repeat distortion parameters or to set autoDistortion -->
+          </plugin>
+        </sensor>
   </gazebo>
   <ros2_control name="GazeboSystem" type="system">

Commit message: Added GPS

File: urc_gazebo/urdf/wallii.xacro (robot description, xacro)
@@ -149,4 +149,50 @@
     </sensor>
   </gazebo>
+  <!-- gps -->
+  <link name="gps">
+    <visual>
+      <geometry>
+        <box size="0.1 0.1 0.1"/>
+      </geometry>
+    </visual>
+    <collision>
+      <geometry>
+        <box size="0.1 0.1 0.1"/>
+      </geometry>
+    </collision>
+    <xacro:box_inertia m="0.1" w="0.1" d="0.1" h="0.1"/>
+  </link>
+   <joint name="gps_joint" type="fixed">
+		<axis xyz="1 0 0"/>
+		<origin xyz="0 0 0.05"/>
+		<parent link="base_link"/>
+		<child link="gps"/>
+	</joint>
+  <gazebo reference="gps">
+    <sensor name="gps" type="gps">
+      <plugin filename="libgazebo_ros_gps_sensor.so" name="gps_plugin">
+          <ros>
+            <namespace>/gps</namespace>
+            <remapping>~/out:=data</remapping>
+          </ros>
+          <initial_orientation_as_reference>false</initial_orientation_as_reference>
+        </plugin>
+        <always_on>true</always_on>
+        <updateRate>100000.0</updateRate>
+        <bodyName>base_link</bodyName>
+        <frameId>base_link</frameId>
+        <topicName>/fix</topicName>
+        <velocityTopicName>/fix_velocity</velocityTopicName>
+        <referenceLatitude>33.774497</referenceLatitude>
+        <referenceLongitude>-84.405001</referenceLongitude>
+        <referenceHeading>90</referenceHeading>
+        <referenceAltitude>309.0</referenceAltitude>
+        <drift>0.001 0.001 0.001</drift>
+        <gaussianNoise>0.0001 0.0001 0.0001</gaussianNoise>
+        <velocityDrift>0 0 0</velocityDrift>
+        <velocityGaussianNoise>0.005 0.005 0.05</velocityGaussianNoise>
+    </sensor>
+  </gazebo>
+  <!-- cameras -->
   <link name="cam/center">
     <visual>

Commit message: lidar integration

File: urc_gazebo/urdf/wallii.xacro (robot description, xacro)
@@ -194,4 +194,53 @@
     </sensor>
   </gazebo>
+  <!-- Lidar -->
+ <link name="lidar">
+    <visual>
+      <geometry>
+        <box size="0.1 0.1 0.1"/>
+      </geometry>
+    </visual>
+    <collision>
+      <geometry>
+        <box size="0.1 0.1 0.1"/>
+      </geometry>
+    </collision>
+    <xacro:box_inertia m="0.1" w="0.1" d="0.1" h="0.1"/>
+  </link>
+  <joint name="lidar_joint" type="fixed">
+		<axis xyz="1 0 0"/>
+		<origin xyz="0 0 0.05"/>
+		<parent link="base_link"/>
+		<child link="lidar"/>
+	</joint>
+  <gazebo reference="lidar">
+        <material>Gazebo/Red</material>
+        <sensor name="laser" type="ray">
+            <pose> 0 0 0 0 0 0 </pose>
+            <visualize>true</visualize>
+            <update_rate>10</update_rate>
+            <ray>
+                <scan>
+                    <horizontal>
+                        <samples>360</samples>
+                        <min_angle>-3.14</min_angle>
+                        <max_angle>3.14</max_angle>
+                    </horizontal>
+                </scan>
+                <range>
+                    <min>0.3</min>
+                    <max>12</max>
+                </range>
+            </ray>
+            <plugin name="laser_controller" filename="libgazebo_ros_ray_sensor.so">
+                <ros>
+                  <namespace>/lidar</namespace>
+                  <remapping>~/out:=data</remapping>
+                </ros>
+                <output_type>sensor_msgs/LaserScan</output_type>
+                <frame_name>lidar</frame_name>
+            </plugin>
+        </sensor>
+    </gazebo>
   <!-- cameras -->
   <link name="cam/center">
