Commit message: updated lidar integration

File: urc_gazebo/urdf/wallii.xacro (robot description, xacro)
@@ -181,5 +181,5 @@
         <updateRate>100000.0</updateRate>
         <bodyName>base_link</bodyName>
-        <frameId>base_link</frameId>
+        <frameId>gps</frameId>
         <topicName>/fix</topicName>
         <velocityTopicName>/fix_velocity</velocityTopicName>
@@ -215,32 +215,40 @@
 	</joint>
   <gazebo reference="lidar">
-        <material>Gazebo/Red</material>
-        <sensor name="laser" type="ray">
-            <pose> 0 0 0 0 0 0 </pose>
-            <visualize>true</visualize>
-            <update_rate>10</update_rate>
-            <ray>
-                <scan>
-                    <horizontal>
-                        <samples>360</samples>
-                        <min_angle>-3.14</min_angle>
-                        <max_angle>3.14</max_angle>
-                    </horizontal>
-                </scan>
-                <range>
-                    <min>0.3</min>
-                    <max>12</max>
-                </range>
-            </ray>
-            <plugin name="laser_controller" filename="libgazebo_ros_ray_sensor.so">
-                <ros>
-                  <namespace>/lidar</namespace>
-                  <remapping>~/out:=data</remapping>
-                </ros>
-                <output_type>sensor_msgs/LaserScan</output_type>
-                <frame_name>lidar</frame_name>
-            </plugin>
-        </sensor>
-    </gazebo>
+    <sensor name="lidar" type="ray">
+        <always_on>true</always_on>
+        <visualize>false</visualize>
+        <pose>0.0 0 0.0 0 0 0</pose>
+        <update_rate>15</update_rate>
+        <ray>
+          <scan>
+            <horizontal>
+              <samples>667</samples>
+              <resolution>0.54</resolution>
+              <min_angle>0.000000</min_angle>
+              <max_angle>6.280000</max_angle>
+            </horizontal>
+          </scan>
+          <range>
+            <min>0.120000</min>
+            <max>20</max>
+            <resolution>0.54</resolution>
+          </range>
+          <noise>
+            <type>gaussian</type>
+            <mean>0.0</mean>
+            <stddev>0.01</stddev>
+          </noise>
+        </ray>
+        <plugin name="bytes_laserscan" filename="libgazebo_ros_ray_sensor.so">
+          <ros>
+              <namespace>lidar</namespace>
+            <remapping>~/out:=scan</remapping>
+          </ros>
+          <output_type>sensor_msgs/LaserScan</output_type>
+          <frame_name>lidar</frame_name>
+        </plugin>
+    </sensor>
+    <material>Gazebo/Purple</material>
+</gazebo>
   <!-- cameras -->
   <link name="cam/center">

Commit message: upgraded_robot model. Includes imu, left right center cameras, gps, lidar, and ground truth plugins.

File: urc_gazebo/urdf/wallii.xacro (robot description, xacro)
@@ -194,9 +194,9 @@
         <parent link="base_link"/>
         <child link="lidar_support"/>
-        <origin xyz="${lidar_x/2} 0.0 ${lidar_z-lidar_support_z_dim/2}" rpy="0.0 0.0 0.0"/>
+        <origin xyz="0.0 0.0 0.0" rpy="0.0 0.0 0.0"/>
     </joint>
     <!-- collision range = min sensing distance -->
     <!-- gpu does gpu acceleration -->
-    <xacro:VLP-16 parent="lidar_support" name="lidar" topic="/velodyne_points" hz="${lidar_hz}" samples="${lidar_samples}" gpu="false">
+    <xacro:VLP-16 parent="lidar_support" name="lidar" topic="/scan" hz="${lidar_hz}" samples="${lidar_samples}" gpu="false">
         <origin xyz="${lidar_x} 0.0 ${lidar_z}" rpy="0 ${lidar_pitch} 0" />
     </xacro:VLP-16>
@@ -476,4 +476,17 @@
           </plugin>
         </sensor>
+      <plugin name="gazebo_ros_p3d" filename="libgazebo_ros_p3d.so">
+        <alwaysOn>true</alwaysOn>
+        <update_rate>200.0</update_rate>
+        <ros>
+          <namespace>/ground_truth</namespace>
+          <argument>odom:=state_raw</argument>
+        </ros>
+        <body_name>base_link</body_name>
+        <frame_name>world</frame_name>
+        <xyz_offset>0 0 0</xyz_offset>
+        <rpy_offset>0.0 0.0 0.0</rpy_offset>
+        <gaussian_noise>0.00</gaussian_noise>
+      </plugin>
   </gazebo>
   <ros2_control name="GazeboSystem" type="system">

Commit message: Feat/arm2 (#121)
* Added moveit

* Added arm URDF

* arm urdf and associated urdf files

* Removed moveit from packages

* Load broken arm URDF

* slightly better arm urdf, still rotation issues with bicep, elbow and end effector joints

* ARM WORKING HOOOLY

* Robot Arm moveit files, test functionality somehow

* Fix arm displaying in gazebo

* ros2 control small fix

* the robot got a little excited

* mounted properly but front camera is mounted up for some reason

* add joint state broadcaster and arm controller for arm, yaml issue

* Arm copy to test ros2 control on arm only

* I made a helicopter lol

* unexpected behavior between active joints

* accidentally built in src

* joint breaking issue fixed

* urc manipulation launch file changes

* small plugin fix in launch file

* arm config and ros2 control uncertainty

* god I literally hate ros2 so much

* trying to reverse engineer servo node interface

* servo node interface communicating but still broken

* this is so sick our robot responds to the controller now

* manual servo controls works in gazebo now

* manual control arm integrated onto current rover

* clean up before PR

* delete unwanted folders

* 🥵

* 🥵🥵

* 🥵🥵🥵

* 🥵🥵🥵🥵

* 🥵🥵🥵🥵🥵

* revert python formatting attempt

* 🤠

* 🤠🤠

* 🤠🤠🤠🤠

* and I wonder

* if you know

* what it means

* 🤠🤠🤠

* what it means to find your dreams

* These dreams be waking me up at night

* Im a star how could I not shine

* 🤠 bye build error

* 🤠 auf wiedersehen build error

* and the weather so breezy

* google search how to blackmail your ci pipeline

* ci p😵

* ...

* 🐵

* classic 🦍

* 👉👈 work??? 🤪

* version check

* hmm

* idk

* 😩

* couldnt hurt to try ig

* 🤠🤠🤠🤠🤠

---------

Co-authored-by: Harris Nesteruk <harrislegobrick@gmail.com>

File: urc_gazebo/urdf/wallii.xacro (robot description, xacro)
@@ -4,28 +4,9 @@
   <xacro:include filename="walli_inertials.xacro"/>
   <xacro:include filename="$(find velodyne_description)/urdf/VLP-16.urdf.xacro"/>
+  <!-- Import wallii arm urdf to walli's urdf. -->
+  <xacro:include filename="WalliiArmV3.urdf"/>
+  <!--- Something about this macro breaks the urdf parser. -->
   <!-- The "wheel" macro defines an axle carrier, axle, and wheel. -->
   <xacro:macro name="wheel" params="lr_prefix fr_prefix lr_pos fr_pos">
-    <joint name="${lr_prefix}_${fr_prefix}_axle" type="continuous">
-      <parent link="base_link"/>
-      <child link="${lr_prefix}_${fr_prefix}_wheel"/>
-      <origin xyz="${fr_pos}
-                   ${lr_pos}
-                   ${- body_clearance}"
-              rpy="${degrees_90} 0 0"/>
-      <axis xyz="0 0 -1"/>
-      <limit effort="${axle_eff_limit}" velocity="${axle_vel_limit}"/>
-    </joint>
-    <ros2_control name="GazeboSystem" type="system">
-      <transmission name="${lr_prefix}_${fr_prefix}_axle_trans">
-        <type>transmission_interface/SimpleTransmission</type>
-        <joint name="${lr_prefix}_${fr_prefix}_axle">
-          <hardwareInterface>VelocityJointInterface</hardwareInterface>
-        </joint>
-        <actuator name="${lr_prefix}_${fr_prefix}_axle_act">
-          <hardwareInterface>VelocityJointInterface</hardwareInterface>
-          <mechanicalReduction>1</mechanicalReduction>
-        </actuator>
-      </transmission>
-    </ros2_control>
     <link name="${lr_prefix}_${fr_prefix}_wheel">
       <visual>
@@ -46,4 +27,17 @@
           height="${tire_width}" mass="${wheel_mass}"/>
     </link>
+    <joint name="${lr_prefix}_${fr_prefix}_axle" type="continuous">
+      <parent link="base_link"/>
+      <child link="${lr_prefix}_${fr_prefix}_wheel"/>
+      <origin xyz="${fr_pos}
+                   ${lr_pos}
+                   ${- body_clearance}"
+              rpy="${degrees_90} 0 0"/>
+      <axis xyz="0 0 -1"/>
+      <limit effort="${axle_eff_limit}" velocity="${axle_vel_limit}"/>
+      <dynamics
+      damping="0"
+      friction="4.0" />
+    </joint>
     <gazebo reference="${lr_prefix}_${fr_prefix}_wheel">
       <material>Gazebo/Black</material>
@@ -63,20 +57,155 @@
     <material>Gazebo/Green</material>
   </gazebo>
+    <!-- body -->
+  <link name="body">
+    <visual>
+      <origin xyz="0 0 ${-body_height / 2}"/>
+      <geometry>
+        <box size="${body_length} ${body_width} ${body_height}"/>
+      </geometry>
+      <material name="body_mat"/>
+    </visual>
+    <collision>
+      <origin xyz="0 0 ${-body_height / 2}"/>
+      <geometry>
+        <box size="${body_length} ${body_width} ${body_height}"/>
+      </geometry>
+    </collision>
+    <xacro:solid_cuboid_inertial
+        width="${body_length}" depth="${body_width}"
+        height="${body_height}" mass="${body_mass}">
+      <origin xyz="0 0 ${-body_height / 2}"/>
+    </xacro:solid_cuboid_inertial>
+  </link>
+  <gazebo reference="body">
+    <material>Gazebo/Grey</material>
+  </gazebo>
+  <joint name="base_link_to_chasis" type="fixed">
+    <parent link="base_link"/>
+    <child link="body"/>
+  </joint>
+  <!-- Wheels    -->
+  <xacro:wheel lr_prefix="left_bogie" fr_prefix="front"
+               lr_pos="${track / 2}"
+               fr_pos="${x_center_bogie + wheelbase_bogie / 2}"
+               />
+  <xacro:wheel lr_prefix="left_bogie" fr_prefix="rear"
+               lr_pos="${track / 2}"
+               fr_pos="${x_center_bogie - wheelbase_bogie / 2}"
+               />
+  <xacro:wheel lr_prefix="left_rocker" fr_prefix="rear"
+               lr_pos="${track / 2}"
+               fr_pos="${x_center_rocker - wheelbase_rocker / 2}"
+               />
+  <xacro:wheel lr_prefix="right_bogie" fr_prefix="front"
+               lr_pos="${- track / 2}"
+               fr_pos="${x_center_bogie + wheelbase_bogie / 2}"
+               />
+  <xacro:wheel lr_prefix="right_bogie" fr_prefix="rear"
+               lr_pos="${- track / 2}"
+               fr_pos="${x_center_bogie - wheelbase_bogie / 2}"
+               />
+  <xacro:wheel lr_prefix="right_rocker" fr_prefix="rear"
+               lr_pos="${- track / 2}"
+               fr_pos="${x_center_rocker - wheelbase_rocker / 2}"
+               />
+  <!-- connect rover and arm -->
+  <joint name="arm_to_rover" type="fixed">
+    <origin rpy="0 0 0" xyz="0 0 0"/>
+    <parent link="base_link"/>
+    <child link="arm_base_link"/>
+    <dynamics damping="60.0" friction="4.0"/>
+  </joint>
+    <!--
+    Mock/Untested ros2 control scheme for operating the rover with ros2 control.
+    This matches how the control is supposed to be set up, but is commented out
+    because the way the urdf is designed, it interferes with the arm control.
+    -->
+    <!--
+    <ros2_control name="rover_control" type="system">
+    <hardware>
+      <plugin>ros2_control_demo_hardware/VelocityActuatorHardware</plugin>
+    </hardware>
+    <joint name="left_bogie_front_axle">
+      <command_interface name="velocity">
+        <param name="min">-1</param>
+        <param name="max">1</param>
+      </command_interface>
+      <state_interface name="velocity"/>
+    </joint>
+    <joint name="left_bogie_rear_axle">
+      <command_interface name="velocity">
+        <param name="min">-1</param>
+        <param name="max">1</param>
+      </command_interface>
+      <state_interface name="velocity"/>
+    </joint>
+    <joint name="left_rocker_rear_axle">
+      <command_interface name="velocity">
+        <param name="min">-1</param>
+        <param name="max">1</param>
+      </command_interface>
+      <state_interface name="velocity"/>
+    </joint>
+    <joint name="right_bogie_front_axle">
+      <command_interface name="velocity">
+        <param name="min">-1</param>
+        <param name="max">1</param>
+      </command_interface>
+      <state_interface name="velocity"/>
+    </joint>
+    <joint name="right_bogie_rear_axle">
+      <command_interface name="velocity">
+        <param name="min">-1</param>
+        <param name="max">1</param>
+      </command_interface>
+      <state_interface name="velocity"/>
+    </joint>
+    <joint name="right_rocker_rear_axle">
+      <command_interface name="velocity">
+        <param name="min">-1</param>
+        <param name="max">1</param>
+      </command_interface>
+      <state_interface name="velocity"/>
+    </joint>
+    <transmission name="rover_transmission">
+      <plugin>transmission_interface/SimpleTransmission</plugin>
+      <joint name="left_bogie_front_axle" role="left_bogie_front_axle">
+        <mechanical_reduction>1</mechanical_reduction>
+      </joint>
+      <joint name="left_bogie_rear_axle" role="left_bogie_rear_axle">
+        <mechanical_reduction>1</mechanical_reduction>
+      </joint>
+      <joint name="left_rocker_rear_axle" role="left_rocker_rear_axle">
+        <mechanical_reduction>1</mechanical_reduction>
+      </joint>
+      <joint name="right_bogie_front_axle" role="right_bogie_front_axle">
+        <mechanical_reduction>1</mechanical_reduction>
+      </joint>
+      <joint name="right_bogie_rear_axle" role="right_bogie_rear_axle">
+        <mechanical_reduction>1</mechanical_reduction>
+      </joint>
+      <joint name="right_rocker_rear_axle" role="right_rocket_rear_axle">
+        <mechanical_reduction>1</mechanical_reduction>
+      </joint>
+    </transmission>
+    </ros2_control>
+    -->
   <link name="imu">
     <visual>
       <geometry>
-        <box size="0.1 0.1 0.1"/>
+        <box size="0.01 0.01 0.01"/>
       </geometry>
     </visual>
     <collision>
       <geometry>
-        <box size="0.1 0.1 0.1"/>
+        <box size="0.01 0.01 0.01"/>
       </geometry>
     </collision>
-    <xacro:box_inertia m="0.1" w="0.1" d="0.1" h="0.1"/>
+    <xacro:box_inertia m="0.01" w="0.01" d="0.01" h="0.01"/>
   </link>
   <joint name="imu_joint" type="fixed">
 		<axis xyz="1 0 0"/>
-		<origin xyz="0 0 0.05"/>
+		<origin xyz="0 0 0.1"/>
 		<parent link="base_link"/>
 		<child link="imu"/>
@@ -154,13 +283,13 @@
     <visual>
       <geometry>
-        <box size="0.1 0.1 0.1"/>
+        <box size="0.01 0.01 0.01"/>
       </geometry>
     </visual>
     <collision>
       <geometry>
-        <box size="0.1 0.1 0.1"/>
+        <box size="0.01 0.01 0.01"/>
       </geometry>
     </collision>
-    <xacro:box_inertia m="0.1" w="0.1" d="0.1" h="0.1"/>
+    <xacro:box_inertia m="0.01" w="0.01" d="0.01" h="0.01"/>
   </link>
    <joint name="gps_joint" type="fixed">
@@ -205,18 +334,18 @@
     <visual>
       <geometry>
-        <box size="0.1 0.1 0.1"/>
+        <box size="0.01 0.01 0.01"/>
       </geometry>
     </visual>
     <collision>
       <geometry>
-        <box size="0.1 0.1 0.1"/>
+        <box size="0.01 0.01 0.01"/>
       </geometry>
     </collision>
-    <xacro:box_inertia m="0.1" w="0.1" d="0.1" h="0.1"/>
+    <xacro:box_inertia m="0.01" w="0.01" d="0.01" h="0.01"/>
   </link>
   <joint name="center_cam_joint" type="fixed">
 	<axis xyz="1 0 0"/>
 	<!-- Edit these parameters to change camera orientation -->
-	<origin xyz="0 0 0.05" rpy = "0 0 -.14"/>
+	<origin xyz="0.15 0 -0.1" rpy = "0 0 -.14"/>
 	<parent link="imu"/>
 	<child link="cam/center"/>
@@ -257,18 +386,18 @@
     <visual>
       <geometry>
-        <box size="0.1 0.1 0.1"/>
+        <box size="0.01 0.01 0.01"/>
       </geometry>
     </visual>
     <collision>
       <geometry>
-        <box size="0.1 0.1 0.1"/>
+        <box size="0.01 0.01 0.01"/>
       </geometry>
     </collision>
-    <xacro:box_inertia m="0.1" w="0.1" d="0.1" h="0.1"/>
+    <xacro:box_inertia m="0.01" w="0.01" d="0.01" h="0.01"/>
   </link>
   <joint name="left_cam_joint" type="fixed">
 	<axis xyz="1 0 0"/>
 	<!-- Edit these parameters to change camera orientation -->
-	<origin xyz="0 0 0.05" rpy = "0 0 1.5"/>
+	<origin xyz="0 0.1 0.0" rpy = "0 0 1.5"/>
 	<parent link="base_link"/>
 	<child link="cam/left"/>
@@ -309,18 +438,18 @@
     <visual>
       <geometry>
-        <box size="0.1 0.1 0.1"/>
+        <box size="0.01 0.01 0.01"/>
       </geometry>
     </visual>
     <collision>
       <geometry>
-        <box size="0.1 0.1 0.1"/>
+        <box size="0.01 0.01 0.01"/>
       </geometry>
     </collision>
-    <xacro:box_inertia m="0.1" w="0.1" d="0.1" h="0.1"/>
+    <xacro:box_inertia m="0.01" w="0.01" d="0.01" h="0.01"/>
   </link>
   <joint name="right_cam_joint" type="fixed">
 	<axis xyz="1 0 0"/>
 	<!-- Edit these parameters to change camera orientation -->
-	<origin xyz="0 0 0.05" rpy = "0 0 -1.5"/>
+	<origin xyz="0 -0.1 0.0" rpy = "0 0 -1.5"/>
 	<parent link="base_link"/>
 	<child link="cam/right"/>
@@ -358,57 +487,4 @@
     </sensor>
   </gazebo>
-  <!-- body -->
-  <link name="body">
-    <visual>
-      <origin xyz="0 0 ${-body_height / 2}"/>
-      <geometry>
-        <box size="${body_length} ${body_width} ${body_height}"/>
-      </geometry>
-      <material name="body_mat"/>
-    </visual>
-    <collision>
-      <origin xyz="0 0 ${-body_height / 2}"/>
-      <geometry>
-        <box size="${body_length} ${body_width} ${body_height}"/>
-      </geometry>
-    </collision>
-    <xacro:solid_cuboid_inertial
-        width="${body_length}" depth="${body_width}"
-        height="${body_height}" mass="${body_mass}">
-      <origin xyz="0 0 ${-body_height / 2}"/>
-    </xacro:solid_cuboid_inertial>
-  </link>
-  <gazebo reference="body">
-    <material>Gazebo/Grey</material>
-  </gazebo>
-  <joint name="base_link_to_chasis" type="fixed">
-    <parent link="base_link"/>
-    <child link="body"/>
-  </joint>
-  <!-- Wheels -->
-  <xacro:wheel lr_prefix="left_bogie" fr_prefix="front"
-               lr_pos="${track / 2}"
-               fr_pos="${x_center_bogie + wheelbase_bogie / 2}"
-               />
-  <xacro:wheel lr_prefix="left_bogie" fr_prefix="rear"
-               lr_pos="${track / 2}"
-               fr_pos="${x_center_bogie - wheelbase_bogie / 2}"
-               />
-  <xacro:wheel lr_prefix="left_rocker" fr_prefix="rear"
-               lr_pos="${track / 2}"
-               fr_pos="${x_center_rocker - wheelbase_rocker / 2}"
-               />
-  <xacro:wheel lr_prefix="right_bogie" fr_prefix="front"
-               lr_pos="${- track / 2}"
-               fr_pos="${x_center_bogie + wheelbase_bogie / 2}"
-               />
-  <xacro:wheel lr_prefix="right_bogie" fr_prefix="rear"
-               lr_pos="${- track / 2}"
-               fr_pos="${x_center_bogie - wheelbase_bogie / 2}"
-               />
-  <xacro:wheel lr_prefix="right_rocker" fr_prefix="rear"
-               lr_pos="${- track / 2}"
-               fr_pos="${x_center_rocker - wheelbase_rocker / 2}"
-               />
   <gazebo>
     <sensor name="imu" type="imu">
@@ -511,8 +587,3 @@
       </plugin>
   </gazebo>
-  <ros2_control name="GazeboSystem" type="system">
-    <hardware>
-      <plugin>gazebo_ros2_control/GazeboSystem</plugin>
-    </hardware>
-  </ros2_control>
 </robot>
