Commit message: Fix arm buggit add .!

File: urc_gazebo/urdf/walli_arm_v3.urdf (robot description, URDF)
Before this commit: robot walli_arm_v3, 9 links, 8 joints
Links:
- link arm_base_link: geometry collision mesh filename=file://$(find urc_gazebo)/urdf/meshes/base_link_collision.S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; visual mesh filename=file://$(find urc_gazebo)/urdf/meshes/base_link.STL
- link bicep: geometry collision mesh filename=file://$(find urc_gazebo)/urdf/meshes/bicep_collision.STL; visual mesh filename=file://$(find urc_gazebo)/urdf/meshes/bicep.STL
- link claw: geometry collision mesh filename=file://$(find urc_gazebo)/urdf/meshes/claw_collision.STL; visual mesh filename=file://$(find urc_gazebo)/urdf/meshes/claw.STL
- link elbow: geometry collision mesh filename=file://$(find urc_gazebo)/urdf/meshes/elbow_collision.STL; visual mesh filename=file://$(find urc_gazebo)/urdf/meshes/elbow.STL
- link forearm: geometry collision mesh filename=file://$(find urc_gazebo)/urdf/meshes/forearm_collision.STL; visual mesh filename=file://$(find urc_gazebo)/urdf/meshes/forearm.STL
- link leftgripper: geometry collision mesh filename=file://$(find urc_gazebo)/urdf/meshes/leftgripper_collision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; visual mesh filename=file://$(find urc_gazebo)/urdf/meshes/leftgripper.STL
- link rightgripper: geometry collision mesh filename=file://$(find urc_gazebo)/urdf/meshes/rightgripper_collisio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; visual mesh filename=file://$(find urc_gazebo)/urdf/meshes/rightgripper.STL
- link shoulder: geometry collision mesh filename=file://$(find urc_gazebo)/urdf/meshes/shoulder_collision.STL; visual mesh filename=file://$(find urc_gazebo)/urdf/meshes/shoulder.STL
- link wrist: geometry collision mesh filename=file://$(find urc_gazebo)/urdf/meshes/wrist_collision.STL; visual mesh filename=file://$(find urc_gazebo)/urdf/meshes/wrist.STL
