Commit message: unknown changes

File: urc_gazebo/urdf/ros2_control.xacro (robot description, xacro)
@@ -5,5 +5,5 @@
             <plugin>gazebo_ros2_control/GazeboSystem</plugin>
         </hardware>
-        <joint name="left_wheel_joint">
+        <joint name="left_front_wheel_joint">
             <command_interface name="velocity">
                 <param name="min">-10</param>
@@ -13,5 +13,37 @@
             <state_interface name="position"/>
         </joint>
-        <joint name="right_wheel_joint">
+        <joint name="right_front_wheel_joint">
+            <command_interface name="velocity">
+                <param name="min">-10</param>
+                <param name="max">10</param>
+            </command_interface>
+            <state_interface name="velocity"/>
+            <state_interface name="position"/>
+        </joint>
+        <joint name="left_center_wheel_joint">
+            <command_interface name="velocity">
+                <param name="min">-10</param>
+                <param name="max">10</param>
+            </command_interface>
+            <state_interface name="velocity"/>
+            <state_interface name="position"/>
+        </joint>
+        <joint name="right_center_wheel_joint">
+            <command_interface name="velocity">
+                <param name="min">-10</param>
+                <param name="max">10</param>
+            </command_interface>
+            <state_interface name="velocity"/>
+            <state_interface name="position"/>
+        </joint>
+        <joint name="left_rear_wheel_joint">
+            <command_interface name="velocity">
+                <param name="min">-10</param>
+                <param name="max">10</param>
+            </command_interface>
+            <state_interface name="velocity"/>
+            <state_interface name="position"/>
+        </joint>
+        <joint name="right_rear_wheel_joint">
             <command_interface name="velocity">
                 <param name="min">-10</param>
@@ -23,6 +55,6 @@
     </ros2_control>
     <gazebo>
-        <plugin name="gazebo_ros2_control" filename="libgazebo_ros2_control.so">
-            <parameters>$(find articubot_one)/config/my_controllers.yaml</parameters>
+        <plugin name="gazebo_ros2_control/user" filename="libgazebo_ros2_control.so">
+            <parameters>$(find urc_gazebo)/config/my_controllers.yaml</parameters>
         </plugin>
     </gazebo>

File: urc_gazebo/urdf/walli.xacro (robot description, xacro)
@@ -5,4 +5,5 @@
   <xacro:include filename="$(find velodyne_description)/urdf/VLP-16.urdf.xacro"/>
   <xacro:include filename="walli_arm.urdf"/>
+  <xacro:include filename="ros2_control.xacro"/>
   <!-- Rover Base Link -->
   <link name="base_link">

Commit message: Editing some configs to make ros2 control work

File: urc_gazebo/urdf/ros2_control.xacro (robot description, xacro)
@@ -3,10 +3,15 @@
     <ros2_control name="GazeboSystem" type="system">
         <hardware>
+            <!-- TODO make a launch param to switch between real/fake hardware. You can only use ONE. -->
+            <!--Use for functionality in Gazebo, also needed for drivetrain-->
             <plugin>gazebo_ros2_control/GazeboSystem</plugin>
+            <!--Use for functionality in RViz-->
+            <!-- <plugin>mock_components/GenericSystem</plugin> -->
+            <!-- <plugin>ros2_control_demo_hardware/VelocityActuatorHardware</plugin> -->
         </hardware>
         <joint name="left_front_wheel_joint">
             <command_interface name="velocity">
-                <param name="min">-10</param>
-                <param name="max">10</param>
+                <param name="min">-0.05</param>
+                <param name="max">0.05</param>
             </command_interface>
             <state_interface name="velocity"/>
@@ -15,6 +20,6 @@
         <joint name="right_front_wheel_joint">
             <command_interface name="velocity">
-                <param name="min">-10</param>
-                <param name="max">10</param>
+                <param name="min">-0.05</param>
+                <param name="max">0.05</param>
             </command_interface>
             <state_interface name="velocity"/>
@@ -23,6 +28,6 @@
         <joint name="left_center_wheel_joint">
             <command_interface name="velocity">
-                <param name="min">-10</param>
-                <param name="max">10</param>
+                <param name="min">-0.05</param>
+                <param name="max">0.05</param>
             </command_interface>
             <state_interface name="velocity"/>
@@ -31,6 +36,6 @@
         <joint name="right_center_wheel_joint">
             <command_interface name="velocity">
-                <param name="min">-10</param>
-                <param name="max">10</param>
+                <param name="min">-0.05</param>
+                <param name="max">0.05</param>
             </command_interface>
             <state_interface name="velocity"/>
@@ -39,6 +44,6 @@
         <joint name="left_rear_wheel_joint">
             <command_interface name="velocity">
-                <param name="min">-10</param>
-                <param name="max">10</param>
+                <param name="min">-0.05</param>
+                <param name="max">0.05</param>
             </command_interface>
             <state_interface name="velocity"/>
@@ -47,14 +52,81 @@
         <joint name="right_rear_wheel_joint">
             <command_interface name="velocity">
-                <param name="min">-10</param>
-                <param name="max">10</param>
+                <param name="min">-0.05</param>
+                <param name="max">0.05</param>
             </command_interface>
             <state_interface name="velocity"/>
             <state_interface name="position"/>
         </joint>
+<!--
+      <joint name ="shoulderjoint">
+        <command_interface name="position" />
+        <state_interface name="position">
+          <param name="initial_value">0.0</param>
+        </state_interface>
+        <state_interface name="velocity"/>
+        <state_interface name="effort"/>
+      </joint>
+      <joint name ="bicepjoint">
+        <command_interface name="position" />
+        <state_interface name="position">
+          <param name="initial_value">0.0</param>
+        </state_interface>
+        <state_interface name="velocity"/>
+        <state_interface name="effort"/>
+      </joint>
+      <joint name ="elbowjoint">
+        <command_interface name="position" />
+        <state_interface name="position">
+          <param name="initial_value">0.0</param>
+        </state_interface>
+        <state_interface name="velocity"/>
+        <state_interface name="effort"/>
+      </joint>
+	<joint name ="forearmjoint">
+        <command_interface name="position" />
+        <state_interface name="position">
+          <param name="initial_value">0.0</param>
+        </state_interface>
+        <state_interface name="velocity"/>
+        <state_interface name="effort"/>
+      </joint>
+	<joint name ="wristjoint">
+        <command_interface name="position" />
+        <state_interface name="position">
+          <param name="initial_value">0.0</param>
+        </state_interface>
+        <state_interface name="velocity"/>
+        <state_interface name="effort"/>
+      </joint>
+      <joint name ="clawjoint">
+        <command_interface name="position" />
+        <state_interface name="position">
+          <param name="initial_value">0.0</param>
+        </state_interface>
+        <state_interface name="velocity"/>
+        <state_interface name="effort"/>
+      </joint>
+      <joint name ="leftgripperjoint">
+        <command_interface name="position" />
+        <state_interface name="position">
+          <param name="initial_value">0.0</param>
+        </state_interface>
+        <state_interface name="velocity"/>
+        <state_interface name="effort"/>
+      </joint>
+      <joint name ="rightgripperjoint">
+        <command_interface name="position" />
+        <state_interface name="position">
+          <param name="initial_value">0.0</param>
+        </state_interface>
+        <state_interface name="velocity"/>
+        <state_interface name="effort"/>
+      </joint> -->
     </ros2_control>
     <gazebo>
         <plugin name="gazebo_ros2_control" filename="libgazebo_ros2_control.so">
             <parameters>$(find urc_gazebo)/config/my_controllers.yaml</parameters>
+            <!-- Below is the one needed for the arm -->
+            <!-- <parameters>file://$(find urc_gazebo)/urdf/config/RoboticArm_params.yaml</parameters> -->
         </plugin>
     </gazebo>

File: urc_gazebo/urdf/walli.xacro (robot description, xacro)
@@ -4,5 +4,5 @@
   <xacro:include filename="walli_inertials.xacro"/>
   <xacro:include filename="$(find velodyne_description)/urdf/VLP-16.urdf.xacro"/>
-  <xacro:include filename="walli_arm.urdf"/>
+  <!-- <xacro:include filename="walli_arm.urdf"/> -->
   <xacro:include filename="ros2_control.xacro"/>
   <!-- Rover Base Link -->
@@ -30,5 +30,5 @@
     <link name="${prefix}_link">
       <visual>
-        <origin xyz="0 0 0" rpy="${pi/2} 0 0" />
+        <!-- <origin xyz="0 0 0" rpy="${y_reflect * pi/2} 0 0" /> -->
         <geometry>
           <cylinder radius="${wheel_radius}" length="${wheel_width}"/>
@@ -39,5 +39,5 @@
       </visual>
       <collision>
-        <origin xyz="0 0 0" rpy="${pi/2} 0 0"/>
+        <!-- <origin xyz="0 0 0" rpy="${y_reflect * pi/2} 0 0"/> -->
         <geometry>
           <cylinder radius="${wheel_radius}" length="${wheel_width}"/>
@@ -49,8 +49,8 @@
       <parent link="base_link"/>
       <child link="${prefix}_link"/>
-      <origin xyz="${x_reflect*wheel_xoff} ${y_reflect*(base_width/2+wheel_ygap)} ${-wheel_zoff}" rpy="0 0 0"/>
-      <axis xyz="0 1 0"/>
-      <limit effort="${axle_eff_limit}" velocity="${axle_vel_limit}"/>
-      <dynamics damping="0" friction="4.0" />
+      <origin xyz="${x_reflect*wheel_xoff} ${y_reflect*(base_width/2+wheel_ygap)} ${-wheel_zoff}" rpy="${pi/2} 0 0"/>
+      <axis xyz="0 0 1"/>
+      <!-- <limit effort="${axle_eff_limit}" velocity="${axle_vel_limit}"/>
+      <dynamics damping="0" friction="4.0" /> -->
     </joint>
     <gazebo reference="${prefix}_link">
@@ -70,11 +70,4 @@
     <child link="base_footprint"/>
     <origin xyz="0.0 0.0 ${-(wheel_radius+wheel_zoff)}" rpy="0 0 0"/>
-  </joint>
-  <!-- Arm Joint -->
-  <joint name="arm_to_rover" type="fixed">
-    <origin rpy="0 0 0" xyz="0 0 0"/>
-    <parent link="base_link"/>
-    <child link="arm_base_link"/>
-    <dynamics damping="60.0" friction="4.0"/>
   </joint>
   <!-- IMU -->

File: urc_gazebo/urdf/walli_arm.urdf (robot description, URDF)
Before this commit: robot walli_arm, 9 links, 8 joints
Joints:
- added joint arm_to_rover: type fixed, parent base_link, child arm_base_link, origin xyz=0 0 0 rpy=0 0 0

File: urc_gazebo/urdf/walli_prop.xacro (robot description, xacro)
@@ -7,14 +7,14 @@
   <xacro:property name="degrees_90" value="1.57079633"/>
   <!-- New Properties from NAV2-->
-  <xacro:property name="base_length"    value="0.300"/>
+  <xacro:property name="base_length"    value="0.600"/>
   <xacro:property name="base_width"     value="0.250"/>
-  <xacro:property name="base_height"    value="0.050"/>
-  <xacro:property name="base_mass"      value="3.000"/>
+  <xacro:property name="base_height"    value="0.100"/>
+  <xacro:property name="base_mass"      value="30.000"/>
   <xacro:property name="base_clearance" value="0.200"/>
-  <xacro:property name="wheel_radius" value="0.05"/>
-  <xacro:property name="wheel_width" value="0.075"/>
+  <xacro:property name="wheel_radius" value="0.03"/>
+  <xacro:property name="wheel_width" value="0.03"/>
   <xacro:property name="wheel_ygap" value="0.025"/>
   <xacro:property name="wheel_zoff" value="0.05"/>
-  <xacro:property name="wheel_xoff" value="0.12"/>
+  <xacro:property name="wheel_xoff" value="0.2"/>
   <!-- body_length is measured along the x axis, body_width
        along the y axis, and body_height along the z axis. -->

Commit message: MUncommented out arm things

File: urc_gazebo/urdf/ros2_control.xacro (robot description, xacro)
@@ -58,5 +58,4 @@
             <state_interface name="position"/>
         </joint>
-<!--
       <joint name ="shoulderjoint">
         <command_interface name="position" />
@@ -122,5 +121,5 @@
         <state_interface name="velocity"/>
         <state_interface name="effort"/>
-      </joint> -->
+      </joint>
     </ros2_control>
     <gazebo>
