Commit message: Made camera macro

File: urc_gazebo/urdf/walli.xacro (robot description, xacro)
@@ -298,9 +298,9 @@
    <!-- LIDAR -->
    <link name="lidar_support">
-        <visual>
-            <geometry>
-                <box size="${lidar_support_x_dim} ${lidar_support_y_dim} ${lidar_support_z_dim}"/>
-            </geometry>
-        </visual>
+      <visual>
+          <geometry>
+              <box size="${lidar_support_x_dim} ${lidar_support_y_dim} ${lidar_support_z_dim}"/>
+          </geometry>
+      </visual>
     </link>
     <joint name="base_link_to_lidar_support" type="fixed">
@@ -314,161 +314,61 @@
         <origin xyz="${lidar_x} 0.0 ${lidar_z}" rpy="0 ${lidar_pitch} 0" />
     </xacro:VLP-16>
-  <!-- cameras -->
-  <link name="cam/center">
-    <visual>
-      <geometry>
-        <box size="0.01 0.01 0.01"/>
-      </geometry>
-    </visual>
-    <collision>
-      <geometry>
-        <box size="0.01 0.01 0.01"/>
-      </geometry>
-    </collision>
-    <xacro:box_inertia m="0.01" w="0.01" d="0.01" h="0.01"/>
-  </link>
-  <joint name="center_cam_joint" type="fixed">
-	<axis xyz="1 0 0"/>
-	<!-- Edit these parameters to change camera orientation -->
-	<origin xyz="0.15 0 -0.1" rpy = "0 0 -.14"/>
-	<parent link="imu_link"/>
-	<child link="cam/center"/>
-   </joint>
-   <gazebo reference="cam/center">
-    <sensor name="center_sensor" type="camera">
-        <plugin name="center_sensor" filename="libgazebo_ros_camera.so">
+  <xacro:macro name="camera" params="orientation origin_x origin_y origin_z yaw">
+    <link name="cam/${orientation}">
+      <visual>
+        <geometry>
+          <box size="0.01 0.01 0.01"/>
+        </geometry>
+      </visual>
+      <collision>
+        <geometry>
+          <box size="0.01 0.01 0.01"/>
+        </geometry>
+      </collision>
+      <xacro:box_inertia m="0.01" w="0.01" d="0.01" h="0.01"/>
+    </link>
+    <joint name="${orientation}_cam_joint" type="fixed">
+  	  <axis xyz="1 0 0"/>
+      <!-- Camera Orientation-->
+	    <origin xyz="${origin_x} ${origin_y} ${origin_z}" rpy = "0 0 ${yaw}"/>
+	    <parent link="base_link"/>
+	    <child link="cam/${orientation}"/>
+    </joint>
+    <gazebo reference="cam/${orientation}">
+      <sensor name="${orientation}_sensor" type="camera">
+        <plugin name="${orientation}_sensor" filename="libgazebo_ros_camera.so">
         <ros>
           <namespace>/image</namespace>
-          <remapping>~/image_raw:=center_img</remapping>
+          <remapping>~/image_raw:=${orientation}_img</remapping>
           <remapping>~/camera_info:=camera_info</remapping>
         </ros>
         <initial_orientation_as_reference>false</initial_orientation_as_reference>
-      </plugin>
-      <always_on>true</always_on>
-      <update_rate>100</update_rate>
-      <visualize>true</visualize>
-      <camera name="cam/center">
-	<horizontal_fov>1.3962634</horizontal_fov>
-	<image>
-	<width>800</width>
-	<height>800</height>
-	<format>R8G8B8</format>
-	</image>
-	<clip>
-	<near>0.02</near>
-	<far>300</far>
-	</clip>
-	<noise>
-	<type>gaussian</type>
-	<mean>0</mean>
-	<stddev>0.007</stddev>
-	</noise>
-      </camera>
-    </sensor>
-  </gazebo>
-  <link name="cam/left">
-    <visual>
-      <geometry>
-        <box size="0.01 0.01 0.01"/>
-      </geometry>
-    </visual>
-    <collision>
-      <geometry>
-        <box size="0.01 0.01 0.01"/>
-      </geometry>
-    </collision>
-    <xacro:box_inertia m="0.01" w="0.01" d="0.01" h="0.01"/>
-  </link>
-  <joint name="left_cam_joint" type="fixed">
-	<axis xyz="1 0 0"/>
-	<!-- Edit these parameters to change camera orientation -->
-	<origin xyz="0 0.1 0.0" rpy = "0 0 1.5"/>
-	<parent link="base_link"/>
-	<child link="cam/left"/>
-   </joint>
-   <gazebo reference="cam/left">
-    <sensor name="left_sensor" type="camera">
-        <plugin name="left_sensor" filename="libgazebo_ros_camera.so">
-        <ros>
-          <namespace>/image</namespace>
-          <remapping>~/image_raw:=left_img</remapping>
-          <remapping>~/camera_info:=camera_info</remapping>
-        </ros>
-        <initial_orientation_as_reference>false</initial_orientation_as_reference>
-      </plugin>
-      <always_on>true</always_on>
-      <update_rate>100</update_rate>
-      <visualize>true</visualize>
-      <camera name="cam/left">
-        <horizontal_fov>1.3962634</horizontal_fov>
-	<image>
-	<width>800</width>
-	<height>800</height>
-	<format>R8G8B8</format>
-	</image>
-	<clip>
-	<near>0.02</near>
-	<far>300</far>
-	</clip>
-	<noise>
-	<type>gaussian</type>
-	<mean>0</mean>
-	<stddev>0.007</stddev>
-	</noise>
-      </camera>
-    </sensor>
-  </gazebo>
-  <link name="cam/right">
-    <visual>
-      <geometry>
-        <box size="0.01 0.01 0.01"/>
-      </geometry>
-    </visual>
-    <collision>
-      <geometry>
-        <box size="0.01 0.01 0.01"/>
-      </geometry>
-    </collision>
-    <xacro:box_inertia m="0.01" w="0.01" d="0.01" h="0.01"/>
-  </link>
-  <joint name="right_cam_joint" type="fixed">
-	<axis xyz="1 0 0"/>
-	<!-- Edit these parameters to change camera orientation -->
-	<origin xyz="0 -0.1 0.0" rpy = "0 0 -1.5"/>
-	<parent link="base_link"/>
-	<child link="cam/right"/>
-   </joint>
-   <gazebo reference="cam/right">
-    <sensor name="right_sensor" type="camera">
-        <plugin name="right_sensor" filename="libgazebo_ros_camera.so">
-        <ros>
-          <namespace>/image</namespace>
-          <remapping>~/image_raw:=right_img</remapping>
-          <remapping>~/camera_info:=camera_info</remapping>
-        </ros>
-        <initial_orientation_as_reference>false</initial_orientation_as_reference>
-      </plugin>
-      <always_on>true</always_on>
-      <update_rate>100</update_rate>
-      <visualize>true</visualize>
-      <camera name="cam/right">
-        <horizontal_fov>1.3962634</horizontal_fov>
-	<image>
-	<width>800</width>
-	<height>800</height>
-	<format>R8G8B8</format>
-	</image>
-	<clip>
-	<near>0.02</near>
-	<far>300</far>
-	</clip>
-	<noise>
-	<type>gaussian</type>
-	<mean>0</mean>
-	<stddev>0.007</stddev>
-	</noise>
-      </camera>
-    </sensor>
-  </gazebo>
+        </plugin>
+        <always_on>true</always_on>
+        <update_rate>100</update_rate>
+        <visualize>true</visualize>
+        <camera name="cam/${orientation}">
+          <horizontal_fov>1.3962634</horizontal_fov>
+          <image>
+            <width>800</width>
+            <height>800</height>
+            <format>R8G8B8</format>
+          </image>
+          <clip>
+            <near>0.02</near>
+            <far>300</far>
+          </clip>
+          <noise>
+            <type>gaussian</type>
+            <mean>0</mean>
+            <stddev>0.007</stddev>
+          </noise>
+        </camera>
+      </sensor>
+    </gazebo>
+  </xacro:macro>
+  <xacro:camera orientation="center" origin_x="0.15" origin_y="0"    origin_z="-0.1" yaw="-0.14"/>
+  <xacro:camera orientation="left"   origin_x="0"    origin_y="0.1"  origin_z="0"    yaw="1.5"/>
+  <xacro:camera orientation="right"  origin_x="0"    origin_y="-0.1" origin_z="0"    yaw="-1.5"/>
   <gazebo>
     <sensor name="imu" type="imu">

Commit message: Cleanup unnecessary repeated camera sensor info

File: urc_gazebo/urdf/walli.xacro (robot description, xacro)
@@ -57,5 +57,4 @@
     </gazebo>
   </xacro:macro>
-    <!-- Wheels    -->
   <xacro:wheel prefix="left_front_wheel"   x_reflect="1" y_reflect="-1"/>
   <xacro:wheel prefix="left_center_wheel"  x_reflect="0" y_reflect="-1"/>
@@ -78,79 +77,4 @@
     <dynamics damping="60.0" friction="4.0"/>
   </joint>
-    <!--
-    Mock/Untested ros2 control scheme for operating the rover with ros2 control.
-    This matches how the control is supposed to be set up, but is commented out
-    because the way the urdf is designed, it interferes with the arm control.
-    -->
-    <!--
-    <ros2_control name="rover_control" type="system">
-    <hardware>
-      <plugin>ros2_control_demo_hardware/VelocityActuatorHardware</plugin>
-    </hardware>
-    <joint name="left_bogie_front_axle">
-      <command_interface name="velocity">
-        <param name="min">-1</param>
-        <param name="max">1</param>
-      </command_interface>
-      <state_interface name="velocity"/>
-    </joint>
-    <joint name="left_bogie_rear_axle">
-      <command_interface name="velocity">
-        <param name="min">-1</param>
-        <param name="max">1</param>
-      </command_interface>
-      <state_interface name="velocity"/>
-    </joint>
-    <joint name="left_rocker_rear_axle">
-      <command_interface name="velocity">
-        <param name="min">-1</param>
-        <param name="max">1</param>
-      </command_interface>
-      <state_interface name="velocity"/>
-    </joint>
-    <joint name="right_bogie_front_axle">
-      <command_interface name="velocity">
-        <param name="min">-1</param>
-        <param name="max">1</param>
-      </command_interface>
-      <state_interface name="velocity"/>
-    </joint>
-    <joint name="right_bogie_rear_axle">
-      <command_interface name="velocity">
-        <param name="min">-1</param>
-        <param name="max">1</param>
-      </command_interface>
-      <state_interface name="velocity"/>
-    </joint>
-    <joint name="right_rocker_rear_axle">
-      <command_interface name="velocity">
-        <param name="min">-1</param>
-        <param name="max">1</param>
-      </command_interface>
-      <state_interface name="velocity"/>
-    </joint>
-    <transmission name="rover_transmission">
-      <plugin>transmission_interface/SimpleTransmission</plugin>
-      <joint name="left_bogie_front_axle" role="left_bogie_front_axle">
-        <mechanical_reduction>1</mechanical_reduction>
-      </joint>
-      <joint name="left_bogie_rear_axle" role="left_bogie_rear_axle">
-        <mechanical_reduction>1</mechanical_reduction>
-      </joint>
-      <joint name="left_rocker_rear_axle" role="left_rocker_rear_axle">
-        <mechanical_reduction>1</mechanical_reduction>
-      </joint>
-      <joint name="right_bogie_front_axle" role="right_bogie_front_axle">
-        <mechanical_reduction>1</mechanical_reduction>
-      </joint>
-      <joint name="right_bogie_rear_axle" role="right_bogie_rear_axle">
-        <mechanical_reduction>1</mechanical_reduction>
-      </joint>
-      <joint name="right_rocker_rear_axle" role="right_rocket_rear_axle">
-        <mechanical_reduction>1</mechanical_reduction>
-      </joint>
-    </transmission>
-    </ros2_control>
-    -->
   <!-- IMU -->
   <link name="imu_link">
@@ -338,10 +262,13 @@
       <sensor name="${orientation}_sensor" type="camera">
         <plugin name="${orientation}_sensor" filename="libgazebo_ros_camera.so">
-        <ros>
-          <namespace>/image</namespace>
-          <remapping>~/image_raw:=${orientation}_img</remapping>
-          <remapping>~/camera_info:=camera_info</remapping>
-        </ros>
-        <initial_orientation_as_reference>false</initial_orientation_as_reference>
+          <ros>
+            <namespace>/image</namespace>
+            <remapping>~/image_raw:=${orientation}_img</remapping>
+            <remapping>~/camera_info:=${orientation}_camera_info</remapping>
+          </ros>
+          <initial_orientation_as_reference>false</initial_orientation_as_reference>
+          <camera_name>${orientation}_camera</camera_name>
+          <frame_name>${orientation}_tf</frame_name>
+          <hack_baseline>0.07</hack_baseline>
         </plugin>
         <always_on>true</always_on>
@@ -374,9 +301,7 @@
     <sensor name="imu" type="imu">
       <always_on>true</always_on>
-      <!-- Publish at 30 hz -->
       <update_rate>30</update_rate>
       <plugin name="imu" filename="libgazebo_ros_imu_sensor.so">
         <ros>
-          <!-- Will publish to /imu/data -->
           <namespace>/imu</namespace>
           <argument>~/out:=data</argument>
@@ -385,89 +310,90 @@
       </plugin>
     </sensor>
-    <sensor type="camera" name="center_sensor">
-          <!-- Set always_on only sensor, not on plugin -->
-          <always_on>0</always_on>
-          <!-- Set update_rate only sensor, not on plugin -->
-          <update_rate>1</update_rate>
-          <!-- Use camera, not camera_triggered -->
-          <plugin name="center_sensor" filename="libgazebo_ros_camera.so">
-            <!-- Change namespace, camera name and topics so:
-                 * Images are published to: /custom_ns/custom_camera/custom_image
-                 * Camera info is published to: /custom_ns/custom_camera/custom_info
-            -->
-            <ros>
-              <namespace>/image</namespace>
-              <argument>~/image_raw:=center_img</argument>
-              <argument>~/camera_info:=center_info</argument>
-            </ros>
-            <!-- Set camera name. If empty, defaults to sensor name (i.e. "sensor_name") -->
-            <camera_name>center_camera</camera_name>
-            <!-- Set TF frame name. If empty, defaults to link name (i.e. "link_name") -->
-            <frame_name>center_tf</frame_name>
-            <hack_baseline>0.07</hack_baseline>
-            <!-- No need to repeat distortion parameters or to set autoDistortion -->
-          </plugin>
-        </sensor>
-     <sensor type="camera" name="left_sensor">
-          <!-- Set always_on only sensor, not on plugin -->
-          <always_on>0</always_on>
-          <!-- Set update_rate only sensor, not on plugin -->
-          <update_rate>1</update_rate>
-          <!-- Use camera, not camera_triggered -->
-          <plugin name="left_sensor" filename="libgazebo_ros_camera.so">
-            <!-- Change namespace, camera name and topics so:
-                 * Images are published to: /custom_ns/custom_camera/custom_image
-                 * Camera info is published to: /custom_ns/custom_camera/custom_info
-            -->
-            <ros>
-              <namespace>/image</namespace>
-              <argument>~/image_raw:=left_img</argument>
-              <argument>~/camera_info:=left_info</argument>
-            </ros>
-            <!-- Set camera name. If empty, defaults to sensor name (i.e. "sensor_name") -->
-            <camera_name>left_camera</camera_name>
-            <!-- Set TF frame name. If empty, defaults to link name (i.e. "link_name") -->
-            <frame_name>left_tf</frame_name>
-            <hack_baseline>0.07</hack_baseline>
-            <!-- No need to repeat distortion parameters or to set autoDistortion -->
-          </plugin>
-        </sensor>
-      <sensor type="camera" name="right_sensor">
-          <!-- Set always_on only sensor, not on plugin -->
-          <always_on>0</always_on>
-          <!-- Set update_rate only sensor, not on plugin -->
-          <update_rate>1</update_rate>
-          <!-- Use camera, not camera_triggered -->
-          <plugin name="right_sensor" filename="libgazebo_ros_camera.so">
-            <!-- Change namespace, camera name and topics so:
-                 * Images are published to: /custom_ns/custom_camera/custom_image
-                 * Camera info is published to: /custom_ns/custom_camera/custom_info
-            -->
-            <ros>
-              <namespace>/image</namespace>
-              <argument>~/image_raw:=right_img</argument>
-              <argument>~/camera_info:=right_info</argument>
-            </ros>
-            <!-- Set camera name. If empty, defaults to sensor name (i.e. "sensor_name") -->
-            <camera_name>right_camera</camera_name>
-            <!-- Set TF frame name. If empty, defaults to link name (i.e. "link_name") -->
-            <frame_name>right_tf</frame_name>
-            <hack_baseline>0.07</hack_baseline>
-            <!-- No need to repeat distortion parameters or to set autoDistortion -->
-          </plugin>
-        </sensor>
-      <plugin name="gazebo_ros_p3d" filename="libgazebo_ros_p3d.so">
-        <alwaysOn>true</alwaysOn>
-        <update_rate>30.0</update_rate>
-        <ros>
-          <namespace>/ground_truth</namespace>
-          <remapping>odom:=state_raw</remapping>
-        </ros>
-        <body_name>base_link</body_name>
-        <frame_name>world</frame_name>
-        <xyz_offset>0 0 0</xyz_offset>
-        <rpy_offset>0.0 0.0 0.0</rpy_offset>
-        <gaussian_noise>0.00</gaussian_noise>
-      </plugin>
+    <plugin name="gazebo_ros_p3d" filename="libgazebo_ros_p3d.so">
+      <alwaysOn>true</alwaysOn>
+      <update_rate>30.0</update_rate>
+      <ros>
+        <namespace>/ground_truth</namespace>
+        <remapping>odom:=state_raw</remapping>
+      </ros>
+      <body_name>base_link</body_name>
+      <frame_name>world</frame_name>
+      <xyz_offset>0 0 0</xyz_offset>
+      <rpy_offset>0.0 0.0 0.0</rpy_offset>
+      <gaussian_noise>0.00</gaussian_noise>
+    </plugin>
   </gazebo>
 </robot>
+    <!-- Mock/Untested ros2 control scheme for operating the rover with ros2 control.
+    This matches how the control is supposed to be set up, but is commented out
+    because the way the urdf is designed, it interferes with the arm control. -->
+    <!--
+    <ros2_control name="rover_control" type="system">
+    <hardware>
+      <plugin>ros2_control_demo_hardware/VelocityActuatorHardware</plugin>
+    </hardware>
+    <joint name="left_bogie_front_axle">
+      <command_interface name="velocity">
+        <param name="min">-1</param>
+        <param name="max">1</param>
+      </command_interface>
+      <state_interface name="velocity"/>
+    </joint>
+    <joint name="left_bogie_rear_axle">
+      <command_interface name="velocity">
+        <param name="min">-1</param>
+        <param name="max">1</param>
+      </command_interface>
+      <state_interface name="velocity"/>
+    </joint>
+    <joint name="left_rocker_rear_axle">
+      <command_interface name="velocity">
+        <param name="min">-1</param>
+        <param name="max">1</param>
+      </command_interface>
+      <state_interface name="velocity"/>
+    </joint>
+    <joint name="right_bogie_front_axle">
+      <command_interface name="velocity">
+        <param name="min">-1</param>
+        <param name="max">1</param>
+      </command_interface>
+      <state_interface name="velocity"/>
+    </joint>
+    <joint name="right_bogie_rear_axle">
+      <command_interface name="velocity">
+        <param name="min">-1</param>
+        <param name="max">1</param>
+      </command_interface>
+      <state_interface name="velocity"/>
+    </joint>
+    <joint name="right_rocker_rear_axle">
+      <command_interface name="velocity">
+        <param name="min">-1</param>
+        <param name="max">1</param>
+      </command_interface>
+      <state_interface name="velocity"/>
+    </joint>
+    <transmission name="rover_transmission">
+      <plugin>transmission_interface/SimpleTransmission</plugin>
+      <joint name="left_bogie_front_axle" role="left_bogie_front_axle">
+        <mechanical_reduction>1</mechanical_reduction>
+      </joint>
+      <joint name="left_bogie_rear_axle" role="left_bogie_rear_axle">
+        <mechanical_reduction>1</mechanical_reduction>
+      </joint>
+      <joint name="left_rocker_rear_axle" role="left_rocker_rear_axle">
+        <mechanical_reduction>1</mechanical_reduction>
+      </joint>
+      <joint name="right_bogie_front_axle" role="right_bogie_front_axle">
+        <mechanical_reduction>1</mechanical_reduction>
+      </joint>
+      <joint name="right_bogie_rear_axle" role="right_bogie_rear_axle">
+        <mechanical_reduction>1</mechanical_reduction>
+      </joint>
+      <joint name="right_rocker_rear_axle" role="right_rocket_rear_axle">
+        <mechanical_reduction>1</mechanical_reduction>
+      </joint>
+    </transmission>
+    </ros2_control>
+    -->
