Commit message: Fixed lidar somewhat but not enough

File: urc_gazebo/urdf/walli.xacro (robot description, xacro)
@@ -221,21 +221,66 @@
   </gazebo>
    <!-- LIDAR -->
-   <link name="lidar_support">
-      <visual>
-          <geometry>
-              <box size="${lidar_support_x_dim} ${lidar_support_y_dim} ${lidar_support_z_dim}"/>
-          </geometry>
-      </visual>
-    </link>
-    <joint name="base_link_to_lidar_support" type="fixed">
-        <parent link="base_link"/>
-        <child link="lidar_support"/>
-        <origin xyz="0.0 0.0 0.0" rpy="0.0 0.0 0.0"/>
-    </joint>
-    <!-- collision range = min sensing distance -->
-    <!-- gpu does gpu acceleration -->
-    <xacro:VLP-16 parent="lidar_support" name="lidar" topic="/scan" hz="${lidar_hz}" samples="${lidar_samples}" gpu="false">
-        <origin xyz="${lidar_x} 0.0 ${lidar_z}" rpy="0 ${lidar_pitch} 0" />
-    </xacro:VLP-16>
+  <link name="lidar_link">
+    <inertial>
+      <origin xyz="0 0 0" rpy="0 0 0"/>
+      <mass value="0.125"/>
+      <inertia ixx="0.001"  ixy="0"  ixz="0" iyy="0.001" iyz="0" izz="0.001" />
+    </inertial>
+    <collision>
+      <origin xyz="0 0 0" rpy="0 0 0"/>
+      <geometry>
+        <cylinder radius="0.0508" length="0.055"/>
+      </geometry>
+    </collision>
+    <visual>
+      <origin xyz="0 0 0" rpy="0 0 0"/>
+      <geometry>
+        <cylinder radius="0.0508" length="0.055"/>
+      </geometry>
+    </visual>
+  </link>
+  <joint name="lidar_joint" type="fixed">
+    <parent link="base_link"/>
+    <child link="lidar_link"/>
+    <origin xyz="0.0 0.0 0.0" rpy="0.0 0.0 0.0"/>
+  </joint>
+  <xacro:VLP-16 parent="lidar_link" name="lidar" topic="/scan" hz="${lidar_hz}" samples="${lidar_samples}" gpu="false">
+    <origin xyz="${lidar_x} 0.0 ${lidar_z}" rpy="0 ${lidar_pitch} 0" />
+  </xacro:VLP-16>
+  <gazebo reference="lidar_link">
+  <sensor name="lidar" type="ray">
+    <always_on>true</always_on>
+    <visualize>true</visualize>
+    <update_rate>5</update_rate>
+    <ray>
+      <scan>
+        <horizontal>
+          <samples>360</samples>
+          <resolution>1.000000</resolution>
+          <min_angle>0.000000</min_angle>
+          <max_angle>6.280000</max_angle>
+        </horizontal>
+      </scan>
+      <range>
+        <min>0.120000</min>
+        <max>3.5</max>
+        <resolution>0.015000</resolution>
+      </range>
+      <noise>
+        <type>gaussian</type>
+        <mean>0.0</mean>
+        <stddev>0.01</stddev>
+      </noise>
+    </ray>
+    <plugin name="scan" filename="libgazebo_ros_ray_sensor.so">
+      <ros>
+        <remapping>~/out:=scan</remapping>
+      </ros>
+      <output_type>sensor_msgs/LaserScan</output_type>
+      <frame_name>lidar_link</frame_name>
+    </plugin>
+  </sensor>
+</gazebo>
+  <!-- May want to change this to a depth camera -->
   <xacro:macro name="camera" params="orientation origin_x origin_y origin_z yaw">
     <link name="cam/${orientation}">

File: urc_gazebo/urdf/walli_prop.xacro (robot description, xacro)
@@ -54,10 +54,7 @@
    <!-- Lidar -->
     <xacro:property name="lidar_pitch" value="0.0"/>
-    <xacro:property name="lidar_x" value="0.127"/>
-    <xacro:property name="lidar_z" value="0.8486"/>
+    <xacro:property name="lidar_x" value="0.12"/>
+    <xacro:property name="lidar_z" value="0.12"/>
     <xacro:property name="lidar_hz" value="10"/>
     <xacro:property name="lidar_samples" value="500"/>
-    <xacro:property name="lidar_support_x_dim" value="0.2"/>
-    <xacro:property name="lidar_support_y_dim" value="0.08"/>
-    <xacro:property name="lidar_support_z_dim" value="0.01"/>
 </robot>

Commit message: Almost finalized config

File: urc_gazebo/urdf/walli.xacro (robot description, xacro)
@@ -57,10 +57,10 @@
     </gazebo>
   </xacro:macro>
-  <xacro:wheel prefix="left_front_wheel"   x_reflect="1" y_reflect="-1"/>
-  <xacro:wheel prefix="left_center_wheel"  x_reflect="0" y_reflect="-1"/>
-  <xacro:wheel prefix="left_rear_wheel"    x_reflect="-1" y_reflect="-1"/>
-  <xacro:wheel prefix="right_front_wheel"  x_reflect="1" y_reflect="1"/>
-  <xacro:wheel prefix="right_center_wheel" x_reflect="0" y_reflect="1"/>
-  <xacro:wheel prefix="right_rear_wheel"   x_reflect="-1" y_reflect="1"/>
+  <xacro:wheel prefix="left_front_wheel"   x_reflect="1" y_reflect="1"/>
+  <xacro:wheel prefix="left_center_wheel"  x_reflect="0" y_reflect="1"/>
+  <xacro:wheel prefix="left_rear_wheel"    x_reflect="-1" y_reflect="1"/>
+  <xacro:wheel prefix="right_front_wheel"  x_reflect="1" y_reflect="-1"/>
+  <xacro:wheel prefix="right_center_wheel" x_reflect="0" y_reflect="-1"/>
+  <xacro:wheel prefix="right_rear_wheel"   x_reflect="-1" y_reflect="-1"/>
   <!-- Robot Footprint -->
   <link name="base_footprint"/>
@@ -243,9 +243,9 @@
     <parent link="base_link"/>
     <child link="lidar_link"/>
-    <origin xyz="0.0 0.0 0.0" rpy="0.0 0.0 0.0"/>
+    <origin xyz="0.0 0.0 0.1" rpy="0.0 0.0 0.0"/>
   </joint>
-  <xacro:VLP-16 parent="lidar_link" name="lidar" topic="/scan" hz="${lidar_hz}" samples="${lidar_samples}" gpu="false">
+  <!-- <xacro:VLP-16 parent="lidar_link" name="lidar" topic="/scan" hz="${lidar_hz}" samples="${lidar_samples}" gpu="false">
     <origin xyz="${lidar_x} 0.0 ${lidar_z}" rpy="0 ${lidar_pitch} 0" />
-  </xacro:VLP-16>
+  </xacro:VLP-16> -->
   <gazebo reference="lidar_link">
   <sensor name="lidar" type="ray">
@@ -263,5 +263,5 @@
       </scan>
       <range>
-        <min>0.120000</min>
+        <min>0.12</min>
         <max>3.5</max>
         <resolution>0.015000</resolution>
@@ -343,4 +343,71 @@
   <xacro:camera orientation="left"   origin_x="0"    origin_y="0.1"  origin_z="0"    yaw="1.5"/>
   <xacro:camera orientation="right"  origin_x="0"    origin_y="-0.1" origin_z="0"    yaw="-1.5"/>
+<!-- Depth Camera (addition for Nav2) -->
+<link name="camera_link">
+  <visual>
+    <origin xyz="0 0 0" rpy="0 0 0"/>
+    <geometry>
+      <box size="0.015 0.130 0.022"/>
+    </geometry>
+  </visual>
+  <collision>
+    <origin xyz="0 0 0" rpy="0 0 0"/>
+    <geometry>
+      <box size="0.015 0.130 0.022"/>
+    </geometry>
+  </collision>
+  <inertial>
+    <origin xyz="0 0 0" rpy="0 0 0"/>
+    <mass value="0.035"/>
+    <inertia ixx="0.001"  ixy="0"  ixz="0" iyy="0.001" iyz="0" izz="0.001" />
+  </inertial>
+</link>
+<joint name="camera_joint" type="fixed">
+  <parent link="base_link"/>
+  <child link="camera_link"/>
+  <origin xyz="0.215 0 0.05" rpy="0 0 0"/>
+</joint>
+<link name="camera_depth_frame"/>
+<joint name="camera_depth_joint" type="fixed">
+  <origin xyz="0 0 0" rpy="${-pi/2} 0 ${-pi/2}"/>
+  <parent link="camera_link"/>
+  <child link="camera_depth_frame"/>
+</joint>
+<gazebo reference="camera_link">
+  <sensor name="depth_camera" type="depth">
+    <visualize>true</visualize>
+    <update_rate>30.0</update_rate>
+    <camera name="camera">
+      <horizontal_fov>1.047198</horizontal_fov>
+      <image>
+        <width>640</width>
+        <height>480</height>
+        <format>R8G8B8</format>
+      </image>
+      <clip>
+        <near>0.05</near>
+        <far>3</far>
+      </clip>
+    </camera>
+    <plugin name="depth_camera_controller" filename="libgazebo_ros_camera.so">
+      <baseline>0.2</baseline>
+      <alwaysOn>true</alwaysOn>
+      <updateRate>0.0</updateRate>
+      <frame_name>camera_depth_frame</frame_name>
+      <pointCloudCutoff>0.5</pointCloudCutoff>
+      <pointCloudCutoffMax>3.0</pointCloudCutoffMax>
+      <distortionK1>0</distortionK1>
+      <distortionK2>0</distortionK2>
+      <distortionK3>0</distortionK3>
+      <distortionT1>0</distortionT1>
+      <distortionT2>0</distortionT2>
+      <CxPrime>0</CxPrime>
+      <Cx>0</Cx>
+      <Cy>0</Cy>
+      <focalLength>0</focalLength>
+      <hackBaseline>0</hackBaseline>
+    </plugin>
+  </sensor>
+</gazebo>
   <gazebo>
     <sensor name="imu" type="imu">

Commit message: sensor origin fixes

File: urc_gazebo/urdf/walli.xacro (robot description, xacro)
@@ -340,5 +340,5 @@
     </gazebo>
   </xacro:macro>
-  <xacro:camera orientation="center" origin_x="0.15" origin_y="0"    origin_z="-0.1" yaw="-0.14"/>
+  <xacro:camera orientation="center" origin_x="0.1" origin_y="0"    origin_z="0" yaw="-0.14"/>
   <xacro:camera orientation="left"   origin_x="0"    origin_y="0.1"  origin_z="0"    yaw="1.5"/>
   <xacro:camera orientation="right"  origin_x="0"    origin_y="-0.1" origin_z="0"    yaw="-1.5"/>
@@ -366,5 +366,5 @@
   <parent link="base_link"/>
   <child link="camera_link"/>
-  <origin xyz="0.215 0 0.05" rpy="0 0 0"/>
+  <origin xyz="0.1 0 0.03" rpy="0 0 0"/>
 </joint>
 <link name="camera_depth_frame"/>

Commit message: fixed issues as addressed by Yashas Ambati

File: urc_gazebo/urdf/walli.xacro (robot description, xacro)
@@ -27,8 +27,8 @@
   </gazebo>
   <!-- Wheels -->
-  <xacro:macro name="wheel" params="prefix x_reflect y_reflect">
+  <xacro:macro name="wheel" params="prefix x_reflect y_reflect z_reflect">
     <link name="${prefix}_link">
       <visual>
-        <!-- <origin xyz="0 0 0" rpy="${y_reflect * pi/2} 0 0" /> -->
+        <origin xyz="0 0 0" rpy="0 0 ${z_reflect * pi}" />
         <geometry>
           <cylinder radius="${wheel_radius}" length="${wheel_width}"/>
@@ -39,5 +39,5 @@
       </visual>
       <collision>
-        <!-- <origin xyz="0 0 0" rpy="${y_reflect * pi/2} 0 0"/> -->
+        <origin xyz="0 0 0" rpy="0 0 ${z_reflect * pi}" />
         <geometry>
           <cylinder radius="${wheel_radius}" length="${wheel_width}"/>
@@ -51,6 +51,4 @@
       <origin xyz="${x_reflect*wheel_xoff} ${y_reflect*(base_width/2+wheel_ygap)} ${-wheel_zoff}" rpy="${pi/2} 0 0"/>
       <axis xyz="0 0 1"/>
-      <!-- <limit effort="${axle_eff_limit}" velocity="${axle_vel_limit}"/>
-      <dynamics damping="0" friction="4.0" /> -->
     </joint>
     <gazebo reference="${prefix}_link">
@@ -58,10 +56,10 @@
     </gazebo>
   </xacro:macro>
-  <xacro:wheel prefix="left_front_wheel"   x_reflect="1" y_reflect="1"/>
-  <xacro:wheel prefix="left_center_wheel"  x_reflect="0" y_reflect="1"/>
-  <xacro:wheel prefix="left_rear_wheel"    x_reflect="-1" y_reflect="1"/>
-  <xacro:wheel prefix="right_front_wheel"  x_reflect="1" y_reflect="-1"/>
-  <xacro:wheel prefix="right_center_wheel" x_reflect="0" y_reflect="-1"/>
-  <xacro:wheel prefix="right_rear_wheel"   x_reflect="-1" y_reflect="-1"/>
+  <xacro:wheel prefix="left_front_wheel"   x_reflect="1" y_reflect="1" z_reflect="0"/>
+  <xacro:wheel prefix="left_center_wheel"  x_reflect="0" y_reflect="1" z_reflect="0"/>
+  <xacro:wheel prefix="left_rear_wheel"    x_reflect="-1" y_reflect="1" z_reflect="0"/>
+  <xacro:wheel prefix="right_front_wheel"  x_reflect="1" y_reflect="-1" z_reflect="1"/>
+  <xacro:wheel prefix="right_center_wheel" x_reflect="0" y_reflect="-1" z_reflect="1"/>
+  <xacro:wheel prefix="right_rear_wheel"   x_reflect="-1" y_reflect="-1" z_reflect="1"/>
   <!-- Robot Footprint -->
   <link name="base_footprint"/>
