Commit message: this is so sick our robot responds to the controller now

File: urc_arm_moveit_config/config/WalliiArmV3.urdf.xacro (robot description, xacro)
@@ -6,4 +6,4 @@
     <!-- Import control_xacro -->
     <xacro:include filename="WalliiArmV3.ros2_control.xacro" />
-    <xacro:WalliiArmV3_ros2_control name="FakeSystem" initial_positions_file="$(arg initial_positions_file)"/>
+    <xacro:WalliiArmV3_ros2_control name="GazeboSystem" initial_positions_file="$(arg initial_positions_file)"/>
 </robot>

File: urc_gazebo/urdf/WalliiArmV3.urdf (robot description, URDF)
Before this commit: robot WalliiArmV3, 10 links, 9 joints
Links:
- link base_link: geometry collision mesh filename=package://urc_gazebo/urdf/meshes/base_link_collision.STL; visual mesh filename=package://urc_gazebo/urdf/meshes/base_link.STL
- link bicep: geometry collision mesh filename=package://urc_gazebo/urdf/meshes/bicep_collision.STL; visual mesh filename=package://urc_gazebo/urdf/meshes/bicep.STL
- link claw: geometry collision mesh filename=package://urc_gazebo/urdf/meshes/claw_collision.STL; visual mesh filename=package://urc_gazebo/urdf/meshes/claw.STL
- link elbow: geometry collision mesh filename=package://urc_gazebo/urdf/meshes/elbow_collision.STL; visual mesh filename=package://urc_gazebo/urdf/meshes/elbow.STL
- link forearm: geometry collision mesh filename=package://urc_gazebo/urdf/meshes/forearm_collision.STL; visual mesh filename=package://urc_gazebo/urdf/meshes/forearm.STL
- link leftgripper: geometry collision mesh filename=package://urc_gazebo/urdf/meshes/leftgripper_collision.STL; visual mesh filename=package://urc_gazebo/urdf/meshes/leftgripper.STL
- link rightgripper: geometry collision mesh filename=package://urc_gazebo/urdf/meshes/rightgripper_collision.STL; visual mesh filename=package://urc_gazebo/urdf/meshes/rightgripper.STL
- link shoulder: geometry collision mesh filename=package://urc_gazebo/urdf/meshes/shoulder_collision.STL; visual mesh filename=package://urc_gazebo/urdf/meshes/shoulder.STL
- link wrist: geometry collision mesh filename=package://urc_gazebo/urdf/meshes/wrist_collision.STL; visual mesh filename=package://urc_gazebo/urdf/meshes/wrist.STL

Commit message: manual control arm integrated onto current rover

File: urc_arm_moveit_config/config/WalliiArmV3.urdf.xacro (robot description, xacro)
@@ -3,5 +3,5 @@
     <xacro:arg name="initial_positions_file" default="initial_positions.yaml" />
     <!-- Import WalliiArmV3 urdf file -->
-    <xacro:include filename="$(find urc_gazebo)/urdf/WalliiArmV3.urdf" />
+    <xacro:include filename="$(find urc_gazebo)/urdf/wallii.xacro" />
     <!-- Import control_xacro -->
     <xacro:include filename="WalliiArmV3.ros2_control.xacro" />

File: urc_gazebo/urdf/WalliiArmV3.urdf (robot description, URDF)
Before this commit: robot WalliiArmV3, 10 links, 9 joints
Links:
- removed link base_link
- removed link world
- added link arm_base_link, mass 0.56817; collision mesh filename=package://urc_gazebo/urdf/meshes/base_link_collision.STL; visual mesh filename=package://urc_gazebo/urdf/meshes/base_link.STL
Joints:
- removed joint world_to_base
- joint shoulderjoint: parent base_link -> arm_base_link

File: urc_gazebo/urdf/walli_prop.xacro (robot description, xacro)
@@ -10,5 +10,5 @@
   <xacro:property name="body_width"     value="0.250"/>
   <xacro:property name="body_height"    value="0.050"/>
-  <xacro:property name="body_mass"      value="3.000"/>
+  <xacro:property name="body_mass"      value="50.000"/>
   <xacro:property name="body_clearance" value="0.200"/>
   <xacro:property name="wheelbase_rocker" value="0.350"/>

File: urc_gazebo/urdf/wallii.xacro (robot description, xacro)
@@ -4,29 +4,8 @@
   <xacro:include filename="walli_inertials.xacro"/>
   <xacro:include filename="$(find velodyne_description)/urdf/VLP-16.urdf.xacro"/>
-  <xacro:include filename="RoboticArm.urdf"/>
+  <xacro:include filename="WalliiArmV3.urdf"/>
+  <!--- Something about this macro breaks the urdf parser. -->
   <!-- The "wheel" macro defines an axle carrier, axle, and wheel. -->
   <xacro:macro name="wheel" params="lr_prefix fr_prefix lr_pos fr_pos">
-    <joint name="${lr_prefix}_${fr_prefix}_axle" type="continuous">
-      <parent link="base_link"/>
-      <child link="${lr_prefix}_${fr_prefix}_wheel"/>
-      <origin xyz="${fr_pos}
-                   ${lr_pos}
-                   ${- body_clearance}"
-              rpy="${degrees_90} 0 0"/>
-      <axis xyz="0 0 -1"/>
-      <limit effort="${axle_eff_limit}" velocity="${axle_vel_limit}"/>
-    </joint>
-    <ros2_control name="GazeboSystem" type="system">
-      <transmission name="${lr_prefix}_${fr_prefix}_axle_trans">
-        <type>transmission_interface/SimpleTransmission</type>
-        <joint name="${lr_prefix}_${fr_prefix}_axle">
-          <hardwareInterface>VelocityJointInterface</hardwareInterface>
-        </joint>
-        <actuator name="${lr_prefix}_${fr_prefix}_axle_act">
-          <hardwareInterface>VelocityJointInterface</hardwareInterface>
-          <mechanicalReduction>1</mechanicalReduction>
-        </actuator>
-      </transmission>
-    </ros2_control>
     <link name="${lr_prefix}_${fr_prefix}_wheel">
       <visual>
@@ -47,4 +26,14 @@
           height="${tire_width}" mass="${wheel_mass}"/>
     </link>
+    <joint name="${lr_prefix}_${fr_prefix}_axle" type="continuous">
+      <parent link="base_link"/>
+      <child link="${lr_prefix}_${fr_prefix}_wheel"/>
+      <origin xyz="${fr_pos}
+                   ${lr_pos}
+                   ${- body_clearance}"
+              rpy="${degrees_90} 0 0"/>
+      <axis xyz="0 0 -1"/>
+      <limit effort="${axle_eff_limit}" velocity="${axle_vel_limit}"/>
+    </joint>
     <gazebo reference="${lr_prefix}_${fr_prefix}_wheel">
       <material>Gazebo/Black</material>
@@ -64,20 +53,151 @@
     <material>Gazebo/Green</material>
   </gazebo>
+    <!-- body -->
+  <link name="body">
+    <visual>
+      <origin xyz="0 0 ${-body_height / 2}"/>
+      <geometry>
+        <box size="${body_length} ${body_width} ${body_height}"/>
+      </geometry>
+      <material name="body_mat"/>
+    </visual>
+    <collision>
+      <origin xyz="0 0 ${-body_height / 2}"/>
+      <geometry>
+        <box size="${body_length} ${body_width} ${body_height}"/>
+      </geometry>
+    </collision>
+    <xacro:solid_cuboid_inertial
+        width="${body_length}" depth="${body_width}"
+        height="${body_height}" mass="${body_mass}">
+      <origin xyz="0 0 ${-body_height / 2}"/>
+    </xacro:solid_cuboid_inertial>
+  </link>
+  <gazebo reference="body">
+    <material>Gazebo/Grey</material>
+  </gazebo>
+  <joint name="base_link_to_chasis" type="fixed">
+    <parent link="base_link"/>
+    <child link="body"/>
+  </joint>
+    <!-- breaking urdf parser -->
+  <!-- Wheels    -->
+  <xacro:wheel lr_prefix="left_bogie" fr_prefix="front"
+               lr_pos="${track / 2}"
+               fr_pos="${x_center_bogie + wheelbase_bogie / 2}"
+               />
+  <xacro:wheel lr_prefix="left_bogie" fr_prefix="rear"
+               lr_pos="${track / 2}"
+               fr_pos="${x_center_bogie - wheelbase_bogie / 2}"
+               />
+  <xacro:wheel lr_prefix="left_rocker" fr_prefix="rear"
+               lr_pos="${track / 2}"
+               fr_pos="${x_center_rocker - wheelbase_rocker / 2}"
+               />
+  <xacro:wheel lr_prefix="right_bogie" fr_prefix="front"
+               lr_pos="${- track / 2}"
+               fr_pos="${x_center_bogie + wheelbase_bogie / 2}"
+               />
+  <xacro:wheel lr_prefix="right_bogie" fr_prefix="rear"
+               lr_pos="${- track / 2}"
+               fr_pos="${x_center_bogie - wheelbase_bogie / 2}"
+               />
+  <xacro:wheel lr_prefix="right_rocker" fr_prefix="rear"
+               lr_pos="${- track / 2}"
+               fr_pos="${x_center_rocker - wheelbase_rocker / 2}"
+               />
+  <!-- connect rover and arm -->
+  <joint name="arm_to_rover" type="fixed">
+    <origin rpy="0 0 0" xyz="0 0 0"/>
+    <parent link="base_link"/>
+    <child link="arm_base_link"/>
+    <dynamics damping="60.0" friction="4.0"/>
+  </joint>
+    <!--
+    <ros2_control name="rover_control" type="system">
+    <hardware>
+      <plugin>ros2_control_demo_hardware/VelocityActuatorHardware</plugin>
+    </hardware>
+    <joint name="left_bogie_front_axle">
+      <command_interface name="velocity">
+        <param name="min">-1</param>
+        <param name="max">1</param>
+      </command_interface>
+      <state_interface name="velocity"/>
+    </joint>
+    <joint name="left_bogie_rear_axle">
+      <command_interface name="velocity">
+        <param name="min">-1</param>
+        <param name="max">1</param>
+      </command_interface>
+      <state_interface name="velocity"/>
+    </joint>
+    <joint name="left_rocker_rear_axle">
+      <command_interface name="velocity">
+        <param name="min">-1</param>
+        <param name="max">1</param>
+      </command_interface>
+      <state_interface name="velocity"/>
+    </joint>
+    <joint name="right_bogie_front_axle">
+      <command_interface name="velocity">
+        <param name="min">-1</param>
+        <param name="max">1</param>
+      </command_interface>
+      <state_interface name="velocity"/>
+    </joint>
+    <joint name="right_bogie_rear_axle">
+      <command_interface name="velocity">
+        <param name="min">-1</param>
+        <param name="max">1</param>
+      </command_interface>
+      <state_interface name="velocity"/>
+    </joint>
+    <joint name="right_rocker_rear_axle">
+      <command_interface name="velocity">
+        <param name="min">-1</param>
+        <param name="max">1</param>
+      </command_interface>
+      <state_interface name="velocity"/>
+    </joint>
+    <transmission name="rover_transmission">
+      <plugin>transmission_interface/SimpleTransmission</plugin>
+      <joint name="left_bogie_front_axle" role="left_bogie_front_axle">
+        <mechanical_reduction>1</mechanical_reduction>
+      </joint>
+      <joint name="left_bogie_rear_axle" role="left_bogie_rear_axle">
+        <mechanical_reduction>1</mechanical_reduction>
+      </joint>
+      <joint name="left_rocker_rear_axle" role="left_rocker_rear_axle">
+        <mechanical_reduction>1</mechanical_reduction>
+      </joint>
+      <joint name="right_bogie_front_axle" role="right_bogie_front_axle">
+        <mechanical_reduction>1</mechanical_reduction>
+      </joint>
+      <joint name="right_bogie_rear_axle" role="right_bogie_rear_axle">
+        <mechanical_reduction>1</mechanical_reduction>
+      </joint>
+      <joint name="right_rocker_rear_axle" role="right_rocket_rear_axle">
+        <mechanical_reduction>1</mechanical_reduction>
+      </joint>
+    </transmission>
+    </ros2_control>
+    -->
   <link name="imu">
     <visual>
       <geometry>
-        <box size="0.1 0.1 0.1"/>
+        <box size="0.01 0.01 0.01"/>
       </geometry>
     </visual>
     <collision>
       <geometry>
-        <box size="0.1 0.1 0.1"/>
+        <box size="0.01 0.01 0.01"/>
       </geometry>
     </collision>
-    <xacro:box_inertia m="0.1" w="0.1" d="0.1" h="0.1"/>
+    <xacro:box_inertia m="0.01" w="0.01" d="0.01" h="0.01"/>
   </link>
   <joint name="imu_joint" type="fixed">
 		<axis xyz="1 0 0"/>
-		<origin xyz="0 0 .4"/>
+		<origin xyz="0 0 0.1"/>
 		<parent link="base_link"/>
 		<child link="imu"/>
@@ -155,13 +275,13 @@
     <visual>
       <geometry>
-        <box size="0.1 0.1 0.1"/>
+        <box size="0.01 0.01 0.01"/>
       </geometry>
     </visual>
     <collision>
       <geometry>
-        <box size="0.1 0.1 0.1"/>
+        <box size="0.01 0.01 0.01"/>
       </geometry>
     </collision>
-    <xacro:box_inertia m="0.1" w="0.1" d="0.1" h="0.1"/>
+    <xacro:box_inertia m="0.01" w="0.01" d="0.01" h="0.01"/>
   </link>
    <joint name="gps_joint" type="fixed">
@@ -199,20 +319,20 @@
     <!-- collision range = min sensing distance -->
     <!-- gpu does gpu acceleration -->
-    <xacro:VLP-16 parent="lidar_support" name="lidar" topic="/scan" hz="${lidar_hz}" samples="${lidar_samples}" gpu="false">
+    <!-- <xacro:VLP-16 parent="lidar_support" name="lidar" topic="/scan" hz="${lidar_hz}" samples="${lidar_samples}" gpu="false">
         <origin xyz="${lidar_x} 0.0 ${lidar_z}" rpy="0 ${lidar_pitch} 0" />
-    </xacro:VLP-16>
+    </xacro:VLP-16> -->
   <!-- cameras -->
   <link name="cam/center">
     <visual>
       <geometry>
-        <box size="0.1 0.1 0.1"/>
+        <box size="0.01 0.01 0.01"/>
       </geometry>
     </visual>
     <collision>
       <geometry>
-        <box size="0.1 0.1 0.1"/>
+        <box size="0.01 0.01 0.01"/>
       </geometry>
     </collision>
-    <xacro:box_inertia m="0.1" w="0.1" d="0.1" h="0.1"/>
+    <xacro:box_inertia m="0.01" w="0.01" d="0.01" h="0.01"/>
   </link>
   <joint name="center_cam_joint" type="fixed">
@@ -258,13 +378,13 @@
     <visual>
       <geometry>
-        <box size="0.1 0.1 0.1"/>
+        <box size="0.01 0.01 0.01"/>
       </geometry>
     </visual>
     <collision>
       <geometry>
-        <box size="0.1 0.1 0.1"/>
+        <box size="0.01 0.01 0.01"/>
       </geometry>
     </collision>
-    <xacro:box_inertia m="0.1" w="0.1" d="0.1" h="0.1"/>
+    <xacro:box_inertia m="0.01" w="0.01" d="0.01" h="0.01"/>
   </link>
   <joint name="left_cam_joint" type="fixed">
@@ -310,13 +430,13 @@
     <visual>
       <geometry>
-        <box size="0.1 0.1 0.1"/>
+        <box size="0.01 0.01 0.01"/>
       </geometry>
     </visual>
     <collision>
       <geometry>
-        <box size="0.1 0.1 0.1"/>
+        <box size="0.01 0.01 0.01"/>
       </geometry>
     </collision>
-    <xacro:box_inertia m="0.1" w="0.1" d="0.1" h="0.1"/>
+    <xacro:box_inertia m="0.01" w="0.01" d="0.01" h="0.01"/>
   </link>
   <joint name="right_cam_joint" type="fixed">
@@ -359,57 +479,4 @@
     </sensor>
   </gazebo>
-  <!-- body -->
-  <link name="body">
-    <visual>
-      <origin xyz="0 0 ${-body_height / 2}"/>
-      <geometry>
-        <box size="${body_length} ${body_width} ${body_height}"/>
-      </geometry>
-      <material name="body_mat"/>
-    </visual>
-    <collision>
-      <origin xyz="0 0 ${-body_height / 2}"/>
-      <geometry>
-        <box size="${body_length} ${body_width} ${body_height}"/>
-      </geometry>
-    </collision>
-    <xacro:solid_cuboid_inertial
-        width="${body_length}" depth="${body_width}"
-        height="${body_height}" mass="${body_mass}">
-      <origin xyz="0 0 ${-body_height / 2}"/>
-    </xacro:solid_cuboid_inertial>
-  </link>
-  <gazebo reference="body">
-    <material>Gazebo/Grey</material>
-  </gazebo>
-  <joint name="base_link_to_chasis" type="fixed">
-    <parent link="base_link"/>
-    <child link="body"/>
-  </joint>
-  <!-- Wheels -->
-  <xacro:wheel lr_prefix="left_bogie" fr_prefix="front"
-               lr_pos="${track / 2}"
-               fr_pos="${x_center_bogie + wheelbase_bogie / 2}"
-               />
-  <xacro:wheel lr_prefix="left_bogie" fr_prefix="rear"
-               lr_pos="${track / 2}"
-               fr_pos="${x_center_bogie - wheelbase_bogie / 2}"
-               />
-  <xacro:wheel lr_prefix="left_rocker" fr_prefix="rear"
-               lr_pos="${track / 2}"
-               fr_pos="${x_center_rocker - wheelbase_rocker / 2}"
-               />
-  <xacro:wheel lr_prefix="right_bogie" fr_prefix="front"
-               lr_pos="${- track / 2}"
-               fr_pos="${x_center_bogie + wheelbase_bogie / 2}"
-               />
-  <xacro:wheel lr_prefix="right_bogie" fr_prefix="rear"
-               lr_pos="${- track / 2}"
-               fr_pos="${x_center_bogie - wheelbase_bogie / 2}"
-               />
-  <xacro:wheel lr_prefix="right_rocker" fr_prefix="rear"
-               lr_pos="${- track / 2}"
-               fr_pos="${x_center_rocker - wheelbase_rocker / 2}"
-               />
   <gazebo>
     <sensor name="imu" type="imu">
@@ -512,8 +579,3 @@
       </plugin>
   </gazebo>
-  <ros2_control name="GazeboSystem" type="system">
-    <hardware>
-      <plugin>gazebo_ros2_control/GazeboSystem</plugin>
-    </hardware>
-  </ros2_control>
 </robot>
