Commit message: configured wheels and imu

File: urc_arm_moveit_config/config/WalliiArmV3.ros2_control.xacro (robot description, xacro)
@@ -1,5 +1,5 @@
 <?xml version="1.0"?>
 <robot xmlns:xacro="http://www.ros.org/wiki/xacro">
-    <xacro:macro name="WalliiArmV3_ros2_control" params="name initial_positions_file">
+    <xacro:macro name="walliArmV3_ros2_control" params="name initial_positions_file">
         <xacro:property name="initial_positions" value="${load_yaml(initial_positions_file)['initial_positions']}"/>
         <ros2_control name="${name}" type="system">

File: urc_arm_moveit_config/config/WalliiArmV3.urdf.xacro (robot description, xacro)
@@ -1,9 +1,9 @@
 <?xml version="1.0"?>
-<robot xmlns:xacro="http://www.ros.org/wiki/xacro" name="WalliiArmV3">
+<robot xmlns:xacro="http://www.ros.org/wiki/xacro" name="walliArmV3">
     <xacro:arg name="initial_positions_file" default="initial_positions.yaml" />
-    <!-- Import WalliiArmV3 urdf file -->
-    <xacro:include filename="$(find urc_gazebo)/urdf/wallii.xacro" />
+    <!-- Import walliArmV3 urdf file -->
+    <xacro:include filename="$(find urc_gazebo)/urdf/walli.xacro" />
     <!-- Import control_xacro -->
-    <xacro:include filename="WalliiArmV3.ros2_control.xacro" />
-    <xacro:WalliiArmV3_ros2_control name="GazeboSimSystem" initial_positions_file="$(arg initial_positions_file)"/>
+    <xacro:include filename="walliArmV3.ros2_control.xacro" />
+    <xacro:walliArmV3_ros2_control name="GazeboSimSystem" initial_positions_file="$(arg initial_positions_file)"/>
 </robot>

File: urc_gazebo/urdf/walli.xacro (robot description, xacro)
@@ -1,114 +1,75 @@
 <?xml version='1.0'?>
-<robot name="wallii" xmlns:xacro="http://www.ros.org/wiki/xacro">
+<robot name="walli" xmlns:xacro="http://www.ros.org/wiki/xacro">
   <xacro:include filename="walli_prop.xacro"/>
   <xacro:include filename="walli_inertials.xacro"/>
   <xacro:include filename="$(find velodyne_description)/urdf/VLP-16.urdf.xacro"/>
-  <!-- Import wallii arm urdf to walli's urdf. -->
-  <xacro:include filename="WalliiArmV3.urdf"/>
-  <!--- Something about this macro breaks the urdf parser. -->
-  <!-- The "wheel" macro defines an axle carrier, axle, and wheel. -->
-  <xacro:macro name="wheel" params="lr_prefix fr_prefix lr_pos fr_pos">
-    <link name="${lr_prefix}_${fr_prefix}_wheel">
+  <xacro:include filename="walliArmV3.urdf"/>
+  <!-- Rover Base Link -->
+  <link name="base_link">
+    <visual>
+      <geometry>
+        <box size="${base_length} ${base_width} ${base_height}"/>
+      </geometry>
+      <material name="Cyan">
+        <color rgba="0 1.0 1.0 1.0"/>
+      </material>
+    </visual>
+    <collision>
+      <geometry>
+        <box size="${base_length} ${base_width} ${base_height}"/>
+      </geometry>
+    </collision>
+    <xacro:box_inertia m="15" w="${base_width}" d="${base_length}" h="${base_height}"/>
+  </link>
+  <gazebo reference="base_link">
+    <material>Gazebo/Red</material>
+  </gazebo>
+  <!-- Wheels -->
+  <xacro:macro name="wheel" params="prefix x_reflect y_reflect">
+    <link name="${prefix}_link">
       <visual>
-        <origin xyz="0 0 0"/>
+        <origin xyz="0 0 0" rpy="${pi/2} 0 0" />
         <geometry>
-          <cylinder radius="${tire_dia / 2}" length="${tire_width}"/>
+          <cylinder radius="${wheel_radius}" length="${wheel_width}"/>
         </geometry>
-        <material name="tire_mat"/>
+        <material name="Gray">
+          <color rgba="0.5 0.5 0.5 1.0"/>
+        </material>
       </visual>
       <collision>
-        <origin xyz="0 0 0"/>
+        <origin xyz="0 0 0" rpy="${pi/2} 0 0"/>
         <geometry>
-          <cylinder radius="${tire_dia / 2}" length="${tire_width}"/>
+          <cylinder radius="${wheel_radius}" length="${wheel_width}"/>
         </geometry>
       </collision>
-      <xacro:thick_walled_tube_inertial
-          inner_rad="${hub_dia / 2}" outer_rad="${tire_dia / 2}"
-          height="${tire_width}" mass="${wheel_mass}"/>
+      <xacro:cylinder_inertia m="0.5" r="${wheel_radius}" h="${wheel_width}"/>
     </link>
-    <joint name="${lr_prefix}_${fr_prefix}_axle" type="continuous">
+    <joint name="${prefix}_joint" type="continuous">
       <parent link="base_link"/>
-      <child link="${lr_prefix}_${fr_prefix}_wheel"/>
-      <origin xyz="${fr_pos}
-                   ${lr_pos}
-                   ${- body_clearance}"
-              rpy="${degrees_90} 0 0"/>
-      <axis xyz="0 0 -1"/>
+      <child link="${prefix}_link"/>
+      <origin xyz="${x_reflect*wheel_xoff} ${y_reflect*(base_width/2+wheel_ygap)} ${-wheel_zoff}" rpy="0 0 0"/>
+      <axis xyz="0 1 0"/>
       <limit effort="${axle_eff_limit}" velocity="${axle_vel_limit}"/>
-      <dynamics
-      damping="0"
-      friction="4.0" />
-    </joint>
-    <gazebo reference="${lr_prefix}_${fr_prefix}_wheel">
+      <dynamics damping="0" friction="4.0" />
+    </joint>
+    <gazebo reference="${prefix}_link">
       <material>Gazebo/Black</material>
     </gazebo>
   </xacro:macro>
-  <!-- base_link must have geometry so that its axes can be displayed in
-       rviz. -->
-  <link name="base_link">
-    <visual>
-      <geometry>
-        <box size="0.05 0.05 0.01"/>
-      </geometry>
-      <material name="body_mat"/>
-    </visual>
-  </link>
-  <gazebo reference="base_link">
-    <material>Gazebo/Green</material>
-  </gazebo>
-    <!-- body -->
-  <link name="body">
-    <visual>
-      <origin xyz="0 0 ${-body_height / 2}"/>
-      <geometry>
-        <box size="${body_length} ${body_width} ${body_height}"/>
-      </geometry>
-      <material name="body_mat"/>
-    </visual>
-    <collision>
-      <origin xyz="0 0 ${-body_height / 2}"/>
-      <geometry>
-        <box size="${body_length} ${body_width} ${body_height}"/>
-      </geometry>
-    </collision>
-    <xacro:solid_cuboid_inertial
-        width="${body_length}" depth="${body_width}"
-        height="${body_height}" mass="${body_mass}">
-      <origin xyz="0 0 ${-body_height / 2}"/>
-    </xacro:solid_cuboid_inertial>
-  </link>
-  <gazebo reference="body">
-    <material>Gazebo/Grey</material>
-  </gazebo>
-  <joint name="base_link_to_chasis" type="fixed">
+    <!-- Wheels    -->
+  <xacro:wheel prefix="left_front_wheel"   x_reflect="1" y_reflect="-1"/>
+  <xacro:wheel prefix="left_center_wheel"  x_reflect="0" y_reflect="-1"/>
+  <xacro:wheel prefix="left_rear_wheel"    x_reflect="-1" y_reflect="-1"/>
+  <xacro:wheel prefix="right_front_wheel"  x_reflect="1" y_reflect="1"/>
+  <xacro:wheel prefix="right_center_wheel" x_reflect="0" y_reflect="1"/>
+  <xacro:wheel prefix="right_rear_wheel"   x_reflect="-1" y_reflect="1"/>
+  <!-- Robot Footprint -->
+  <link name="base_footprint"/>
+  <joint name="base_joint" type="fixed">
     <parent link="base_link"/>
-    <child link="body"/>
+    <child link="base_footprint"/>
+    <origin xyz="0.0 0.0 ${-(wheel_radius+wheel_zoff)}" rpy="0 0 0"/>
   </joint>
-  <!-- Wheels    -->
-  <xacro:wheel lr_prefix="left_bogie" fr_prefix="front"
-               lr_pos="${track / 2}"
-               fr_pos="${x_center_bogie + wheelbase_bogie / 2}"
-               />
-  <xacro:wheel lr_prefix="left_bogie" fr_prefix="rear"
-               lr_pos="${track / 2}"
-               fr_pos="${x_center_bogie - wheelbase_bogie / 2}"
-               />
-  <xacro:wheel lr_prefix="left_rocker" fr_prefix="rear"
-               lr_pos="${track / 2}"
-               fr_pos="${x_center_rocker - wheelbase_rocker / 2}"
-               />
-  <xacro:wheel lr_prefix="right_bogie" fr_prefix="front"
-               lr_pos="${- track / 2}"
-               fr_pos="${x_center_bogie + wheelbase_bogie / 2}"
-               />
-  <xacro:wheel lr_prefix="right_bogie" fr_prefix="rear"
-               lr_pos="${- track / 2}"
-               fr_pos="${x_center_bogie - wheelbase_bogie / 2}"
-               />
-  <xacro:wheel lr_prefix="right_rocker" fr_prefix="rear"
-               lr_pos="${- track / 2}"
-               fr_pos="${x_center_rocker - wheelbase_rocker / 2}"
-               />
-  <!-- connect rover and arm -->
+  <!-- Arm Joint -->
   <joint name="arm_to_rover" type="fixed">
     <origin rpy="0 0 0" xyz="0 0 0"/>
@@ -192,24 +153,25 @@
     </ros2_control>
     -->
-  <link name="imu">
+  <!-- IMU -->
+  <link name="imu_link">
     <visual>
       <geometry>
-        <box size="0.01 0.01 0.01"/>
+        <box size="0.1 0.1 0.1"/>
       </geometry>
     </visual>
     <collision>
       <geometry>
-        <box size="0.01 0.01 0.01"/>
+        <box size="0.1 0.1 0.1"/>
       </geometry>
     </collision>
-    <xacro:box_inertia m="0.01" w="0.01" d="0.01" h="0.01"/>
+    <xacro:box_inertia m="0.1" w="0.1" d="0.1" h="0.1"/>
   </link>
   <joint name="imu_joint" type="fixed">
 		<axis xyz="1 0 0"/>
-		<origin xyz="0 0 0.1"/>
+		<origin xyz="0 0 0.05"/>
 		<parent link="base_link"/>
-		<child link="imu"/>
+		<child link="imu_link"/>
 	</joint>
-	<gazebo reference="imu">
+	<gazebo reference="imu_link">
     <sensor name="imu_sensor" type="imu">
       <plugin filename="libgazebo_ros_imu_sensor.so" name="imu_plugin">
@@ -279,17 +241,39 @@
     </sensor>
   </gazebo>
-  <!-- gps -->
+  <gazebo>
+  <plugin name='diff_drive' filename='libgazebo_ros_diff_drive.so'>
+    <ros>
+      <namespace>/sensor</namespace>
+    </ros>
+    <!-- wheels -->
+    <left_joint>left_front_wheel_joint</left_joint>
+    <right_joint>right_front_wheel_joint</right_joint>
+    <!-- kinematics -->
+    <wheel_separation>0.4</wheel_separation>
+    <wheel_diameter>0.2</wheel_diameter>
+    <!-- limits -->
+    <max_wheel_torque>20</max_wheel_torque>
+    <max_wheel_acceleration>1.0</max_wheel_acceleration>
+    <!-- output -->
+    <publish_odom>true</publish_odom>
+    <publish_odom_tf>false</publish_odom_tf>
+    <publish_wheel_tf>true</publish_wheel_tf>
+    <odometry_frame>odom</odometry_frame>
+    <robot_base_frame>base_link</robot_base_frame>
+  </plugin>
+</gazebo>
+  <!-- GPS -->
   <link name="gps">
     <visual>
       <geometry>
-        <box size="0.01 0.01 0.01"/>
+        <box size="0.1 0.1 0.1"/>
       </geometry>
     </visual>
     <collision>
       <geometry>
-        <box size="0.01 0.01 0.01"/>
+        <box size="0.1 0.1 0.1"/>
       </geometry>
     </collision>
-    <xacro:box_inertia m="0.01" w="0.01" d="0.01" h="0.01"/>
+    <xacro:box_inertia m="0.1" w="0.1" d="0.1" h="0.1"/>
   </link>
    <joint name="gps_joint" type="fixed">
@@ -348,5 +332,5 @@
 	<!-- Edit these parameters to change camera orientation -->
 	<origin xyz="0.15 0 -0.1" rpy = "0 0 -.14"/>
-	<parent link="imu"/>
+	<parent link="imu_link"/>
 	<child link="cam/center"/>
    </joint>

File: urc_gazebo/urdf/walli_prop.xacro (robot description, xacro)
@@ -5,11 +5,17 @@
   <xacro:property name="degrees_45" value="0.785398163"/>
   <xacro:property name="degrees_90" value="1.57079633"/>
+  <!-- New Properties from NAV2-->
+  <xacro:property name="base_length"    value="0.300"/>
+  <xacro:property name="base_width"     value="0.250"/>
+  <xacro:property name="base_height"    value="0.050"/>
+  <xacro:property name="base_mass"      value="3.000"/>
+  <xacro:property name="base_clearance" value="0.200"/>
+  <xacro:property name="wheel_radius" value="0.05"/>
+  <xacro:property name="wheel_width" value="0.075"/>
+  <xacro:property name="wheel_ygap" value="0.025"/>
+  <xacro:property name="wheel_zoff" value="0.05"/>
+  <xacro:property name="wheel_xoff" value="0.12"/>
   <!-- body_length is measured along the x axis, body_width
        along the y axis, and body_height along the z axis. -->
-  <xacro:property name="body_length"    value="0.300"/>
-  <xacro:property name="body_width"     value="0.250"/>
-  <xacro:property name="body_height"    value="0.050"/>
-  <xacro:property name="body_mass"      value="50.000"/>
-  <xacro:property name="body_clearance" value="0.200"/>
   <xacro:property name="wheelbase_rocker" value="0.350"/>
   <xacro:property name="wheelbase_bogie"  value="0.200"/>

Commit message: minor fixes

File: urc_arm_moveit_config/config/WalliiArmV3.ros2_control.xacro (robot description, xacro)
@@ -7,5 +7,5 @@
                 <!-- gazebo_ros2_control/GazeboSystem -->
                 <!-- mock_components/GenericSystem -->
-                <plugin>gazebo_ros2_control/GazeboSystem</plugin>
+                <plugin>mock_components/GenericSystem</plugin>
             </hardware>
             <joint name="shoulderjoint">

File: urc_arm_moveit_config/config/WalliiArmV3.urdf.xacro (robot description, xacro)
@@ -2,4 +2,6 @@
 <robot xmlns:xacro="http://www.ros.org/wiki/xacro" name="WalliiArmV3">
     <xacro:arg name="initial_positions_file" default="initial_positions.yaml" />
+    <!-- mock_components/GenericSystem -->
+    <xacro:arg name="use_hardware" default="gazebo_ros2_control/GazeboSystem"/>
     <!-- Import WalliiArmV3 urdf file -->
     <!-- wallii.xacro -->

File: urc_gazebo/urdf/walli_prop.xacro (robot description, xacro)
@@ -2,4 +2,5 @@
  -->
 <robot name="walli_prop" xmlns:xacro="http://ros.org/wiki/xacro">
+  <xacro:property name="realhardware" value="false"/>
    <!-- Degree-to-radian conversions -->
   <xacro:property name="degrees_45" value="0.785398163"/>
