Commit message: Nav2 Configuration  (#125)
* Changed flat world texture

* Added new nodes for joint state publisher

* configured wheels and imu

* Made camera macro

* Cleanup unnecessary repeated camera sensor info

* Fixed lidar somewhat but not enough

* Almost finalized config

* Fix CI bs part 1

* Fix CI bs part 2

* Configured spacing of aruco tags

* Fixed world configuration

* removed objects from sim

* sensor origin fixes

* fix state transform issue for rviz

* unnecessary import I added now removed

* linting 😫

---------

Co-authored-by: Matthew Kerner <mkerner3@gatech.edu>

File: urc_arm_moveit_config/config/walli_arm_v3.ros2_control.xacro (robot description, xacro)
@@ -1,5 +1,5 @@
 <?xml version="1.0"?>
 <robot xmlns:xacro="http://www.ros.org/wiki/xacro">
-    <xacro:macro name="WalliiArmV3_ros2_control" params="name initial_positions_file">
+    <xacro:macro name="walli_arm_v3_ros2_control" params="name initial_positions_file">
         <xacro:property name="initial_positions" value="${load_yaml(initial_positions_file)['initial_positions']}"/>
         <ros2_control name="${name}" type="system">

File: urc_gazebo/urdf/walli_prop.xacro (robot description, xacro)
@@ -6,11 +6,17 @@
   <xacro:property name="degrees_45" value="0.785398163"/>
   <xacro:property name="degrees_90" value="1.57079633"/>
+  <!-- New Properties from NAV2-->
+  <xacro:property name="base_length"    value="0.300"/>
+  <xacro:property name="base_width"     value="0.250"/>
+  <xacro:property name="base_height"    value="0.050"/>
+  <xacro:property name="base_mass"      value="3.000"/>
+  <xacro:property name="base_clearance" value="0.200"/>
+  <xacro:property name="wheel_radius" value="0.05"/>
+  <xacro:property name="wheel_width" value="0.075"/>
+  <xacro:property name="wheel_ygap" value="0.025"/>
+  <xacro:property name="wheel_zoff" value="0.05"/>
+  <xacro:property name="wheel_xoff" value="0.12"/>
   <!-- body_length is measured along the x axis, body_width
        along the y axis, and body_height along the z axis. -->
-  <xacro:property name="body_length"    value="0.300"/>
-  <xacro:property name="body_width"     value="0.250"/>
-  <xacro:property name="body_height"    value="0.050"/>
-  <xacro:property name="body_mass"      value="50.000"/>
-  <xacro:property name="body_clearance" value="0.200"/>
   <xacro:property name="wheelbase_rocker" value="0.350"/>
   <xacro:property name="wheelbase_bogie"  value="0.200"/>
@@ -49,10 +55,7 @@
    <!-- Lidar -->
     <xacro:property name="lidar_pitch" value="0.0"/>
-    <xacro:property name="lidar_x" value="0.127"/>
-    <xacro:property name="lidar_z" value="0.8486"/>
+    <xacro:property name="lidar_x" value="0.12"/>
+    <xacro:property name="lidar_z" value="0.12"/>
     <xacro:property name="lidar_hz" value="10"/>
     <xacro:property name="lidar_samples" value="500"/>
-    <xacro:property name="lidar_support_x_dim" value="0.2"/>
-    <xacro:property name="lidar_support_y_dim" value="0.08"/>
-    <xacro:property name="lidar_support_z_dim" value="0.01"/>
 </robot>
