Commit message: removed v3 naming convention

File: urc_arm_moveit_config/config/walli_arm.ros2_control.xacro (robot description, xacro)
@@ -1,5 +1,5 @@
 <?xml version="1.0"?>
 <robot xmlns:xacro="http://www.ros.org/wiki/xacro">
-    <xacro:macro name="walli_arm_v3_ros2_control" params="name initial_positions_file">
+    <xacro:macro name="walli_arm_ros2_control" params="name initial_positions_file">
         <xacro:property name="initial_positions" value="${load_yaml(initial_positions_file)['initial_positions']}"/>
         <ros2_control name="${name}" type="system">

File: urc_gazebo/urdf/walli.xacro (robot description, xacro)
@@ -4,5 +4,5 @@
   <xacro:include filename="walli_inertials.xacro"/>
   <xacro:include filename="$(find velodyne_description)/urdf/VLP-16.urdf.xacro"/>
-  <xacro:include filename="walli_arm_v3.urdf"/>
+  <xacro:include filename="walli_arm.urdf"/>
   <!-- Rover Base Link -->
   <link name="base_link">
