Commit message: rewrite ekf yaml

File: urc_hw_description/urdf/six_wheel_simplified.xacro (robot description, xacro)
@@ -169,5 +169,5 @@
     <joint name="gps_joint" type="fixed">
         <axis xyz="1 0 0" />
-        <origin xyz="0.05 -0.1 0.2" />
+        <origin xyz="00 0 0" />
         <parent link="base_link" />
         <child link="gps" />
