Commit message: Add config variable to choose between full and simplified robot model

File: urc_hw_description/urdf/robot.xacro (robot description, xacro)
@@ -2,8 +2,14 @@
 <robot name="sam_bot" xmlns:xacro="http://ros.org/wiki/xacro">
     <xacro:property name="config_file" value="$(find urc_bringup)/config/hardware_config.yaml" />
-   <xacro:property name="config_data" value="${load_yaml(config_file)}"></xacro:property>
-   <xacro:property name="use_simulation" value="${config_data['hardware_config']['use_simulation']}" />
-   <!-- Pick either walli hardware or simplified hardware -->
-   <!-- <xacro:include filename="$(find urc_hw_description)/urdf/walli.xacro" /> -->
-   <xacro:include filename="$(find urc_hw_description)/urdf/diff_drive.xacro" />
+    <xacro:property name="config_data" value="${xacro.load_yaml(config_file)}"></xacro:property>
+    <xacro:property name="use_simulation"
+        value="${config_data['hardware_config']['use_simulation']}" />
+    <xacro:property name="use_simplified_model"
+        value="${config_data['hardware_config']['use_simplified_model']}" />
+    <xacro:if value="${use_simplified_model}">
+        <xacro:include filename="$(find urc_hw_description)/urdf/diff_drive.xacro" />
+    </xacro:if>
+    <xacro:if value="${not use_simplified_model}">
+        <xacro:include filename="$(find urc_hw_description)/urdf/walli.xacro" />
+    </xacro:if>
 </robot>

File: urc_hw_description/urdf/walli.xacro (robot description, xacro)
@@ -3,5 +3,5 @@
    <xacro:property name="config_file"
       value="$(find urc_bringup)/config/hardware_config.yaml" />
-   <xacro:property name="config_data" value="${load_yaml(config_file)}"></xacro:property>
+   <xacro:property name="config_data" value="${xacro.load_yaml(config_file)}"></xacro:property>
    <xacro:property name="use_simulation" value="${config_data['hardware_config']['use_simulation']}" />
    <xacro:include filename="$(find urc_hw_description)/urdf/walli_prop.xacro" />

Commit message: Lots of cleanup and changes to try and get the simplified model to work. Still won't respond to angular velocity for some reason

File: urc_hw_description/urdf/robot.xacro (robot description, xacro)
@@ -8,5 +8,6 @@
         value="${config_data['hardware_config']['use_simplified_model']}" />
     <xacro:if value="${use_simplified_model}">
-        <xacro:include filename="$(find urc_hw_description)/urdf/six_wheel_simplified.xacro" />
+        <xacro:include
+            filename="$(find urc_hw_description)/urdf/simplified_model/simplified_model.xacro" />
     </xacro:if>
     <xacro:if value="${not use_simplified_model}">

File: urc_hw_description/urdf/simplified_model/simplified_model.xacro (robot description, xacro)
@@ -5,33 +5,13 @@
     <xacro:property name="base_length" value="0.8" />
     <xacro:property name="base_height" value="0.18" />
+    <xacro:property name="base_mass" value="1.0" />
     <xacro:property name="wheel_radius" value="0.10" />
-    <xacro:property name="wheel_width" value="0.04" />
-    <xacro:property name="wheel_ygap" value="0.025" />
-    <xacro:property name="wheel_zoff" value="0.05" />
-    <xacro:property name="wheel_xoff" value="0.12" />
-    <!-- Define some commonly used intertial properties  -->
-    <xacro:macro name="box_inertia" params="m w h d">
-        <inertial>
-            <origin xyz="0 0 0" rpy="${pi/2} 0 ${pi/2}" />
-            <mass value="${m}" />
-            <inertia ixx="${(m/12) * (h*h + d*d)}" ixy="0.0" ixz="0.0" iyy="${(m/12) * (w*w + d*d)}"
-                iyz="0.0" izz="${(m/12) * (w*w + h*h)}" />
-        </inertial>
-    </xacro:macro>
-    <xacro:macro name="cylinder_inertia" params="m r h">
-        <inertial>
-            <origin xyz="0 0 0" rpy="${pi/2} 0 0" />
-            <mass value="${m}" />
-            <inertia ixx="${(m/12) * (3*r*r + h*h)}" ixy="0" ixz="0" iyy="${(m/12) * (3*r*r + h*h)}"
-                iyz="0" izz="${(m/2) * (r*r)}" />
-        </inertial>
-    </xacro:macro>
-    <xacro:macro name="sphere_inertia" params="m r">
-        <inertial>
-            <mass value="${m}" />
-            <inertia ixx="${(2/5) * m * (r*r)}" ixy="0.0" ixz="0.0" iyy="${(2/5) * m * (r*r)}"
-                iyz="0.0" izz="${(2/5) * m * (r*r)}" />
-        </inertial>
-    </xacro:macro>
+    <xacro:property name="wheel_thickness" value="0.04" />
+    <xacro:property name="wheel_mass" value="0.05" />
+    <xacro:property name="wheel_gap_y" value="0.025" />
+    <xacro:property name="wheel_offset_z" value="0.05" />
+    <xacro:property name="wheel_offset_x" value="0.12" />
+    <xacro:include filename="inertial_macros.xacro" />
+    <!-- Define gazebo system joints -->
     <ros2_control name="GazeboSystem" type="system">
         <hardware>
@@ -40,6 +20,6 @@
         <joint name="left_front_wheel_joint">
             <command_interface name="velocity">
-                <param name="min">-0.05</param>
-                <param name="max">0.05</param>
+                <param name="min">-10</param>
+                <param name="max">10</param>
             </command_interface>
             <state_interface name="velocity" />
@@ -48,6 +28,6 @@
         <joint name="right_front_wheel_joint">
             <command_interface name="velocity">
-                <param name="min">-0.05</param>
-                <param name="max">0.05</param>
+                <param name="min">-10</param>
+                <param name="max">10</param>
             </command_interface>
             <state_interface name="velocity" />
@@ -56,6 +36,6 @@
         <joint name="left_center_wheel_joint">
             <command_interface name="velocity">
-                <param name="min">-0.05</param>
-                <param name="max">0.05</param>
+                <param name="min">-10</param>
+                <param name="max">10</param>
             </command_interface>
             <state_interface name="velocity" />
@@ -64,6 +44,6 @@
         <joint name="right_center_wheel_joint">
             <command_interface name="velocity">
-                <param name="min">-0.05</param>
-                <param name="max">0.05</param>
+                <param name="min">-10</param>
+                <param name="max">10</param>
             </command_interface>
             <state_interface name="velocity" />
@@ -72,6 +52,6 @@
         <joint name="left_rear_wheel_joint">
             <command_interface name="velocity">
-                <param name="min">-0.05</param>
-                <param name="max">0.05</param>
+                <param name="min">-10</param>
+                <param name="max">10</param>
             </command_interface>
             <state_interface name="velocity" />
@@ -80,6 +60,6 @@
         <joint name="right_rear_wheel_joint">
             <command_interface name="velocity">
-                <param name="min">-0.05</param>
-                <param name="max">0.05</param>
+                <param name="min">-10</param>
+                <param name="max">10</param>
             </command_interface>
             <state_interface name="velocity" />
@@ -91,24 +71,4 @@
             <parameters>$(find urc_bringup)/config/ros2_control_walli.yaml</parameters>
         </plugin>
-        <plugin name='diff_drive' filename='libgazebo_ros_diff_drive.so'>
-            <ros>
-            <namespace>/wheel</namespace>
-            </ros>
-            <!-- wheels -->
-            <left_joint>left_front_wheel_joint</left_joint>
-            <right_joint>right_front_wheel_joint</right_joint>
-            <!-- kinematics -->
-            <wheel_separation>0.4</wheel_separation>
-            <wheel_diameter>0.2</wheel_diameter>
-            <!-- limits -->
-            <max_wheel_torque>20</max_wheel_torque>
-            <max_wheel_acceleration>1.0</max_wheel_acceleration>
-            <!-- output -->
-            <publish_odom>true</publish_odom>
-            <publish_odom_tf>true</publish_odom_tf>
-            <publish_wheel_tf>true</publish_wheel_tf>
-            <odometry_frame>odom</odometry_frame>
-            <robot_base_frame>base_link</robot_base_frame>
-        </plugin>
     </gazebo>
     <!-- Robot Base -->
@@ -127,22 +87,28 @@
             </geometry>
         </collision>
-        <xacro:box_inertia m="15" w="${base_width}" d="${base_length}" h="${base_height}" />
+        <xacro:box_inertia m="${base_mass}" w="${base_width}" d="${base_length}" h="${base_height}" />
     </link>
     <!-- Robot Footprint -->
     <link name="base_footprint">
-        <xacro:box_inertia m="5" w="${base_width}" d="${base_width}" h="${base_width}" />
     </link>
     <joint name="base_joint" type="fixed">
         <parent link="base_link" />
         <child link="base_footprint" />
-        <origin xyz="0.0 0.0 ${-(wheel_radius+wheel_zoff)}" rpy="0 0 0" />
+        <origin xyz="0.0 0.0 ${-(wheel_radius+wheel_offset_z)}" rpy="0 0 0" />
     </joint>
     <!-- Wheels -->
-    <xacro:macro name="wheel" params="prefix x_reflect y_reflect">
+    <xacro:macro name="wheel" params="prefix x_mult y_reflect">
+        <joint name="${prefix}_joint" type="continuous">
+            <parent link="base_link" />
+            <child link="${prefix}_link" />
+            <origin
+                xyz="${x_mult*wheel_offset_x} ${-y_reflect*(base_width/2+wheel_gap_y)} ${-wheel_offset_z}"
+                rpy="${y_reflect*pi/2} 0 0" />
+            <axis xyz="0 0 ${y_reflect}" />
+        </joint>
         <link name="${prefix}_link">
             <visual>
-                <origin xyz="0 0 0" rpy="${pi/2} 0 0" />
                 <geometry>
-                    <cylinder radius="${wheel_radius}" length="${wheel_width}" />
+                    <cylinder radius="${wheel_radius}" length="${wheel_thickness}" />
                 </geometry>
                 <material name="Gray">
@@ -151,26 +117,17 @@
             </visual>
             <collision>
-                <origin xyz="0 0 0" rpy="${pi/2} 0 0" />
                 <geometry>
-                    <cylinder radius="${wheel_radius}" length="${wheel_width}" />
+                    <cylinder radius="${wheel_radius}" length="${wheel_thickness}" />
                 </geometry>
             </collision>
-            <xacro:cylinder_inertia m="0.5" r="${wheel_radius}" h="${wheel_width}" />
+            <xacro:cylinder_inertia m="${wheel_mass}" r="${wheel_radius}" h="${wheel_thickness}" />
         </link>
-        <joint name="${prefix}_joint" type="continuous">
-            <parent link="base_link" />
-            <child link="${prefix}_link" />
-            <origin
-                xyz="${x_reflect*wheel_xoff} ${y_reflect*(base_width/2+wheel_ygap)} ${-wheel_zoff}"
-                rpy="0 0 0" />
-            <axis xyz="0 1 0" />
-        </joint>
     </xacro:macro>
-    <xacro:wheel prefix="left_front_wheel" x_reflect="-2" y_reflect="1" />
-    <xacro:wheel prefix="left_center_wheel" x_reflect="0" y_reflect="1" />
-    <xacro:wheel prefix="left_rear_wheel" x_reflect="2" y_reflect="1" />
-    <xacro:wheel prefix="right_front_wheel" x_reflect="-2" y_reflect="-1" />
-    <xacro:wheel prefix="right_center_wheel" x_reflect="0" y_reflect="-1" />
-    <xacro:wheel prefix="right_rear_wheel" x_reflect="2" y_reflect="-1" />
+    <xacro:wheel prefix="left_front_wheel" x_mult="-2" y_reflect="1" />
+    <xacro:wheel prefix="left_center_wheel" x_mult="0" y_reflect="1" />
+    <xacro:wheel prefix="left_rear_wheel" x_mult="2" y_reflect="1" />
+    <xacro:wheel prefix="right_front_wheel" x_mult="-2" y_reflect="-1" />
+    <xacro:wheel prefix="right_center_wheel" x_mult="0" y_reflect="-1" />
+    <xacro:wheel prefix="right_rear_wheel" x_mult="2" y_reflect="-1" />
     <!-- GPS -->
     <link name="gps">
@@ -185,5 +142,4 @@
             </geometry>
         </collision>
-        <xacro:box_inertia m="0.1" w="0.1" d="0.1" h="0.1" />
     </link>
     <joint name="gps_joint" type="fixed">
@@ -217,5 +173,4 @@
             </geometry>
         </collision>
-        <xacro:box_inertia m="0.1" w="0.1" d="0.1" h="0.1" />
     </link>
     <joint name="imu_joint" type="fixed">
