Commit message: Fix friction

File: urc_hw_description/urdf/new_drivebase.xacro (robot description, xacro)
@@ -54,5 +54,5 @@
             <axis xyz="0 1 0" />
             <limit effort="100.0" lower="-0.24" upper="0.24" velocity="100.0" />
-            <dynamics friction="3.0" damping="0.1" />
+            <dynamics friction="1.0" damping="0.1" />
         </joint>
         <link name="leftrocker">

Commit message: Decrease wheel separation

File: urc_hw_description/urdf/new_drivebase.xacro (robot description, xacro)
@@ -168,5 +168,5 @@
         </link>
         <joint name="right_rear_wheel_joint" type="continuous">
-            <origin xyz="-0.36316 -0.08 -0.19158" rpy="0 0 0" />
+            <origin xyz="-0.36316 -0.04 -0.19158" rpy="0 0 0" />
             <parent link="rightrocker" />
             <child link="right_rear_wheel" />
@@ -195,5 +195,5 @@
         </link>
         <joint name="right_front_wheel_joint" type="continuous">
-            <origin xyz="0.20139 -0.08 -0.11671" rpy="0 0 0" />
+            <origin xyz="0.20139 -0.04 -0.11671" rpy="0 0 0" />
             <parent link="rightbogie" />
             <child link="right_front_wheel" />
@@ -222,5 +222,5 @@
         </link>
         <joint name="right_center_wheel_joint" type="continuous">
-            <origin xyz="-0.20177 -0.08 -0.11606" rpy="0 0 0" />
+            <origin xyz="-0.20177 -0.04 -0.11606" rpy="0 0 0" />
             <parent link="rightbogie" />
             <child link="right_center_wheel" />
@@ -249,5 +249,5 @@
         </link>
         <joint name="left_rear_wheel_joint" type="continuous">
-            <origin xyz="-0.36266 0.08 -0.19248" rpy="0 0 0" />
+            <origin xyz="-0.36266 0.04 -0.19248" rpy="0 0 0" />
             <parent link="leftrocker" />
             <child link="left_rear_wheel" />
@@ -276,5 +276,5 @@
         </link>
         <joint name="left_front_wheel_joint" type="continuous">
-            <origin xyz="0.20177 0.08 -0.11606" rpy="0 0 0" />
+            <origin xyz="0.20177 0.04 -0.11606" rpy="0 0 0" />
             <parent link="leftbogie" />
             <child link="left_front_wheel" />
@@ -303,5 +303,5 @@
         </link>
         <joint name="left_center_wheel_joint" type="continuous">
-            <origin xyz="-0.20139 0.08 -0.11671" rpy="0 0 0" />
+            <origin xyz="-0.20139 0.04 -0.11671" rpy="0 0 0" />
             <parent link="leftbogie" />
             <child link="left_center_wheel" />

File: urc_hw_description/urdf/walli.xacro (robot description, xacro)
@@ -11,5 +11,5 @@
    <xacro:include filename="$(find urc_hw_description)/urdf/new_drivebase.xacro" />
    <xacro:include filename="$(find urc_hw_description)/urdf/arm.xacro" />
-   <xacro:drivebase mu="1.0" mu2="0.25" wheel_radius="0.1" wheel_thickness="0.05"
+   <xacro:drivebase mu="1.0" mu2="0.25" wheel_radius="0.1" wheel_thickness="0.08"
       approximate="false" />
    <!-- <xacro:arm /> -->

Commit message: Various fixes

File: urc_hw_description/urdf/new_drivebase.xacro (robot description, xacro)
@@ -53,5 +53,5 @@
             <child link="rightrocker" />
             <axis xyz="0 1 0" />
-            <limit effort="100.0" lower="-0.24" upper="0.24" velocity="100.0" />
+            <limit effort="0.0" lower="-0.24" upper="0.24" velocity="100.0" />
             <dynamics friction="1.0" damping="0.1" />
         </joint>
@@ -84,5 +84,5 @@
             <child link="leftrocker" />
             <axis xyz="0 1 0" />
-            <limit effort="100.0" lower="-0.24" upper="0.24" velocity="100.0" />
+            <limit effort="0.0" lower="-0.24" upper="0.24" velocity="100.0" />
             <dynamics friction="1.0" damping="0.1" />
         </joint>
@@ -114,5 +114,5 @@
             <child link="rightbogie" />
             <axis xyz="0 1 0" />
-            <limit effort="100.0" lower="-0.24" upper="0.24" velocity="100.0" />
+            <limit effort="0.0" lower="-0.24" upper="0.24" velocity="100.0" />
             <dynamics friction="1.0" damping="0.1" />
         </joint>
@@ -143,5 +143,5 @@
             <child link="leftbogie" />
             <axis xyz="0 1 0" />
-            <limit effort="100.0" lower="-0.24" upper="0.24" velocity="100.0" />
+            <limit effort="0.0" lower="-0.24" upper="0.24" velocity="100.0" />
             <dynamics friction="1.0" damping="0.1" />
         </joint>
