Commit message: fix: urdf axis inversion

File: urc_hw_description/urdf/drivebase.xacro (robot description, xacro)
@@ -1,5 +1,5 @@
 <?xml version="1.0"?>
 <robot xmlns:xacro="http://www.ros.org/wiki/xacro">
-    <xacro:macro name="drivebase" params="wheel_friction">
+    <xacro:macro name="drivebase" params="wheel_radius wheel_thickness wheel_friction ">
         <link name="base_link">
             <inertial>
@@ -50,5 +50,5 @@
             <child link="rightrocker" />
             <axis xyz="0 0 0" />
-            <dynamics damping="60" friction="4" />
+            <dynamics damping="0.01" friction="0.01" />
         </joint>
         <link name="right_rear_wheel">
@@ -71,4 +71,5 @@
                     <mesh
                         filename="file://$(find urc_gazebo)/urdf/meshes/collision/right_rear_wheel_collision.STL" />
+                    <!-- <cylinder radius="${wheel_radius}" length="${wheel_thickness}" /> -->
                 </geometry>
             </collision>
@@ -86,5 +87,5 @@
             <parent link="rightrocker" />
             <child link="right_rear_wheel" />
-            <axis xyz="0 -1 0" />
+            <axis xyz="0 1 0" />
             <dynamics damping="0.01" friction="0.01" />
         </joint>
@@ -136,4 +137,5 @@
                     <mesh
                         filename="file://$(find urc_gazebo)/urdf/meshes/collision/right_front_wheel_collision.STL" />
+                    <!-- <cylinder radius="${wheel_radius}" length="${wheel_thickness}" /> -->
                 </geometry>
             </collision>
@@ -159,5 +161,5 @@
             <parent link="rightbogie" />
             <child link="right_front_wheel" />
-            <axis xyz="0 -1 0" />
+            <axis xyz="0 1 0" />
             <dynamics damping="0.01" friction="0.01" />
         </joint>
@@ -181,4 +183,5 @@
                     <mesh
                         filename="file://$(find urc_gazebo)/urdf/meshes/collision/right_center_wheel_collision.STL" />
+                    <!-- <cylinder radius="${wheel_radius}" length="${wheel_thickness}" /> -->
                 </geometry>
             </collision>
@@ -196,5 +199,5 @@
             <parent link="rightbogie" />
             <child link="right_center_wheel" />
-            <axis xyz="0 -1 0" />
+            <axis xyz="0 1 0" />
             <dynamics damping="0.01" friction="0.01" />
         </joint>
@@ -246,4 +249,5 @@
                     <mesh
                         filename="file://$(find urc_gazebo)/urdf/meshes/collision/left_rear_wheel_collision.STL" />
+                    <!-- <cylinder radius="${wheel_radius}" length="${wheel_thickness}" /> -->
                 </geometry>
             </collision>
@@ -311,4 +315,5 @@
                     <mesh
                         filename="file://$(find urc_gazebo)/urdf/meshes/collision/left_front_wheel_collision.STL" />
+                    <!-- <cylinder radius="${wheel_radius}" length="${wheel_thickness}" /> -->
                 </geometry>
             </collision>
@@ -348,4 +353,5 @@
                     <mesh
                         filename="file://$(find urc_gazebo)/urdf/meshes/collision/left_center_wheel_collision.STL" />
+                    <!-- <cylinder radius="${wheel_radius}" length="${wheel_thickness}" /> -->
                 </geometry>
             </collision>

File: urc_hw_description/urdf/walli.xacro (robot description, xacro)
@@ -8,5 +8,5 @@
    <xacro:include filename="$(find urc_hw_description)/urdf/drivebase.xacro" />
    <xacro:include filename="$(find urc_hw_description)/urdf/arm.xacro" />
-   <xacro:drivebase wheel_friction="0.01" />
+   <xacro:drivebase wheel_friction="0.012" wheel_radius="0.35" wheel_thickness="0.03" />
    <xacro:arm />
    <xacro:ros2_control use_simulation="${use_simulation}"

Commit message: feat: one file control for simulation
- control simulation from hardware_config.yaml

File: urc_hw_description/urdf/drivebase.xacro (robot description, xacro)
@@ -1,5 +1,5 @@
 <?xml version="1.0"?>
 <robot xmlns:xacro="http://www.ros.org/wiki/xacro">
-    <xacro:macro name="drivebase" params="wheel_radius wheel_thickness wheel_friction ">
+    <xacro:macro name="drivebase" params="wheel_radius wheel_thickness wheel_friction approximate">
         <link name="base_link">
             <inertial>
@@ -69,7 +69,11 @@
                 <origin xyz="0 0 0" rpy="0 0 0" />
                 <geometry>
-                    <mesh
-                        filename="file://$(find urc_gazebo)/urdf/meshes/collision/right_rear_wheel_collision.STL" />
-                    <!-- <cylinder radius="${wheel_radius}" length="${wheel_thickness}" /> -->
+                    <xacro:if value="${approximate}">
+                        <cylinder radius="${wheel_radius}" length="${wheel_thickness}" />
+                    </xacro:if>
+                    <xacro:if value="${not approximate}">
+                        <mesh
+                            filename="file://$(find urc_gazebo)/urdf/meshes/collision/right_rear_wheel_collision.STL" />
+                    </xacro:if>
                 </geometry>
             </collision>
@@ -116,5 +120,5 @@
             <child link="rightbogie" />
             <axis xyz="0 0 0" />
-            <dynamics damping="60" friction="4" />
+            <dynamics damping="0.02" friction="0" />
         </joint>
         <link name="right_front_wheel">
@@ -135,7 +139,11 @@
                 <origin xyz="0 0 0" rpy="0 0 0" />
                 <geometry>
-                    <mesh
-                        filename="file://$(find urc_gazebo)/urdf/meshes/collision/right_front_wheel_collision.STL" />
-                    <!-- <cylinder radius="${wheel_radius}" length="${wheel_thickness}" /> -->
+                    <xacro:if value="${approximate}">
+                        <cylinder radius="${wheel_radius}" length="${wheel_thickness}" />
+                    </xacro:if>
+                    <xacro:if value="${not approximate}">
+                        <mesh
+                            filename="file://$(find urc_gazebo)/urdf/meshes/collision/right_rear_wheel_collision.STL" />
+                    </xacro:if>
                 </geometry>
             </collision>

File: urc_hw_description/urdf/walli.xacro (robot description, xacro)
@@ -1,5 +1,8 @@
 <?xml version="1.0" encoding="UTF-8"?>
 <robot name="walli" xmlns:xacro="http://ros.org/wiki/xacro">
-   <xacro:property name="use_simulation" value="true"></xacro:property>
+   <xacro:property name="config_file"
+      value="$(find urc_bringup)/config/hardware_config.yaml" />
+   <xacro:property name="config_data" value="${load_yaml(config_file)}"></xacro:property>
+   <xacro:property name="use_simulation" value="${config_data['hardware_config']['use_simulation']}" />
    <xacro:include filename="$(find urc_hw_description)/urdf/walli_prop.xacro" />
    <xacro:include filename="$(find urc_hw_description)/urdf/walli_inertials.xacro" />
@@ -8,5 +11,6 @@
    <xacro:include filename="$(find urc_hw_description)/urdf/drivebase.xacro" />
    <xacro:include filename="$(find urc_hw_description)/urdf/arm.xacro" />
-   <xacro:drivebase wheel_friction="0.012" wheel_radius="0.35" wheel_thickness="0.03" />
+   <xacro:drivebase wheel_friction="0.012" wheel_radius="0.10" wheel_thickness="0.05"
+      approximate="true" />
    <xacro:arm />
    <xacro:ros2_control use_simulation="${use_simulation}"

Commit message: fix: minor updates

File: urc_hw_description/urdf/drivebase.xacro (robot description, xacro)
@@ -139,11 +139,6 @@
                 <origin xyz="0 0 0" rpy="0 0 0" />
                 <geometry>
-                    <xacro:if value="${approximate}">
-                        <cylinder radius="${wheel_radius}" length="${wheel_thickness}" />
-                    </xacro:if>
-                    <xacro:if value="${not approximate}">
-                        <mesh
-                            filename="file://$(find urc_gazebo)/urdf/meshes/collision/right_rear_wheel_collision.STL" />
-                    </xacro:if>
+                    <mesh
+                        filename="file://$(find urc_gazebo)/urdf/meshes/collision/right_rear_wheel_collision.STL" />
                 </geometry>
             </collision>
@@ -191,5 +186,4 @@
                     <mesh
                         filename="file://$(find urc_gazebo)/urdf/meshes/collision/right_center_wheel_collision.STL" />
-                    <!-- <cylinder radius="${wheel_radius}" length="${wheel_thickness}" /> -->
                 </geometry>
             </collision>
@@ -257,5 +251,4 @@
                     <mesh
                         filename="file://$(find urc_gazebo)/urdf/meshes/collision/left_rear_wheel_collision.STL" />
-                    <!-- <cylinder radius="${wheel_radius}" length="${wheel_thickness}" /> -->
                 </geometry>
             </collision>
@@ -323,5 +316,4 @@
                     <mesh
                         filename="file://$(find urc_gazebo)/urdf/meshes/collision/left_front_wheel_collision.STL" />
-                    <!-- <cylinder radius="${wheel_radius}" length="${wheel_thickness}" /> -->
                 </geometry>
             </collision>
@@ -361,5 +353,4 @@
                     <mesh
                         filename="file://$(find urc_gazebo)/urdf/meshes/collision/left_center_wheel_collision.STL" />
-                    <!-- <cylinder radius="${wheel_radius}" length="${wheel_thickness}" /> -->
                 </geometry>
             </collision>

Commit message: added xacro ifs

File: urc_hw_description/urdf/drivebase.xacro (robot description, xacro)
@@ -1,4 +1,24 @@
 <?xml version="1.0"?>
 <robot xmlns:xacro="http://www.ros.org/wiki/xacro">
+    <!-- Approximated Wheel -->
+    <!-- <xacro:macro name="approximate_wheel" params="prefix x_reflect y_reflect">
+        <link name="${prefix}_link">
+        <visual>
+            <origin xyz="0 0 0" rpy="${pi/2} 0 0"/>
+            <geometry>
+                <cylinder radius="${wheel_radius}" length="${wheel_width}"/>
+            </geometry>
+            <material name="Gray">
+            <color rgba="0.5 0.5 0.5 1.0"/>
+            </material>
+        </visual>
+        </link>
+        <joint name="${prefix}_joint" type="continuous">
+        <parent link="base_link"/>
+        <child link="${prefix}_link"/>
+        <origin xyz="${x_reflect*wheel_xoff} ${y_reflect*(base_width/2+wheel_ygap)} ${-wheel_zoff}" rpy="0 0 0"/>
+        <axis xyz="0 1 0"/>
+        </joint>
+    </xacro:macro> -->
     <xacro:macro name="drivebase" params="wheel_radius wheel_thickness wheel_friction approximate">
         <link name="base_link">
@@ -52,4 +72,5 @@
             <dynamics damping="0.01" friction="0.01" />
         </joint>
+        <!-- Wheel 1 -->
         <link name="right_rear_wheel">
             <inertial>
@@ -139,6 +160,11 @@
                 <origin xyz="0 0 0" rpy="0 0 0" />
                 <geometry>
+                <xacro:if value="${approximate}">
+                        <cylinder radius="${wheel_radius}" length="${wheel_thickness}" />
+                    </xacro:if>
+                    <xacro:if value="${not approximate}">
                     <mesh
                         filename="file://$(find urc_gazebo)/urdf/meshes/collision/right_rear_wheel_collision.STL" />
+                    </xacro:if>
                 </geometry>
             </collision>
@@ -184,6 +210,11 @@
                 <origin xyz="0 0 0" rpy="0 0 0" />
                 <geometry>
+                <xacro:if value="${approximate}">
+                        <cylinder radius="${wheel_radius}" length="${wheel_thickness}" />
+                    </xacro:if>
+                    <xacro:if value="${not approximate}">
                     <mesh
                         filename="file://$(find urc_gazebo)/urdf/meshes/collision/right_center_wheel_collision.STL" />
+                    </xacro:if>
                 </geometry>
             </collision>
@@ -249,6 +280,11 @@
                 <origin xyz="0 0 0" rpy="0 0 0" />
                 <geometry>
+                <xacro:if value="${approximate}">
+                        <cylinder radius="${wheel_radius}" length="${wheel_thickness}" />
+                    </xacro:if>
+                    <xacro:if value="${not approximate}">
                     <mesh
                         filename="file://$(find urc_gazebo)/urdf/meshes/collision/left_rear_wheel_collision.STL" />
+                    </xacro:if>
                 </geometry>
             </collision>
@@ -314,6 +350,11 @@
                 <origin xyz="0 0 0" rpy="0 0 0" />
                 <geometry>
+                <xacro:if value="${approximate}">
+                        <cylinder radius="${wheel_radius}" length="${wheel_thickness}" />
+                    </xacro:if>
+                    <xacro:if value="${not approximate}">
                     <mesh
                         filename="file://$(find urc_gazebo)/urdf/meshes/collision/left_front_wheel_collision.STL" />
+                    </xacro:if>
                 </geometry>
             </collision>
@@ -351,6 +392,11 @@
                 <origin xyz="0 0 0" rpy="0 0 0" />
                 <geometry>
+                <xacro:if value="${approximate}">
+                        <cylinder radius="${wheel_radius}" length="${wheel_thickness}" />
+                    </xacro:if>
+                    <xacro:if value="${not approximate}">
                     <mesh
                         filename="file://$(find urc_gazebo)/urdf/meshes/collision/left_center_wheel_collision.STL" />
+                    </xacro:if>
                 </geometry>
             </collision>

Commit message: Made simplifies cylinders for collisions and visuals

File: urc_hw_description/urdf/drivebase.xacro (robot description, xacro)
@@ -24,5 +24,5 @@
         <link name="base_link">
             <inertial>
-                <origin xyz="-0.22771 0.0020794 0.13424" rpy="0 0 0" />
+                <origin xyz="-0.22771 0.0020794 1" rpy="0 0 0" />
                 <mass value="2.485" />
                 <inertia ixx="0.017201" ixy="-2.0986E-11" ixz="5.8899E-06" iyy="0.0028906"
@@ -81,12 +81,13 @@
             </inertial>
             <visual>
-                <origin xyz="0 0 0" rpy="0 0 0" />
-                <geometry>
-                    <mesh
-                        filename="file://$(find urc_gazebo)/urdf/meshes/visual/right_rear_wheel.STL" />
-                </geometry>
-            </visual>
-            <collision>
-                <origin xyz="0 0 0" rpy="0 0 0" />
+                <origin xyz="0 0 0" rpy="${pi/2} 0 0" />
+                <geometry>
+                    <!-- <mesh
+                        filename="file://$(find urc_gazebo)/urdf/meshes/visual/right_rear_wheel.STL" /> -->
+                        <cylinder radius="${wheel_radius}" length="${wheel_thickness}" />
+                </geometry>
+            </visual>
+            <collision>
+                <origin xyz="0 0 0" rpy="${pi/2} 0 0" />
                 <geometry>
                     <xacro:if value="${approximate}">
@@ -143,4 +144,5 @@
             <dynamics damping="0.02" friction="0" />
         </joint>
+        <!-- Wheel 2 -->
         <link name="right_front_wheel">
             <inertial>
@@ -151,12 +153,13 @@
             </inertial>
             <visual>
-                <origin xyz="0 0 0" rpy="0 0 0" />
-                <geometry>
-                    <mesh
-                        filename="file://$(find urc_gazebo)/urdf/meshes/visual/right_front_wheel.STL" />
-                </geometry>
-            </visual>
-            <collision>
-                <origin xyz="0 0 0" rpy="0 0 0" />
+                <origin xyz="0 0 0" rpy="${pi/2} 0 0" />
+                <geometry>
+                <cylinder radius="${wheel_radius}" length="${wheel_thickness}" />
+                    <!-- <mesh
+                        filename="file://$(find urc_gazebo)/urdf/meshes/visual/right_front_wheel.STL" /> -->
+                </geometry>
+            </visual>
+            <collision>
+                <origin xyz="${pi/2} 0 0" rpy="0 0 0" />
                 <geometry>
                 <xacro:if value="${approximate}">
@@ -193,4 +196,5 @@
             <dynamics damping="0.01" friction="0.01" />
         </joint>
+        <!-- Wheel 3 -->
         <link name="right_center_wheel">
             <inertial>
@@ -201,12 +205,13 @@
             </inertial>
             <visual>
-                <origin xyz="0 0 0" rpy="0 0 0" />
-                <geometry>
-                    <mesh
-                        filename="file://$(find urc_gazebo)/urdf/meshes/visual/right_center_wheel.STL" />
-                </geometry>
-            </visual>
-            <collision>
-                <origin xyz="0 0 0" rpy="0 0 0" />
+                <origin xyz="0 0 0" rpy="${pi/2} 0 0" />
+                <geometry>
+                    <cylinder radius="${wheel_radius}" length="${wheel_thickness}" />
+                    <!-- <mesh
+                        filename="file://$(find urc_gazebo)/urdf/meshes/visual/right_center_wheel.STL" /> -->
+                </geometry>
+            </visual>
+            <collision>
+                <origin xyz="0 0 0" rpy="${pi/2} 0 0" />
                 <geometry>
                 <xacro:if value="${approximate}">
@@ -263,4 +268,5 @@
             <dynamics damping="60" friction="4" />
         </joint>
+        <!-- Wheel 4 -->
         <link name="left_rear_wheel">
             <inertial>
@@ -271,12 +277,13 @@
             </inertial>
             <visual>
-                <origin xyz="0 0 0" rpy="0 0 0" />
-                <geometry>
-                    <mesh
-                        filename="file://$(find urc_gazebo)/urdf/meshes/visual/left_rear_wheel.STL" />
-                </geometry>
-            </visual>
-            <collision>
-                <origin xyz="0 0 0" rpy="0 0 0" />
+                <origin xyz="0 0 0" rpy="${pi/2} 0 0" />
+                <geometry>
+                <cylinder radius="${wheel_radius}" length="${wheel_thickness}" />
+                    <!-- <mesh
+                        filename="file://$(find urc_gazebo)/urdf/meshes/visual/left_rear_wheel.STL" /> -->
+                </geometry>
+            </visual>
+            <collision>
+                <origin xyz="0 0 0" rpy="${pi/2} 0 0" />
                 <geometry>
                 <xacro:if value="${approximate}">
@@ -333,4 +340,5 @@
             <dynamics damping="60" friction="4" />
         </joint>
+        <!-- Wheel 5 -->
         <link name="left_front_wheel">
             <inertial>
@@ -341,12 +349,13 @@
             </inertial>
             <visual>
-                <origin xyz="0 0 0" rpy="0 0 0" />
-                <geometry>
-                    <mesh
-                        filename="file://$(find urc_gazebo)/urdf/meshes/visual/left_front_wheel.STL" />
-                </geometry>
-            </visual>
-            <collision>
-                <origin xyz="0 0 0" rpy="0 0 0" />
+                <origin xyz="0 0 0" rpy="${pi/2} 0 0" />
+                <geometry>
+                <cylinder radius="${wheel_radius}" length="${wheel_thickness}" />
+                    <!-- <mesh
+                        filename="file://$(find urc_gazebo)/urdf/meshes/visual/left_front_wheel.STL" /> -->
+                </geometry>
+            </visual>
+            <collision>
+                <origin xyz="0 0 0" rpy="${pi/2} 0 0" />
                 <geometry>
                 <xacro:if value="${approximate}">
@@ -375,4 +384,5 @@
             <dynamics damping="0.01" friction="0.01" />
         </joint>
+        <!-- Wheel 6 -->
         <link name="left_center_wheel">
             <inertial>
@@ -383,12 +393,13 @@
             </inertial>
             <visual>
-                <origin xyz="0 0 0" rpy="0 0 0" />
-                <geometry>
-                    <mesh
-                        filename="file://$(find urc_gazebo)/urdf/meshes/visual/left_center_wheel.STL" />
-                </geometry>
-            </visual>
-            <collision>
-                <origin xyz="0 0 0" rpy="0 0 0" />
+                <origin xyz="0 0 0" rpy="${pi/2} 0 0" />
+                <geometry>
+                <cylinder radius="${wheel_radius}" length="${wheel_thickness}" />
+                    <!-- <mesh
+                        filename="file://$(find urc_gazebo)/urdf/meshes/visual/left_center_wheel.STL" /> -->
+                </geometry>
+            </visual>
+            <collision>
+                <origin xyz="0 0 0" rpy="${pi/2} 0 0" />
                 <geometry>
                 <xacro:if value="${approximate}">

File: urc_hw_description/urdf/walli.xacro (robot description, xacro)
@@ -11,5 +11,5 @@
    <xacro:include filename="$(find urc_hw_description)/urdf/drivebase.xacro" />
    <xacro:include filename="$(find urc_hw_description)/urdf/arm.xacro" />
-   <xacro:drivebase wheel_friction="0.012" wheel_radius="0.10" wheel_thickness="0.05"
+   <xacro:drivebase wheel_friction="0.012" wheel_radius="0.05" wheel_thickness="0.025"
       approximate="true" />
    <xacro:arm />
