Commit message: fix: updating arm simulation and moveit

File: urc_hw_description/urdf/drivebase.xacro (robot description, xacro)
@@ -17,5 +17,6 @@
         <parent link="base_link"/>
         <child link="${prefix}_link"/>
-        <origin xyz="${x_reflect*wheel_xoff} ${y_reflect*(base_width/2+wheel_ygap)} ${-wheel_zoff}" rpy="0 0 0"/>
+        <origin xyz="${x_reflect*wheel_xoff} ${y_reflect*(base_width/2+wheel_ygap)} ${-wheel_zoff}" rpy="0
+    0 0"/>
         <axis xyz="0 1 0"/>
         </joint>
@@ -160,10 +161,10 @@
                 <origin xyz="0 0 0" rpy="0 0 0" />
                 <geometry>
-                <xacro:if value="${approximate}">
-                        <cylinder radius="${wheel_radius}" length="${wheel_thickness}" />
-                    </xacro:if>
-                    <xacro:if value="${not approximate}">
-                    <mesh
-                        filename="file://$(find urc_gazebo)/urdf/meshes/collision/right_rear_wheel_collision.STL" />
+                    <xacro:if value="${approximate}">
+                        <cylinder radius="${wheel_radius}" length="${wheel_thickness}" />
+                    </xacro:if>
+                    <xacro:if value="${not approximate}">
+                        <mesh
+                            filename="file://$(find urc_gazebo)/urdf/meshes/collision/right_rear_wheel_collision.STL" />
                     </xacro:if>
                 </geometry>
@@ -210,10 +211,10 @@
                 <origin xyz="0 0 0" rpy="0 0 0" />
                 <geometry>
-                <xacro:if value="${approximate}">
-                        <cylinder radius="${wheel_radius}" length="${wheel_thickness}" />
-                    </xacro:if>
-                    <xacro:if value="${not approximate}">
-                    <mesh
-                        filename="file://$(find urc_gazebo)/urdf/meshes/collision/right_center_wheel_collision.STL" />
+                    <xacro:if value="${approximate}">
+                        <cylinder radius="${wheel_radius}" length="${wheel_thickness}" />
+                    </xacro:if>
+                    <xacro:if value="${not approximate}">
+                        <mesh
+                            filename="file://$(find urc_gazebo)/urdf/meshes/collision/right_center_wheel_collision.STL" />
                     </xacro:if>
                 </geometry>
@@ -280,10 +281,10 @@
                 <origin xyz="0 0 0" rpy="0 0 0" />
                 <geometry>
-                <xacro:if value="${approximate}">
-                        <cylinder radius="${wheel_radius}" length="${wheel_thickness}" />
-                    </xacro:if>
-                    <xacro:if value="${not approximate}">
-                    <mesh
-                        filename="file://$(find urc_gazebo)/urdf/meshes/collision/left_rear_wheel_collision.STL" />
+                    <xacro:if value="${approximate}">
+                        <cylinder radius="${wheel_radius}" length="${wheel_thickness}" />
+                    </xacro:if>
+                    <xacro:if value="${not approximate}">
+                        <mesh
+                            filename="file://$(find urc_gazebo)/urdf/meshes/collision/left_rear_wheel_collision.STL" />
                     </xacro:if>
                 </geometry>
@@ -350,10 +351,10 @@
                 <origin xyz="0 0 0" rpy="0 0 0" />
                 <geometry>
-                <xacro:if value="${approximate}">
-                        <cylinder radius="${wheel_radius}" length="${wheel_thickness}" />
-                    </xacro:if>
-                    <xacro:if value="${not approximate}">
-                    <mesh
-                        filename="file://$(find urc_gazebo)/urdf/meshes/collision/left_front_wheel_collision.STL" />
+                    <xacro:if value="${approximate}">
+                        <cylinder radius="${wheel_radius}" length="${wheel_thickness}" />
+                    </xacro:if>
+                    <xacro:if value="${not approximate}">
+                        <mesh
+                            filename="file://$(find urc_gazebo)/urdf/meshes/collision/left_front_wheel_collision.STL" />
                     </xacro:if>
                 </geometry>
@@ -392,10 +393,10 @@
                 <origin xyz="0 0 0" rpy="0 0 0" />
                 <geometry>
-                <xacro:if value="${approximate}">
-                        <cylinder radius="${wheel_radius}" length="${wheel_thickness}" />
-                    </xacro:if>
-                    <xacro:if value="${not approximate}">
-                    <mesh
-                        filename="file://$(find urc_gazebo)/urdf/meshes/collision/left_center_wheel_collision.STL" />
+                    <xacro:if value="${approximate}">
+                        <cylinder radius="${wheel_radius}" length="${wheel_thickness}" />
+                    </xacro:if>
+                    <xacro:if value="${not approximate}">
+                        <mesh
+                            filename="file://$(find urc_gazebo)/urdf/meshes/collision/left_center_wheel_collision.STL" />
                     </xacro:if>
                 </geometry>

File: urc_hw_description/urdf/walli.xacro (robot description, xacro)
@@ -1,3 +1,3 @@
-<?xml version="1.0" encoding="UTF-8"?>
+<?xml version="1.0"?>
 <robot name="walli" xmlns:xacro="http://ros.org/wiki/xacro">
    <xacro:property name="config_file"
@@ -12,5 +12,5 @@
    <xacro:include filename="$(find urc_hw_description)/urdf/arm.xacro" />
    <xacro:drivebase wheel_friction="0.012" wheel_radius="0.10" wheel_thickness="0.05"
-      approximate="true" />
+      approximate="false" />
    <xacro:arm />
    <xacro:ros2_control use_simulation="${use_simulation}"

Commit message: feat: arm pinocchio implementation

File: urc_hw_description/urdf/drivebase.xacro (robot description, xacro)
@@ -23,8 +23,14 @@
     </xacro:macro> -->
     <xacro:macro name="drivebase" params="wheel_radius wheel_thickness wheel_friction approximate">
+        <link name="world" />
+        <joint name="fixed" type="fixed">
+            <parent link="world" />
+            <child link="base_link" />
+            <origin xyz="0.0 0.0 0.0" rpy="0.0 0.0 0.0" />
+        </joint>
         <link name="base_link">
             <inertial>
                 <origin xyz="-0.22771 0.0020794 0.13424" rpy="0 0 0" />
-                <mass value="2.485" />
+                <mass value="4.0" />
                 <inertia ixx="0.017201" ixy="-2.0986E-11" ixz="5.8899E-06" iyy="0.0028906"
                     iyz="5.0336E-07"

File: urc_hw_description/urdf/ros2_control.xacro (robot description, xacro)
@@ -111,4 +111,13 @@
         </joint>
         <joint name="rightgripperjoint">
+          <command_interface name="position" />
+          <command_interface name="velocity" />
+          <command_interface name="effort" />
+          <state_interface name="position">
+            <param name="initial_value">${initial_positions['rightgripperjoint']}</param>
+          </state_interface>
+          <state_interface name="velocity" />
+        </joint>
+        <joint name="leftgripperjoint">
           <command_interface name="position" />
           <command_interface name="velocity" />

Commit message: fix: diff_drive_controller params

File: urc_hw_description/urdf/drivebase.xacro (robot description, xacro)
@@ -23,10 +23,4 @@
     </xacro:macro> -->
     <xacro:macro name="drivebase" params="wheel_radius wheel_thickness wheel_friction approximate">
-        <link name="world" />
-        <joint name="fixed" type="fixed">
-            <parent link="world" />
-            <child link="base_link" />
-            <origin xyz="0.0 0.0 0.0" rpy="0.0 0.0 0.0" />
-        </joint>
         <link name="base_link">
             <inertial>

File: urc_hw_description/urdf/ros2_control.xacro (robot description, xacro)
@@ -153,6 +153,6 @@
         <hardware>
           <plugin>urc_hw/RoverDrivetrain</plugin>
-          <param name="udp_address">127.0.0.1</param>
-          <param name="udp_port">5000</param>
+          <param name="udp_address">192.168.1.100</param>
+          <param name="udp_port">8443</param>
         </hardware>
         <joint name="left_wheel">
