Commit message: Better sim

File: urc_hw_description/urdf/drivebase.xacro (robot description, xacro)
@@ -1,25 +1,4 @@
 <?xml version="1.0"?>
 <robot xmlns:xacro="http://www.ros.org/wiki/xacro">
-    <!-- Approximated Wheel -->
-    <!-- <xacro:macro name="approximate_wheel" params="prefix x_reflect y_reflect">
-        <link name="${prefix}_link">
-        <visual>
-            <origin xyz="0 0 0" rpy="${pi/2} 0 0"/>
-            <geometry>
-                <cylinder radius="${wheel_radius}" length="${wheel_width}"/>
-            </geometry>
-            <material name="Gray">
-            <color rgba="0.5 0.5 0.5 1.0"/>
-            </material>
-        </visual>
-        </link>
-        <joint name="${prefix}_joint" type="continuous">
-        <parent link="base_link"/>
-        <child link="${prefix}_link"/>
-        <origin xyz="${x_reflect*wheel_xoff} ${y_reflect*(base_width/2+wheel_ygap)} ${-wheel_zoff}" rpy="0
-    0 0"/>
-        <axis xyz="0 1 0"/>
-        </joint>
-    </xacro:macro> -->
     <xacro:macro name="drivebase" params="wheel_radius wheel_thickness wheel_friction approximate">
         <link name="base_link">
@@ -27,7 +6,7 @@
                 <origin xyz="-0.22771 0.0020794 0.13424" rpy="0 0 0" />
                 <mass value="4.0" />
-                <inertia ixx="0.017201" ixy="-2.0986E-11" ixz="5.8899E-06" iyy="0.0028906"
+                <inertia ixx="0.17201" ixy="-2.0986E-11" ixz="5.8899E-06" iyy="0.028906"
                     iyz="5.0336E-07"
-                    izz="0.019124" />
+                    izz="0.19124" />
             </inertial>
             <visual>
@@ -49,6 +28,6 @@
                 <origin xyz="0.062687 0.034616 -0.016048" rpy="0 0 0" />
                 <mass value="0.57523" />
-                <inertia ixx="0.00040232" ixy="-8.4972E-11" ixz="-0.00023706" iyy="0.00095582"
-                    iyz="-4.2951E-08" izz="0.00061776" />
+                <inertia ixx="0.0040232" ixy="-8.4972E-11" ixz="-0.00023706" iyy="0.0095582"
+                    iyz="-4.2951E-08" izz="0.0061776" />
             </inertial>
             <visual>
@@ -70,6 +49,7 @@
             <parent link="base_link" />
             <child link="rightrocker" />
-            <axis xyz="0 0 0" />
-            <dynamics damping="0.01" friction="0.01" />
+            <axis xyz="0 1 0" />
+            <dynamics damping="0.9" friction="0.01" />
+            <limit effort="1000.0" lower="${-pi/20}" upper="${pi/20}" velocity="0.1" />
         </joint>
         <!-- Wheel 1 -->
@@ -101,4 +81,10 @@
             </collision>
             <surface>
+                <contact>
+                    <ode>
+                        <kp>1e15</kp>
+                        <kd>1</kd>
+                    </ode>
+                </contact>
                 <friction>
                     <ode>
@@ -120,6 +106,6 @@
                 <origin xyz="-6.8787E-09 0.032385 -0.015429" rpy="0 0 0" />
                 <mass value="0.66758" />
-                <inertia ixx="0.00019756" ixy="-5.9804E-10" ixz="9.4624E-11" iyy="0.00044836"
-                    iyz="2.6509E-13" izz="0.0003846" />
+                <inertia ixx="0.019756" ixy="-5.9804E-10" ixz="9.4624E-11" iyy="0.044836"
+                    iyz="2.6509E-13" izz="0.03846" />
             </inertial>
             <visual>
@@ -141,6 +127,7 @@
             <parent link="rightrocker" />
             <child link="rightbogie" />
-            <axis xyz="0 0 0" />
-            <dynamics damping="0.02" friction="0" />
+            <axis xyz="0 1 0" />
+            <dynamics damping="0.9" friction="0.01" />
+            <limit effort="1000.0" lower="${-pi/20}" upper="${pi/20}" velocity="0.1" />
         </joint>
         <link name="right_front_wheel">
@@ -171,12 +158,10 @@
             </collision>
             <surface>
-                <friction>
-                    <ode>
-                        <mu>${wheel_friction}</mu>
-                        <mu2>${wheel_friction}</mu2>
-                    </ode>
-                </friction>
-            </surface>
-            <surface>
+                <contact>
+                    <ode>
+                        <kp>1e15</kp>
+                        <kd>1</kd>
+                    </ode>
+                </contact>
                 <friction>
                     <ode>
@@ -221,4 +206,10 @@
             </collision>
             <surface>
+                <contact>
+                    <ode>
+                        <kp>1e15</kp>
+                        <kd>1</kd>
+                    </ode>
+                </contact>
                 <friction>
                     <ode>
@@ -240,5 +231,5 @@
                 <origin xyz="0.065435 -0.034981 -0.01685" rpy="0 0 0" />
                 <mass value="0.58415" />
-                <inertia ixx="0.0004044" ixy="-5.259E-11" ixz="-0.00023722" iyy="0.00095925"
+                <inertia ixx="0.004044" ixy="-5.259E-11" ixz="-0.0023722" iyy="0.0095925"
                     iyz="-4.2951E-08" izz="0.00061912" />
             </inertial>
@@ -261,6 +252,7 @@
             <parent link="base_link" />
             <child link="leftrocker" />
-            <axis xyz="0 0 0" />
-            <dynamics damping="60" friction="4" />
+            <axis xyz="0 1 0" />
+            <dynamics damping="0.9" friction="0.01" />
+            <limit effort="1000.0" lower="${-pi/20}" upper="${pi/20}" velocity="0.1" />
         </joint>
         <link name="left_rear_wheel">
@@ -291,4 +283,10 @@
             </collision>
             <surface>
+                <contact>
+                    <ode>
+                        <kp>1e15</kp>
+                        <kd>1</kd>
+                    </ode>
+                </contact>
                 <friction>
                     <ode>
@@ -310,6 +308,6 @@
                 <origin xyz="-6.8787E-09 -0.032385 -0.015429" rpy="0 0 0" />
                 <mass value="0.66758" />
-                <inertia ixx="0.00019756" ixy="-5.9804E-10" ixz="9.4624E-11" iyy="0.00044836"
-                    iyz="2.6509E-13" izz="0.0003846" />
+                <inertia ixx="0.019756" ixy="-5.9804E-10" ixz="9.4624E-11" iyy="0.044836"
+                    iyz="2.6509E-13" izz="0.03846" />
             </inertial>
             <visual>
@@ -331,6 +329,7 @@
             <parent link="leftrocker" />
             <child link="leftbogie" />
-            <axis xyz="0 0 0" />
-            <dynamics damping="60" friction="4" />
+            <axis xyz="0 1 0" />
+            <dynamics damping="0.9" friction="0.01" />
+            <limit effort="1000.0" lower="${-pi/20}" upper="${pi/20}" velocity="0.1" />
         </joint>
         <link name="left_front_wheel">
@@ -343,8 +342,15 @@
             <visual>
                 <origin xyz="0 0 0" rpy="0 0 0" />
-                <geometry>
-                    <mesh
-                        filename="file://$(find urc_gazebo)/urdf/meshes/visual/left_front_wheel.STL" />
-                </geometry>
+                <xacro:if value="${approximate}">
+                    <geometry>
+                        <cylinder radius="${wheel_radius}" length="${wheel_thickness}" />
+                    </geometry>
+                </xacro:if>
+                <xacro:if value="${not approximate}">
+                    <geometry>
+                        <mesh
+                            filename="file://$(find urc_gazebo)/urdf/meshes/visual/left_front_wheel.STL" />
+                    </geometry>
+                </xacro:if>
             </visual>
             <collision>
@@ -361,4 +367,10 @@
             </collision>
             <surface>
+                <contact>
+                    <ode>
+                        <kp>1e15</kp>
+                        <kd>1</kd>
+                    </ode>
+                </contact>
                 <friction>
                     <ode>
@@ -403,4 +415,10 @@
             </collision>
             <surface>
+                <contact>
+                    <ode>
+                        <kp>1e15</kp>
+                        <kd>1</kd>
+                    </ode>
+                </contact>
                 <friction>
                     <ode>

File: urc_hw_description/urdf/walli.xacro (robot description, xacro)
@@ -9,7 +9,7 @@
    <xacro:include filename="$(find urc_hw_description)/urdf/walli_sensors.xacro" />
    <xacro:include filename="$(find urc_hw_description)/urdf/ros2_control.xacro" />
-   <xacro:include filename="$(find urc_hw_description)/urdf/drivebase.xacro" />
+   <xacro:include filename="$(find urc_hw_description)/urdf/new_drivebase.xacro" />
    <xacro:include filename="$(find urc_hw_description)/urdf/arm.xacro" />
-   <xacro:drivebase wheel_friction="0.012" wheel_radius="0.10" wheel_thickness="0.05"
+   <xacro:drivebase mu="1.0" mu2="0.25" wheel_radius="0.1" wheel_thickness="0.05"
       approximate="false" />
    <!-- <xacro:arm /> -->

File: urc_hw_description/urdf/walli_drivebase.xacro (robot description, xacro)
@@ -1,4 +1,25 @@
 <?xml version="1.0"?>
 <robot xmlns:xacro="http://www.ros.org/wiki/xacro">
+    <!-- Approximated Wheel -->
+    <!-- <xacro:macro name="approximate_wheel" params="prefix x_reflect y_reflect">
+        <link name="${prefix}_link">
+        <visual>
+            <origin xyz="0 0 0" rpy="${pi/2} 0 0"/>
+            <geometry>
+                <cylinder radius="${wheel_radius}" length="${wheel_width}"/>
+            </geometry>
+            <material name="Gray">
+            <color rgba="0.5 0.5 0.5 1.0"/>
+            </material>
+        </visual>
+        </link>
+        <joint name="${prefix}_joint" type="continuous">
+        <parent link="base_link"/>
+        <child link="${prefix}_link"/>
+        <origin xyz="${x_reflect*wheel_xoff} ${y_reflect*(base_width/2+wheel_ygap)} ${-wheel_zoff}" rpy="0
+    0 0"/>
+        <axis xyz="0 1 0"/>
+        </joint>
+    </xacro:macro> -->
     <xacro:macro name="drivebase" params="wheel_radius wheel_thickness wheel_friction approximate">
         <link name="base_link">
@@ -65,5 +86,5 @@
                     <!-- <mesh
                         filename="file://$(find urc_gazebo)/urdf/meshes/visual/right_rear_wheel.STL" /> -->
-                        <cylinder radius="${wheel_radius}" length="${wheel_thickness}" />
+                    <cylinder radius="${wheel_radius}" length="${wheel_thickness}" />
                 </geometry>
             </visual>
@@ -135,5 +156,5 @@
                 <origin xyz="0 0 0" rpy="${pi/2} 0 0" />
                 <geometry>
-                <cylinder radius="${wheel_radius}" length="${wheel_thickness}" />
+                    <cylinder radius="${wheel_radius}" length="${wheel_thickness}" />
                     <!-- <mesh
                         filename="file://$(find urc_gazebo)/urdf/meshes/visual/right_front_wheel.STL" /> -->
@@ -143,10 +164,10 @@
                 <origin xyz="${pi/2} 0 0" rpy="0 0 0" />
                 <geometry>
-                <xacro:if value="${approximate}">
-                        <cylinder radius="${wheel_radius}" length="${wheel_thickness}" />
-                    </xacro:if>
-                    <xacro:if value="${not approximate}">
-                    <mesh
-                        filename="file://$(find urc_gazebo)/urdf/meshes/collision/right_rear_wheel_collision.STL" />
+                    <xacro:if value="${approximate}">
+                        <cylinder radius="${wheel_radius}" length="${wheel_thickness}" />
+                    </xacro:if>
+                    <xacro:if value="${not approximate}">
+                        <mesh
+                            filename="file://$(find urc_gazebo)/urdf/meshes/collision/right_rear_wheel_collision.STL" />
                     </xacro:if>
                 </geometry>
@@ -195,10 +216,10 @@
                 <origin xyz="0 0 0" rpy="${pi/2} 0 0" />
                 <geometry>
-                <xacro:if value="${approximate}">
-                        <cylinder radius="${wheel_radius}" length="${wheel_thickness}" />
-                    </xacro:if>
-                    <xacro:if value="${not approximate}">
-                    <mesh
-                        filename="file://$(find urc_gazebo)/urdf/meshes/collision/right_center_wheel_collision.STL" />
+                    <xacro:if value="${approximate}">
+                        <cylinder radius="${wheel_radius}" length="${wheel_thickness}" />
+                    </xacro:if>
+                    <xacro:if value="${not approximate}">
+                        <mesh
+                            filename="file://$(find urc_gazebo)/urdf/meshes/collision/right_center_wheel_collision.STL" />
                     </xacro:if>
                 </geometry>
@@ -259,5 +280,5 @@
                 <origin xyz="0 0 0" rpy="${pi/2} 0 0" />
                 <geometry>
-                <cylinder radius="${wheel_radius}" length="${wheel_thickness}" />
+                    <cylinder radius="${wheel_radius}" length="${wheel_thickness}" />
                     <!-- <mesh
                         filename="file://$(find urc_gazebo)/urdf/meshes/visual/left_rear_wheel.STL" /> -->
@@ -267,10 +288,10 @@
                 <origin xyz="0 0 0" rpy="${pi/2} 0 0" />
                 <geometry>
-                <xacro:if value="${approximate}">
-                        <cylinder radius="${wheel_radius}" length="${wheel_thickness}" />
-                    </xacro:if>
-                    <xacro:if value="${not approximate}">
-                    <mesh
-                        filename="file://$(find urc_gazebo)/urdf/meshes/collision/left_rear_wheel_collision.STL" />
+                    <xacro:if value="${approximate}">
+                        <cylinder radius="${wheel_radius}" length="${wheel_thickness}" />
+                    </xacro:if>
+                    <xacro:if value="${not approximate}">
+                        <mesh
+                            filename="file://$(find urc_gazebo)/urdf/meshes/collision/left_rear_wheel_collision.STL" />
                     </xacro:if>
                 </geometry>
@@ -331,5 +352,5 @@
                 <origin xyz="0 0 0" rpy="${pi/2} 0 0" />
                 <geometry>
-                <cylinder radius="${wheel_radius}" length="${wheel_thickness}" />
+                    <cylinder radius="${wheel_radius}" length="${wheel_thickness}" />
                     <!-- <mesh
                         filename="file://$(find urc_gazebo)/urdf/meshes/visual/left_front_wheel.STL" /> -->
@@ -339,10 +360,10 @@
                 <origin xyz="0 0 0" rpy="${pi/2} 0 0" />
                 <geometry>
-                <xacro:if value="${approximate}">
-                        <cylinder radius="${wheel_radius}" length="${wheel_thickness}" />
-                    </xacro:if>
-                    <xacro:if value="${not approximate}">
-                    <mesh
-                        filename="file://$(find urc_gazebo)/urdf/meshes/collision/left_front_wheel_collision.STL" />
+                    <xacro:if value="${approximate}">
+                        <cylinder radius="${wheel_radius}" length="${wheel_thickness}" />
+                    </xacro:if>
+                    <xacro:if value="${not approximate}">
+                        <mesh
+                            filename="file://$(find urc_gazebo)/urdf/meshes/collision/left_front_wheel_collision.STL" />
                     </xacro:if>
                 </geometry>
@@ -375,5 +396,5 @@
                 <origin xyz="0 0 0" rpy="${pi/2} 0 0" />
                 <geometry>
-                <cylinder radius="${wheel_radius}" length="${wheel_thickness}" />
+                    <cylinder radius="${wheel_radius}" length="${wheel_thickness}" />
                     <!-- <mesh
                         filename="file://$(find urc_gazebo)/urdf/meshes/visual/left_center_wheel.STL" /> -->
@@ -383,10 +404,10 @@
                 <origin xyz="0 0 0" rpy="${pi/2} 0 0" />
                 <geometry>
-                <xacro:if value="${approximate}">
-                        <cylinder radius="${wheel_radius}" length="${wheel_thickness}" />
-                    </xacro:if>
-                    <xacro:if value="${not approximate}">
-                    <mesh
-                        filename="file://$(find urc_gazebo)/urdf/meshes/collision/left_center_wheel_collision.STL" />
+                    <xacro:if value="${approximate}">
+                        <cylinder radius="${wheel_radius}" length="${wheel_thickness}" />
+                    </xacro:if>
+                    <xacro:if value="${not approximate}">
+                        <mesh
+                            filename="file://$(find urc_gazebo)/urdf/meshes/collision/left_center_wheel_collision.STL" />
                     </xacro:if>
                 </geometry>
