Commit message: Cleanup

File: urc_hw_description/urdf/drivebase.xacro (robot description, xacro)
@@ -1,30 +1,9 @@
 <?xml version="1.0"?>
 <robot xmlns:xacro="http://www.ros.org/wiki/xacro">
-    <!-- Approximated Wheel -->
-    <!-- <xacro:macro name="approximate_wheel" params="prefix x_reflect y_reflect">
-        <link name="${prefix}_link">
-        <visual>
-            <origin xyz="0 0 0" rpy="${pi/2} 0 0"/>
-            <geometry>
-                <cylinder radius="${wheel_radius}" length="${wheel_width}"/>
-            </geometry>
-            <material name="Gray">
-            <color rgba="0.5 0.5 0.5 1.0"/>
-            </material>
-        </visual>
-        </link>
-        <joint name="${prefix}_joint" type="continuous">
-        <parent link="base_link"/>
-        <child link="${prefix}_link"/>
-        <origin xyz="${x_reflect*wheel_xoff} ${y_reflect*(base_width/2+wheel_ygap)} ${-wheel_zoff}" rpy="0
-    0 0"/>
-        <axis xyz="0 1 0"/>
-        </joint>
-    </xacro:macro> -->
-    <xacro:macro name="drivebase" params="wheel_radius wheel_thickness wheel_friction approximate">
+    <xacro:macro name="drivebase" params="wheel_radius wheel_thickness mu mu2 approximate">
         <link name="base_link">
             <inertial>
                 <origin xyz="-0.22771 0.0020794 0.13424" rpy="0 0 0" />
-                <mass value="4.0" />
+                <mass value="1.584994" />
                 <inertia ixx="0.017201" ixy="-2.0986E-11" ixz="5.8899E-06" iyy="0.0028906"
                     iyz="5.0336E-07"
@@ -45,10 +24,13 @@
             </collision>
         </link>
+        <!-- ROCKERS -->
         <link name="rightrocker">
             <inertial>
                 <origin xyz="0.062687 0.034616 -0.016048" rpy="0 0 0" />
-                <mass value="0.57523" />
-                <inertia ixx="0.00040232" ixy="-8.4972E-11" ixz="-0.00023706" iyy="0.00095582"
-                    iyz="-4.2951E-08" izz="0.00061776" />
+                <mass value="1.387336" />
+                <inertia
+                    ixx="0.002956" ixy="-0.000001489324" ixz="-0.000008103407"
+                    iyy="0.02924" iyz="0.00007112"
+                    izz="0.02832" />
             </inertial>
             <visual>
@@ -66,60 +48,50 @@
             </collision>
         </link>
-        <joint name="rightrockerjoint" type="fixed">
+        <joint name="rightrockerjoint" type="revolute">
             <origin xyz="-0.194 -0.33715 0.080295" rpy="0 0 0" />
             <parent link="base_link" />
             <child link="rightrocker" />
-            <axis xyz="0 0 0" />
-            <dynamics damping="0.01" friction="0.01" />
-        </joint>
-        <!-- Wheel 1 -->
-        <link name="right_rear_wheel">
-            <inertial>
-                <origin xyz="0.0010497 0.10248 0.00012788" rpy="0 0 0" />
-                <mass value="0.65429" />
-                <inertia ixx="0.00040499" ixy="-2.9713E-08" ixz="-2.8347E-07" iyy="0.00055081"
-                    iyz="2.6154E-08" izz="0.00040532" />
-            </inertial>
-            <visual>
-                <origin xyz="0 0 0" rpy="0 0 0" />
-                <geometry>
-                    <mesh
-                        filename="file://$(find urc_gazebo)/urdf/meshes/visual/right_rear_wheel.STL" />
-                </geometry>
-            </visual>
-            <collision>
-                <origin xyz="0 0 0" rpy="0 0 0" />
-                <geometry>
-                    <xacro:if value="${approximate}">
-                        <cylinder radius="${wheel_radius}" length="${wheel_thickness}" />
-                    </xacro:if>
-                    <xacro:if value="${not approximate}">
-                        <mesh
-                            filename="file://$(find urc_gazebo)/urdf/meshes/collision/right_rear_wheel_collision.STL" />
-                    </xacro:if>
-                </geometry>
-            </collision>
-            <surface>
-                <friction>
-                    <ode>
-                        <mu>${wheel_friction}</mu>
-                        <mu2>${wheel_friction}</mu2>
-                    </ode>
-                </friction>
-            </surface>
-        </link>
-        <joint name="right_rear_wheel_joint" type="continuous">
-            <origin xyz="-0.36316 -0.17103 -0.19158" rpy="0 0 0" />
-            <parent link="rightrocker" />
-            <child link="right_rear_wheel" />
-            <axis xyz="0 1 0" />
-            <dynamics damping="0.01" friction="0.01" />
-        </joint>
+            <axis xyz="0 1 0" />
+            <limit effort="0.0" lower="-0.24" upper="0.24" velocity="100.0" />
+            <dynamics friction="1.0" damping="0.1" />
+        </joint>
+        <link name="leftrocker">
+            <inertial>
+                <origin xyz="0.065435 -0.034981 -0.01685" rpy="0 0 0" />
+                <mass value="1.387336" />
+                <inertia
+                    ixx="0.002956" ixy="-0.000001489324" ixz="-0.000008103407"
+                    iyy="0.02924" iyz="0.00007112"
+                    izz="0.02832" />
+            </inertial>
+            <visual>
+                <origin xyz="0 0 0" rpy="0 0 0" />
+                <geometry>
+                    <mesh filename="file://$(find urc_gazebo)/urdf/meshes/visual/leftrocker.STL" />
+                </geometry>
+            </visual>
+            <collision>
+                <origin xyz="0 0 0" rpy="0 0 0" />
+                <geometry>
+                    <mesh
+                        filename="file://$(find urc_gazebo)/urdf/meshes/collision/leftrocker_collision.STL" />
+                </geometry>
+            </collision>
+        </link>
+        <joint name="leftrockerjoint" type="revolute">
+            <origin xyz="-0.19241 0.33715 0.080257" rpy="0 0 0" />
+            <parent link="base_link" />
+            <child link="leftrocker" />
+            <axis xyz="0 1 0" />
+            <limit effort="0.0" lower="-0.24" upper="0.24" velocity="100.0" />
+            <dynamics friction="1.0" damping="0.1" />
+        </joint>
+        <!-- BOGIES -->
         <link name="rightbogie">
             <inertial>
                 <origin xyz="-6.8787E-09 0.032385 -0.015429" rpy="0 0 0" />
                 <mass value="0.66758" />
-                <inertia ixx="0.00019756" ixy="-5.9804E-10" ixz="9.4624E-11" iyy="0.00044836"
-                    iyz="2.6509E-13" izz="0.0003846" />
+                <inertia ixx="0.0019756" ixy="-5.9804E-10" ixz="9.4624E-11" iyy="0.0044836"
+                    iyz="2.6509E-13" izz="0.003846" />
             </inertial>
             <visual>
@@ -137,172 +109,11 @@
             </collision>
         </link>
-        <joint name="rightbogiejoint" type="fixed">
+        <joint name="rightbogiejoint" type="revolute">
             <origin xyz="0.24177 -0.00254 -0.074203" rpy="0 0 0" />
             <parent link="rightrocker" />
             <child link="rightbogie" />
-            <axis xyz="0 0 0" />
-            <dynamics damping="0.02" friction="0" />
-        </joint>
-        <link name="right_front_wheel">
-            <inertial>
-                <origin xyz="-0.00066285 0.10248 0.00082496" rpy="0 0 0" />
-                <mass value="0.65429" />
-                <inertia ixx="0.000405" ixy="-2.1882E-08" ixz="2.5112E-07" iyy="0.00055081"
-                    iyz="-4.9845E-08" izz="0.00040531" />
-            </inertial>
-            <visual>
-                <origin xyz="0 0 0" rpy="0 0 0" />
-                <geometry>
-                    <mesh
-                        filename="file://$(find urc_gazebo)/urdf/meshes/visual/right_front_wheel.STL" />
-                </geometry>
-            </visual>
-            <collision>
-                <origin xyz="0 0 0" rpy="0 0 0" />
-                <geometry>
-                    <xacro:if value="${approximate}">
-                        <cylinder radius="${wheel_radius}" length="${wheel_thickness}" />
-                    </xacro:if>
-                    <xacro:if value="${not approximate}">
-                        <mesh
-                            filename="file://$(find urc_gazebo)/urdf/meshes/collision/right_rear_wheel_collision.STL" />
-                    </xacro:if>
-                </geometry>
-            </collision>
-            <surface>
-                <friction>
-                    <ode>
-                        <mu>${wheel_friction}</mu>
-                        <mu2>${wheel_friction}</mu2>
-                    </ode>
-                </friction>
-            </surface>
-            <surface>
-                <friction>
-                    <ode>
-                        <mu>${wheel_friction}</mu>
-                        <mu2>${wheel_friction}</mu2>
-                    </ode>
-                </friction>
-            </surface>
-        </link>
-        <joint name="right_front_wheel_joint" type="continuous">
-            <origin xyz="0.20139 -0.16849 -0.11671" rpy="0 0 0" />
-            <parent link="rightbogie" />
-            <child link="right_front_wheel" />
-            <axis xyz="0 1 0" />
-            <dynamics damping="0.01" friction="0.01" />
-        </joint>
-        <link name="right_center_wheel">
-            <inertial>
-                <origin xyz="0.0010444 0.10248 0.00016665" rpy="0 0 0" />
-                <mass value="0.65429" />
-                <inertia ixx="0.00040501" ixy="-3.1023E-08" ixz="-2.9568E-07" iyy="0.00055081"
-                    iyz="2.5206E-08" izz="0.0004053" />
-            </inertial>
-            <visual>
-                <origin xyz="0 0 0" rpy="0 0 0" />
-                <geometry>
-                    <mesh
-                        filename="file://$(find urc_gazebo)/urdf/meshes/visual/right_center_wheel.STL" />
-                </geometry>
-            </visual>
-            <collision>
-                <origin xyz="0 0 0" rpy="0 0 0" />
-                <geometry>
-                    <xacro:if value="${approximate}">
-                        <cylinder radius="${wheel_radius}" length="${wheel_thickness}" />
-                    </xacro:if>
-                    <xacro:if value="${not approximate}">
-                        <mesh
-                            filename="file://$(find urc_gazebo)/urdf/meshes/collision/right_center_wheel_collision.STL" />
-                    </xacro:if>
-                </geometry>
-            </collision>
-            <surface>
-                <friction>
-                    <ode>
-                        <mu>${wheel_friction}</mu>
-                        <mu2>${wheel_friction}</mu2>
-                    </ode>
-                </friction>
-            </surface>
-        </link>
-        <joint name="right_center_wheel_joint" type="continuous">
-            <origin xyz="-0.20177 -0.16849 -0.11606" rpy="0 0 0" />
-            <parent link="rightbogie" />
-            <child link="right_center_wheel" />
-            <axis xyz="0 1 0" />
-            <dynamics damping="0.01" friction="0.01" />
-        </joint>
-        <link name="leftrocker">
-            <inertial>
-                <origin xyz="0.065435 -0.034981 -0.01685" rpy="0 0 0" />
-                <mass value="0.58415" />
-                <inertia ixx="0.0004044" ixy="-5.259E-11" ixz="-0.00023722" iyy="0.00095925"
-                    iyz="-4.2951E-08" izz="0.00061912" />
-            </inertial>
-            <visual>
-                <origin xyz="0 0 0" rpy="0 0 0" />
-                <geometry>
-                    <mesh filename="file://$(find urc_gazebo)/urdf/meshes/visual/leftrocker.STL" />
-                </geometry>
-            </visual>
-            <collision>
-                <origin xyz="0 0 0" rpy="0 0 0" />
-                <geometry>
-                    <mesh
-                        filename="file://$(find urc_gazebo)/urdf/meshes/collision/leftrocker_collision.STL" />
-                </geometry>
-            </collision>
-        </link>
-        <joint name="leftrockerjoint" type="fixed">
-            <origin xyz="-0.19241 0.33715 0.080257" rpy="0 0 0" />
-            <parent link="base_link" />
-            <child link="leftrocker" />
-            <axis xyz="0 0 0" />
-            <dynamics damping="60" friction="4" />
-        </joint>
-        <link name="left_rear_wheel">
-            <inertial>
-                <origin xyz="0.00069452 -0.10248 0.00079886" rpy="0 0 0" />
-                <mass value="0.65433" />
-                <inertia ixx="0.00040509" ixy="-4.8144E-09" ixz="-2.5925E-07" iyy="0.00055097"
-                    iyz="4.0749E-08" izz="0.00040552" />
-            </inertial>
-            <visual>
-                <origin xyz="0 0 0" rpy="0 0 0" />
-                <geometry>
-                    <mesh
-                        filename="file://$(find urc_gazebo)/urdf/meshes/visual/left_rear_wheel.STL" />
-                </geometry>
-            </visual>
-            <collision>
-                <origin xyz="0 0 0" rpy="0 0 0" />
-                <geometry>
-                    <xacro:if value="${approximate}">
-                        <cylinder radius="${wheel_radius}" length="${wheel_thickness}" />
-                    </xacro:if>
-                    <xacro:if value="${not approximate}">
-                        <mesh
-                            filename="file://$(find urc_gazebo)/urdf/meshes/collision/left_rear_wheel_collision.STL" />
-                    </xacro:if>
-                </geometry>
-            </collision>
-            <surface>
-                <friction>
-                    <ode>
-                        <mu>${wheel_friction}</mu>
-                        <mu2>${wheel_friction}</mu2>
-                    </ode>
-                </friction>
-            </surface>
-        </link>
-        <joint name="left_rear_wheel_joint" type="continuous">
-            <origin xyz="-0.36266 0.17103 -0.19248" rpy="0 0 0" />
-            <parent link="leftrocker" />
-            <child link="left_rear_wheel" />
-            <axis xyz="0 1 0" />
-            <dynamics damping="0.01" friction="0.01" />
+            <axis xyz="0 1 0" />
+            <limit effort="0.0" lower="-0.24" upper="0.24" velocity="100.0" />
+            <dynamics friction="1.0" damping="0.1" />
         </joint>
         <link name="leftbogie">
@@ -310,6 +121,6 @@
                 <origin xyz="-6.8787E-09 -0.032385 -0.015429" rpy="0 0 0" />
                 <mass value="0.66758" />
-                <inertia ixx="0.00019756" ixy="-5.9804E-10" ixz="9.4624E-11" iyy="0.00044836"
-                    iyz="2.6509E-13" izz="0.0003846" />
+                <inertia ixx="0.0019756" ixy="-5.9804E-10" ixz="9.4624E-11" iyy="0.0044836"
+                    iyz="2.6509E-13" izz="0.003846" />
             </inertial>
             <visual>
@@ -327,94 +138,174 @@
             </collision>
         </link>
-        <joint name="leftbogiejoint" type="fixed">
+        <joint name="leftbogiejoint" type="revolute">
             <origin xyz="0.24182 0.00254 -0.073984" rpy="0 0 0" />
             <parent link="leftrocker" />
             <child link="leftbogie" />
-            <axis xyz="0 0 0" />
-            <dynamics damping="60" friction="4" />
+            <axis xyz="0 1 0" />
+            <limit effort="0.0" lower="-0.24" upper="0.24" velocity="100.0" />
+            <dynamics friction="1.0" damping="0.1" />
+        </joint>
+        <!-- WHEELS -->
+        <link name="right_rear_wheel">
+            <inertial>
+                <origin xyz="0 0 0" rpy="0 0 0" />
+                <mass value="0.283642" />
+                <inertia ixx="0.000391" ixy="0.00000123962" ixz="5.52582e-7" iyy="0.0004716"
+                    iyz="-0.000002082042" izz="0.000391" />
+            </inertial>
+            <visual>
+                <origin xyz="0 0 0" rpy="${pi/2} 0 0" />
+                <geometry>
+                    <cylinder radius="${wheel_radius}" length="${wheel_thickness}" />
+                </geometry>
+            </visual>
+            <collision>
+                <origin xyz="0 0 0" rpy="${pi/2} 0 0" />
+                <geometry>
+                    <cylinder radius="${wheel_radius}" length="${wheel_thickness}" />
+                </geometry>
+            </collision>
+        </link>
+        <joint name="right_rear_wheel_joint" type="continuous">
+            <origin xyz="-0.36316 -0.04 -0.19158" rpy="0 0 0" />
+            <parent link="rightrocker" />
+            <child link="right_rear_wheel" />
+            <axis xyz="0 1 0" />
+            <dynamics friction="0.3125" damping="0.1" />
+        </joint>
+        <link name="right_front_wheel">
+            <inertial>
+                <origin xyz="0 0 0" rpy="0 0 0" />
+                <mass value="0.283642" />
+                <inertia ixx="0.000391" ixy="0.00000123962" ixz="5.52582e-7" iyy="0.0004716"
+                    iyz="-0.000002082042" izz="0.000391" />
+            </inertial>
+            <visual>
+                <origin xyz="0 0 0" rpy="${pi/2} 0 0" />
+                <geometry>
+                    <cylinder radius="${wheel_radius}" length="${wheel_thickness}" />
+                </geometry>
+            </visual>
+            <collision>
+                <origin xyz="0 0 0" rpy="${pi/2} 0 0" />
+                <geometry>
+                    <cylinder radius="${wheel_radius}" length="${wheel_thickness}" />
+                </geometry>
+            </collision>
+        </link>
+        <joint name="right_front_wheel_joint" type="continuous">
+            <origin xyz="0.20139 -0.04 -0.11671" rpy="0 0 0" />
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
File: urc_hw_description/urdf/ros2_control.xacro (robot description, xacro)
@@ -8,12 +8,5 @@
       <ros2_control name="GazeboSystem" type="system">
         <hardware>
-          <!-- TODO make a launch param to switch between real/fake hardware. You can only use ONE. -->
-          <!--Use
-          for functionality in Gazebo, also needed for drivetrain-->
           <plugin>gazebo_ros2_control/GazeboSystem</plugin>
-          <!--Use
-          for functionality in RViz-->
-          <!-- <plugin>mock_components/GenericSystem</plugin> -->
-          <!-- <plugin>ros2_control_demo_hardware/VelocityActuatorHardware</plugin> -->
         </hardware>
         <joint name="leftbogiejoint">

File: urc_hw_description/urdf/walli.xacro (robot description, xacro)
@@ -1,13 +1,15 @@
 <?xml version="1.0"?>
 <robot name="walli" xmlns:xacro="http://ros.org/wiki/xacro">
-   <xacro:property name="config_file"
+   <!-- <xacro:property name="config_file"
       value="$(find urc_bringup)/config/hardware_config.yaml" />
    <xacro:property name="config_data" value="${load_yaml(config_file)}"></xacro:property>
-   <xacro:property name="use_simulation" value="${config_data['hardware_config']['use_simulation']}" />
+   <xacro:property name="use_simulation" value="${config_data['hardware_config']['use_simulation']}"
+   /> -->
+   <xacro:arg name="use_simulation" default="true" />
    <xacro:include filename="$(find urc_hw_description)/urdf/walli_prop.xacro" />
    <xacro:include filename="$(find urc_hw_description)/urdf/walli_inertials.xacro" />
    <xacro:include filename="$(find urc_hw_description)/urdf/walli_sensors.xacro" />
    <xacro:include filename="$(find urc_hw_description)/urdf/ros2_control.xacro" />
-   <xacro:include filename="$(find urc_hw_description)/urdf/new_drivebase.xacro" />
+   <xacro:include filename="$(find urc_hw_description)/urdf/drivebase.xacro" />
    <xacro:include filename="$(find urc_hw_description)/urdf/arm.xacro" />
    <xacro:drivebase mu="1.0" mu2="0.25" wheel_radius="0.1" wheel_thickness="0.08"
