Commit message: Cleanup

File: urc_hw_description/urdf/walli_drivebase.xacro (robot description, xacro)
@@ -1,29 +1,9 @@
 <?xml version="1.0"?>
 <robot xmlns:xacro="http://www.ros.org/wiki/xacro">
-    <!-- Approximated Wheel -->
-    <!-- <xacro:macro name="approximate_wheel" params="prefix x_reflect y_reflect">
-        <link name="${prefix}_link">
-        <visual>
-            <origin xyz="0 0 0" rpy="${pi/2} 0 0"/>
-            <geometry>
-                <cylinder radius="${wheel_radius}" length="${wheel_width}"/>
-            </geometry>
-            <material name="Gray">
-            <color rgba="0.5 0.5 0.5 1.0"/>
-            </material>
-        </visual>
-        </link>
-        <joint name="${prefix}_joint" type="continuous">
-        <parent link="base_link"/>
-        <child link="${prefix}_link"/>
-        <origin xyz="${x_reflect*wheel_xoff} ${y_reflect*(base_width/2+wheel_ygap)} ${-wheel_zoff}" rpy="0 0 0"/>
-        <axis xyz="0 1 0"/>
-        </joint>
-    </xacro:macro> -->
     <xacro:macro name="drivebase" params="wheel_radius wheel_thickness wheel_friction approximate">
         <link name="base_link">
             <inertial>
-                <origin xyz="-0.22771 0.0020794 1" rpy="0 0 0" />
-                <mass value="2.485" />
+                <origin xyz="-0.22771 0.0020794 0.13424" rpy="0 0 0" />
+                <mass value="4.0" />
                 <inertia ixx="0.017201" ixy="-2.0986E-11" ixz="5.8899E-06" iyy="0.0028906"
                     iyz="5.0336E-07"
@@ -81,13 +61,12 @@
             </inertial>
             <visual>
-                <origin xyz="0 0 0" rpy="${pi/2} 0 0" />
-                <geometry>
-                    <!-- <mesh
-                        filename="file://$(find urc_gazebo)/urdf/meshes/visual/right_rear_wheel.STL" /> -->
-                        <cylinder radius="${wheel_radius}" length="${wheel_thickness}" />
-                </geometry>
-            </visual>
-            <collision>
-                <origin xyz="0 0 0" rpy="${pi/2} 0 0" />
+                <origin xyz="0 0 0" rpy="0 0 0" />
+                <geometry>
+                    <mesh
+                        filename="file://$(find urc_gazebo)/urdf/meshes/visual/right_rear_wheel.STL" />
+                </geometry>
+            </visual>
+            <collision>
+                <origin xyz="0 0 0" rpy="0 0 0" />
                 <geometry>
                     <xacro:if value="${approximate}">
@@ -144,5 +123,4 @@
             <dynamics damping="0.02" friction="0" />
         </joint>
-        <!-- Wheel 2 -->
         <link name="right_front_wheel">
             <inertial>
@@ -153,20 +131,19 @@
             </inertial>
             <visual>
-                <origin xyz="0 0 0" rpy="${pi/2} 0 0" />
-                <geometry>
-                <cylinder radius="${wheel_radius}" length="${wheel_thickness}" />
-                    <!-- <mesh
-                        filename="file://$(find urc_gazebo)/urdf/meshes/visual/right_front_wheel.STL" /> -->
-                </geometry>
-            </visual>
-            <collision>
-                <origin xyz="${pi/2} 0 0" rpy="0 0 0" />
-                <geometry>
-                <xacro:if value="${approximate}">
-                        <cylinder radius="${wheel_radius}" length="${wheel_thickness}" />
-                    </xacro:if>
-                    <xacro:if value="${not approximate}">
-                    <mesh
-                        filename="file://$(find urc_gazebo)/urdf/meshes/collision/right_rear_wheel_collision.STL" />
+                <origin xyz="0 0 0" rpy="0 0 0" />
+                <geometry>
+                    <mesh
+                        filename="file://$(find urc_gazebo)/urdf/meshes/visual/right_front_wheel.STL" />
+                </geometry>
+            </visual>
+            <collision>
+                <origin xyz="0 0 0" rpy="0 0 0" />
+                <geometry>
+                    <xacro:if value="${approximate}">
+                        <cylinder radius="${wheel_radius}" length="${wheel_thickness}" />
+                    </xacro:if>
+                    <xacro:if value="${not approximate}">
+                        <mesh
+                            filename="file://$(find urc_gazebo)/urdf/meshes/collision/right_rear_wheel_collision.STL" />
                     </xacro:if>
                 </geometry>
@@ -196,5 +173,4 @@
             <dynamics damping="0.01" friction="0.01" />
         </joint>
-        <!-- Wheel 3 -->
         <link name="right_center_wheel">
             <inertial>
@@ -205,20 +181,19 @@
             </inertial>
             <visual>
-                <origin xyz="0 0 0" rpy="${pi/2} 0 0" />
-                <geometry>
-                    <cylinder radius="${wheel_radius}" length="${wheel_thickness}" />
-                    <!-- <mesh
-                        filename="file://$(find urc_gazebo)/urdf/meshes/visual/right_center_wheel.STL" /> -->
-                </geometry>
-            </visual>
-            <collision>
-                <origin xyz="0 0 0" rpy="${pi/2} 0 0" />
-                <geometry>
-                <xacro:if value="${approximate}">
-                        <cylinder radius="${wheel_radius}" length="${wheel_thickness}" />
-                    </xacro:if>
-                    <xacro:if value="${not approximate}">
-                    <mesh
-                        filename="file://$(find urc_gazebo)/urdf/meshes/collision/right_center_wheel_collision.STL" />
+                <origin xyz="0 0 0" rpy="0 0 0" />
+                <geometry>
+                    <mesh
+                        filename="file://$(find urc_gazebo)/urdf/meshes/visual/right_center_wheel.STL" />
+                </geometry>
+            </visual>
+            <collision>
+                <origin xyz="0 0 0" rpy="0 0 0" />
+                <geometry>
+                    <xacro:if value="${approximate}">
+                        <cylinder radius="${wheel_radius}" length="${wheel_thickness}" />
+                    </xacro:if>
+                    <xacro:if value="${not approximate}">
+                        <mesh
+                            filename="file://$(find urc_gazebo)/urdf/meshes/collision/right_center_wheel_collision.STL" />
                     </xacro:if>
                 </geometry>
@@ -268,5 +243,4 @@
             <dynamics damping="60" friction="4" />
         </joint>
-        <!-- Wheel 4 -->
         <link name="left_rear_wheel">
             <inertial>
@@ -277,20 +251,19 @@
             </inertial>
             <visual>
-                <origin xyz="0 0 0" rpy="${pi/2} 0 0" />
-                <geometry>
-                <cylinder radius="${wheel_radius}" length="${wheel_thickness}" />
-                    <!-- <mesh
-                        filename="file://$(find urc_gazebo)/urdf/meshes/visual/left_rear_wheel.STL" /> -->
-                </geometry>
-            </visual>
-            <collision>
-                <origin xyz="0 0 0" rpy="${pi/2} 0 0" />
-                <geometry>
-                <xacro:if value="${approximate}">
-                        <cylinder radius="${wheel_radius}" length="${wheel_thickness}" />
-                    </xacro:if>
-                    <xacro:if value="${not approximate}">
-                    <mesh
-                        filename="file://$(find urc_gazebo)/urdf/meshes/collision/left_rear_wheel_collision.STL" />
+                <origin xyz="0 0 0" rpy="0 0 0" />
+                <geometry>
+                    <mesh
+                        filename="file://$(find urc_gazebo)/urdf/meshes/visual/left_rear_wheel.STL" />
+                </geometry>
+            </visual>
+            <collision>
+                <origin xyz="0 0 0" rpy="0 0 0" />
+                <geometry>
+                    <xacro:if value="${approximate}">
+                        <cylinder radius="${wheel_radius}" length="${wheel_thickness}" />
+                    </xacro:if>
+                    <xacro:if value="${not approximate}">
+                        <mesh
+                            filename="file://$(find urc_gazebo)/urdf/meshes/collision/left_rear_wheel_collision.STL" />
                     </xacro:if>
                 </geometry>
@@ -340,5 +313,4 @@
             <dynamics damping="60" friction="4" />
         </joint>
-        <!-- Wheel 5 -->
         <link name="left_front_wheel">
             <inertial>
@@ -349,20 +321,19 @@
             </inertial>
             <visual>
-                <origin xyz="0 0 0" rpy="${pi/2} 0 0" />
-                <geometry>
-                <cylinder radius="${wheel_radius}" length="${wheel_thickness}" />
-                    <!-- <mesh
-                        filename="file://$(find urc_gazebo)/urdf/meshes/visual/left_front_wheel.STL" /> -->
-                </geometry>
-            </visual>
-            <collision>
-                <origin xyz="0 0 0" rpy="${pi/2} 0 0" />
-                <geometry>
-                <xacro:if value="${approximate}">
-                        <cylinder radius="${wheel_radius}" length="${wheel_thickness}" />
-                    </xacro:if>
-                    <xacro:if value="${not approximate}">
-                    <mesh
-                        filename="file://$(find urc_gazebo)/urdf/meshes/collision/left_front_wheel_collision.STL" />
+                <origin xyz="0 0 0" rpy="0 0 0" />
+                <geometry>
+                    <mesh
+                        filename="file://$(find urc_gazebo)/urdf/meshes/visual/left_front_wheel.STL" />
+                </geometry>
+            </visual>
+            <collision>
+                <origin xyz="0 0 0" rpy="0 0 0" />
+                <geometry>
+                    <xacro:if value="${approximate}">
+                        <cylinder radius="${wheel_radius}" length="${wheel_thickness}" />
+                    </xacro:if>
+                    <xacro:if value="${not approximate}">
+                        <mesh
+                            filename="file://$(find urc_gazebo)/urdf/meshes/collision/left_front_wheel_collision.STL" />
                     </xacro:if>
                 </geometry>
@@ -384,5 +355,4 @@
             <dynamics damping="0.01" friction="0.01" />
         </joint>
-        <!-- Wheel 6 -->
         <link name="left_center_wheel">
             <inertial>
@@ -393,20 +363,19 @@
             </inertial>
             <visual>
-                <origin xyz="0 0 0" rpy="${pi/2} 0 0" />
-                <geometry>
-                <cylinder radius="${wheel_radius}" length="${wheel_thickness}" />
-                    <!-- <mesh
-                        filename="file://$(find urc_gazebo)/urdf/meshes/visual/left_center_wheel.STL" /> -->
-                </geometry>
-            </visual>
-            <collision>
-                <origin xyz="0 0 0" rpy="${pi/2} 0 0" />
-                <geometry>
-                <xacro:if value="${approximate}">
-                        <cylinder radius="${wheel_radius}" length="${wheel_thickness}" />
-                    </xacro:if>
-                    <xacro:if value="${not approximate}">
-                    <mesh
-                        filename="file://$(find urc_gazebo)/urdf/meshes/collision/left_center_wheel_collision.STL" />
+                <origin xyz="0 0 0" rpy="0 0 0" />
+                <geometry>
+                    <mesh
+                        filename="file://$(find urc_gazebo)/urdf/meshes/visual/left_center_wheel.STL" />
+                </geometry>
+            </visual>
+            <collision>
+                <origin xyz="0 0 0" rpy="0 0 0" />
+                <geometry>
+                    <xacro:if value="${approximate}">
+                        <cylinder radius="${wheel_radius}" length="${wheel_thickness}" />
+                    </xacro:if>
+                    <xacro:if value="${not approximate}">
+                        <mesh
+                            filename="file://$(find urc_gazebo)/urdf/meshes/collision/left_center_wheel_collision.STL" />
                     </xacro:if>
                 </geometry>
