Commit message: Hardware Interface & ROS2 Control (#149)
* feat: implementation in progress

* feat: finish urc_hw, adding urc_description

* feat: simple controller and robot description

* feat: working example of hardware interface (no eth)

* fix: urc control bringup error partially resolved

* fix building

* Create common_issues.md

Signed-off-by: David Calderon <davidcalderon03@hotmail.com>

* fix: error during configuration

* fix: crappy minimal working version

* fix: minor updates

* feat: async udp, working example

* fix: add parameter choice for udp address and port

* Added udp tester

* Changed packet size to 1024 instead of 4096 bytes

* feat: refactor & start writing imu

* feat: add status light and imu

* fix: imu and status light bug, add readme

* fix: include bug

* feat: nanopb and implementation in status light

* Added small package.xml modification to allow everything to build

* Added rover hardware interface information from other branch

* refactor: seperate to imu & status light

* refactor: reduce info logging & change cmd name

* fix: update udp_test, working nanopb

* fix: usable nanopb for status light, test imu

* feat: battery management

* Started code for rover hardware interface

* Finished rough version of drivetrain hardware interface

* Corrected some issues with rover drivetrai

* Added science module hardware interface

* feat: bms broadcaster

* Ported urdf to hardware description

* other changes

* feat: diff drive controller

* fix: minor updates

* fix: udp test update (verified working version)

* uncrustify 1

* uncrustify 2

* uncrustify 3

* redid python file formatting

* auto format

* manual linting

* more manual linting

* linting mk4

* cmake linting

* added ros2 control xacro

* added ros2 control xacro

---------

Signed-off-by: David Calderon <davidcalderon03@hotmail.com>
Co-authored-by: Harris Nesteruk <harrislegobrick@gmail.com>
Co-authored-by: David Calderon <davidcalderon03@hotmail.com>

File: urc_hw_description/urdf/walli.xacro (robot description, xacro)
@@ -1,25 +1,24 @@
 <?xml version='1.0'?>
 <robot name="walli" xmlns:xacro="http://www.ros.org/wiki/xacro">
-  <xacro:include filename="walli_prop.xacro"/>
-  <xacro:include filename="walli_inertials.xacro"/>
-  <xacro:include filename="$(find velodyne_description)/urdf/VLP-16.urdf.xacro"/>
-  <xacro:include filename="walli_arm.urdf"/>
-  <xacro:include filename="ros2_control.xacro"/>
+  <xacro:include filename="$(find urc_hw_description)/urdf/walli_prop.xacro" />
+  <xacro:include filename="$(find urc_hw_description)/urdf/walli_inertials.xacro" />
+  <xacro:include filename="$(find velodyne_description)/urdf/VLP-16.urdf.xacro" />
+  <xacro:include filename="$(find urc_hw_description)/urdf/walli_arm.urdf" />
   <!-- Rover Base Link -->
   <link name="base_link">
     <visual>
       <geometry>
-        <box size="${base_length} ${base_width} ${base_height}"/>
+        <box size="${base_length} ${base_width} ${base_height}" />
       </geometry>
       <material name="Cyan">
-        <color rgba="0 1.0 1.0 1.0"/>
+        <color rgba="0 1.0 1.0 1.0" />
       </material>
     </visual>
     <collision>
       <geometry>
-        <box size="${base_length} ${base_width} ${base_height}"/>
+        <box size="${base_length} ${base_width} ${base_height}" />
       </geometry>
     </collision>
-    <xacro:box_inertia m="15" w="${base_width}" d="${base_length}" h="${base_height}"/>
+    <xacro:box_inertia m="15" w="${base_width}" d="${base_length}" h="${base_height}" />
   </link>
   <gazebo reference="base_link">
@@ -32,24 +31,25 @@
         <origin xyz="0 0 0" rpy="${pi/2} 0 0" />
         <geometry>
-          <cylinder radius="${wheel_radius}" length="${wheel_width}"/>
+          <cylinder radius="${wheel_radius}" length="${wheel_width}" />
         </geometry>
         <material name="Gray">
-          <color rgba="0.5 0.5 0.5 1.0"/>
+          <color rgba="0.5 0.5 0.5 1.0" />
         </material>
       </visual>
       <collision>
-        <origin xyz="0 0 0" rpy="${pi/2} 0 0"/>
+        <origin xyz="0 0 0" rpy="${pi/2} 0 0" />
         <geometry>
-          <cylinder radius="${wheel_radius}" length="${wheel_width}"/>
+          <cylinder radius="${wheel_radius}" length="${wheel_width}" />
         </geometry>
       </collision>
-      <xacro:cylinder_inertia m="0.5" r="${wheel_radius}" h="${wheel_width}"/>
+      <xacro:cylinder_inertia m="0.5" r="${wheel_radius}" h="${wheel_width}" />
     </link>
     <joint name="${prefix}_joint" type="continuous">
-      <parent link="base_link"/>
-      <child link="${prefix}_link"/>
-      <origin xyz="${x_reflect*wheel_xoff} ${y_reflect*(base_width/2+wheel_ygap)} ${-wheel_zoff}" rpy="0 0 0"/>
-      <axis xyz="0 1 0"/>
-      <limit effort="${axle_eff_limit}" velocity="${axle_vel_limit}"/>
+      <parent link="base_link" />
+      <child link="${prefix}_link" />
+      <origin xyz="${x_reflect*wheel_xoff} ${y_reflect*(base_width/2+wheel_ygap)} ${-wheel_zoff}"
+        rpy="0 0 0" />
+      <axis xyz="0 1 0" />
+      <limit effort="${axle_eff_limit}" velocity="${axle_vel_limit}" />
       <dynamics damping="0" friction="4.0" />
     </joint>
@@ -58,23 +58,23 @@
     </gazebo>
   </xacro:macro>
-  <xacro:wheel prefix="left_front_wheel"   x_reflect="1" y_reflect="1"/>
-  <xacro:wheel prefix="left_center_wheel"  x_reflect="0" y_reflect="1"/>
-  <xacro:wheel prefix="left_rear_wheel"    x_reflect="-1" y_reflect="1"/>
-  <xacro:wheel prefix="right_front_wheel"  x_reflect="1" y_reflect="-1"/>
-  <xacro:wheel prefix="right_center_wheel" x_reflect="0" y_reflect="-1"/>
-  <xacro:wheel prefix="right_rear_wheel"   x_reflect="-1" y_reflect="-1"/>
+  <xacro:wheel prefix="left_front_wheel" x_reflect="1" y_reflect="1" />
+  <xacro:wheel prefix="left_center_wheel" x_reflect="0" y_reflect="1" />
+  <xacro:wheel prefix="left_rear_wheel" x_reflect="-1" y_reflect="1" />
+  <xacro:wheel prefix="right_front_wheel" x_reflect="1" y_reflect="-1" />
+  <xacro:wheel prefix="right_center_wheel" x_reflect="0" y_reflect="-1" />
+  <xacro:wheel prefix="right_rear_wheel" x_reflect="-1" y_reflect="-1" />
   <!-- Robot Footprint -->
-  <link name="base_footprint"/>
+  <link name="base_footprint" />
   <joint name="base_joint" type="fixed">
-    <parent link="base_link"/>
-    <child link="base_footprint"/>
-    <origin xyz="0.0 0.0 ${-(wheel_radius+wheel_zoff)}" rpy="0 0 0"/>
+    <parent link="base_link" />
+    <child link="base_footprint" />
+    <origin xyz="0.0 0.0 ${-(wheel_radius+wheel_zoff)}" rpy="0 0 0" />
   </joint>
   <!-- Arm Joint -->
   <joint name="arm_to_rover" type="fixed">
-    <origin rpy="0 0 0" xyz="0 0 0"/>
-    <parent link="base_link"/>
-    <child link="arm_base_link"/>
-    <dynamics damping="60.0" friction="4.0"/>
+    <origin rpy="0 0 0" xyz="0 0 0" />
+    <parent link="base_link" />
+    <child link="arm_base_link" />
+    <dynamics damping="60.0" friction="4.0" />
   </joint>
   <!-- IMU -->
@@ -82,21 +82,21 @@
     <visual>
       <geometry>
-        <box size="0.1 0.1 0.1"/>
+        <box size="0.1 0.1 0.1" />
       </geometry>
     </visual>
     <collision>
       <geometry>
-        <box size="0.1 0.1 0.1"/>
+        <box size="0.1 0.1 0.1" />
       </geometry>
     </collision>
-    <xacro:box_inertia m="0.1" w="0.1" d="0.1" h="0.1"/>
+    <xacro:box_inertia m="0.1" w="0.1" d="0.1" h="0.1" />
   </link>
   <joint name="imu_joint" type="fixed">
-		<axis xyz="1 0 0"/>
-		<origin xyz="0 0 0.05"/>
-		<parent link="base_link"/>
-		<child link="imu_link"/>
-	</joint>
-	<gazebo reference="imu_link">
+    <axis xyz="1 0 0" />
+    <origin xyz="0 0 0.05" />
+    <parent link="base_link" />
+    <child link="imu_link" />
+  </joint>
+  <gazebo reference="imu_link">
     <sensor name="imu_sensor" type="imu">
       <plugin filename="libgazebo_ros_imu_sensor.so" name="imu_plugin">
@@ -110,8 +110,8 @@
       <update_rate>100</update_rate>
       <visualize>true</visualize>
-     <imu>
-     	<angular_velocity>
-     	  <x>
-     	    <noise type="gaussian">
+      <imu>
+        <angular_velocity>
+          <x>
+            <noise type="gaussian">
               <mean>0.0</mean>
               <stddev>2e-4</stddev>
@@ -167,120 +167,121 @@
   </gazebo>
   <gazebo>
-  <plugin name='diff_drive' filename='libgazebo_ros_diff_drive.so'>
-    <ros>
-      <namespace>/sensor</namespace>
-    </ros>
-    <!-- wheels -->
-    <left_joint>left_front_wheel_joint</left_joint>
-    <right_joint>right_front_wheel_joint</right_joint>
-    <!-- kinematics -->
-    <wheel_separation>0.4</wheel_separation>
-    <wheel_diameter>0.2</wheel_diameter>
-    <!-- limits -->
-    <max_wheel_torque>20</max_wheel_torque>
-    <max_wheel_acceleration>1.0</max_wheel_acceleration>
-    <!-- output -->
-    <publish_odom>true</publish_odom>
-    <publish_odom_tf>false</publish_odom_tf>
-    <publish_wheel_tf>true</publish_wheel_tf>
-    <odometry_frame>odom</odometry_frame>
-    <robot_base_frame>base_link</robot_base_frame>
-  </plugin>
-</gazebo>
+    <plugin name='diff_drive' filename='libgazebo_ros_diff_drive.so'>
+      <ros>
+        <namespace>/sensor</namespace>
+      </ros>
+      <!-- wheels -->
+      <left_joint>left_front_wheel_joint</left_joint>
+      <right_joint>right_front_wheel_joint</right_joint>
+      <!-- kinematics -->
+      <wheel_separation>0.4</wheel_separation>
+      <wheel_diameter>0.2</wheel_diameter>
+      <!-- limits -->
+      <max_wheel_torque>20</max_wheel_torque>
+      <max_wheel_acceleration>1.0</max_wheel_acceleration>
+      <!-- output -->
+      <publish_odom>true</publish_odom>
+      <publish_odom_tf>false</publish_odom_tf>
+      <publish_wheel_tf>true</publish_wheel_tf>
+      <odometry_frame>odom</odometry_frame>
+      <robot_base_frame>base_link</robot_base_frame>
+    </plugin>
+  </gazebo>
   <!-- GPS -->
   <link name="gps">
     <visual>
       <geometry>
-        <box size="0.1 0.1 0.1"/>
+        <box size="0.1 0.1 0.1" />
       </geometry>
     </visual>
     <collision>
       <geometry>
-        <box size="0.1 0.1 0.1"/>
+        <box size="0.1 0.1 0.1" />
       </geometry>
     </collision>
-    <xacro:box_inertia m="0.1" w="0.1" d="0.1" h="0.1"/>
+    <xacro:box_inertia m="0.1" w="0.1" d="0.1" h="0.1" />
   </link>
-   <joint name="gps_joint" type="fixed">
-		<axis xyz="1 0 0"/>
-		<origin xyz="0 0 0.05"/>
-		<parent link="base_link"/>
-		<child link="gps"/>
-	</joint>
+  <joint name="gps_joint" type="fixed">
+    <axis xyz="1 0 0" />
+    <origin xyz="0 0 0.05" />
+    <parent link="base_link" />
+    <child link="gps" />
+  </joint>
   <gazebo reference="gps">
     <sensor name="gps" type="gps">
       <plugin filename="libgazebo_ros_gps_sensor.so" name="gps_plugin">
-          <ros>
-            <namespace>/gps</namespace>
-            <remapping>~/out:=data</remapping>
-          </ros>
-          <frame_name>gps</frame_name>
-        </plugin>
-        <always_on>true</always_on>
-        <updateRate>30</updateRate>
+        <ros>
+          <namespace>/gps</namespace>
+          <remapping>~/out:=data</remapping>
+        </ros>
+        <frame_name>gps</frame_name>
+      </plugin>
+      <always_on>true</always_on>
+      <updateRate>30</updateRate>
     </sensor>
   </gazebo>
-   <!-- LIDAR -->
+  <!-- LIDAR -->
   <link name="lidar_link">
     <inertial>
-      <origin xyz="0 0 0" rpy="0 0 0"/>
-      <mass value="0.125"/>
-      <inertia ixx="0.001"  ixy="0"  ixz="0" iyy="0.001" iyz="0" izz="0.001" />
+      <origin xyz="0 0 0" rpy="0 0 0" />
+      <mass value="0.125" />
+      <inertia ixx="0.001" ixy="0" ixz="0" iyy="0.001" iyz="0" izz="0.001" />
     </inertial>
     <collision>
-      <origin xyz="0 0 0" rpy="0 0 0"/>
-      <geometry>
-        <cylinder radius="0.0508" length="0.055"/>
+      <origin xyz="0 0 0" rpy="0 0 0" />
+      <geometry>
+        <cylinder radius="0.0508" length="0.055" />
       </geometry>
     </collision>
     <visual>
-      <origin xyz="0 0 0" rpy="0 0 0"/>
-      <geometry>
-        <cylinder radius="0.0508" length="0.055"/>
+      <origin xyz="0 0 0" rpy="0 0 0" />
+      <geometry>
+        <cylinder radius="0.0508" length="0.055" />
       </geometry>
     </visual>
   </link>
   <joint name="lidar_joint" type="fixed">
-    <parent link="base_link"/>
-    <child link="lidar_link"/>
-    <origin xyz="0.0 0.0 0.1" rpy="0.0 0.0 0.0"/>
-  </joint>
-  <!-- <xacro:VLP-16 parent="lidar_link" name="lidar" topic="/scan" hz="${lidar_hz}" samples="${lidar_samples}" gpu="false">
+    <parent link="base_link" />
+    <child link="lidar_link" />
+    <origin xyz="0.0 0.0 0.1" rpy="0.0 0.0 0.0" />
+  </joint>
+  <!-- <xacro:VLP-16 parent="lidar_link" name="lidar" topic="/scan" hz="${lidar_hz}"
+  samples="${lidar_samples}" gpu="false">
     <origin xyz="${lidar_x} 0.0 ${lidar_z}" rpy="0 ${lidar_pitch} 0" />
   </xacro:VLP-16> -->
   <gazebo reference="lidar_link">
-  <sensor name="lidar" type="ray">
-    <always_on>true</always_on>
-    <visualize>true</visualize>
-    <update_rate>5</update_rate>
-    <ray>
-      <scan>
-        <horizontal>
-          <samples>360</samples>
-          <resolution>1.000000</resolution>
-          <min_angle>0.000000</min_angle>
-          <max_angle>6.280000</max_angle>
-        </horizontal>
-      </scan>
-      <range>
-        <min>0.12</min>
-        <max>3.5</max>
-        <resolution>0.015000</resolution>
-      </range>
-      <noise>
-        <type>gaussian</type>
-        <mean>0.0</mean>
-        <stddev>0.01</stddev>
-      </noise>
-    </ray>
-    <plugin name="scan" filename="libgazebo_ros_ray_sensor.so">
-      <ros>
-        <remapping>~/out:=scan</remapping>
-      </ros>
-      <output_type>sensor_msgs/LaserScan</output_type>
-      <frame_name>lidar_link</frame_name>
-    </plugin>
-  </sensor>
-</gazebo>
+    <sensor name="lidar" type="ray">
+      <always_on>true</always_on>
+      <visualize>true</visualize>
+      <update_rate>5</update_rate>
+      <ray>
+        <scan>
+          <horizontal>
+            <samples>360</samples>
+            <resolution>1.000000</resolution>
+            <min_angle>0.000000</min_angle>
+            <max_angle>6.280000</max_angle>
+          </horizontal>
+        </scan>
+        <range>
+          <min>0.12</min>
+          <max>3.5</max>
+          <resolution>0.015000</resolution>
+        </range>
+        <noise>
+          <type>gaussian</type>
+          <mean>0.0</mean>
+          <stddev>0.01</stddev>
+        </noise>
+      </ray>
+      <plugin name="scan" filename="libgazebo_ros_ray_sensor.so">
+        <ros>
+          <remapping>~/out:=scan</remapping>
+        </ros>
+        <output_type>sensor_msgs/LaserScan</output_type>
+        <frame_name>lidar_link</frame_name>
+      </plugin>
+    </sensor>
+  </gazebo>
   <!-- May want to change this to a depth camera -->
   <xacro:macro name="camera" params="orientation origin_x origin_y origin_z yaw">
@@ -288,20 +289,20 @@
       <visual>
         <geometry>
-          <box size="0.01 0.01 0.01"/>
+          <box size="0.01 0.01 0.01" />
         </geometry>
       </visual>
       <collision>
         <geometry>
-          <box size="0.01 0.01 0.01"/>
+          <box size="0.01 0.01 0.01" />
         </geometry>
       </collision>
-      <xacro:box_inertia m="0.01" w="0.01" d="0.01" h="0.01"/>
+      <xacro:box_inertia m="0.01" w="0.01" d="0.01" h="0.01" />
     </link>
     <joint name="${orientation}_cam_joint" type="fixed">
-  	  <axis xyz="1 0 0"/>
+      <axis xyz="1 0 0" />
       <!-- Camera Orientation-->
-	    <origin xyz="${origin_x} ${origin_y} ${origin_z}" rpy = "0 0 ${yaw}"/>
-	    <parent link="base_link"/>
-	    <child link="cam/${orientation}"/>
+      <origin xyz="${origin_x} ${origin_y} ${origin_z}" rpy="0 0 ${yaw}" />
+      <parent link="base_link" />
+      <child link="cam/${orientation}" />
     </joint>
     <gazebo reference="cam/${orientation}">
@@ -341,74 +342,74 @@
     </gazebo>
   </xacro:macro>
-  <xacro:camera orientation="center" origin_x="0.1" origin_y="0"    origin_z="0" yaw="-0.14"/>
-  <xacro:camera orientation="left"   origin_x="0"    origin_y="0.1"  origin_z="0"    yaw="1.5"/>
-  <xacro:camera orientation="right"  origin_x="0"    origin_y="-0.1" origin_z="0"    yaw="-1.5"/>
-<!-- Depth Camera (addition for Nav2) -->
-<link name="camera_link">
-  <visual>
-    <origin xyz="0 0 0" rpy="0 0 0"/>
-    <geometry>
-      <box size="0.015 0.130 0.022"/>
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