Commit message: [cleanup] deleted files which may not be needed anymore (#225)
* Deleted files which I believe we do not need anymore

* readded urc scripts

* linting

File: urc_hw_description/urdf/arm.xacro (robot description, xacro)
@@ -13,12 +13,12 @@
                 <origin xyz="0 0 0" rpy="0 0 0" />
                 <geometry>
-                    <mesh filename="file://$(find urc_gazebo)/urdf/meshes/visual/spine.STL" />
-                </geometry>
-            </visual>
-            <collision>
-                <origin xyz="0 0 0" rpy="0 0 0" />
-                <geometry>
-                    <mesh
-                        filename="file://$(find urc_gazebo)/urdf/meshes/collision/spine_collision.STL" />
+                    <mesh filename="file://$(find urc_hw_description)/urdf/meshes/visual/spine.STL" />
+                </geometry>
+            </visual>
+            <collision>
+                <origin xyz="0 0 0" rpy="0 0 0" />
+                <geometry>
+                    <mesh
+                        filename="file://$(find urc_hw_description)/urdf/meshes/collision/spine_collision.STL" />
                 </geometry>
             </collision>
@@ -40,12 +40,12 @@
                 <origin xyz="0 0 0" rpy="0 0 0" />
                 <geometry>
-                    <mesh filename="file://$(find urc_gazebo)/urdf/meshes/visual/shoulder.STL" />
-                </geometry>
-            </visual>
-            <collision>
-                <origin xyz="0 0 0" rpy="0 0 0" />
-                <geometry>
-                    <mesh
-                        filename="file://$(find urc_gazebo)/urdf/meshes/collision/shoulder_collision.STL" />
+                    <mesh filename="file://$(find urc_hw_description)/urdf/meshes/visual/shoulder.STL" />
+                </geometry>
+            </visual>
+            <collision>
+                <origin xyz="0 0 0" rpy="0 0 0" />
+                <geometry>
+                    <mesh
+                        filename="file://$(find urc_hw_description)/urdf/meshes/collision/shoulder_collision.STL" />
                 </geometry>
             </collision>
@@ -69,12 +69,12 @@
                 <origin xyz="0 0 0" rpy="0 0 0" />
                 <geometry>
-                    <mesh filename="file://$(find urc_gazebo)/urdf/meshes/visual/bicep.STL" />
-                </geometry>
-            </visual>
-            <collision>
-                <origin xyz="0 0 0" rpy="0 0 0" />
-                <geometry>
-                    <mesh
-                        filename="file://$(find urc_gazebo)/urdf/meshes/collision/bicep_collision.STL" />
+                    <mesh filename="file://$(find urc_hw_description)/urdf/meshes/visual/bicep.STL" />
+                </geometry>
+            </visual>
+            <collision>
+                <origin xyz="0 0 0" rpy="0 0 0" />
+                <geometry>
+                    <mesh
+                        filename="file://$(find urc_hw_description)/urdf/meshes/collision/bicep_collision.STL" />
                 </geometry>
             </collision>
@@ -98,12 +98,12 @@
                 <origin xyz="0 0 0" rpy="0 0 0" />
                 <geometry>
-                    <mesh filename="file://$(find urc_gazebo)/urdf/meshes/visual/elbow.STL" />
-                </geometry>
-            </visual>
-            <collision>
-                <origin xyz="0 0 0" rpy="0 0 0" />
-                <geometry>
-                    <mesh
-                        filename="file://$(find urc_gazebo)/urdf/meshes/collision/elbow_collision.STL" />
+                    <mesh filename="file://$(find urc_hw_description)/urdf/meshes/visual/elbow.STL" />
+                </geometry>
+            </visual>
+            <collision>
+                <origin xyz="0 0 0" rpy="0 0 0" />
+                <geometry>
+                    <mesh
+                        filename="file://$(find urc_hw_description)/urdf/meshes/collision/elbow_collision.STL" />
                 </geometry>
             </collision>
@@ -127,12 +127,12 @@
                 <origin xyz="0 0 0" rpy="0 0 0" />
                 <geometry>
-                    <mesh filename="file://$(find urc_gazebo)/urdf/meshes/visual/wrist.STL" />
-                </geometry>
-            </visual>
-            <collision>
-                <origin xyz="0 0 0" rpy="0 0 0" />
-                <geometry>
-                    <mesh
-                        filename="file://$(find urc_gazebo)/urdf/meshes/collision/wrist_collision.STL" />
+                    <mesh filename="file://$(find urc_hw_description)/urdf/meshes/visual/wrist.STL" />
+                </geometry>
+            </visual>
+            <collision>
+                <origin xyz="0 0 0" rpy="0 0 0" />
+                <geometry>
+                    <mesh
+                        filename="file://$(find urc_hw_description)/urdf/meshes/collision/wrist_collision.STL" />
                 </geometry>
             </collision>
@@ -156,12 +156,12 @@
                 <origin xyz="0 0 0" rpy="0 0 0" />
                 <geometry>
-                    <mesh filename="file://$(find urc_gazebo)/urdf/meshes/visual/claw.STL" />
-                </geometry>
-            </visual>
-            <collision>
-                <origin xyz="0 0 0" rpy="0 0 0" />
-                <geometry>
-                    <mesh
-                        filename="file://$(find urc_gazebo)/urdf/meshes/collision/claw_collision.STL" />
+                    <mesh filename="file://$(find urc_hw_description)/urdf/meshes/visual/claw.STL" />
+                </geometry>
+            </visual>
+            <collision>
+                <origin xyz="0 0 0" rpy="0 0 0" />
+                <geometry>
+                    <mesh
+                        filename="file://$(find urc_hw_description)/urdf/meshes/collision/claw_collision.STL" />
                 </geometry>
             </collision>
@@ -185,12 +185,12 @@
                 <origin xyz="0 0 0" rpy="0 0 0" />
                 <geometry>
-                    <mesh filename="file://$(find urc_gazebo)/urdf/meshes/visual/rightgripper.STL" />
-                </geometry>
-            </visual>
-            <collision>
-                <origin xyz="0 0 0" rpy="0 0 0" />
-                <geometry>
-                    <mesh
-                        filename="file://$(find urc_gazebo)/urdf/meshes/collision/rightgripper_collision.STL" />
+                    <mesh filename="file://$(find urc_hw_description)/urdf/meshes/visual/rightgripper.STL" />
+                </geometry>
+            </visual>
+            <collision>
+                <origin xyz="0 0 0" rpy="0 0 0" />
+                <geometry>
+                    <mesh
+                        filename="file://$(find urc_hw_description)/urdf/meshes/collision/rightgripper_collision.STL" />
                 </geometry>
             </collision>
@@ -214,12 +214,12 @@
                 <origin xyz="0 0 0" rpy="0 0 0" />
                 <geometry>
-                    <mesh filename="file://$(find urc_gazebo)/urdf/meshes/visual/leftgripper.STL" />
-                </geometry>
-            </visual>
-            <collision>
-                <origin xyz="0 0 0" rpy="0 0 0" />
-                <geometry>
-                    <mesh
-                        filename="file://$(find urc_gazebo)/urdf/meshes/collision/leftgripper_collision.STL" />
+                    <mesh filename="file://$(find urc_hw_description)/urdf/meshes/visual/leftgripper.STL" />
+                </geometry>
+            </visual>
+            <collision>
+                <origin xyz="0 0 0" rpy="0 0 0" />
+                <geometry>
+                    <mesh
+                        filename="file://$(find urc_hw_description)/urdf/meshes/collision/leftgripper_collision.STL" />
                 </geometry>
             </collision>

File: urc_hw_description/urdf/drivebase.xacro (robot description, xacro)
@@ -13,12 +13,12 @@
                 <origin xyz="0 0 0" rpy="0 0 0" />
                 <geometry>
-                    <mesh filename="file://$(find urc_gazebo)/urdf/meshes/visual/base_link.STL" />
-                </geometry>
-            </visual>
-            <collision>
-                <origin xyz="0 0 0" rpy="0 0 0" />
-                <geometry>
-                    <mesh
-                        filename="file://$(find urc_gazebo)/urdf/meshes/collision/base_link_collision.STL" />
+                    <mesh filename="file://$(find urc_hw_description)/urdf/meshes/visual/base_link.STL" />
+                </geometry>
+            </visual>
+            <collision>
+                <origin xyz="0 0 0" rpy="0 0 0" />
+                <geometry>
+                    <mesh
+                        filename="file://$(find urc_hw_description)/urdf/meshes/collision/base_link_collision.STL" />
                 </geometry>
             </collision>
@@ -37,12 +37,12 @@
                 <origin xyz="0 0 0" rpy="0 0 0" />
                 <geometry>
-                    <mesh filename="file://$(find urc_gazebo)/urdf/meshes/visual/rightrocker.STL" />
-                </geometry>
-            </visual>
-            <collision>
-                <origin xyz="0 0 0" rpy="0 0 0" />
-                <geometry>
-                    <mesh
-                        filename="file://$(find urc_gazebo)/urdf/meshes/collision/rightrocker_collision.STL" />
+                    <mesh filename="file://$(find urc_hw_description)/urdf/meshes/visual/rightrocker.STL" />
+                </geometry>
+            </visual>
+            <collision>
+                <origin xyz="0 0 0" rpy="0 0 0" />
+                <geometry>
+                    <mesh
+                        filename="file://$(find urc_hw_description)/urdf/meshes/collision/rightrocker_collision.STL" />
                 </geometry>
             </collision>
@@ -68,12 +68,12 @@
                 <origin xyz="0 0 0" rpy="0 0 0" />
                 <geometry>
-                    <mesh filename="file://$(find urc_gazebo)/urdf/meshes/visual/leftrocker.STL" />
-                </geometry>
-            </visual>
-            <collision>
-                <origin xyz="0 0 0" rpy="0 0 0" />
-                <geometry>
-                    <mesh
-                        filename="file://$(find urc_gazebo)/urdf/meshes/collision/leftrocker_collision.STL" />
+                    <mesh filename="file://$(find urc_hw_description)/urdf/meshes/visual/leftrocker.STL" />
+                </geometry>
+            </visual>
+            <collision>
+                <origin xyz="0 0 0" rpy="0 0 0" />
+                <geometry>
+                    <mesh
+                        filename="file://$(find urc_hw_description)/urdf/meshes/collision/leftrocker_collision.STL" />
                 </geometry>
             </collision>
@@ -98,12 +98,12 @@
                 <origin xyz="0 0 0" rpy="0 0 0" />
                 <geometry>
-                    <mesh filename="file://$(find urc_gazebo)/urdf/meshes/visual/rightbogie.STL" />
-                </geometry>
-            </visual>
-            <collision>
-                <origin xyz="0 0 0" rpy="0 0 0" />
-                <geometry>
-                    <mesh
-                        filename="file://$(find urc_gazebo)/urdf/meshes/collision/rightbogie_collision.STL" />
+                    <mesh filename="file://$(find urc_hw_description)/urdf/meshes/visual/rightbogie.STL" />
+                </geometry>
+            </visual>
+            <collision>
+                <origin xyz="0 0 0" rpy="0 0 0" />
+                <geometry>
+                    <mesh
+                        filename="file://$(find urc_hw_description)/urdf/meshes/collision/rightbogie_collision.STL" />
                 </geometry>
             </collision>
@@ -127,12 +127,12 @@
                 <origin xyz="0 0 0" rpy="0 0 0" />
                 <geometry>
-                    <mesh filename="file://$(find urc_gazebo)/urdf/meshes/visual/leftbogie.STL" />
-                </geometry>
-            </visual>
-            <collision>
-                <origin xyz="0 0 0" rpy="0 0 0" />
-                <geometry>
-                    <mesh
-                        filename="file://$(find urc_gazebo)/urdf/meshes/collision/leftbogie_collision.STL" />
+                    <mesh filename="file://$(find urc_hw_description)/urdf/meshes/visual/leftbogie.STL" />
+                </geometry>
+            </visual>
+            <collision>
+                <origin xyz="0 0 0" rpy="0 0 0" />
+                <geometry>
+                    <mesh
+                        filename="file://$(find urc_hw_description)/urdf/meshes/collision/leftbogie_collision.STL" />
                 </geometry>
             </collision>

File: urc_hw_description/urdf/panda.urdf (robot description, URDF)
Before this commit: robot panda, 14 links, 13 joints
Links:
- link panda_hand: geometry collision mesh filename=$(find urc_hw_description)/urdf/meshes/collision/hand.obj; visual mesh filename=$(find urc_hw_description)/urdf/meshes/visual/hand.obj
- link panda_leftfinger: geometry collision mesh filename=$(find urc_hw_description)/urdf/meshes/collision/finger.obj; visual mesh filename=$(find urc_hw_description)/urdf/meshes/visual/finger.obj
- link panda_link0: geometry collision mesh filename=$(find urc_hw_description)/urdf/meshes/collision/link0.obj; visual mesh filename=$(find urc_hw_description)/urdf/meshes/collision/link0.obj
- link panda_link1: geometry collision mesh filename=$(find urc_hw_description)/urdf/meshes/collision/link1.obj; visual mesh filename=$(find urc_hw_description)/urdf/meshes/visual/link1.obj
- link panda_link2: geometry collision mesh filename=$(find urc_hw_description)/urdf/meshes/collision/link2.obj; visual mesh filename=$(find urc_hw_description)/urdf/meshes/visual/link2.obj
- link panda_link3: geometry collision mesh filename=$(find urc_hw_description)/urdf/meshes/collision/link3.obj; visual mesh filename=$(find urc_hw_description)/urdf/meshes/visual/link3.obj
- link panda_link4: geometry collision mesh filename=$(find urc_hw_description)/urdf/meshes/collision/link4.obj; visual mesh filename=$(find urc_hw_description)/urdf/meshes/visual/link4.obj
- link panda_link5: geometry collision mesh filename=$(find urc_hw_description)/urdf/meshes/collision/link5.obj; visual mesh filename=$(find urc_hw_description)/urdf/meshes/visual/link5.obj
- link panda_link6: geometry collision mesh filename=$(find urc_hw_description)/urdf/meshes/collision/link6.obj; visual mesh filename=$(find urc_hw_description)/urdf/meshes/visual/link6.obj
- link panda_link7: geometry collision mesh filename=$(find urc_hw_description)/urdf/meshes/collision/link7.obj; visual mesh filename=$(find urc_hw_description)/urdf/meshes/collision/link7.obj
- link panda_rightfinger: geometry collision mesh filename=$(find urc_hw_description)/urdf/meshes/collision/finger.obj; visual mesh filename=$(find urc_hw_description)/urdf/meshes/visual/finger.obj
