Commit message: [cleanup] deleted files which may not be needed anymore (#225)
* Deleted files which I believe we do not need anymore

* readded urc scripts

* linting

File: urc_hw_description/urdf/walli_drivebase.xacro (robot description, xacro)
@@ -13,12 +13,12 @@
                 <origin xyz="0 0 0" rpy="0 0 0" />
                 <geometry>
-                    <mesh filename="file://$(find urc_gazebo)/urdf/meshes/visual/base_link.STL" />
-                </geometry>
-            </visual>
-            <collision>
-                <origin xyz="0 0 0" rpy="0 0 0" />
-                <geometry>
-                    <mesh
-                        filename="file://$(find urc_gazebo)/urdf/meshes/collision/base_link_collision.STL" />
+                    <mesh filename="file://$(find urc_hw_description)/urdf/meshes/visual/base_link.STL" />
+                </geometry>
+            </visual>
+            <collision>
+                <origin xyz="0 0 0" rpy="0 0 0" />
+                <geometry>
+                    <mesh
+                        filename="file://$(find urc_hw_description)/urdf/meshes/collision/base_link_collision.STL" />
                 </geometry>
             </collision>
@@ -34,12 +34,12 @@
                 <origin xyz="0 0 0" rpy="0 0 0" />
                 <geometry>
-                    <mesh filename="file://$(find urc_gazebo)/urdf/meshes/visual/rightrocker.STL" />
-                </geometry>
-            </visual>
-            <collision>
-                <origin xyz="0 0 0" rpy="0 0 0" />
-                <geometry>
-                    <mesh
-                        filename="file://$(find urc_gazebo)/urdf/meshes/collision/rightrocker_collision.STL" />
+                    <mesh filename="file://$(find urc_hw_description)/urdf/meshes/visual/rightrocker.STL" />
+                </geometry>
+            </visual>
+            <collision>
+                <origin xyz="0 0 0" rpy="0 0 0" />
+                <geometry>
+                    <mesh
+                        filename="file://$(find urc_hw_description)/urdf/meshes/collision/rightrocker_collision.STL" />
                 </geometry>
             </collision>
@@ -64,16 +64,16 @@
                 <geometry>
                     <mesh
-                        filename="file://$(find urc_gazebo)/urdf/meshes/visual/right_rear_wheel.STL" />
-                </geometry>
-            </visual>
-            <collision>
-                <origin xyz="0 0 0" rpy="0 0 0" />
-                <geometry>
-                    <xacro:if value="${approximate}">
-                        <cylinder radius="${wheel_radius}" length="${wheel_thickness}" />
-                    </xacro:if>
-                    <xacro:if value="${not approximate}">
-                        <mesh
-                            filename="file://$(find urc_gazebo)/urdf/meshes/collision/right_rear_wheel_collision.STL" />
+                        filename="file://$(find urc_hw_description)/urdf/meshes/visual/right_rear_wheel.STL" />
+                </geometry>
+            </visual>
+            <collision>
+                <origin xyz="0 0 0" rpy="0 0 0" />
+                <geometry>
+                    <xacro:if value="${approximate}">
+                        <cylinder radius="${wheel_radius}" length="${wheel_thickness}" />
+                    </xacro:if>
+                    <xacro:if value="${not approximate}">
+                        <mesh
+                            filename="file://$(find urc_hw_description)/urdf/meshes/collision/right_rear_wheel_collision.STL" />
                     </xacro:if>
                 </geometry>
@@ -105,12 +105,12 @@
                 <origin xyz="0 0 0" rpy="0 0 0" />
                 <geometry>
-                    <mesh filename="file://$(find urc_gazebo)/urdf/meshes/visual/rightbogie.STL" />
-                </geometry>
-            </visual>
-            <collision>
-                <origin xyz="0 0 0" rpy="0 0 0" />
-                <geometry>
-                    <mesh
-                        filename="file://$(find urc_gazebo)/urdf/meshes/collision/rightbogie_collision.STL" />
+                    <mesh filename="file://$(find urc_hw_description)/urdf/meshes/visual/rightbogie.STL" />
+                </geometry>
+            </visual>
+            <collision>
+                <origin xyz="0 0 0" rpy="0 0 0" />
+                <geometry>
+                    <mesh
+                        filename="file://$(find urc_hw_description)/urdf/meshes/collision/rightbogie_collision.STL" />
                 </geometry>
             </collision>
@@ -134,16 +134,16 @@
                 <geometry>
                     <mesh
-                        filename="file://$(find urc_gazebo)/urdf/meshes/visual/right_front_wheel.STL" />
-                </geometry>
-            </visual>
-            <collision>
-                <origin xyz="0 0 0" rpy="0 0 0" />
-                <geometry>
-                    <xacro:if value="${approximate}">
-                        <cylinder radius="${wheel_radius}" length="${wheel_thickness}" />
-                    </xacro:if>
-                    <xacro:if value="${not approximate}">
-                        <mesh
-                            filename="file://$(find urc_gazebo)/urdf/meshes/collision/right_rear_wheel_collision.STL" />
+                        filename="file://$(find urc_hw_description)/urdf/meshes/visual/right_front_wheel.STL" />
+                </geometry>
+            </visual>
+            <collision>
+                <origin xyz="0 0 0" rpy="0 0 0" />
+                <geometry>
+                    <xacro:if value="${approximate}">
+                        <cylinder radius="${wheel_radius}" length="${wheel_thickness}" />
+                    </xacro:if>
+                    <xacro:if value="${not approximate}">
+                        <mesh
+                            filename="file://$(find urc_hw_description)/urdf/meshes/collision/right_rear_wheel_collision.STL" />
                     </xacro:if>
                 </geometry>
@@ -184,16 +184,16 @@
                 <geometry>
                     <mesh
-                        filename="file://$(find urc_gazebo)/urdf/meshes/visual/right_center_wheel.STL" />
-                </geometry>
-            </visual>
-            <collision>
-                <origin xyz="0 0 0" rpy="0 0 0" />
-                <geometry>
-                    <xacro:if value="${approximate}">
-                        <cylinder radius="${wheel_radius}" length="${wheel_thickness}" />
-                    </xacro:if>
-                    <xacro:if value="${not approximate}">
-                        <mesh
-                            filename="file://$(find urc_gazebo)/urdf/meshes/collision/right_center_wheel_collision.STL" />
+                        filename="file://$(find urc_hw_description)/urdf/meshes/visual/right_center_wheel.STL" />
+                </geometry>
+            </visual>
+            <collision>
+                <origin xyz="0 0 0" rpy="0 0 0" />
+                <geometry>
+                    <xacro:if value="${approximate}">
+                        <cylinder radius="${wheel_radius}" length="${wheel_thickness}" />
+                    </xacro:if>
+                    <xacro:if value="${not approximate}">
+                        <mesh
+                            filename="file://$(find urc_hw_description)/urdf/meshes/collision/right_center_wheel_collision.STL" />
                     </xacro:if>
                 </geometry>
@@ -225,12 +225,12 @@
                 <origin xyz="0 0 0" rpy="0 0 0" />
                 <geometry>
-                    <mesh filename="file://$(find urc_gazebo)/urdf/meshes/visual/leftrocker.STL" />
-                </geometry>
-            </visual>
-            <collision>
-                <origin xyz="0 0 0" rpy="0 0 0" />
-                <geometry>
-                    <mesh
-                        filename="file://$(find urc_gazebo)/urdf/meshes/collision/leftrocker_collision.STL" />
+                    <mesh filename="file://$(find urc_hw_description)/urdf/meshes/visual/leftrocker.STL" />
+                </geometry>
+            </visual>
+            <collision>
+                <origin xyz="0 0 0" rpy="0 0 0" />
+                <geometry>
+                    <mesh
+                        filename="file://$(find urc_hw_description)/urdf/meshes/collision/leftrocker_collision.STL" />
                 </geometry>
             </collision>
@@ -254,16 +254,16 @@
                 <geometry>
                     <mesh
-                        filename="file://$(find urc_gazebo)/urdf/meshes/visual/left_rear_wheel.STL" />
-                </geometry>
-            </visual>
-            <collision>
-                <origin xyz="0 0 0" rpy="0 0 0" />
-                <geometry>
-                    <xacro:if value="${approximate}">
-                        <cylinder radius="${wheel_radius}" length="${wheel_thickness}" />
-                    </xacro:if>
-                    <xacro:if value="${not approximate}">
-                        <mesh
-                            filename="file://$(find urc_gazebo)/urdf/meshes/collision/left_rear_wheel_collision.STL" />
+                        filename="file://$(find urc_hw_description)/urdf/meshes/visual/left_rear_wheel.STL" />
+                </geometry>
+            </visual>
+            <collision>
+                <origin xyz="0 0 0" rpy="0 0 0" />
+                <geometry>
+                    <xacro:if value="${approximate}">
+                        <cylinder radius="${wheel_radius}" length="${wheel_thickness}" />
+                    </xacro:if>
+                    <xacro:if value="${not approximate}">
+                        <mesh
+                            filename="file://$(find urc_hw_description)/urdf/meshes/collision/left_rear_wheel_collision.STL" />
                     </xacro:if>
                 </geometry>
@@ -295,12 +295,12 @@
                 <origin xyz="0 0 0" rpy="0 0 0" />
                 <geometry>
-                    <mesh filename="file://$(find urc_gazebo)/urdf/meshes/visual/leftbogie.STL" />
-                </geometry>
-            </visual>
-            <collision>
-                <origin xyz="0 0 0" rpy="0 0 0" />
-                <geometry>
-                    <mesh
-                        filename="file://$(find urc_gazebo)/urdf/meshes/collision/leftbogie_collision.STL" />
+                    <mesh filename="file://$(find urc_hw_description)/urdf/meshes/visual/leftbogie.STL" />
+                </geometry>
+            </visual>
+            <collision>
+                <origin xyz="0 0 0" rpy="0 0 0" />
+                <geometry>
+                    <mesh
+                        filename="file://$(find urc_hw_description)/urdf/meshes/collision/leftbogie_collision.STL" />
                 </geometry>
             </collision>
@@ -324,16 +324,16 @@
                 <geometry>
                     <mesh
-                        filename="file://$(find urc_gazebo)/urdf/meshes/visual/left_front_wheel.STL" />
-                </geometry>
-            </visual>
-            <collision>
-                <origin xyz="0 0 0" rpy="0 0 0" />
-                <geometry>
-                    <xacro:if value="${approximate}">
-                        <cylinder radius="${wheel_radius}" length="${wheel_thickness}" />
-                    </xacro:if>
-                    <xacro:if value="${not approximate}">
-                        <mesh
-                            filename="file://$(find urc_gazebo)/urdf/meshes/collision/left_front_wheel_collision.STL" />
+                        filename="file://$(find urc_hw_description)/urdf/meshes/visual/left_front_wheel.STL" />
+                </geometry>
+            </visual>
+            <collision>
+                <origin xyz="0 0 0" rpy="0 0 0" />
+                <geometry>
+                    <xacro:if value="${approximate}">
+                        <cylinder radius="${wheel_radius}" length="${wheel_thickness}" />
+                    </xacro:if>
+                    <xacro:if value="${not approximate}">
+                        <mesh
+                            filename="file://$(find urc_hw_description)/urdf/meshes/collision/left_front_wheel_collision.STL" />
                     </xacro:if>
                 </geometry>
@@ -366,16 +366,16 @@
                 <geometry>
                     <mesh
-                        filename="file://$(find urc_gazebo)/urdf/meshes/visual/left_center_wheel.STL" />
-                </geometry>
-            </visual>
-            <collision>
-                <origin xyz="0 0 0" rpy="0 0 0" />
-                <geometry>
-                    <xacro:if value="${approximate}">
-                        <cylinder radius="${wheel_radius}" length="${wheel_thickness}" />
-                    </xacro:if>
-                    <xacro:if value="${not approximate}">
-                        <mesh
-                            filename="file://$(find urc_gazebo)/urdf/meshes/collision/left_center_wheel_collision.STL" />
+                        filename="file://$(find urc_hw_description)/urdf/meshes/visual/left_center_wheel.STL" />
+                </geometry>
+            </visual>
+            <collision>
+                <origin xyz="0 0 0" rpy="0 0 0" />
+                <geometry>
+                    <xacro:if value="${approximate}">
+                        <cylinder radius="${wheel_radius}" length="${wheel_thickness}" />
+                    </xacro:if>
+                    <xacro:if value="${not approximate}">
+                        <mesh
+                            filename="file://$(find urc_hw_description)/urdf/meshes/collision/left_center_wheel_collision.STL" />
                     </xacro:if>
                 </geometry>
