Commit message: inertia fixes

File: urc_hw_description/urdf/wallii.xacro (robot description, xacro)
@@ -4,10 +4,9 @@
    <xacro:include filename="$(find urc_hw_description)/urdf/inertials.xacro" />
    <xacro:include filename="$(find urc_hw_description)/urdf/wallii_drivebase.xacro" />
-   <xacro:include filename="$(find urc_hw_description)/urdf/walli_sensors.xacro" />
-   <xacro:include filename="$(find urc_hw_description)/urdf/ros2_control.xacro" />
+   <!-- <xacro:include filename="$(find urc_hw_description)/urdf/walli_sensors.xacro" /> -->
+   <!-- <xacro:include filename="$(find urc_hw_description)/urdf/ros2_control.xacro" /> -->
    <xacro:drivebase mu="1.0" mu2="0.25" />
-   <!-- <xacro:arm /> -->
-   <xacro:ros2_control use_simulation="$(arg use_simulation)"
-      config_file_path="$(find urc_bringup)/config/controller_config.yaml"
-      arm_initial_positions_file="$(find urc_hw_description)/config/initial_positions.yaml" />
+   <!-- <xacro:ros2_control use_simulation="$(arg use_simulation)" -->
+   <!--    config_file_path="$(find urc_bringup)/config/controller_config.yaml" -->
+   <!--    arm_initial_positions_file="$(find urc_hw_description)/config/initial_positions.yaml" /> -->
 </robot>

File: urc_hw_description/urdf/wallii_drivebase.xacro (robot description, xacro)
@@ -9,15 +9,15 @@
       <inertial>
         <origin
-          xyz="-0.014317225327403 0.0104296335321108 0.153421389255203"
-          rpy="0 0 0" />
-        <mass
-          value="4.16872664819669" />
-        <inertia
-          ixx="0.0133014161912341"
-          ixy="9.61058451240803E-06"
-          ixz="3.78220834652181E-09"
-          iyy="0.0282864040971226"
-          iyz="-5.32294329059233E-06"
-          izz="0.0262313272124921" />
+          xyz="0.0 0.0 -0.5"
+          rpy="0 0 0" />
+        <mass
+          value="18.7" />
+        <inertia
+          ixx="0.5"
+          ixy="0.0"
+          ixz="0.0"
+          iyy="0.62"
+          iyz="0.0"
+          izz="1.0" />
       </inertial>
       <visual>
@@ -52,12 +52,12 @@
           rpy="0 0 0" />
         <mass
-          value="1.51922550428194" />
-        <inertia
-          ixx="0.0172747101435764"
-          ixy="1.95090448894846E-06"
-          ixz="2.77456502210212E-08"
-          iyy="0.016672008092978"
-          iyz="-0.000130959848654314"
-          izz="0.00134369269865275" />
+          value="3.79806376070485" />
+        <inertia
+          ixx="0.043186775358941"
+          ixy="4.87726122237115E-06"
+          ixz="6.9364125552553E-08"
+          iyy="0.041680020232445"
+          iyz="-0.000327399621635785"
+          izz="0.00335923174663188" />
       </inertial>
       <visual>
@@ -96,5 +96,5 @@
         link="Left_Leg" />
       <axis
-        xyz="0 0 0" />
+        xyz="0 1 0" />
       <limit
         lower="0"
@@ -111,12 +111,12 @@
           rpy="0 0 0" />
         <mass
-          value="1.13616610202435" />
-        <inertia
-          ixx="0.00583600145685734"
-          ixy="-3.78138840894905E-09"
-          ixz="3.44212174951375E-08"
-          iyy="0.0108465522742051"
-          iyz="4.91733251357684E-09"
-          izz="0.00583602395506444" />
+          value="2.84041525506088" />
+        <inertia
+          ixx="0.0145900036421434"
+          ixy="-9.45347102237263E-09"
+          ixz="8.60530437378438E-08"
+          iyy="0.0271163806855128"
+          iyz="1.22933312839421E-08"
+          izz="0.0145900598876611" />
       </inertial>
       <visual>
@@ -172,12 +172,12 @@
           rpy="0 0 0" />
         <mass
-          value="1.1361661167724" />
-        <inertia
-          ixx="0.00583600145988187"
-          ixy="-3.78130385122974E-09"
-          ixz="3.44208561048418E-08"
-          iyy="0.010846552274239"
-          iyz="4.91663609733339E-09"
-          izz="0.00583602395841195" />
+          value="2.8404152919431" />
+        <inertia
+          ixx="0.0145900036497047"
+          ixy="-9.45325962807435E-09"
+          ixz="8.60521402621045E-08"
+          iyy="0.0271163806855975"
+          iyz="1.22915902433335E-08"
+          izz="0.0145900598960299" />
       </inertial>
       <visual>
@@ -233,12 +233,12 @@
           rpy="0 0 0" />
         <mass
-          value="0.35481398078544" />
-        <inertia
-          ixx="0.000118183325221152"
-          ixy="2.50308247601608E-05"
-          ixz="1.74352465550517E-08"
-          iyy="0.00260829860640953"
-          iyz="-8.05543749773572E-08"
-          izz="0.00271714842544938" />
+          value="0.8870349519636" />
+        <inertia
+          ixx="0.00029545831305288"
+          ixy="6.25770619004021E-05"
+          ixz="4.35881163876293E-08"
+          iyy="0.00652074651602383"
+          iyz="-2.01385937443393E-07"
+          izz="0.00679287106362345" />
       </inertial>
       <visual>
@@ -292,12 +292,12 @@
           rpy="0 0 0" />
         <mass
-          value="1.51922403384041" />
-        <inertia
-          ixx="0.0172747098040692"
-          ixy="-1.95088285599865E-06"
-          ixz="-2.76912278959164E-08"
-          iyy="0.016672007901523"
-          iyz="-0.000130959797312506"
-          izz="0.00134369248974745" />
+          value="3.79806008460103" />
+        <inertia
+          ixx="0.043186774510173"
+          ixy="-4.87720713999662E-06"
+          ixz="-6.9228069739791E-08"
+          iyy="0.0416800197538075"
+          iyz="-0.000327399493281265"
+          izz="0.00335923122436863" />
       </inertial>
       <visual>
@@ -336,5 +336,5 @@
         link="Right_Leg" />
       <axis
-        xyz="0 0 0" />
+        xyz="0 1 0" />
       <limit
         lower="0"
@@ -351,12 +351,12 @@
           rpy="0 0 0" />
         <mass
-          value="1.13616589675483" />
-        <inertia
-          ixx="0.00583600369475276"
-          ixy="-3.78178980764489E-09"
-          ixz="3.44207610191845E-08"
-          iyy="0.0108465504538541"
-          iyz="4.91693676653181E-09"
-          izz="0.00583602619264686" />
+          value="2.84041474188708" />
+        <inertia
+          ixx="0.0145900092368819"
+          ixy="-9.45447451911223E-09"
+          ixz="8.60519025479613E-08"
+          iyy="0.0271163761346353"
+          iyz="1.22923419163295E-08"
+          izz="0.0145900654816172" />
       </inertial>
       <visual>
@@ -412,12 +412,12 @@
           rpy="0 0 0" />
         <mass
-          value="1.13616589718668" />
-        <inertia
-          ixx="0.00583600369447215"
-          ixy="-3.7820831107468E-09"
-          ixz="3.44209450267363E-08"
-          iyy="0.0108465504538551"
-          iyz="4.91681588687628E-09"
-          izz="0.00583602619308218" />
+          value="2.8404147429667" />
+        <inertia
+          ixx="0.0145900092361804"
+          ixy="-9.4552077768867E-09"
+          ixz="8.60523625668408E-08"
+          iyy="0.0271163761346378"
+          iyz="1.22920397171907E-08"
+          izz="0.0145900654827055" />
       </inertial>
       <visual>
