Commit message: inertia fixes

File: urc_hw_description/urdf/wallii_drivebase.xacro (robot description, xacro)
@@ -49,15 +49,15 @@
       <inertial>
         <origin
-          xyz="-0.314720519412685 -0.267228491093624 0.0144844412176535"
-          rpy="0 0 0" />
-        <mass
-          value="3.79806376070485" />
-        <inertia
-          ixx="0.043186775358941"
-          ixy="4.87726122237115E-06"
-          ixz="6.9364125552553E-08"
-          iyy="0.041680020232445"
-          iyz="-0.000327399621635785"
-          izz="0.00335923174663188" />
+          xyz="0.0 0.0 0.12"
+          rpy="0 0 0" />
+        <mass
+          value="3.2" />
+        <inertia
+          ixx="0.0"
+          ixy="0.0"
+          ixz="0.0"
+          iyy="0.62"
+          iyz="0.0"
+          izz="0.62" />
       </inertial>
       <visual>
@@ -108,15 +108,15 @@
       <inertial>
         <origin
-          xyz="-9.85643131612424E-07 -0.0424756514469604 1.28618891753751E-06"
-          rpy="0 0 0" />
-        <mass
-          value="2.84041525506088" />
-        <inertia
-          ixx="0.0145900036421434"
-          ixy="-9.45347102237263E-09"
-          ixz="8.60530437378438E-08"
-          iyy="0.0271163806855128"
-          iyz="1.22933312839421E-08"
-          izz="0.0145900598876611" />
+          xyz="-9.85790539753673E-07 -0.0424756522296364 1.28556895756526E-06"
+          rpy="0 0 0" />
+        <mass
+          value="2.8404147429667" />
+        <inertia
+          ixx="0.0145900092361804"
+          ixy="-9.4552077768867E-09"
+          ixz="8.60523625668408E-08"
+          iyy="0.0271163761346378"
+          iyz="1.22920397171907E-08"
+          izz="0.0145900654827055" />
       </inertial>
       <visual>
@@ -169,15 +169,15 @@
       <inertial>
         <origin
-          xyz="-9.85722509394549E-07 -0.0424756513980336 1.28528277876239E-06"
-          rpy="0 0 0" />
-        <mass
-          value="2.8404152919431" />
-        <inertia
-          ixx="0.0145900036497047"
-          ixy="-9.45325962807435E-09"
-          ixz="8.60521402621045E-08"
-          iyy="0.0271163806855975"
-          iyz="1.22915902433335E-08"
-          izz="0.0145900598960299" />
+          xyz="0.0 0.0 0.0"
+          rpy="0 0 0" />
+        <mass
+          value="1.4" />
+        <inertia
+          ixx="0.005"
+          ixy="0.0"
+          ixz="0"
+          iyy="0.01"
+          iyz="0.0"
+          izz="0.005" />
       </inertial>
       <visual>
@@ -226,56 +226,115 @@
         xyz="0 1 0" />
     </joint>
-    <link
-      name="Differential_Bar">
-      <inertial>
-        <origin
-          xyz="0.0001696304329344 0.0146364855896726 0.0184524262584146"
-          rpy="0 0 0" />
-        <mass
-          value="0.8870349519636" />
-        <inertia
-          ixx="0.00029545831305288"
-          ixy="6.25770619004021E-05"
-          ixz="4.35881163876293E-08"
-          iyy="0.00652074651602383"
-          iyz="-2.01385937443393E-07"
-          izz="0.00679287106362345" />
-      </inertial>
-      <visual>
-        <origin
-          xyz="0 0 0"
-          rpy="0 0 0" />
-        <geometry>
-          <mesh
-            filename="file://$(find urc_hw_description)/urdf/meshes/Differential_Bar.STL" />
-        </geometry>
-        <material
-          name="">
-          <color
-            rgba="0.792156862745098 0.819607843137255 0.933333333333333 1" />
-        </material>
-      </visual>
-      <collision>
-        <origin
-          xyz="0 0 0"
-          rpy="0 0 0" />
-        <geometry>
-          <mesh
-            filename="file://$(find urc_hw_description)/urdf/meshes/Differential_Bar.STL" />
-        </geometry>
-      </collision>
-    </link>
-    <joint
-      name="Differential_Bar_Shaft"
+    <!-- <link -->
+    <!--   name="Differential_Bar"> -->
+    <!--   <inertial> -->
+    <!--     <origin -->
+    <!--       xyz="0.0001696304329344 0.0146364855896726 0.0184524262584146" -->
+    <!--       rpy="0 0 0" /> -->
+    <!--     <mass -->
+    <!--       value="0.8870349519636" /> -->
+    <!--     <inertia -->
+    <!--       ixx="0.00029545831305288" -->
+    <!--       ixy="6.25770619004021E-05" -->
+    <!--       ixz="4.35881163876293E-08" -->
+    <!--       iyy="0.00652074651602383" -->
+    <!--       iyz="-2.01385937443393E-07" -->
+    <!--       izz="0.00679287106362345" /> -->
+    <!--   </inertial> -->
+    <!--   <visual> -->
+    <!--     <origin -->
+    <!--       xyz="0 0 0" -->
+    <!--       rpy="0 0 0" /> -->
+    <!--     <geometry> -->
+    <!--       <mesh -->
+    <!--         filename="file://$(find urc_hw_description)/urdf/meshes/Differential_Bar.STL" /> -->
+    <!--     </geometry> -->
+    <!--     <material -->
+    <!--       name=""> -->
+    <!--       <color -->
+    <!--         rgba="0.792156862745098 0.819607843137255 0.933333333333333 1" /> -->
+    <!--     </material> -->
+    <!--   </visual> -->
+    <!--   <collision> -->
+    <!--     <origin -->
+    <!--       xyz="0 0 0" -->
+    <!--       rpy="0 0 0" /> -->
+    <!--     <geometry> -->
+    <!--       <mesh -->
+    <!--         filename="file://$(find urc_hw_description)/urdf/meshes/Differential_Bar.STL" /> -->
+    <!--     </geometry> -->
+    <!--   </collision> -->
+    <!-- </link> -->
+    <!-- <joint -->
+    <!--   name="Differential_Bar_Shaft" -->
+    <!--   type="revolute"> -->
+    <!--   <origin -->
+    <!--     xyz="0 -0.37445 -0.070294" -->
+    <!--     rpy="1.5708 0 0" /> -->
+    <!--   <parent -->
+    <!--     link="base_link" /> -->
+    <!--   <child -->
+    <!--     link="Differential_Bar" /> -->
+    <!--   <axis -->
+    <!--     xyz="0 0 1" /> -->
+    <!--   <limit -->
+    <!--     lower="0" -->
+    <!--     upper="0" -->
+    <!--     effort="0" -->
+    <!--     velocity="0" /> -->
+    <!--     <dynamics damping="0.01" friction="0.01" /> -->
+    <!-- </joint> -->
+    <link
+      name="Right_Leg">
+      <inertial>
+        <origin
+          xyz="0.0 0.0 0.12"
+          rpy="0 0 0" />
+        <mass
+          value="3.2" />
+        <inertia
+          ixx="0.0"
+          ixy="0.0"
+          ixz="0.0"
+          iyy="0.62"
+          iyz="0.0"
+          izz="0.62" />
+      </inertial>
+      <visual>
+        <origin
+          xyz="0 0 0"
+          rpy="0 0 0" />
+        <geometry>
+          <mesh
+            filename="file://$(find urc_hw_description)/urdf/meshes/Right_Leg.STL" />
+        </geometry>
+        <material
+          name="">
+          <color
+            rgba="0.792156862745098 0.819607843137255 0.933333333333333 1" />
+        </material>
+      </visual>
+      <collision>
+        <origin
+          xyz="0 0 0"
+          rpy="0 0 0" />
+        <geometry>
+          <mesh
+            filename="file://$(find urc_hw_description)/urdf/meshes/Right_Leg.STL" />
+        </geometry>
+      </collision>
+    </link>
+    <joint
+      name="Right_Leg_Shaft"
       type="revolute">
       <origin
-        xyz="0 -0.37445 -0.070294"
-        rpy="1.5708 0 0" />
+        xyz="0 -0.0011403 0.0099997"
+        rpy="1.5791 0 0" />
       <parent
         link="base_link" />
       <child
-        link="Differential_Bar" />
-      <axis
-        xyz="0 0 1" />
+        link="Right_Leg" />
+      <axis
+        xyz="0 1 0" />
       <limit
         lower="0"
@@ -286,77 +345,18 @@
     </joint>
     <link
-      name="Right_Leg">
-      <inertial>
-        <origin
-          xyz="0.314720537608315 -0.27732042463059 0.00342777397828535"
-          rpy="0 0 0" />
-        <mass
-          value="3.79806008460103" />
-        <inertia
-          ixx="0.043186774510173"
-          ixy="-4.87720713999662E-06"
-          ixz="-6.9228069739791E-08"
-          iyy="0.0416800197538075"
-          iyz="-0.000327399493281265"
-          izz="0.00335923122436863" />
-      </inertial>
-      <visual>
-        <origin
-          xyz="0 0 0"
-          rpy="0 0 0" />
-        <geometry>
-          <mesh
-            filename="file://$(find urc_hw_description)/urdf/meshes/Right_Leg.STL" />
-        </geometry>
-        <material
-          name="">
-          <color
-            rgba="0.792156862745098 0.819607843137255 0.933333333333333 1" />
-        </material>
-      </visual>
-      <collision>
-        <origin
-          xyz="0 0 0"
-          rpy="0 0 0" />
-        <geometry>
-          <mesh
-            filename="file://$(find urc_hw_description)/urdf/meshes/Right_Leg.STL" />
-        </geometry>
-      </collision>
-    </link>
-    <joint
-      name="Right_Leg_Shaft"
-      type="revolute">
-      <origin
-        xyz="0 -0.0011403 0.0099997"
-        rpy="1.5791 0 0" />
-      <parent
-        link="base_link" />
-      <child
-        link="Right_Leg" />
-      <axis
-        xyz="0 1 0" />
-      <limit
-        lower="0"
-        upper="0"
-        effort="0"
-        velocity="0" />
-        <dynamics damping="0.01" friction="0.01" />
-    </joint>
-    <link
       name="Front_Right_Wheel">
       <inertial>
         <origin
-          xyz="-9.8607342807755E-07 -0.0424756522332874 1.28600934945489E-06"
-          rpy="0 0 0" />
-        <mass
-          value="2.84041474188708" />
-        <inertia
-          ixx="0.0145900092368819"
-          ixy="-9.45447451911223E-09"
-          ixz="8.60519025479613E-08"
-          iyy="0.0271163761346353"
-          iyz="1.22923419163295E-08"
-          izz="0.0145900654816172" />
+          xyz="0.0 0.0 0.0"
+          rpy="0 0 0" />
+        <mass
+          value="1.4" />
+        <inertia
+          ixx="0.005"
+          ixy="0.0"
+          ixz="0"
+          iyy="0.01"
+          iyz="0.0"
+          izz="0.005" />
       </inertial>
       <visual>
@@ -409,15 +409,15 @@
       <inertial>
         <origin
-          xyz="-9.85790539753673E-07 -0.0424756522296364 1.28556895756526E-06"
-          rpy="0 0 0" />
-        <mass
-          value="2.8404147429667" />
-        <inertia
-          ixx="0.0145900092361804"
-          ixy="-9.4552077768867E-09"
-          ixz="8.60523625668408E-08"
-          iyy="0.0271163761346378"
-          iyz="1.22920397171907E-08"
-          izz="0.0145900654827055" />
+          xyz="-9.8607342807755E-07 -0.0424756522332874 1.28600934945489E-06"
+          rpy="0 0 0" />
+        <mass
+          value="2.84041474188708" />
+        <inertia
+          ixx="0.0145900092368819"
+          ixy="-9.45447451911223E-09"
+          ixz="8.60519025479613E-08"
+          iyy="0.0271163761346353"
+          iyz="1.22923419163295E-08"
+          izz="0.0145900654816172" />
       </inertial>
       <visual>

Commit message: added joint between diff bar and rocker

File: urc_hw_description/urdf/wallii_drivebase.xacro (robot description, xacro)
@@ -278,4 +278,26 @@
       <dynamics damping="0.01" friction="0.01" />
     </joint>
+    <joint
+      name="diff_bar_right_rocker"
+      type="fixed">
+      <origin
+        xyz="-0.26 -0.253 0.05"
+        rpy="" />
+      <parent
+        link="differential_bar" />
+      <child
+        link="right_rocker" />
+      </joint>
+    <joint
+      name="diff_bar_left_rocker"
+      type="fixed">
+      <origin
+        xyz="0.26 -0.253 0.05"
+        rpy="" />
+      <parent
+        link="differential_bar" />
+      <child
+        link="left_rocker" />
+      </joint>
     <link
       name="right_rocker">

Commit message: simplified collision logic

File: urc_hw_description/urdf/wallii_drivebase.xacro (robot description, xacro)
@@ -132,6 +132,5 @@
           rpy="0 0 0" />
         <geometry>
-          <mesh
-            filename="file://$(find urc_hw_description)/urdf/meshes/Front_Left_Wheel.STL" />
+          <cylinder length="3.25" radius="4.75"/>
         </geometry>
       </collision>
@@ -193,6 +192,5 @@
           rpy="0 0 0" />
         <geometry>
-          <mesh
-            filename="file://$(find urc_hw_description)/urdf/meshes/Back_Left_Wheel.STL" />
+          <cylinder length="3.25" radius="4.75"/>
         </geometry>
       </collision>
@@ -390,6 +388,5 @@
           rpy="0 0 0" />
         <geometry>
-          <mesh
-            filename="file://$(find urc_hw_description)/urdf/meshes/Front_Right_Wheel.STL" />
+            <cylinder length="3.25" radius="4.75"/>
         </geometry>
       </collision>
@@ -451,6 +448,5 @@
           rpy="0 0 0" />
         <geometry>
-          <mesh
-            filename="file://$(find urc_hw_description)/urdf/meshes/Back_Right_Wheel.STL" />
+          <cylinder length="3.25" radius="4.75"/>
         </geometry>
       </collision>

Commit message: conversion goof

File: urc_hw_description/urdf/wallii_drivebase.xacro (robot description, xacro)
@@ -132,5 +132,5 @@
           rpy="0 0 0" />
         <geometry>
-          <cylinder length="3.25" radius="4.75"/>
+          <cylinder length="0.083" radius="0.1207"/>
         </geometry>
       </collision>
@@ -192,5 +192,5 @@
           rpy="0 0 0" />
         <geometry>
-          <cylinder length="3.25" radius="4.75"/>
+          <cylinder length="0.083" radius="0.1207"/>
         </geometry>
       </collision>
@@ -388,5 +388,5 @@
           rpy="0 0 0" />
         <geometry>
-            <cylinder length="3.25" radius="4.75"/>
+            <cylinder length="0.083" radius="0.1207"/>
         </geometry>
       </collision>
@@ -448,5 +448,5 @@
           rpy="0 0 0" />
         <geometry>
-          <cylinder length="3.25" radius="4.75"/>
+          <cylinder length="0.083" radius="0.1207"/>
         </geometry>
       </collision>

Commit message: simplified collision logic

File: urc_hw_description/urdf/wallii_drivebase.xacro (robot description, xacro)
@@ -118,6 +118,5 @@
           rpy="0 0 0" />
         <geometry>
-          <mesh
-            filename="file://$(find urc_hw_description)/urdf/meshes/Front_Left_Wheel.STL" />
+          <cylinder length="0.083" radius="0.1207"/>
         </geometry>
         <material
@@ -178,6 +177,5 @@
           rpy="0 0 0" />
         <geometry>
-          <mesh
-            filename="file://$(find urc_hw_description)/urdf/meshes/Back_Left_Wheel.STL" />
+          <cylinder length="0.083" radius="0.1207"/>
         </geometry>
         <material
@@ -374,6 +372,5 @@
           rpy="0 0 0" />
         <geometry>
-          <mesh
-            filename="file://$(find urc_hw_description)/urdf/meshes/Front_Right_Wheel.STL" />
+          <cylinder length="0.083" radius="0.1207"/>
         </geometry>
         <material
@@ -434,6 +431,5 @@
           rpy="0 0 0" />
         <geometry>
-          <mesh
-            filename="file://$(find urc_hw_description)/urdf/meshes/Back_Right_Wheel.STL" />
+          <cylinder length="0.083" radius="0.1207"/>
         </geometry>
         <material

Commit message: maybe some collision stuff?

File: urc_hw_description/urdf/wallii_drivebase.xacro (robot description, xacro)
@@ -37,6 +37,5 @@
           rpy="0 0 0" />
         <geometry>
-          <mesh
-            filename="file://$(find urc_hw_description)/urdf/meshes/base_link.STL" />
+          <box size="21 24.5 8"/>
         </geometry>
       </collision>
@@ -77,6 +76,5 @@
           rpy="0 0 0" />
         <geometry>
-          <mesh
-            filename="file://$(find urc_hw_description)/urdf/meshes/Left_Leg.STL" />
+          <box size="2 30.25 2"/>
         </geometry>
       </collision>
@@ -250,6 +248,5 @@
           rpy="0 0 0" />
         <geometry>
-          <mesh
-            filename="file://$(find urc_hw_description)/urdf/meshes/Differential_Bar.STL" />
+          <box size="21 1 3">
         </geometry>
       </collision>
@@ -329,6 +326,5 @@
           rpy="0 0 0" />
         <geometry>
-          <mesh
-            filename="file://$(find urc_hw_description)/urdf/meshes/Right_Leg.STL" />
+          <box size="2 30.25 2"/>
         </geometry>
       </collision>

Commit message: bugfix

File: urc_hw_description/urdf/wallii_drivebase.xacro (robot description, xacro)
@@ -248,5 +248,5 @@
           rpy="0 0 0" />
         <geometry>
-          <box size="21 1 3">
+          <box size="21 1 3" />
         </geometry>
       </collision>
