Commit message: added 3D LIDAR functionality

File: urc_hw_description/urdf/walli_sensors.xacro (robot description, xacro)
@@ -123,8 +123,8 @@
   </gazebo>
   <!-- LIDAR -->
-  <!-- <link name="lidar_link">
+  <link name="lidar_link">
     <inertial>
       <origin xyz="0 0 0" rpy="0 0 0" />
-      <mass value="0.125" />
+      <mass value="0.025" />
       <inertia ixx="0.001" ixy="0" ixz="0" iyy="0.001" iyz="0" izz="0.001" />
     </inertial>
@@ -160,4 +160,10 @@
             <max_angle>6.280000</max_angle>
           </horizontal>
+          <vertical>
+            <samples>10</samples>
+            <resolution>1.000000</resolution>
+            <min_angle>0.000000</min_angle>
+            <max_angle>0.5000</max_angle>
+          </vertical>
         </scan>
         <range>
@@ -176,9 +182,9 @@
           <remapping>~/out:=scan</remapping>
         </ros>
-        <output_type>sensor_msgs/LaserScan</output_type>
+        <output_type>sensor_msgs/PointCloud2</output_type>
         <frame_name>lidar_link</frame_name>
       </plugin>
     </sensor>
-  </gazebo> -->
+  </gazebo>
   <!-- May want to change this to a depth camera -->
   <xacro:macro name="camera" params="orientation origin_x origin_y origin_z yaw">

Commit message: modified real values of LIDAR but not done yet.

File: urc_hw_description/urdf/walli_sensors.xacro (robot description, xacro)
@@ -126,5 +126,5 @@
     <inertial>
       <origin xyz="0 0 0" rpy="0 0 0" />
-      <mass value="0.025" />
+      <mass value="0.7" />
       <inertia ixx="0.001" ixy="0" ixz="0" iyy="0.001" iyz="0" izz="0.001" />
     </inertial>
@@ -161,8 +161,8 @@
           </horizontal>
           <vertical>
-            <samples>10</samples>
+            <samples>16</samples>
             <resolution>1.000000</resolution>
-            <min_angle>0.000000</min_angle>
-            <max_angle>0.5000</max_angle>
+            <min_angle>-.12566</min_angle>
+            <max_angle>0.59865</max_angle>
           </vertical>
         </scan>

Commit message: editted mass, geometry, min/max angles to match spec sheet

File: urc_hw_description/urdf/walli_sensors.xacro (robot description, xacro)
@@ -138,5 +138,5 @@
       <origin xyz="0 0 0" rpy="0 0 0" />
       <geometry>
-        <cylinder radius="0.0508" length="0.055" />
+        <cylinder radius="0.05" length="0.0985" />
       </geometry>
     </visual>
@@ -150,5 +150,5 @@
     <sensor name="lidar" type="ray">
       <always_on>true</always_on>
-      <visualize>true</visualize>
+      <visualize>false</visualize>
       <update_rate>5</update_rate>
       <ray>

Commit message: minor fixes

File: urc_hw_description/urdf/walli_sensors.xacro (robot description, xacro)
@@ -17,5 +17,5 @@
   <joint name="imu_joint" type="fixed">
     <axis xyz="1 0 0" />
-    <origin xyz="0.05 0.1 0.2" />
+    <origin xyz="0.05 0.1 0.2" rpy="0 -0.095 0"/>
     <parent link="base_link" />
     <child link="imu_link" />

Commit message: update sensor positions

File: urc_hw_description/urdf/walli_sensors.xacro (robot description, xacro)
@@ -17,5 +17,5 @@
   <joint name="imu_joint" type="fixed">
     <axis xyz="1 0 0" />
-    <origin xyz="0.05 0.1 0.2" />
+    <origin xyz="-0.32 -0.09 0.0" />
     <parent link="base_link" />
     <child link="imu_link" />
@@ -105,5 +105,5 @@
   <joint name="gps_joint" type="fixed">
     <axis xyz="1 0 0" />
-    <origin xyz="0.05 -0.1 0.2" />
+    <origin xyz="-0.39 -0.27 0.34" />
     <parent link="base_link" />
     <child link="gps" />

Commit message: vectornav frame

File: urc_hw_description/urdf/walli_sensors.xacro (robot description, xacro)
@@ -90,5 +90,5 @@
   </gazebo>
   <!-- GPS -->
-  <link name="gps">
+  <link name="gps_link">
     <visual>
       <geometry>

Commit message: gps link name

File: urc_hw_description/urdf/walli_sensors.xacro (robot description, xacro)
@@ -107,5 +107,5 @@
     <origin xyz="-0.39 -0.27 0.34" />
     <parent link="base_link" />
-    <child link="gps" />
+    <child link="gps_link" />
   </joint>
   <gazebo reference="gps">
@@ -116,5 +116,5 @@
           <remapping>~/out:=data</remapping>
         </ros>
-        <frame_name>gps</frame_name>
+        <frame_name>gps_link</frame_name>
       </plugin>
       <always_on>true</always_on>

Commit message: [misc] update sensor static transformations (#244)

File: urc_hw_description/urdf/walli_sensors.xacro (robot description, xacro)
@@ -17,5 +17,5 @@
   <joint name="imu_joint" type="fixed">
     <axis xyz="1 0 0" />
-    <origin xyz="0.05 0.1 0.2" />
+    <origin xyz="-0.32 -0.09 0.0" />
     <parent link="base_link" />
     <child link="imu_link" />
@@ -90,5 +90,5 @@
   </gazebo>
   <!-- GPS -->
-  <link name="gps">
+  <link name="gps_link">
     <visual>
       <geometry>
@@ -105,7 +105,7 @@
   <joint name="gps_joint" type="fixed">
     <axis xyz="1 0 0" />
-    <origin xyz="0.05 -0.1 0.2" />
+    <origin xyz="-0.39 -0.27 0.34" />
     <parent link="base_link" />
-    <child link="gps" />
+    <child link="gps_link" />
   </joint>
   <gazebo reference="gps">
@@ -116,5 +116,5 @@
           <remapping>~/out:=data</remapping>
         </ros>
-        <frame_name>gps</frame_name>
+        <frame_name>gps_link</frame_name>
       </plugin>
       <always_on>true</always_on>

Commit message: Invoked launch file for multiscan100

File: urc_hw_description/urdf/walli_sensors.xacro (robot description, xacro)
@@ -123,5 +123,5 @@
   </gazebo>
   <!-- LIDAR -->
-  <!-- <link name="lidar_link">
+  <link name="lidar_link">
     <inertial>
       <origin xyz="0 0 0" rpy="0 0 0" />
@@ -147,5 +147,5 @@
     <origin xyz="0.0 0.0 0.25" rpy="0.0 0.0 0.0" />
   </joint>
-  <gazebo reference="lidar_link">
+  <!--<gazebo reference="lidar_link">
     <sensor name="lidar" type="ray">
       <always_on>true</always_on>

Commit message: transform position of lidar joint

File: urc_hw_description/urdf/walli_sensors.xacro (robot description, xacro)
@@ -145,5 +145,5 @@
     <parent link="base_link" />
     <child link="lidar_link" />
-    <origin xyz="0.0 0.0 0.25" rpy="0.0 0.0 0.0" />
+    <origin xyz="0.1778 0.0 0.254"/>
   </joint>
   <!--<gazebo reference="lidar_link">

Commit message: Transformed lidar joint upside down

File: urc_hw_description/urdf/walli_sensors.xacro (robot description, xacro)
@@ -145,5 +145,5 @@
     <parent link="base_link" />
     <child link="lidar_link" />
-    <origin xyz="0.1778 0.0 0.254"/>
+    <origin xyz="0.1778 0.0 0.254" rpy="0 3.14159265358 0"/>
   </joint>
   <!--<gazebo reference="lidar_link">

Commit message: [misc] LiDAR transforms (#248)
* Invoked launch file for multiscan100

* transform point cloud from lidar_link to map frame

* add gridmap dependencies

* Fix sick launch description

* Filter far away points

* Implemented lookup_tranform method

* transform position of lidar joint

* Add lookup_transform to hpp file

* Transformed lidar joint upside down

* Fix launch file

* Launch sick lidar with correct reference frame

* Minor changes

* Formatting

* Missed some stuff in merge

* code formatting

---------

Co-authored-by: Mrinal Jain <2mrinaljain@gmail.com>
Co-authored-by: Yashas Ambati <yashas.amb@gmail.com>

File: urc_hw_description/urdf/walli_sensors.xacro (robot description, xacro)
@@ -123,5 +123,5 @@
   </gazebo>
   <!-- LIDAR -->
-  <!-- <link name="lidar_link">
+  <link name="lidar_link">
     <inertial>
       <origin xyz="0 0 0" rpy="0 0 0" />
@@ -145,7 +145,7 @@
     <parent link="base_link" />
     <child link="lidar_link" />
-    <origin xyz="0.0 0.0 0.25" rpy="0.0 0.0 0.0" />
-  </joint>
-  <gazebo reference="lidar_link">
+    <origin xyz="0.1778 0.0 0.254" rpy="0 3.14159265358 0"/>
+  </joint>
+  <!--<gazebo reference="lidar_link">
     <sensor name="lidar" type="ray">
       <always_on>true</always_on>

Commit message: imu position

File: urc_hw_description/urdf/walli_sensors.xacro (robot description, xacro)
@@ -17,5 +17,5 @@
   <joint name="imu_joint" type="fixed">
     <axis xyz="1 0 0" />
-    <origin xyz="-0.32 -0.09 0.0" />
+    <origin xyz="0.35 0.0 0.25" />
     <parent link="base_link" />
     <child link="imu_link" />

Commit message: update imu pos

File: urc_hw_description/urdf/walli_sensors.xacro (robot description, xacro)
@@ -17,5 +17,5 @@
   <joint name="imu_joint" type="fixed">
     <axis xyz="1 0 0" />
-    <origin xyz="0.35 0.0 0.25" />
+    <origin xyz="0.14 0.0 0.22" />
     <parent link="base_link" />
     <child link="imu_link" />

Commit message: fix imu frame

File: urc_hw_description/urdf/walli_sensors.xacro (robot description, xacro)
@@ -2,22 +2,15 @@
 <robot name="walli_sensors" xmlns:xacro="http://ros.org/wiki/xacro">
   <!-- IMU -->
-  <link name="imu_link">
-    <visual>
-      <geometry>
-        <box size="0.05 0.05 0.05" />
-      </geometry>
-    </visual>
-    <collision>
-      <geometry>
-        <box size="0.05 0.05 0.05" />
-      </geometry>
-    </collision>
-    <xacro:box_inertia m="0.1" w="0.1" d="0.1" h="0.1" />
-  </link>
+  <link name="imu_link"></link>
+  <link name="imu_link_raw"></link>
   <joint name="imu_joint" type="fixed">
-    <axis xyz="1 0 0" />
     <origin xyz="0.14 0.0 0.22" />
     <parent link="base_link" />
     <child link="imu_link" />
+  </joint>
+  <joint name="imu_joint_raw" type="fixed">
+    <origin rpy="3.14159 0 1.5708" />
+    <parent link="imu_link" />
+    <child link="imu_link_raw" />
   </joint>
   <gazebo reference="imu_link">

Commit message: imu ned2enu

File: urc_hw_description/urdf/walli_sensors.xacro (robot description, xacro)
@@ -3,14 +3,8 @@
   <!-- IMU -->
   <link name="imu_link"></link>
-  <link name="imu_link_raw"></link>
   <joint name="imu_joint" type="fixed">
     <origin xyz="0.14 0.0 0.22" />
     <parent link="base_link" />
     <child link="imu_link" />
-  </joint>
-  <joint name="imu_joint_raw" type="fixed">
-    <origin rpy="3.14159 0 1.5708" />
-    <parent link="imu_link" />
-    <child link="imu_link_raw" />
   </joint>
   <gazebo reference="imu_link">

Commit message: localization tuning (#276)
* ekf param tuning

* localization fixes

* imu position

* update imu pos

* update vectornav

* fix yaw offset

* fix imu frame

* imu ned2enu

* fixes

* fixes

* fixes

* fixes

* linting

File: urc_hw_description/urdf/walli_sensors.xacro (robot description, xacro)
@@ -2,20 +2,7 @@
 <robot name="walli_sensors" xmlns:xacro="http://ros.org/wiki/xacro">
   <!-- IMU -->
-  <link name="imu_link">
-    <visual>
-      <geometry>
-        <box size="0.05 0.05 0.05" />
-      </geometry>
-    </visual>
-    <collision>
-      <geometry>
-        <box size="0.05 0.05 0.05" />
-      </geometry>
-    </collision>
-    <xacro:box_inertia m="0.1" w="0.1" d="0.1" h="0.1" />
-  </link>
+  <link name="imu_link"></link>
   <joint name="imu_joint" type="fixed">
-    <axis xyz="1 0 0" />
-    <origin xyz="-0.32 -0.09 0.0" />
+    <origin xyz="0.14 0.0 0.22" />
     <parent link="base_link" />
     <child link="imu_link" />

Commit message: lidar fixes

File: urc_hw_description/urdf/walli_sensors.xacro (robot description, xacro)
@@ -110,5 +110,5 @@
   </gazebo>
   <!-- LIDAR -->
-  <link name="lidar_link">
+  <link name="lidar_link2">
     <inertial>
       <origin xyz="0 0 0" rpy="0 0 0" />
@@ -131,5 +131,5 @@
   <joint name="lidar_joint" type="fixed">
     <parent link="base_link" />
-    <child link="lidar_link" />
+    <child link="lidar_link2" />
     <origin xyz="0.1778 0.0 0.254" rpy="0 3.14159265358 0"/>
   </joint>

Commit message: lidar fixes

File: urc_hw_description/urdf/walli_sensors.xacro (robot description, xacro)
@@ -132,5 +132,5 @@
     <parent link="base_link" />
     <child link="lidar_link2" />
-    <origin xyz="0.1778 0.0 0.254" rpy="0 3.14159265358 0"/>
+    <origin xyz="0.1778 0.0 0.254" rpy="3.14159265358 0 0"/>
   </joint>
   <!--<gazebo reference="lidar_link">

Commit message: Fixes made during URC 2025 (#277)
* remove unecessary code

* manual localization

* register localizer node

* localizer fixes

* update geographic conversions

* map to base_link manual transform

* status light controller udp address

* status light hw interface fix

* fix status light order

* lidar fixes

* lidar fixes

* lidar fixes

* default teleop

* formatting

File: urc_hw_description/urdf/walli_sensors.xacro (robot description, xacro)
@@ -110,5 +110,5 @@
   </gazebo>
   <!-- LIDAR -->
-  <link name="lidar_link">
+  <link name="lidar_link2">
     <inertial>
       <origin xyz="0 0 0" rpy="0 0 0" />
@@ -131,6 +131,6 @@
   <joint name="lidar_joint" type="fixed">
     <parent link="base_link" />
-    <child link="lidar_link" />
-    <origin xyz="0.1778 0.0 0.254" rpy="0 3.14159265358 0"/>
+    <child link="lidar_link2" />
+    <origin xyz="0.1778 0.0 0.254" rpy="3.14159265358 0 0"/>
   </joint>
   <!--<gazebo reference="lidar_link">
