Commit message: Added things from nav2 tutorial in launch script

File: urc_hw_description/urdf/ros2_control.xacro (robot description, xacro)
@@ -154,5 +154,5 @@
           <param name="udp_port">5000</param>
         </hardware>
-        <joint name="left_wheel">
+        <joint name="left_wheel_joint">
           <command_interface name="velocity" />
           <state_interface name="velocity" />
@@ -161,5 +161,5 @@
           <state_interface name="velocity.back" />
         </joint>
-        <joint name="right_wheel">
+        <joint name="right_wheel_joint">
           <command_interface name="velocity" />
           <state_interface name="velocity" />

File: urc_hw_description/urdf/walli.xacro (robot description, xacro)
@@ -9,10 +9,10 @@
    <xacro:include filename="$(find urc_hw_description)/urdf/walli_sensors.xacro" />
    <xacro:include filename="$(find urc_hw_description)/urdf/ros2_control.xacro" />
-   <xacro:include filename="$(find urc_hw_description)/urdf/drivebase.xacro" />
-   <xacro:include filename="$(find urc_hw_description)/urdf/arm.xacro" />
+   <xacro:include filename="$(find urc_hw_description)/urdf/walli_drivebase.xacro" />
+   <xacro:include filename="$(find urc_hw_description)/urdf/walli_arm.xacro" />
    <xacro:drivebase wheel_friction="0.012" wheel_radius="0.05" wheel_thickness="0.025"
       approximate="true" />
    <xacro:arm />
    <xacro:ros2_control use_simulation="${use_simulation}"
-      config_file_path="$(find urc_bringup)/config/controller_config.yaml" />
+      config_file_path="$(find urc_bringup)/config/ros2_control_walli.yaml" />
 </robot>

Commit message: Feat/six wheel simplified model (#160)
* fix: make things work temporarily for sim

* fix: working drivebase simulation

- xacro: fix damping and friction, reorganize
- config file: change config file location to be found only in urc_bringup
- launch files: create simulation.launch.py in urc_bringup for unified access

* fix: urdf axis inversion

* feat: one file control for simulation

- control simulation from hardware_config.yaml

* fix: minor updates

* added xacro ifs

* Made simplifies cylinders for collisions and visuals

* Added things from nav2 tutorial in launch script

* Configured rviz

* Reconfigured urc_navigation package

* Python linting

* Add config variable to choose between full and simplified robot model

* Fix python errors caused by linting

* Add six-wheel simplified model

* rewrite ekf yaml

* working wheel odom - need to change, but good start

* global ekf not working yet

* Lots of cleanup and changes to try and get the simplified model to work. Still won't respond to angular velocity for some reason

* Delete old simplified model

* Fix some params

* working local, global, navsat localization

* add nav to bringup

* rename

* start nav2 bringup

* Fixed navigation launch script

* C++ and Python Reformatting

* Joystick reformmating and automatic bringup + formatting

* Flake8 Linting

* Flake8 Linting 2

* Flake8 Linting 3

* Final fixes

---------

Co-authored-by: KeseterG <zhiwan13579@126.com>
Co-authored-by: davidcalderon03 <davidcalderon03@hotmail.com>
Co-authored-by: Rohan Bansal <bansalrohan18@gmail.com>
Co-authored-by: Saraansh Wadkar <saraanshwadkar@gmail.com>

File: urc_hw_description/urdf/ros2_control.xacro (robot description, xacro)
@@ -1,223 +1,230 @@
 <?xml version="1.0"?>
 <robot xmlns:xacro="http://www.ros.org/wiki/xacro">
-    <!-- Gazebo Configuration -->
-    <ros2_control name="GazeboSystem" type="system">
-        <hardware>
-            <!-- TODO make a launch param to switch between real/fake hardware. You can only use ONE. -->
-            <!--Use for functionality in Gazebo, also needed for drivetrain-->
-            <plugin>gazebo_ros2_control/GazeboSystem</plugin>
-            <!--Use for functionality in RViz-->
-            <!-- <plugin>mock_components/GenericSystem</plugin> -->
-            <!-- <plugin>ros2_control_demo_hardware/VelocityActuatorHardware</plugin> -->
+  <xacro:macro name="ros2_control" params="use_simulation config_file_path">
+    <xacro:if value="${use_simulation}">
+      <ros2_control name="GazeboSystem" type="system">
+        <hardware>
+          <!-- TODO make a launch param to switch between real/fake hardware. You can only use ONE. -->
+          <!--Use
+          for functionality in Gazebo, also needed for drivetrain-->
+          <plugin>gazebo_ros2_control/GazeboSystem</plugin>
+          <!--Use
+          for functionality in RViz-->
+          <!-- <plugin>mock_components/GenericSystem</plugin> -->
+          <!-- <plugin>ros2_control_demo_hardware/VelocityActuatorHardware</plugin> -->
         </hardware>
         <joint name="left_front_wheel_joint">
-            <command_interface name="velocity">
-                <param name="min">-0.05</param>
-                <param name="max">0.05</param>
-            </command_interface>
-            <state_interface name="velocity"/>
-            <state_interface name="position"/>
+          <command_interface name="velocity">
+            <param name="min">-0.05</param>
+            <param name="max">0.05</param>
+          </command_interface>
+          <state_interface name="velocity" />
+          <state_interface name="position" />
         </joint>
         <joint name="right_front_wheel_joint">
-            <command_interface name="velocity">
-                <param name="min">-0.05</param>
-                <param name="max">0.05</param>
-            </command_interface>
-            <state_interface name="velocity"/>
-            <state_interface name="position"/>
+          <command_interface name="velocity">
+            <param name="min">-0.05</param>
+            <param name="max">0.05</param>
+          </command_interface>
+          <state_interface name="velocity" />
+          <state_interface name="position" />
         </joint>
         <joint name="left_center_wheel_joint">
-            <command_interface name="velocity">
-                <param name="min">-0.05</param>
-                <param name="max">0.05</param>
-            </command_interface>
-            <state_interface name="velocity"/>
-            <state_interface name="position"/>
+          <command_interface name="velocity">
+            <param name="min">-0.05</param>
+            <param name="max">0.05</param>
+          </command_interface>
+          <state_interface name="velocity" />
+          <state_interface name="position" />
         </joint>
         <joint name="right_center_wheel_joint">
-            <command_interface name="velocity">
-                <param name="min">-0.05</param>
-                <param name="max">0.05</param>
-            </command_interface>
-            <state_interface name="velocity"/>
-            <state_interface name="position"/>
+          <command_interface name="velocity">
+            <param name="min">-0.05</param>
+            <param name="max">0.05</param>
+          </command_interface>
+          <state_interface name="velocity" />
+          <state_interface name="position" />
         </joint>
         <joint name="left_rear_wheel_joint">
-            <command_interface name="velocity">
-                <param name="min">-0.05</param>
-                <param name="max">0.05</param>
-            </command_interface>
-            <state_interface name="velocity"/>
-            <state_interface name="position"/>
+          <command_interface name="velocity">
+            <param name="min">-0.05</param>
+            <param name="max">0.05</param>
+          </command_interface>
+          <state_interface name="velocity" />
+          <state_interface name="position" />
         </joint>
         <joint name="right_rear_wheel_joint">
-            <command_interface name="velocity">
-                <param name="min">-0.05</param>
-                <param name="max">0.05</param>
-            </command_interface>
-            <state_interface name="velocity"/>
-            <state_interface name="position"/>
-        </joint>
-      <joint name ="shoulderjoint">
-        <command_interface name="position" />
-        <state_interface name="position">
-          <param name="initial_value">0.0</param>
-        </state_interface>
-        <state_interface name="velocity"/>
-        <state_interface name="effort"/>
-      </joint>
-      <joint name ="bicepjoint">
-        <command_interface name="position" />
-        <state_interface name="position">
-          <param name="initial_value">0.0</param>
-        </state_interface>
-        <state_interface name="velocity"/>
-        <state_interface name="effort"/>
-      </joint>
-      <joint name ="elbowjoint">
-        <command_interface name="position" />
-        <state_interface name="position">
-          <param name="initial_value">0.0</param>
-        </state_interface>
-        <state_interface name="velocity"/>
-        <state_interface name="effort"/>
-      </joint>
-	    <joint name ="forearmjoint">
-        <command_interface name="position" />
-        <state_interface name="position">
-          <param name="initial_value">0.0</param>
-        </state_interface>
-        <state_interface name="velocity"/>
-        <state_interface name="effort"/>
-      </joint>
-      <joint name ="wristjoint">
-        <command_interface name="position" />
-        <state_interface name="position">
-          <param name="initial_value">0.0</param>
-        </state_interface>
-        <state_interface name="velocity"/>
-        <state_interface name="effort"/>
-      </joint>
-      <joint name ="clawjoint">
-        <command_interface name="position" />
-        <state_interface name="position">
-          <param name="initial_value">0.0</param>
-        </state_interface>
-        <state_interface name="velocity"/>
-        <state_interface name="effort"/>
-      </joint>
-      <joint name ="leftgripperjoint">
-        <command_interface name="position" />
-        <state_interface name="position">
-          <param name="initial_value">0.0</param>
-        </state_interface>
-        <state_interface name="velocity"/>
-        <state_interface name="effort"/>
-      </joint>
-      <joint name ="rightgripperjoint">
-        <command_interface name="position" />
-        <state_interface name="position">
-          <param name="initial_value">0.0</param>
-        </state_interface>
-        <state_interface name="velocity"/>
-        <state_interface name="effort"/>
-      </joint>
-    </ros2_control>
-    <!-- New ROS2 Control Work-->
-    <ros2_control name="walli_others" type="system">
-        <hardware>
-            <plugin>urc_hw/StatusLight</plugin>
-            <param name="serial_port">/dev/ttyACM0</param>
-            <param name="udp_address">143.215.63.147</param>
-            <param name="udp_port">5000</param>
+          <command_interface name="velocity">
+            <param name="min">-0.05</param>
+            <param name="max">0.05</param>
+          </command_interface>
+          <state_interface name="velocity" />
+          <state_interface name="position" />
+        </joint>
+        <joint name="shoulderjoint">
+          <command_interface name="position" />
+          <state_interface name="position">
+            <param name="initial_value">0.0</param>
+          </state_interface>
+          <state_interface name="velocity" />
+          <state_interface name="effort" />
+        </joint>
+        <joint name="bicepjoint">
+          <command_interface name="position" />
+          <state_interface name="position">
+            <param name="initial_value">0.0</param>
+          </state_interface>
+          <state_interface name="velocity" />
+          <state_interface name="effort" />
+        </joint>
+        <joint name="elbowjoint">
+          <command_interface name="position" />
+          <state_interface name="position">
+            <param name="initial_value">0.0</param>
+          </state_interface>
+          <state_interface name="velocity" />
+          <state_interface name="effort" />
+        </joint>
+        <joint name="forearmjoint">
+          <command_interface name="position" />
+          <state_interface name="position">
+            <param name="initial_value">0.0</param>
+          </state_interface>
+          <state_interface name="velocity" />
+          <state_interface name="effort" />
+        </joint>
+        <joint name="wristjoint">
+          <command_interface name="position" />
+          <state_interface name="position">
+            <param name="initial_value">0.0</param>
+          </state_interface>
+          <state_interface name="velocity" />
+          <state_interface name="effort" />
+        </joint>
+        <joint name="clawjoint">
+          <command_interface name="position" />
+          <state_interface name="position">
+            <param name="initial_value">0.0</param>
+          </state_interface>
+          <state_interface name="velocity" />
+          <state_interface name="effort" />
+        </joint>
+        <joint name="leftgripperjoint">
+          <command_interface name="position" />
+          <state_interface name="position">
+            <param name="initial_value">0.0</param>
+          </state_interface>
+          <state_interface name="velocity" />
+          <state_interface name="effort" />
+        </joint>
+        <joint name="rightgripperjoint">
+          <command_interface name="position" />
+          <state_interface name="position">
+            <param name="initial_value">0.0</param>
+          </state_interface>
+          <state_interface name="velocity" />
+          <state_interface name="effort" />
+        </joint>
+      </ros2_control>
+    </xacro:if>
+    <xacro:if value="${use_simulation}">
+      <gazebo>
+        <plugin filename="libgazebo_ros2_control.so" name="gazebo_ros2_control">
+          <parameters>${config_file_path}</parameters>
+        </plugin>
+      </gazebo>
+    </xacro:if>
+    <xacro:if value="${not use_simulation}">
+      <ros2_control name="walli_others" type="system">
+        <hardware>
+          <plugin>urc_hw/StatusLight</plugin>
+          <param name="serial_port">/dev/ttyACM0</param>
+          <param name="udp_address">143.215.63.147</param>
+          <param name="udp_port">5000</param>
         </hardware>
         <gpio name="status_light">
-            <command_interface name="color" />
-            <command_interface name="display" />
+          <command_interface name="color" />
+          <command_interface name="display" />
         </gpio>
-    </ros2_control>
-    <ros2_control name="rover_drivetrain" type="system">
-          <hardware>
-              <plugin>urc_hw/RoverDrivetrain</plugin>
-              <param name="udp_address">127.0.0.1</param>
-              <param name="udp_port">5000</param>
-          </hardware>
-          <joint name="left_wheel">
-              <command_interface name="velocity" />
-              <state_interface name="velocity" />
-              <state_interface name="velocity.front" />
-              <state_interface name="velocity.mid" />
-              <state_interface name="velocity.back" />
-          </joint>
-          <joint name="right_wheel">
-              <command_interface name="velocity" />
-              <state_interface name="velocity" />
-              <state_interface name="velocity.front" />
-              <state_interface name="velocity.mid" />
-              <state_interface name="velocity.back" />
-          </joint>
+      </ros2_control>
+      <ros2_control name="rover_drivetrain" type="system">
+        <hardware>
+          <plugin>urc_hw/RoverDrivetrain</plugin>
+          <param name="udp_address">127.0.0.1</param>
+          <param name="udp_port">5000</param>
+        </hardware>
+        <joint name="left_wheel_joint">
+          <command_interface name="velocity" />
+          <state_interface name="velocity" />
+          <state_interface name="velocity.front" />
+          <state_interface name="velocity.mid" />
+          <state_interface name="velocity.back" />
+        </joint>
+        <joint name="right_wheel_joint">
+          <command_interface name="velocity" />
+          <state_interface name="velocity" />
+          <state_interface name="velocity.front" />
+          <state_interface name="velocity.mid" />
+          <state_interface name="velocity.back" />
+        </joint>
       </ros2_control>
       <ros2_control name="status_light" type="system">
-          <hardware>
-              <plugin>urc_hw/StatusLight</plugin>
-              <param name="serial_port">/dev/ttyACM0</param>
-              <param name="udp_address">143.215.63.147</param>
-              <param name="udp_port">5000</param>
-          </hardware>
-          <gpio name="status_light">
-              <command_interface name="color" />
-              <command_interface name="display" />
-          </gpio>
+        <hardware>
+          <plugin>urc_hw/StatusLight</plugin>
+          <param name="serial_port">/dev/ttyACM0</param>
+          <param name="udp_address">143.215.63.147</param>
+          <param name="udp_port">5000</param>
+        </hardware>
+        <gpio name="status_light">
+          <command_interface name="color" />
+          <command_interface name="display" />
+        </gpio>
       </ros2_control>
       <ros2_control name="battery_management" type="sensor">
-          <hardware>
-              <plugin>urc_hw/BatteryManagement</plugin>
-              <param name="udp_address">127.0.0.1</param>
-              <param name="udp_port">5000</param>
-              <param name="udp_self_address">127.0.0.1</param>
-              <param name="udp_self_port">7000</param>
-          </hardware>
-          <sensor name="battery_management">
-              <state_interface name="main_voltage" />
-              <state_interface name="charge_percentage" />
-              <state_interface name="discharge_current" />
-              <state_interface name="temperature" />
-              <state_interface name="cell1_voltage" />
-              <state_interface name="cell2_voltage" />
-              <state_interface name="cell3_voltage" />
-              <state_interface name="cell4_voltage" />
-              <state_interface name="cell5_voltage" />
-              <state_interface name="cell6_voltage" />
-              <state_interface name="cell7_voltage" />
-              <state_interface name="cell8_voltage" />
-          </sensor>
+        <hardware>
+          <plugin>urc_hw/BatteryManagement</plugin>
+          <param name="udp_address">127.0.0.1</param>
+          <param name="udp_port">5000</param>
+          <param name="udp_self_address">127.0.0.1</param>
+          <param name="udp_self_port">7000</param>
+        </hardware>
+        <sensor name="battery_management">
+          <state_interface name="main_voltage" />
+          <state_interface name="charge_percentage" />
+          <state_interface name="discharge_current" />
+          <state_interface name="temperature" />
+          <state_interface name="cell1_voltage" />
+          <state_interface name="cell2_voltage" />
+          <state_interface name="cell3_voltage" />
+          <state_interface name="cell4_voltage" />
+          <state_interface name="cell5_voltage" />
+          <state_interface name="cell6_voltage" />
+          <state_interface name="cell7_voltage" />
+          <state_interface name="cell8_voltage" />
+        </sensor>
       </ros2_control>
       <ros2_control name="imu" type="sensor">
-          <hardware>
-              <plugin>urc_hw/IMU</plugin>
-              <param name="udp_address">127.0.0.1</param>
-              <param name="udp_port">5000</param>
-              <param name="udp_self_address">127.0.0.1</param>
-              <param name="udp_self_port">7000</param>
-          </hardware>
-          <sensor name="imu_sensor">
-              <state_interface name="orientation.x" />
-              <state_interface name="orientation.y" />
-              <state_interface name="orientation.z" />
-              <state_interface name="orientation.w" />
-              <state_interface name="linear_acceleration.x" />
-              <state_interface name="linear_acceleration.y" />
-              <state_interface name="linear_acceleration.z" />
-              <state_interface name="angular_velocity.x" />
-              <state_interface name="angular_velocity.y" />
-              <state_interface name="angular_velocity.z" />
-          </sensor>
-      </ros2_control>
-    <gazebo>
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