Commit message: Feat/arm simulation (#159)
* fix: make things work temporarily for sim

* fix: working drivebase simulation

- xacro: fix damping and friction, reorganize
- config file: change config file location to be found only in urc_bringup
- launch files: create simulation.launch.py in urc_bringup for unified access

* fix: urdf axis inversion

* feat: one file control for simulation

- control simulation from hardware_config.yaml

* fix: minor updates

* feat: adding arm simulation

* added xacro ifs

* fix: movegroup launch

* fix: updating arm simulation and moveit

* fix: try to fix moveit but failed

* fix: not working update

* feat: arm pinocchio implementation

* feat: arm feature updates

* fix: diff_drive_controller params

* CI fixes

* Resolve unfound package

* Removed pep257

---------

Co-authored-by: KeseterG <zhiwan13579@126.com>
Co-authored-by: davidcalderon03 <davidcalderon03@hotmail.com>

File: urc_hw_description/urdf/ros2_control.xacro (robot description, xacro)
@@ -1,5 +1,8 @@
 <?xml version="1.0"?>
 <robot xmlns:xacro="http://www.ros.org/wiki/xacro">
-  <xacro:macro name="ros2_control" params="use_simulation config_file_path">
+  <xacro:macro name="ros2_control"
+    params="use_simulation config_file_path arm_initial_positions_file">
+    <xacro:property name="initial_positions"
+      value="${load_yaml(arm_initial_positions_file)['initial_positions']}" />
     <xacro:if value="${use_simulation}">
       <ros2_control name="GazeboSystem" type="system">
@@ -64,65 +67,64 @@
         <joint name="shoulderjoint">
           <command_interface name="position" />
-          <state_interface name="position">
-            <param name="initial_value">0.0</param>
-          </state_interface>
-          <state_interface name="velocity" />
-          <state_interface name="effort" />
+          <command_interface name="velocity" />
+          <command_interface name="effort" />
+          <state_interface name="position">
+            <param name="initial_value">${initial_positions['shoulderjoint']}</param>
+          </state_interface>
+          <state_interface name="velocity" />
         </joint>
         <joint name="bicepjoint">
           <command_interface name="position" />
-          <state_interface name="position">
-            <param name="initial_value">0.0</param>
-          </state_interface>
-          <state_interface name="velocity" />
-          <state_interface name="effort" />
+          <command_interface name="velocity" />
+          <command_interface name="effort" />
+          <state_interface name="position">
+            <param name="initial_value">${initial_positions['bicepjoint']}</param>
+          </state_interface>
+          <state_interface name="velocity" />
         </joint>
         <joint name="elbowjoint">
           <command_interface name="position" />
-          <state_interface name="position">
-            <param name="initial_value">0.0</param>
-          </state_interface>
-          <state_interface name="velocity" />
-          <state_interface name="effort" />
-        </joint>
-        <joint name="forearmjoint">
-          <command_interface name="position" />
-          <state_interface name="position">
-            <param name="initial_value">0.0</param>
-          </state_interface>
-          <state_interface name="velocity" />
-          <state_interface name="effort" />
+          <command_interface name="velocity" />
+          <command_interface name="effort" />
+          <state_interface name="position">
+            <param name="initial_value">${initial_positions['elbowjoint']}</param>
+          </state_interface>
+          <state_interface name="velocity" />
         </joint>
         <joint name="wristjoint">
           <command_interface name="position" />
-          <state_interface name="position">
-            <param name="initial_value">0.0</param>
-          </state_interface>
-          <state_interface name="velocity" />
-          <state_interface name="effort" />
+          <command_interface name="velocity" />
+          <command_interface name="effort" />
+          <state_interface name="position">
+            <param name="initial_value">${initial_positions['wristjoint']}</param>
+          </state_interface>
+          <state_interface name="velocity" />
         </joint>
         <joint name="clawjoint">
           <command_interface name="position" />
-          <state_interface name="position">
-            <param name="initial_value">0.0</param>
-          </state_interface>
-          <state_interface name="velocity" />
-          <state_interface name="effort" />
+          <command_interface name="velocity" />
+          <command_interface name="effort" />
+          <state_interface name="position">
+            <param name="initial_value">${initial_positions['clawjoint']}</param>
+          </state_interface>
+          <state_interface name="velocity" />
+        </joint>
+        <joint name="rightgripperjoint">
+          <command_interface name="position" />
+          <command_interface name="velocity" />
+          <command_interface name="effort" />
+          <state_interface name="position">
+            <param name="initial_value">${initial_positions['rightgripperjoint']}</param>
+          </state_interface>
+          <state_interface name="velocity" />
         </joint>
         <joint name="leftgripperjoint">
           <command_interface name="position" />
-          <state_interface name="position">
-            <param name="initial_value">0.0</param>
-          </state_interface>
-          <state_interface name="velocity" />
-          <state_interface name="effort" />
-        </joint>
-        <joint name="rightgripperjoint">
-          <command_interface name="position" />
-          <state_interface name="position">
-            <param name="initial_value">0.0</param>
-          </state_interface>
-          <state_interface name="velocity" />
-          <state_interface name="effort" />
+          <command_interface name="velocity" />
+          <command_interface name="effort" />
+          <state_interface name="position">
+            <param name="initial_value">${initial_positions['rightgripperjoint']}</param>
+          </state_interface>
+          <state_interface name="velocity" />
         </joint>
       </ros2_control>
@@ -151,8 +153,8 @@
         <hardware>
           <plugin>urc_hw/RoverDrivetrain</plugin>
-          <param name="udp_address">127.0.0.1</param>
-          <param name="udp_port">5000</param>
-        </hardware>
-        <joint name="left_wheel_joint">
+          <param name="udp_address">192.168.1.100</param>
+          <param name="udp_port">8443</param>
+        </hardware>
+        <joint name="left_wheel">
           <command_interface name="velocity" />
           <state_interface name="velocity" />
@@ -161,5 +163,5 @@
           <state_interface name="velocity.back" />
         </joint>
-        <joint name="right_wheel_joint">
+        <joint name="right_wheel">
           <command_interface name="velocity" />
           <state_interface name="velocity" />

File: urc_hw_description/urdf/walli.xacro (robot description, xacro)
@@ -1,7 +1,7 @@
-<?xml version="1.0" encoding="UTF-8"?>
+<?xml version="1.0"?>
 <robot name="walli" xmlns:xacro="http://ros.org/wiki/xacro">
    <xacro:property name="config_file"
       value="$(find urc_bringup)/config/hardware_config.yaml" />
-   <xacro:property name="config_data" value="${xacro.load_yaml(config_file)}"></xacro:property>
+   <xacro:property name="config_data" value="${load_yaml(config_file)}"></xacro:property>
    <xacro:property name="use_simulation" value="${config_data['hardware_config']['use_simulation']}" />
    <xacro:include filename="$(find urc_hw_description)/urdf/walli_prop.xacro" />
@@ -9,10 +9,11 @@
    <xacro:include filename="$(find urc_hw_description)/urdf/walli_sensors.xacro" />
    <xacro:include filename="$(find urc_hw_description)/urdf/ros2_control.xacro" />
-   <xacro:include filename="$(find urc_hw_description)/urdf/walli_drivebase.xacro" />
-   <xacro:include filename="$(find urc_hw_description)/urdf/walli_arm.xacro" />
-   <xacro:drivebase wheel_friction="0.012" wheel_radius="0.05" wheel_thickness="0.025"
-      approximate="true" />
+   <xacro:include filename="$(find urc_hw_description)/urdf/drivebase.xacro" />
+   <xacro:include filename="$(find urc_hw_description)/urdf/arm.xacro" />
+   <xacro:drivebase wheel_friction="0.012" wheel_radius="0.10" wheel_thickness="0.05"
+      approximate="false" />
    <xacro:arm />
    <xacro:ros2_control use_simulation="${use_simulation}"
-      config_file_path="$(find urc_bringup)/config/ros2_control_walli.yaml" />
+      config_file_path="$(find urc_bringup)/config/controller_config.yaml"
+      arm_initial_positions_file="$(find urc_hw_description)/config/initial_positions.yaml" />
 </robot>

Commit message: Add state interface for rocker and bogie joints

File: urc_hw_description/urdf/ros2_control.xacro (robot description, xacro)
@@ -17,4 +17,28 @@
           <!-- <plugin>ros2_control_demo_hardware/VelocityActuatorHardware</plugin> -->
         </hardware>
+        <joint name="leftbogiejoint">
+          <state_interface name="velocity" />
+          <state_interface name="position" />
+        </joint>
+        <joint name="leftrockerjoint">
+          <state_interface name="velocity" />
+          <state_interface name="position" />
+        </joint>
+        <joint name="rightbogiejoint">
+          <state_interface name="velocity" />
+          <state_interface name="position" />
+        </joint>
+        <joint name="rightrockerjoint">
+          <state_interface name="velocity" />
+          <state_interface name="position" />
+        </joint>
+        <joint name="left_front_wheel_joint">
+          <command_interface name="velocity">
+            <param name="min">-0.05</param>
+            <param name="max">0.05</param>
+          </command_interface>
+          <state_interface name="velocity" />
+          <state_interface name="position" />
+        </joint>
         <joint name="left_front_wheel_joint">
           <command_interface name="velocity">

Commit message: Fixed some things, finally getting odometry based on position feedback

File: urc_hw_description/urdf/ros2_control.xacro (robot description, xacro)
@@ -23,12 +23,4 @@
         </joint>
         <joint name="rightrockerjoint">
-          <state_interface name="velocity" />
-          <state_interface name="position" />
-        </joint>
-        <joint name="left_front_wheel_joint">
-          <command_interface name="velocity">
-            <param name="min">-0.05</param>
-            <param name="max">0.05</param>
-          </command_interface>
           <state_interface name="velocity" />
           <state_interface name="position" />
