Commit message: new urdf

File: urc_hw_description/urdf/ros2_control.xacro (robot description, xacro)
@@ -10,21 +10,17 @@
           <plugin>gazebo_ros2_control/GazeboSystem</plugin>
         </hardware>
-        <joint name="leftbogiejoint">
+        <joint name="Left_Leg">
           <state_interface name="velocity" />
           <state_interface name="position" />
         </joint>
-        <joint name="leftrockerjoint">
+        <joint name="Differential_Bar">
           <state_interface name="velocity" />
           <state_interface name="position" />
         </joint>
-        <joint name="rightbogiejoint">
+        <joint name="Right_Leg">
           <state_interface name="velocity" />
           <state_interface name="position" />
         </joint>
-        <joint name="rightrockerjoint">
-          <state_interface name="velocity" />
-          <state_interface name="position" />
-        </joint>
-        <joint name="left_front_wheel_joint">
+        <joint name="Front_Left_Wheel">
           <command_interface name="velocity">
             <param name="min">-0.05</param>
@@ -34,5 +30,5 @@
           <state_interface name="position" />
         </joint>
-        <joint name="right_front_wheel_joint">
+        <joint name="Back_Left_Wheel">
           <command_interface name="velocity">
             <param name="min">-0.05</param>
@@ -42,5 +38,5 @@
           <state_interface name="position" />
         </joint>
-        <joint name="left_center_wheel_joint">
+        <joint name="Front_Right_Wheel">
           <command_interface name="velocity">
             <param name="min">-0.05</param>
@@ -50,5 +46,5 @@
           <state_interface name="position" />
         </joint>
-        <joint name="right_center_wheel_joint">
+        <joint name="Back_Right_Wheel">
           <command_interface name="velocity">
             <param name="min">-0.05</param>
@@ -57,83 +53,4 @@
           <state_interface name="velocity" />
           <state_interface name="position" />
-        </joint>
-        <joint name="left_rear_wheel_joint">
-          <command_interface name="velocity">
-            <param name="min">-0.05</param>
-            <param name="max">0.05</param>
-          </command_interface>
-          <state_interface name="velocity" />
-          <state_interface name="position" />
-        </joint>
-        <joint name="right_rear_wheel_joint">
-          <command_interface name="velocity">
-            <param name="min">-0.05</param>
-            <param name="max">0.05</param>
-          </command_interface>
-          <state_interface name="velocity" />
-          <state_interface name="position" />
-        </joint>
-        <joint name="shoulderjoint">
-          <command_interface name="position" />
-          <command_interface name="velocity" />
-          <command_interface name="effort" />
-          <state_interface name="position">
-            <param name="initial_value">${initial_positions['shoulderjoint']}</param>
-          </state_interface>
-          <state_interface name="velocity" />
-        </joint>
-        <joint name="bicepjoint">
-          <command_interface name="position" />
-          <command_interface name="velocity" />
-          <command_interface name="effort" />
-          <state_interface name="position">
-            <param name="initial_value">${initial_positions['bicepjoint']}</param>
-          </state_interface>
-          <state_interface name="velocity" />
-        </joint>
-        <joint name="elbowjoint">
-          <command_interface name="position" />
-          <command_interface name="velocity" />
-          <command_interface name="effort" />
-          <state_interface name="position">
-            <param name="initial_value">${initial_positions['elbowjoint']}</param>
-          </state_interface>
-          <state_interface name="velocity" />
-        </joint>
-        <joint name="wristjoint">
-          <command_interface name="position" />
-          <command_interface name="velocity" />
-          <command_interface name="effort" />
-          <state_interface name="position">
-            <param name="initial_value">${initial_positions['wristjoint']}</param>
-          </state_interface>
-          <state_interface name="velocity" />
-        </joint>
-        <joint name="clawjoint">
-          <command_interface name="position" />
-          <command_interface name="velocity" />
-          <command_interface name="effort" />
-          <state_interface name="position">
-            <param name="initial_value">${initial_positions['clawjoint']}</param>
-          </state_interface>
-          <state_interface name="velocity" />
-        </joint>
-        <joint name="rightgripperjoint">
-          <command_interface name="position" />
-          <command_interface name="velocity" />
-          <command_interface name="effort" />
-          <state_interface name="position">
-            <param name="initial_value">${initial_positions['rightgripperjoint']}</param>
-          </state_interface>
-          <state_interface name="velocity" />
-        </joint>
-        <joint name="leftgripperjoint">
-          <command_interface name="position" />
-          <command_interface name="velocity" />
-          <command_interface name="effort" />
-          <state_interface name="position">
-            <param name="initial_value">${initial_positions['rightgripperjoint']}</param>
-          </state_interface>
-          <state_interface name="velocity" />
         </joint>
       </ros2_control>
@@ -207,16 +124,4 @@
           <param name="udp_self_port">7000</param>
         </hardware>
-        <sensor name="imu_sensor">
-          <state_interface name="orientation.x" />
-          <state_interface name="orientation.y" />
-          <state_interface name="orientation.z" />
-          <state_interface name="orientation.w" />
-          <state_interface name="linear_acceleration.x" />
-          <state_interface name="linear_acceleration.y" />
-          <state_interface name="linear_acceleration.z" />
-          <state_interface name="angular_velocity.x" />
-          <state_interface name="angular_velocity.y" />
-          <state_interface name="angular_velocity.z" />
-        </sensor>
       </ros2_control>
     </xacro:if>

Commit message: fix joint_state_broadcaster and rover_drivetrain_controller

File: urc_hw_description/urdf/ros2_control.xacro (robot description, xacro)
@@ -2,7 +2,5 @@
 <robot xmlns:xacro="http://www.ros.org/wiki/xacro">
   <xacro:macro name="ros2_control"
-    params="use_simulation config_file_path arm_initial_positions_file">
-    <xacro:property name="initial_positions"
-      value="${load_yaml(arm_initial_positions_file)['initial_positions']}" />
+    params="use_simulation config_file_path">
     <xacro:if value="${use_simulation}">
       <ros2_control name="GazeboSystem" type="system">
@@ -10,17 +8,17 @@
           <plugin>gazebo_ros2_control/GazeboSystem</plugin>
         </hardware>
-        <joint name="Left_Leg">
+        <joint name="Left_Leg_Shaft">
           <state_interface name="velocity" />
           <state_interface name="position" />
         </joint>
-        <joint name="Differential_Bar">
+        <!-- <joint name="Differential_Bar"> -->
+        <!--   <state_interface name="velocity" /> -->
+        <!--   <state_interface name="position" /> -->
+        <!-- </joint> -->
+        <joint name="Right_Leg_Shaft">
           <state_interface name="velocity" />
           <state_interface name="position" />
         </joint>
-        <joint name="Right_Leg">
-          <state_interface name="velocity" />
-          <state_interface name="position" />
-        </joint>
-        <joint name="Front_Left_Wheel">
+        <joint name="Front_Left_Shaft">
           <command_interface name="velocity">
             <param name="min">-0.05</param>
@@ -30,5 +28,5 @@
           <state_interface name="position" />
         </joint>
-        <joint name="Back_Left_Wheel">
+        <joint name="Back_Left_Shaft">
           <command_interface name="velocity">
             <param name="min">-0.05</param>
@@ -38,5 +36,5 @@
           <state_interface name="position" />
         </joint>
-        <joint name="Front_Right_Wheel">
+        <joint name="Front_Right_Shaft">
           <command_interface name="velocity">
             <param name="min">-0.05</param>
@@ -46,5 +44,5 @@
           <state_interface name="position" />
         </joint>
-        <joint name="Back_Right_Wheel">
+        <joint name="Back_Right_Shaft">
           <command_interface name="velocity">
             <param name="min">-0.05</param>

File: urc_hw_description/urdf/wallii.xacro (robot description, xacro)
@@ -5,8 +5,7 @@
    <xacro:include filename="$(find urc_hw_description)/urdf/wallii_drivebase.xacro" />
    <!-- <xacro:include filename="$(find urc_hw_description)/urdf/walli_sensors.xacro" /> -->
-   <!-- <xacro:include filename="$(find urc_hw_description)/urdf/ros2_control.xacro" /> -->
+   <xacro:include filename="$(find urc_hw_description)/urdf/ros2_control.xacro" />
    <xacro:drivebase mu="1.0" mu2="0.25" />
-   <!-- <xacro:ros2_control use_simulation="$(arg use_simulation)" -->
-   <!--    config_file_path="$(find urc_bringup)/config/controller_config.yaml" -->
-   <!--    arm_initial_positions_file="$(find urc_hw_description)/config/initial_positions.yaml" /> -->
+   <xacro:ros2_control use_simulation="$(arg use_simulation)"
+      config_file_path="$(find urc_bringup)/config/ros2_control_walli.yaml" />
 </robot>

Commit message: Clean up joint/link names

File: urc_hw_description/urdf/ros2_control.xacro (robot description, xacro)
@@ -8,5 +8,5 @@
           <plugin>gazebo_ros2_control/GazeboSystem</plugin>
         </hardware>
-        <joint name="Left_Leg_Shaft">
+        <joint name="left_rocker_joint">
           <state_interface name="velocity" />
           <state_interface name="position" />
@@ -16,9 +16,9 @@
         <!--   <state_interface name="position" /> -->
         <!-- </joint> -->
-        <joint name="Right_Leg_Shaft">
+        <joint name="right_rocker_joint">
           <state_interface name="velocity" />
           <state_interface name="position" />
         </joint>
-        <joint name="Front_Left_Shaft">
+        <joint name="front_left_wheel_joint">
           <command_interface name="velocity">
             <param name="min">-0.05</param>
@@ -28,5 +28,5 @@
           <state_interface name="position" />
         </joint>
-        <joint name="Back_Left_Shaft">
+        <joint name="back_left_wheel_joint">
           <command_interface name="velocity">
             <param name="min">-0.05</param>
@@ -36,5 +36,5 @@
           <state_interface name="position" />
         </joint>
-        <joint name="Front_Right_Shaft">
+        <joint name="front_right_wheel_joint">
           <command_interface name="velocity">
             <param name="min">-0.05</param>
@@ -44,5 +44,5 @@
           <state_interface name="position" />
         </joint>
-        <joint name="Back_Right_Shaft">
+        <joint name="back_right_wheel_joint">
           <command_interface name="velocity">
             <param name="min">-0.05</param>

File: urc_hw_description/urdf/wallii_drivebase.xacro (robot description, xacro)
@@ -1,4 +1,5 @@
 <?xml version="1.0" encoding="utf-8"?>
-<!-- This URDF was automatically created by SolidWorks to URDF Exporter! Originally created by Stephen Brawner (brawner@gmail.com)
+<!-- This URDF was automatically created by SolidWorks to URDF Exporter! Originally created by
+Stephen Brawner (brawner@gmail.com)
      Commit Version: 1.6.0-4-g7f85cfe  Build Version: 1.6.7995.38578
      For more information, please see http://wiki.ros.org/sw_urdf_exporter -->
@@ -46,5 +47,5 @@
     </link>
     <link
-      name="Left_Leg">
+      name="left_rocker">
       <inertial>
         <origin
@@ -86,5 +87,5 @@
     </link>
     <joint
-      name="Left_Leg_Shaft"
+      name="left_rocker_joint"
       type="revolute">
       <origin
@@ -94,5 +95,5 @@
         link="base_link" />
       <child
-        link="Left_Leg" />
+        link="left_rocker" />
       <axis
         xyz="0 1 0" />
@@ -105,5 +106,5 @@
     </joint>
     <link
-      name="Front_Left_Wheel">
+      name="front_left_wheel">
       <inertial>
         <origin
@@ -153,5 +154,5 @@
     </link>
     <joint
-      name="Front_Left_Shaft"
+      name="front_left_wheel_joint"
       type="continuous">
       <origin
@@ -159,12 +160,12 @@
         rpy="0 -0.0083213 -1.5708" />
       <parent
-        link="Left_Leg" />
-      <child
-        link="Front_Left_Wheel" />
-      <axis
-        xyz="0 1 0" />
-    </joint>
-    <link
-      name="Back_Left_Wheel">
+        link="left_rocker" />
+      <child
+        link="front_left_wheel" />
+      <axis
+        xyz="0 1 0" />
+    </joint>
+    <link
+      name="back_left_wheel">
       <inertial>
         <origin
@@ -214,5 +215,5 @@
     </link>
     <joint
-      name="Back_Left_Shaft"
+      name="back_left_wheel_joint"
       type="continuous">
       <origin
@@ -220,71 +221,71 @@
         rpy="0 -1.3867 -1.5708" />
       <parent
-        link="Left_Leg" />
-      <child
-        link="Back_Left_Wheel" />
-      <axis
-        xyz="0 1 0" />
-    </joint>
-    <!-- <link -->
-    <!--   name="Differential_Bar"> -->
-    <!--   <inertial> -->
-    <!--     <origin -->
-    <!--       xyz="0.0001696304329344 0.0146364855896726 0.0184524262584146" -->
-    <!--       rpy="0 0 0" /> -->
-    <!--     <mass -->
-    <!--       value="0.8870349519636" /> -->
-    <!--     <inertia -->
-    <!--       ixx="0.00029545831305288" -->
-    <!--       ixy="6.25770619004021E-05" -->
-    <!--       ixz="4.35881163876293E-08" -->
-    <!--       iyy="0.00652074651602383" -->
-    <!--       iyz="-2.01385937443393E-07" -->
-    <!--       izz="0.00679287106362345" /> -->
-    <!--   </inertial> -->
-    <!--   <visual> -->
-    <!--     <origin -->
-    <!--       xyz="0 0 0" -->
-    <!--       rpy="0 0 0" /> -->
-    <!--     <geometry> -->
-    <!--       <mesh -->
-    <!--         filename="file://$(find urc_hw_description)/urdf/meshes/Differential_Bar.STL" /> -->
-    <!--     </geometry> -->
-    <!--     <material -->
-    <!--       name=""> -->
-    <!--       <color -->
-    <!--         rgba="0.792156862745098 0.819607843137255 0.933333333333333 1" /> -->
-    <!--     </material> -->
-    <!--   </visual> -->
-    <!--   <collision> -->
-    <!--     <origin -->
-    <!--       xyz="0 0 0" -->
-    <!--       rpy="0 0 0" /> -->
-    <!--     <geometry> -->
-    <!--       <mesh -->
-    <!--         filename="file://$(find urc_hw_description)/urdf/meshes/Differential_Bar.STL" /> -->
-    <!--     </geometry> -->
-    <!--   </collision> -->
-    <!-- </link> -->
-    <!-- <joint -->
-    <!--   name="Differential_Bar_Shaft" -->
-    <!--   type="revolute"> -->
-    <!--   <origin -->
-    <!--     xyz="0 -0.37445 -0.070294" -->
-    <!--     rpy="1.5708 0 0" /> -->
-    <!--   <parent -->
-    <!--     link="base_link" /> -->
-    <!--   <child -->
-    <!--     link="Differential_Bar" /> -->
-    <!--   <axis -->
-    <!--     xyz="0 0 1" /> -->
-    <!--   <limit -->
-    <!--     lower="0" -->
-    <!--     upper="0" -->
-    <!--     effort="0" -->
-    <!--     velocity="0" /> -->
-    <!--     <dynamics damping="0.01" friction="0.01" /> -->
-    <!-- </joint> -->
-    <link
-      name="Right_Leg">
+        link="left_rocker" />
+      <child
+        link="back_left_wheel" />
+      <axis
+        xyz="0 1 0" />
+    </joint>
+    <link
+      name="differential_bar">
+      <inertial>
+        <origin
+          xyz="0.0001696304329344 0.0146364855896726 0.0184524262584146"
+          rpy="0 0 0" />
+        <mass
+          value="0.8870349519636" />
+        <inertia
+          ixx="0.00029545831305288"
+          ixy="6.25770619004021E-05"
+          ixz="4.35881163876293E-08"
+          iyy="0.00652074651602383"
+          iyz="-2.01385937443393E-07"
+          izz="0.00679287106362345" />
+      </inertial>
+      <visual>
+        <origin
+          xyz="0 0 0"
+          rpy="0 0 0" />
+        <geometry>
+          <mesh
+            filename="file://$(find urc_hw_description)/urdf/meshes/Differential_Bar.STL" />
+        </geometry>
+        <material
+          name="">
+          <color
+            rgba="0.792156862745098 0.819607843137255 0.933333333333333 1" />
+        </material>
+      </visual>
+      <collision>
+        <origin
+          xyz="0 0 0"
+          rpy="0 0 0" />
+        <geometry>
+          <mesh
+            filename="file://$(find urc_hw_description)/urdf/meshes/Differential_Bar.STL" />
+        </geometry>
+      </collision>
+    </link>
+    <joint
+      name="differential_bar_joint"
+      type="revolute">
+      <origin
+        xyz="0 -0.37445 -0.070294"
+        rpy="1.5708 0 0" />
+      <parent
+        link="base_link" />
+      <child
+        link="differential_bar" />
+      <axis
+        xyz="0 0 1" />
+      <limit
+        lower="0"
+        upper="0"
+        effort="0"
+        velocity="0" />
+      <dynamics damping="0.01" friction="0.01" />
+    </joint>
+    <link
+      name="right_rocker">
       <inertial>
         <origin
@@ -326,5 +327,5 @@
     </link>
     <joint
-      name="Right_Leg_Shaft"
+      name="right_rocker_joint"
       type="revolute">
       <origin
@@ -334,5 +335,5 @@
         link="base_link" />
       <child
-        link="Right_Leg" />
+        link="right_rocker" />
       <axis
         xyz="0 1 0" />
@@ -342,8 +343,8 @@
         effort="0"
         velocity="0" />
-        <dynamics damping="0.01" friction="0.01" />
-    </joint>
-    <link
-      name="Front_Right_Wheel">
+      <dynamics damping="0.01" friction="0.01" />
+    </joint>
+    <link
+      name="front_right_wheel">
       <inertial>
         <origin
@@ -393,5 +394,5 @@
     </link>
     <joint
-      name="Front_Right_Shaft"
+      name="front_right_wheel_joint"
       type="continuous">
       <origin
@@ -399,12 +400,12 @@
         rpy="0 0.0083213 1.5708" />
       <parent
-        link="Right_Leg" />
-      <child
-        link="Front_Right_Wheel" />
-      <axis
-        xyz="0 1 0" />
-    </joint>
-    <link
-      name="Back_Right_Wheel">
+        link="right_rocker" />
+      <child
+        link="front_right_wheel" />
+      <axis
+        xyz="0 1 0" />
+    </joint>
+    <link
+      name="back_right_wheel">
       <inertial>
         <origin
@@ -454,5 +455,5 @@
     </link>
     <joint
-      name="Back_Right_Shaft"
+      name="back_right_wheel_joint"
       type="continuous">
       <origin
@@ -460,7 +461,7 @@
         rpy="0 0.0083213063996962 1.57079632679444" />
       <parent
-        link="Right_Leg" />
-      <child
-        link="Back_Right_Wheel" />
+        link="right_rocker" />
+      <child
+        link="back_right_wheel" />
       <axis
         xyz="0 1 0" />
@@ -469,23 +470,23 @@
       <material>Gazebo/Grey</material>
     </gazebo>
-    <gazebo reference="Left_Leg">
+    <gazebo reference="left_rocker">
       <material>Gazebo/Grey</material>
     </gazebo>
-    <gazebo reference="Front_Left_Wheel">
+    <gazebo reference="front_left_wheel">
       <material>Gazebo/Black</material>
     </gazebo>
-    <gazebo reference="Back_Left_Wheel">
+    <gazebo reference="back_left_wheel">
       <material>Gazebo/Black</material>
     </gazebo>
-    <gazebo reference="Differential_Bar">
+    <gazebo reference="differential_bar">
       <material>Gazebo/Grey</material>
     </gazebo>
-    <gazebo reference="Right_Leg">
+    <gazebo reference="right_rocker">
       <material>Gazebo/Grey</material>
     </gazebo>
-    <gazebo reference="Front_Right_Wheel">
+    <gazebo reference="front_right_wheel">
       <material>Gazebo/Black</material>
     </gazebo>
-    <gazebo reference="Back_Right_Wheel">
+    <gazebo reference="back_right_wheel">
       <material>Gazebo/Black</material>
     </gazebo>
