Commit message: Fix joint origins

File: urc_hw_description/urdf/ros2_control.xacro (robot description, xacro)
@@ -12,8 +12,8 @@
           <state_interface name="position" />
         </joint>
-        <!-- <joint name="Differential_Bar"> -->
-        <!--   <state_interface name="velocity" /> -->
-        <!--   <state_interface name="position" /> -->
-        <!-- </joint> -->
+        <joint name="differential_bar_joint">
+          <state_interface name="velocity" />
+          <state_interface name="position" />
+        </joint>
         <joint name="right_rocker_joint">
           <state_interface name="velocity" />

File: urc_hw_description/urdf/wallii_drivebase.xacro (robot description, xacro)
@@ -1,7 +1,3 @@
 <?xml version="1.0" encoding="utf-8"?>
-<!-- This URDF was automatically created by SolidWorks to URDF Exporter! Originally created by
-Stephen Brawner (brawner@gmail.com)
-     Commit Version: 1.6.0-4-g7f85cfe  Build Version: 1.6.7995.38578
-     For more information, please see http://wiki.ros.org/sw_urdf_exporter -->
 <robot xmlns:xacro="http://www.ros.org/wiki/xacro">
   <xacro:macro name="drivebase" params="mu mu2">
@@ -64,5 +60,5 @@
       <visual>
         <origin
-          xyz="0 0 0"
+          xyz="0.26 0.128 -0.01"
           rpy="0 0 0" />
         <geometry>
@@ -78,5 +74,5 @@
       <collision>
         <origin
-          xyz="0 0 0"
+          xyz="0.26 0.128 -0.01"
           rpy="0 0 0" />
         <geometry>
@@ -90,6 +86,6 @@
       type="revolute">
       <origin
-        xyz="0 0.01 0"
-        rpy="1.5791 0 0" />
+        xyz="-0.26 0.0 -0.128"
+        rpy="1.5708 0 0" />
       <parent
         link="base_link" />
@@ -97,11 +93,7 @@
         link="left_rocker" />
       <axis
-        xyz="0 1 0" />
-      <limit
-        lower="0"
-        upper="0"
-        effort="0"
-        velocity="0" />
-      <dynamics damping="0.01" friction="0.01" />
+        xyz="-1 0 0" />
+      <limit effort="0.0" lower="-0.24" upper="0.24" velocity="100.0" />
+      <dynamics friction="1.0" damping="0.1" />
     </joint>
     <link
@@ -157,6 +149,6 @@
       type="continuous">
       <origin
-        xyz="-0.35884 -0.36484 -0.34252"
-        rpy="0 -0.0083213 -1.5708" />
+        xyz="-0.1 -0.236 -0.352"
+        rpy="0.0 0.0 -1.5708" />
       <parent
         link="left_rocker" />
@@ -164,5 +156,5 @@
         link="front_left_wheel" />
       <axis
-        xyz="0 1 0" />
+        xyz="0 -1 0" />
     </joint>
     <link
@@ -218,6 +210,6 @@
       type="continuous">
       <origin
-        xyz="-0.35884 -0.35931 0.36866"
-        rpy="0 -1.3867 -1.5708" />
+        xyz="-0.1 -0.232 0.358"
+        rpy="0.0 -1.5708 -1.5708" />
       <parent
         link="left_rocker" />
@@ -225,5 +217,5 @@
         link="back_left_wheel" />
       <axis
-        xyz="0 1 0" />
+        xyz="0 -1 0" />
     </joint>
     <link
@@ -304,5 +296,5 @@
       <visual>
         <origin
-          xyz="0 0 0"
+          xyz="-0.26 0.138 0"
           rpy="0 0 0" />
         <geometry>
@@ -318,5 +310,5 @@
       <collision>
         <origin
-          xyz="0 0 0"
+          xyz="-0.26 0.138 0"
           rpy="0 0 0" />
         <geometry>
@@ -330,6 +322,6 @@
       type="revolute">
       <origin
-        xyz="0 -0.0011403 0.0099997"
-        rpy="1.5791 0 0" />
+        xyz="0.26 0.0 -0.128"
+        rpy="1.5708 0 0" />
       <parent
         link="base_link" />
@@ -337,11 +329,7 @@
         link="right_rocker" />
       <axis
-        xyz="0 1 0" />
-      <limit
-        lower="0"
-        upper="0"
-        effort="0"
-        velocity="0" />
-      <dynamics damping="0.01" friction="0.01" />
+        xyz="1 0 0" />
+      <limit effort="0.0" lower="-0.24" upper="0.24" velocity="100.0" />
+      <dynamics damping="0.1" friction="1.0" />
     </joint>
     <link
@@ -397,6 +385,6 @@
       type="continuous">
       <origin
-        xyz="0.35884 -0.37493 -0.35357"
-        rpy="0 0.0083213 1.5708" />
+        xyz="0.1 -0.2375 -0.35357"
+        rpy="0.0 0.0 1.5708" />
       <parent
         link="right_rocker" />
@@ -458,6 +446,6 @@
       type="continuous">
       <origin
-        xyz="0.358842224999926 -0.369400178446968 0.357603754666081"
-        rpy="0 0.0083213063996962 1.57079632679444" />
+        xyz="0.1 -0.232 0.357603754666081"
+        rpy="0.0 0.0 1.5708" />
       <parent
         link="right_rocker" />

Commit message: remove old arm urdf code

File: urc_hw_description/urdf/ros2_control.xacro (robot description, xacro)
@@ -2,7 +2,5 @@
 <robot xmlns:xacro="http://www.ros.org/wiki/xacro">
   <xacro:macro name="ros2_control"
-    params="use_simulation config_file_path arm_initial_positions_file">
-    <xacro:property name="initial_positions"
-      value="${load_yaml(arm_initial_positions_file)['initial_positions']}" />
+    params="use_simulation config_file_path">
     <xacro:if value="${use_simulation}">
       <ros2_control name="GazeboSystem" type="system">
@@ -74,67 +72,4 @@
           <state_interface name="position" />
         </joint>
-        <joint name="shoulderjoint">
-          <command_interface name="position" />
-          <command_interface name="velocity" />
-          <command_interface name="effort" />
-          <state_interface name="position">
-            <param name="initial_value">${initial_positions['shoulderjoint']}</param>
-          </state_interface>
-          <state_interface name="velocity" />
-        </joint>
-        <joint name="bicepjoint">
-          <command_interface name="position" />
-          <command_interface name="velocity" />
-          <command_interface name="effort" />
-          <state_interface name="position">
-            <param name="initial_value">${initial_positions['bicepjoint']}</param>
-          </state_interface>
-          <state_interface name="velocity" />
-        </joint>
-        <joint name="elbowjoint">
-          <command_interface name="position" />
-          <command_interface name="velocity" />
-          <command_interface name="effort" />
-          <state_interface name="position">
-            <param name="initial_value">${initial_positions['elbowjoint']}</param>
-          </state_interface>
-          <state_interface name="velocity" />
-        </joint>
-        <joint name="wristjoint">
-          <command_interface name="position" />
-          <command_interface name="velocity" />
-          <command_interface name="effort" />
-          <state_interface name="position">
-            <param name="initial_value">${initial_positions['wristjoint']}</param>
-          </state_interface>
-          <state_interface name="velocity" />
-        </joint>
-        <joint name="clawjoint">
-          <command_interface name="position" />
-          <command_interface name="velocity" />
-          <command_interface name="effort" />
-          <state_interface name="position">
-            <param name="initial_value">${initial_positions['clawjoint']}</param>
-          </state_interface>
-          <state_interface name="velocity" />
-        </joint>
-        <joint name="rightgripperjoint">
-          <command_interface name="position" />
-          <command_interface name="velocity" />
-          <command_interface name="effort" />
-          <state_interface name="position">
-            <param name="initial_value">${initial_positions['rightgripperjoint']}</param>
-          </state_interface>
-          <state_interface name="velocity" />
-        </joint>
-        <joint name="leftgripperjoint">
-          <command_interface name="position" />
-          <command_interface name="velocity" />
-          <command_interface name="effort" />
-          <state_interface name="position">
-            <param name="initial_value">${initial_positions['rightgripperjoint']}</param>
-          </state_interface>
-          <state_interface name="velocity" />
-        </joint>
       </ros2_control>
       <gazebo>

File: urc_hw_description/urdf/walli.xacro (robot description, xacro)
@@ -11,5 +11,4 @@
    <!-- <xacro:arm /> -->
    <xacro:ros2_control use_simulation="$(arg use_simulation)"
-      config_file_path="$(find urc_bringup)/config/controller_config.yaml"
-      arm_initial_positions_file="$(find urc_hw_description)/config/initial_positions.yaml" />
+      config_file_path="$(find urc_bringup)/config/controller_config.yaml" />
 </robot>
