Commit message: feat: update block arm v2 model

File: urc_arm/model/arm_v1/walli_arm.urdf (robot description, URDF)
Before this commit: robot walli, 10 links, 9 joints
Links:
- link bicep: geometry collision mesh filename=package://urc_arm_models/urdf/bicep_collision.STL; visual mesh filename=package://urc_arm_models/urdf/bicep.STL
- link claw: geometry collision mesh filename=package://urc_arm_models/urdf/claw_collision.STL; visual mesh filename=package://urc_arm_models/urdf/claw.STL
- link elbow: geometry collision mesh filename=package://urc_arm_models/urdf/elbow_collision.STL; visual mesh filename=package://urc_arm_models/urdf/elbow.STL
- link leftgripper: geometry collision mesh filename=package://urc_arm_models/urdf/leftgripper_collision.STL; visual mesh filename=package://urc_arm_models/urdf/leftgripper.STL
- link rightgripper: geometry collision mesh filename=package://urc_arm_models/urdf/rightgripper_collision.STL; visual mesh filename=package://urc_arm_models/urdf/rightgripper.STL
- link shoulder: geometry collision mesh filename=package://urc_arm_models/urdf/shoulder_collision.STL; visual mesh filename=package://urc_arm_models/urdf/shoulder.STL
- link spine: geometry collision mesh filename=package://urc_arm_models/urdf/spine_collision.STL; visual mesh filename=package://urc_arm_models/urdf/spine.STL
- link wrist: geometry collision mesh filename=package://urc_arm_models/urdf/wrist_collision.STL; visual mesh filename=package://urc_arm_models/urdf/wrist.STL
