Commit message: fix: change urdf files

File: urc_arm_models/urdf/walli_arm_v2_block/robot.urdf (robot description, URDF)
Before this commit: robot walli_arm_v2_block, 7 links, 6 joints
Links:
- added link base_link
- link base_rotator: geometry collision mesh filename=$(find urc_arm_models)/urdf/walli_arm_v2_block/base_rotator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; visual mesh filename=$(find urc_arm_models)/urdf/walli_arm_v2_block/base_rotator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
- link ee_rod: geometry collision mesh filename=$(find urc_arm_models)/urdf/walli_arm_v2_block/ee_rod_colli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; visual mesh filename=$(find urc_arm_models)/urdf/walli_arm_v2_block/ee_rod_visua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
- link ee_rotary: geometry collision mesh filename=$(find urc_arm_models)/urdf/walli_arm_v2_block/ee_rotary_co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; visual mesh filename=$(find urc_arm_models)/urdf/walli_arm_v2_block/ee_rotary_vi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
- link fore_arm: geometry collision mesh filename=$(find urc_arm_models)/urdf/walli_arm_v2_block/fore_arm_col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; visual mesh filename=$(find urc_arm_models)/urdf/walli_arm_v2_block/fore_arm_vis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
- link spine: geometry collision mesh filename=$(find urc_arm_models)/urdf/walli_arm_v2_block/spine_collis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; visual mesh filename=$(find urc_arm_models)/urdf/walli_arm_v2_block/spine_visual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
- link upper_arm: geometry collision mesh filename=$(find urc_arm_models)/urdf/walli_arm_v2_block/upper_arm_co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; visual mesh filename=$(find urc_arm_models)/urdf/walli_arm_v2_block/upper_arm_vi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
Joints:
- added joint base_connection: type fixed, parent base_link, child spine
- joint ee_roll_jont: type revolute -> continuous

Commit message: fix: commit problem

File: urc_arm_models/urdf/walli_arm_v2_block/robot.urdf (robot description, URDF)
Before this commit: robot walli_arm_v2_block, 8 links, 7 joints
Links:
- removed link base_link
- link base_rotator: geometry collision mesh filename=package://urc_arm_models/urdf/walli_arm_v2_block/base_rotat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; visual mesh filename=package://urc_arm_models/urdf/walli_arm_v2_block/base_rotat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
- link ee_rod: geometry collision mesh filename=package://urc_arm_models/urdf/walli_arm_v2_block/ee_rod_col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; visual mesh filename=package://urc_arm_models/urdf/walli_arm_v2_block/ee_rod_vis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
- link ee_rotary: geometry collision mesh filename=package://urc_arm_models/urdf/walli_arm_v2_block/ee_rotary_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; visual mesh filename=package://urc_arm_models/urdf/walli_arm_v2_block/ee_rotary_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
- link fore_arm: geometry collision mesh filename=package://urc_arm_models/urdf/walli_arm_v2_block/fore_arm_c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; visual mesh filename=package://urc_arm_models/urdf/walli_arm_v2_block/fore_arm_v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
- link spine: geometry collision mesh filename=package://urc_arm_models/urdf/walli_arm_v2_block/spine_coll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; visual mesh filename=package://urc_arm_models/urdf/walli_arm_v2_block/spine_visu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
- link upper_arm: geometry collision mesh filename=package://urc_arm_models/urdf/walli_arm_v2_block/upper_arm_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; visual mesh filename=package://urc_arm_models/urdf/walli_arm_v2_block/upper_arm_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
Joints:
- removed joint base_connection
- joint ee_roll_jont: type continuous -> revolute
