Commit message: feat: new mujoco simulator

File: urc_arm_models/urdf/walli_arm_v2_block_mjcf/robot.urdf (robot description, URDF)
Before this commit: robot walli_arm_v2_block, 7 links, 6 joints
Joints:
- removed joint ee_roll_jont
- added joint ee_roll_joint: type revolute, parent fore_arm, child ee_rotary, origin xyz=-0.48539999999999505764 2.664535259100375697e-7 -0.025399999999999842842 rpy=-3.141592653589793116 -1.5707963267948961139 0, axis 0 0 1, limit effort=60 velocity=20
