Commit message: Minor changes

File: leo_description/urdf/macros.xacro (robot description, xacro)
@@ -2,5 +2,5 @@
 <robot xmlns:xacro="http://www.ros.org/wiki/xacro">
   <xacro:macro name="leo"
-               params="default_antenna:=true
+    params="default_antenna:=true
                        rockers_fixed:=false
                        footprint_link:=true
@@ -12,19 +12,19 @@
       <link name="${link_prefix}rocker_${name}_link">
         <inertial>
-          <mass value="1.387336"/>
-          <origin xyz="0 0.01346 -0.06506"/>
+          <mass value="1.387336" />
+          <origin xyz="0 0.01346 -0.06506" />
           <inertia
             ixx="0.002956" ixy="-0.000001489324" ixz="-0.000008103407"
-            iyy="0.02924"  iyz="0.00007112"
-            izz="0.02832"/>
+            iyy="0.02924" iyz="0.00007112"
+            izz="0.02832" />
         </inertial>
         <visual>
           <geometry>
-            <mesh filename="file://$(find leo_description)/models/Rocker.dae"/>
+            <mesh filename="file://$(find leo_description)/models/Rocker.dae" />
           </geometry>
         </visual>
         <collision>
           <geometry>
-            <mesh filename="file://$(find leo_description)/models/Rocker_outline.stl"/>
+            <mesh filename="file://$(find leo_description)/models/Rocker_outline.stl" />
           </geometry>
         </collision>
@@ -34,32 +34,43 @@
       <link name="${link_prefix}wheel_${name}_link">
         <inertial>
-          <mass value="0.283642"/>
-          <origin xyz="0 0.030026 0"/>
+          <mass value="0.283642" />
+          <origin xyz="0 0.030026 0" />
           <inertia
-            ixx="0.000391"  ixy="0.00000123962" ixz="5.52582e-7"
+            ixx="0.000391" ixy="0.00000123962" ixz="5.52582e-7"
             iyy="0.0004716" iyz="-0.000002082042"
-            izz="0.000391"/>
+            izz="0.000391" />
         </inertial>
         <visual>
           <geometry>
-            <mesh filename="file://$(find leo_description)/models/Wheel${model}.dae"/>
+            <mesh filename="file://$(find leo_description)/models/Wheel${model}.dae" />
           </geometry>
         </visual>
         <collision>
-          <origin xyz="0 0.04485 0" rpy="${pi/2} 0 0"/>
-          <geometry>
-            <cylinder radius="0.057" length="0.07"/>
-          </geometry>
-        </collision>
-        <collision>
-          <origin xyz="0 0.04485 0" rpy="${pi/2} 0 0"/>
-          <geometry>
-            <cylinder radius="0.0625" length="0.04"/>
-          </geometry>
-        </collision>
-        <collision>
-          <geometry>
-            <mesh filename="file://$(find leo_description)/models/Wheel_outline.stl"/>
-          </geometry>
+          <origin xyz="0 0.04485 0" rpy="${pi/2} 0 0" />
+          <geometry>
+            <cylinder radius="0.057" length="0.07" />
+          </geometry>
+        </collision>
+        <collision>
+          <origin xyz="0 0.04485 0" rpy="${pi/2} 0 0" />
+          <geometry>
+            <cylinder radius="0.0625" length="0.04" />
+          </geometry>
+        </collision>
+        <collision>
+          <geometry>
+            <mesh filename="file://$(find leo_description)/models/Wheel_outline.stl" />
+          </geometry>
+          <friction>
+            <ode>
+              <mu>10.0</mu>
+              <mu2>10.0</mu2>
+            </ode>
+          </friction>
+          <contact>
+            <ode>
+              <min_depth>0.01</min_depth>
+            </ode>
+          </contact>
         </collision>
       </link>
@@ -68,25 +79,25 @@
       <link name="${link_prefix}wheel_${name}_link">
         <inertial>
-          <mass value="0.672214"/>
-          <origin xyz="0 -0.036852 0"/>
+          <mass value="0.672214" />
+          <origin xyz="0 -0.036852 0" />
           <inertia
-            ixx="0.0009778"  ixy="-8.10228e-7" ixz="3.2e-11"
+            ixx="0.0009778" ixy="-8.10228e-7" ixz="3.2e-11"
             iyy="0.001321" iyz="5.7e-11"
-            izz="0.0009773"/>
+            izz="0.0009773" />
         </inertial>
         <visual>
           <geometry>
-            <mesh filename="file://$(find leo_description)/models/WheelMecanum${model}.dae"/>
+            <mesh filename="file://$(find leo_description)/models/WheelMecanum${model}.dae" />
           </geometry>
         </visual>
         <collision>
-          <origin xyz="0 -0.0317 0" rpy="${pi/2} 0 0"/>
-          <geometry>
-            <cylinder radius="0.0635" length="0.0515"/>
-          </geometry>
-        </collision>
-        <collision>
-          <geometry>
-            <mesh filename="file://$(find leo_description)/models/Mecanum_wheel_outline.stl"/>
+          <origin xyz="0 -0.0317 0" rpy="${pi/2} 0 0" />
+          <geometry>
+            <cylinder radius="0.0635" length="0.0515" />
+          </geometry>
+        </collision>
+        <collision>
+          <geometry>
+            <mesh filename="file://$(find leo_description)/models/Mecanum_wheel_outline.stl" />
           </geometry>
         </collision>
@@ -95,178 +106,178 @@
     <!-- LINKS -->
     <xacro:if value="${footprint_link}">
-      <link name="${link_prefix}base_footprint"/>
+      <link name="${link_prefix}base_footprint" />
     </xacro:if>
     <link name="${link_prefix}base_link">
       <inertial>
-        <mass value="1.584994"/>
-        <origin xyz="-0.019662 0.011643 -0.031802"/>
+        <mass value="3.0" />
+        <origin xyz="-0.019662 0.011643 -0.031802" />
         <inertia
           ixx="0.01042" ixy="0.001177" ixz="-0.0008871"
           iyy="0.01045" iyz="0.0002226"
-          izz="0.01817"/>
+          izz="0.01817" />
       </inertial>
       <visual>
         <geometry>
-          <mesh filename="file://$(find leo_description)/models/Chassis.dae"/>
+          <mesh filename="file://$(find leo_description)/models/Chassis.dae" />
         </geometry>
       </visual>
       <collision>
         <geometry>
-          <mesh filename="file://$(find leo_description)/models/Chassis_outline.stl"/>
+          <mesh filename="file://$(find leo_description)/models/Chassis_outline.stl" />
         </geometry>
       </collision>
     </link>
-    <xacro:rocker_link name="L"/>
-    <xacro:rocker_link name="R"/>
+    <xacro:rocker_link name="L" />
+    <xacro:rocker_link name="R" />
     <xacro:if value="${mecanum_wheels}">
-      <xacro:mecanum_wheel_link name="FL" model="B"/>
-      <xacro:mecanum_wheel_link name="RL" model="A"/>
-      <xacro:mecanum_wheel_link name="FR" model="A"/>
-      <xacro:mecanum_wheel_link name="RR" model="B"/>
+      <xacro:mecanum_wheel_link name="FL" model="B" />
+      <xacro:mecanum_wheel_link name="RL" model="A" />
+      <xacro:mecanum_wheel_link name="FR" model="A" />
+      <xacro:mecanum_wheel_link name="RR" model="B" />
     </xacro:if>
     <xacro:unless value="${mecanum_wheels}">
-      <xacro:wheel_link name="FL" model="A"/>
-      <xacro:wheel_link name="RL" model="A"/>
-      <xacro:wheel_link name="FR" model="B"/>
-      <xacro:wheel_link name="RR" model="B"/>
+      <xacro:wheel_link name="FL" model="A" />
+      <xacro:wheel_link name="RL" model="A" />
+      <xacro:wheel_link name="FR" model="B" />
+      <xacro:wheel_link name="RR" model="B" />
     </xacro:unless>
     <xacro:if value="${default_antenna}">
       <link name="${link_prefix}antenna_link">
         <inertial>
-          <mass value="0.001237"/>
-          <origin xyz="0 0 0.028828"/>
+          <mass value="0.001237" />
+          <origin xyz="0 0 0.028828" />
           <inertia
             ixx="2.5529e-7" ixy="0.0" ixz="0.0"
             iyy="2.5529e-7" iyz="0.0"
-            izz="1.354e-8"/>
+            izz="1.354e-8" />
         </inertial>
         <visual>
           <geometry>
-            <mesh filename="file://$(find leo_description)/models/Antenna.dae"/>
+            <mesh filename="file://$(find leo_description)/models/Antenna.dae" />
           </geometry>
         </visual>
         <collision>
-          <origin xyz="0 0 0.028"/>
-          <geometry>
-            <cylinder radius="0.0055" length="0.056"/>
+          <origin xyz="0 0 0.028" />
+          <geometry>
+            <cylinder radius="0.0055" length="0.056" />
           </geometry>
         </collision>
       </link>
     </xacro:if>
-    <link name="${link_prefix}camera_frame"/>
-    <link name="${link_prefix}camera_optical_frame"/>
-    <link name="${link_prefix}imu_frame"/>
+    <link name="${link_prefix}camera_frame" />
+    <link name="${link_prefix}camera_optical_frame" />
+    <link name="${link_prefix}imu_frame" />
     <!-- JOINTS -->
     <xacro:if value="${footprint_link}">
       <joint name="${joint_prefix}base_joint" type="fixed">
-        <origin xyz="0 0 0.19783" rpy="0 0 0"/>
-        <parent link="${link_prefix}base_footprint"/>
-        <child link="${link_prefix}base_link"/>
+        <origin xyz="0 0 0.19783" rpy="0 0 0" />
+        <parent link="${link_prefix}base_footprint" />
+        <child link="${link_prefix}base_link" />
       </joint>
     </xacro:if>
     <xacro:if value="${rockers_fixed}">
-      <xacro:property name="rockers_joint_type" value="fixed"/>
+      <xacro:property name="rockers_joint_type" value="fixed" />
     </xacro:if>
     <xacro:unless value="${rockers_fixed}">
-      <xacro:property name="rockers_joint_type" value="revolute"/>
+      <xacro:property name="rockers_joint_type" value="revolute" />
     </xacro:unless>
     <joint name="${joint_prefix}rocker_L_joint" type="${rockers_joint_type}">
-      <origin xyz="0.00263 0.14167 -0.04731" rpy="0 0 ${pi}"/>
-      <parent link="${link_prefix}base_link"/>
-      <child link="${link_prefix}rocker_L_link"/>
-      <axis xyz="0 1 0"/>
-      <limit effort="100.0" lower="-0.24" upper="0.24" velocity="100.0"/>
-      <dynamics friction="1.0" damping="0.1"/>
+      <origin xyz="0.00263 0.14167 -0.04731" rpy="0 0 ${pi}" />
+      <parent link="${link_prefix}base_link" />
+      <child link="${link_prefix}rocker_L_link" />
+      <axis xyz="0 1 0" />
+      <limit effort="100.0" lower="-0.24" upper="0.24" velocity="100.0" />
+      <dynamics friction="1.0" damping="0.1" />
     </joint>
     <joint name="${joint_prefix}rocker_R_joint" type="${rockers_joint_type}">
-      <origin xyz="0.00263 -0.14167 -0.04731" rpy="0 0 0"/>
-      <parent link="${link_prefix}base_link"/>
-      <child link="${link_prefix}rocker_R_link"/>
-      <axis xyz="0 1 0"/>
-      <limit effort="100.0" lower="-0.24" upper="0.24" velocity="100.0"/>
-      <dynamics friction="1.0" damping="0.1"/>
-      <mimic joint="rocker_L_joint"/>
+      <origin xyz="0.00263 -0.14167 -0.04731" rpy="0 0 0" />
+      <parent link="${link_prefix}base_link" />
+      <child link="${link_prefix}rocker_R_link" />
+      <axis xyz="0 1 0" />
+      <limit effort="100.0" lower="-0.24" upper="0.24" velocity="100.0" />
+      <dynamics friction="1.0" damping="0.1" />
+      <mimic joint="rocker_L_joint" />
     </joint>
     <joint name="${joint_prefix}wheel_FL_joint" type="continuous">
       <xacro:if value="${mecanum_wheels}">
-        <origin xyz="-0.15256 -0.00884 -0.08802" rpy="0 0 0"/>
+        <origin xyz="-0.15256 -0.00884 -0.08802" rpy="0 0 0" />
       </xacro:if>
       <xacro:unless value="${mecanum_wheels}">
-        <origin xyz="-0.15256 -0.08214 -0.08802" rpy="0 0 0"/>
+        <origin xyz="-0.15256 -0.08214 -0.08802" rpy="0 0 0" />
       </xacro:unless>
-      <parent link="${link_prefix}rocker_L_link"/>
-      <child link="${link_prefix}wheel_FL_link"/>
-      <axis xyz="0 -1 0"/>
-      <limit effort="2.0" velocity="6.0"/>
-      <dynamics friction="0.3125" damping="0.1"/>
+      <parent link="${link_prefix}rocker_L_link" />
+      <child link="${link_prefix}wheel_FL_link" />
+      <axis xyz="0 -1 0" />
+      <limit effort="2.0" velocity="6.0" />
+      <dynamics friction="0.3125" damping="0.1" />
     </joint>
     <joint name="${joint_prefix}wheel_RL_joint" type="continuous">
       <xacro:if value="${mecanum_wheels}">
-        <origin xyz="0.15256 -0.00884 -0.08802" rpy="0 0 0"/>
+        <origin xyz="0.15256 -0.00884 -0.08802" rpy="0 0 0" />
       </xacro:if>
       <xacro:unless value="${mecanum_wheels}">
-        <origin xyz="0.15256 -0.08214 -0.08802" rpy="0 0 0"/>
+        <origin xyz="0.15256 -0.08214 -0.08802" rpy="0 0 0" />
       </xacro:unless>
-      <parent link="${link_prefix}rocker_L_link"/>
-      <child link="${link_prefix}wheel_RL_link"/>
-      <axis xyz="0 -1 0"/>
-      <limit effort="2.0" velocity="6.0"/>
-      <dynamics friction="0.3125" damping="0.1"/>
+      <parent link="${link_prefix}rocker_L_link" />
+      <child link="${link_prefix}wheel_RL_link" />
+      <axis xyz="0 -1 0" />
+      <limit effort="2.0" velocity="6.0" />
+      <dynamics friction="0.3125" damping="0.1" />
     </joint>
     <joint name="${joint_prefix}wheel_FR_joint" type="continuous">
       <xacro:if value="${mecanum_wheels}">
-        <origin xyz="0.15256 -0.00884 -0.08802" rpy="0 0 0"/>
+        <origin xyz="0.15256 -0.00884 -0.08802" rpy="0 0 0" />
       </xacro:if>
       <xacro:unless value="${mecanum_wheels}">
-        <origin xyz="0.15256 -0.08214 -0.08802" rpy="0 0 0"/>
+        <origin xyz="0.15256 -0.08214 -0.08802" rpy="0 0 0" />
       </xacro:unless>
-      <parent link="${link_prefix}rocker_R_link"/>
-      <child link="${link_prefix}wheel_FR_link"/>
-      <axis xyz="0 1 0"/>
-      <limit effort="2.0" velocity="6.0"/>
-      <dynamics friction="0.3125" damping="0.1"/>
+      <parent link="${link_prefix}rocker_R_link" />
+      <child link="${link_prefix}wheel_FR_link" />
+      <axis xyz="0 1 0" />
+      <limit effort="2.0" velocity="6.0" />
+      <dynamics friction="0.3125" damping="0.1" />
     </joint>
     <joint name="${joint_prefix}wheel_RR_joint" type="continuous">
       <xacro:if value="${mecanum_wheels}">
-        <origin xyz="-0.15256 -0.00884 -0.08802" rpy="0 0 0"/>
+        <origin xyz="-0.15256 -0.00884 -0.08802" rpy="0 0 0" />
       </xacro:if>
       <xacro:unless value="${mecanum_wheels}">
-        <origin xyz="-0.15256 -0.08214 -0.08802" rpy="0 0 0"/>
+        <origin xyz="-0.15256 -0.08214 -0.08802" rpy="0 0 0" />
       </xacro:unless>
-      <parent link="${link_prefix}rocker_R_link"/>
-      <child link="${link_prefix}wheel_RR_link"/>
-      <axis xyz="0 1 0"/>
-      <limit effort="2.0" velocity="6.0"/>
-      <dynamics friction="0.3125" damping="0.1"/>
+      <parent link="${link_prefix}rocker_R_link" />
+      <child link="${link_prefix}wheel_RR_link" />
+      <axis xyz="0 1 0" />
+      <limit effort="2.0" velocity="6.0" />
+      <dynamics friction="0.3125" damping="0.1" />
     </joint>
     <xacro:if value="${default_antenna}">
       <joint name="${joint_prefix}antenna_joint" type="fixed">
-        <origin xyz="-0.0052 0.056 -0.0065" rpy="0 0 0"/>
-        <parent link="${link_prefix}base_link"/>
-        <child link="${link_prefix}antenna_link"/>
+        <origin xyz="-0.0052 0.056 -0.0065" rpy="0 0 0" />
+        <parent link="${link_prefix}base_link" />
+        <child link="${link_prefix}antenna_link" />
       </joint>
     </xacro:if>
     <joint name="${joint_prefix}camera_joint" type="fixed">
-      <origin xyz="0.0971 0 -0.0427" rpy="0 0.2094 0"/>
-      <parent link="${link_prefix}base_link"/>
-      <child link="${link_prefix}camera_frame"/>
+      <origin xyz="0.0971 0 -0.0427" rpy="0 0.2094 0" />
+      <parent link="${link_prefix}base_link" />
+      <child link="${link_prefix}camera_frame" />
     </joint>
     <joint name="${joint_prefix}camera_optical_joint" type="fixed">
-      <origin xyz="0 0 0" rpy="-${pi/2} 0.0 -${pi/2}"/>
-      <parent link="${link_prefix}camera_frame"/>
-      <child link="${link_prefix}camera_optical_frame"/>
+      <origin xyz="0 0 0" rpy="-${pi/2} 0.0 -${pi/2}" />
+      <parent link="${link_prefix}camera_frame" />
+      <child link="${link_prefix}camera_optical_frame" />
     </joint>
     <joint name="${joint_prefix}imu_joint" type="fixed">
-      <origin xyz="${imu_translation}" rpy="0 0 0"/>
-      <parent link="${link_prefix}base_link"/>
-      <child link="${link_prefix}imu_frame"/>
+      <origin xyz="${imu_translation}" rpy="0 0 0" />
+      <parent link="${link_prefix}base_link" />
+      <child link="${link_prefix}imu_frame" />
     </joint>
   </xacro:macro>
   <!-- LEO GAZEBO -->
   <xacro:macro name="leo_gazebo"
-               params="robot_ns:='''">
-    <xacro:property name="link_prefix" value=""/>
+    params="robot_ns:='''">
+    <xacro:property name="link_prefix" value="" />
     <xacro:if value="${robot_ns != '' and robot_ns != '/'}">
-      <xacro:property name="link_prefix" value="${robot_ns}/"/>
+      <xacro:property name="link_prefix" value="${robot_ns}/" />
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
Commit message: Refactor behaviors

File: leo_description/urdf/macros.xacro (robot description, xacro)
@@ -433,5 +433,5 @@
     </gazebo>
     <!-- lidar-->
-    <link name="lidar_link">
+    <!-- <link name="lidar_link">
       <inertial>
         <origin xyz="0 0 0" rpy="0 0 0" />
@@ -496,5 +496,5 @@
         </plugin>
       </sensor>
-    </gazebo>
+    </gazebo> -->
     <!-- camera -->
     <gazebo reference="${link_prefix}camera_frame">
