Commit message: added gps and put all sensor stuff and related plugins in their own xacro files for neatness

File: urc_hw_description/urdf/simplified_swerve/simplified_swerve.urdf.xacro (robot description, xacro)
@@ -10,4 +10,5 @@
   <!-- Include the ROS2 control interfaces -->
   <xacro:include filename="$(find urc_hw_description)/urdf/simplified_swerve/simplified_swerve_ros2_control.xacro" />
+  <!-- Include Sensor interfaces -->
   <!-- Define parameters with defaults -->
   <xacro:arg name="use_sim" default="false" />
@@ -16,4 +17,6 @@
   <!-- Add ROS2 control interfaces -->
   <xacro:simplified_swerve_ros2_control use_sim="$(arg use_sim)" />
+  <!-- Add Sensor interfaces -->
+  <xacro:include filename="$(find urc_hw_description)/urdf/simplified_swerve/simplified_swerve_sensors.xacro" />
   <!-- Add world link for simulation -->
   <xacro:if value="$(arg use_sim)">

File: urc_hw_description/urdf/simplified_swerve/simplified_swerve_macro.xacro (robot description, xacro)
@@ -47,116 +47,4 @@
       </collision>
     </link>
-    <!-- Lidar Link -->
-    <link name="lidar_link">
-      <inertial>
-        <mass value="0.1"/>
-        <origin xyz="0 0 0" rpy="0 0 0"/>
-        <inertia ixx="0.001" ixy="0" ixz="0" iyy="0.001" iyz="0" izz="0.001"/>
-      </inertial>
-      <visual>
-        <origin xyz="0 0 0" rpy="0 0 0"/>
-        <geometry>
-          <cylinder radius="0.03" length="0.05"/>
-        </geometry>
-        <material name="black">
-          <color rgba="0 0 0 1"/>
-        </material>
-      </visual>
-    </link>
-    <!-- Joint to attach lidar to base -->
-    <joint name="lidar_joint" type="fixed">
-      <parent link="base_Link"/>
-      <child link="lidar_link"/>
-      <origin xyz="0 0 0.025" rpy="0 0 0"/>
-    </joint>
-    <!-- Gazebo plugin for lidar -->
-    <gazebo reference="lidar_link">
-      <sensor name="lidar" type="gpu_lidar">
-        <pose>0 0 0 0 0 0</pose>
-        <always_on>true</always_on>
-        <visualize>true</visualize>
-        <update_rate>10</update_rate>
-        <topic>scan</topic>
-        <gz_frame_id>lidar_link</gz_frame_id>
-        <lidar>
-          <scan>
-            <horizontal>
-              <samples>720</samples>
-              <resolution>1</resolution>
-              <min_angle>-3.14</min_angle>
-              <max_angle>3.14</max_angle>
-            </horizontal>
-          </scan>
-          <range>
-            <min>0.05</min>
-            <max>10.0</max>
-            <resolution>0.01</resolution>
-          </range>
-          <noise>
-            <type>gaussian</type>
-            <mean>0.0</mean>
-            <stddev>0.01</stddev>
-          </noise>
-          <frame_id>lidar_link</frame_id>
-        </lidar>
-      </sensor>
-    </gazebo>
-    <link name="imu_link">
-      <inertial>
-        <mass value="0.01"/>
-        <origin xyz="0 0 0" rpy="0 0 0"/>
-        <inertia ixx="0.001" ixy="0" ixz="0" iyy="0.001" iyz="0" izz="0.001"/>
-      </inertial>
-      <collision name="imu_collision">
-        <geometry>
-          <box>
-            <size>0.001 0.001 0.001</size>  <!-- tiny collision -->
-          </box>
-        </geometry>
-      </collision>
-      <visual name="imu_visual">
-        <geometry>
-          <box>
-            <size>0.001 0.001 0.001</size>
-          </box>
-        </geometry>
-      </visual>
-    </link>
-    <joint name="imu_joint" type="fixed">
-      <parent link="base_Link"/>
-      <child link="imu_link"/>
-      <origin xyz="0.1 0 0" rpy="0 0 0"/>
-    </joint>
-    <gazebo reference="imu_link">
-      <sensor name="imu_sensor" type="imu">
-        <always_on>1</always_on>
-        <update_rate>100</update_rate>
-        <visualize>true</visualize>
-        <topic>/imu/data_raw</topic>
-        <imu>
-          <orientation>
-            <noise>
-              <type>gaussian</type>
-              <mean>0.0</mean>
-              <stddev>0.0001</stddev>
-            </noise>
-          </orientation>
-          <angular_velocity>
-            <noise>
-              <type>gaussian</type>
-              <mean>0.0</mean>
-              <stddev>0.0005</stddev>
-            </noise>
-          </angular_velocity>
-          <linear_acceleration>
-            <noise>
-              <type>gaussian</type>
-              <mean>0.0</mean>
-              <stddev>0.01</stddev>
-            </noise>
-          </linear_acceleration>
-        </imu>
-      </sensor>
-    </gazebo>
     <link
       name="L_Rocker_Link">

Commit message: controllers load up!

File: urc_hw_description/urdf/simplified_swerve/simplified_swerve.urdf.xacro (robot description, xacro)
@@ -17,12 +17,12 @@
   <xacro:simplified_swerve_ros2_control use_sim="$(arg use_sim)" />
   <!-- Add world link for simulation -->
-  <xacro:if value="$(arg use_sim)">
-    <link name="world" />
-    <joint name="world_to_base" type="fixed">
-      <parent link="world" />
-      <child link="base_Link" />
-      <origin xyz="0 0 0" rpy="0 0 0" />
-    </joint>
-  </xacro:if>
+  <!-- <xacro:if value="$(arg use_sim)"> -->
+  <!--   <link name="world" /> -->
+  <!--   <joint name="world_to_base" type="fixed"> -->
+  <!--     <parent link="world" /> -->
+  <!--     <child link="base_Link" /> -->
+  <!--     <origin xyz="0 0 0" rpy="0 0 0" /> -->
+  <!--   </joint> -->
+  <!-- </xacro:if> -->
   <!-- Add Gazebo-specific elements for simulation -->
   <xacro:if value="$(arg use_sim)">

Commit message: Merging feat/new-sim into main (#296)
* generate walli.urdf

* Initial simulation framework.

* Walli spawns in leo_world.sdf

* Physics integration

* Additional physics

* Integrate with swervedrive

* modell loads in gz sim

* Controller config file for new sim

* Initial controller config

* Test Controllers Configured

* Updated launch file

* add controller manager to sim launch

* fix controller manager in sim

* controller manager works

* controllers load up!

* ground plane

* urc_nanopb new CMakeList

* added marsyard2020 terrain, rover not appearing anymore?

* marsyard2020 terrain works with walli

* parameter for selecting world type

* fix wheel placement in urdf

* modified some terrain parameters

* Rename file convention

---------

Co-authored-by: Mrinal Jain <2mrinaljain@gmail.com>
Co-authored-by: Marvin Ren <mavren22@gmail.com>

File: urc_hw_description/urdf/simplified_swerve/simplified_swerve.urdf.xacro (robot description, xacro)
@@ -17,22 +17,14 @@
   <xacro:simplified_swerve_ros2_control use_sim="$(arg use_sim)" />
   <!-- Add world link for simulation -->
-  <xacro:if value="$(arg use_sim)">
-    <link name="world" />
-    <joint name="world_to_base" type="fixed">
-      <parent link="world" />
-      <child link="base_Link" />
-      <origin xyz="0 0 0" rpy="0 0 0" />
-    </joint>
-  </xacro:if>
+  <!-- <xacro:if value="$(arg use_sim)"> -->
+  <!--   <link name="world" /> -->
+  <!--   <joint name="world_to_base" type="fixed"> -->
+  <!--     <parent link="world" /> -->
+  <!--     <child link="base_Link" /> -->
+  <!--     <origin xyz="0 0 0" rpy="0 0 0" /> -->
+  <!--   </joint> -->
+  <!-- </xacro:if> -->
   <!-- Add Gazebo-specific elements for simulation -->
   <xacro:if value="$(arg use_sim)">
-    <!-- Gazebo world plugin -->
-    <gazebo>
-      <plugin filename="libgazebo_ros_clock.so" name="gazebo_ros_clock">
-        <ros>
-          <remapping>clock:=/clock</remapping>
-        </ros>
-      </plugin>
-    </gazebo>
     <!-- Gazebo physics settings -->
     <gazebo>

File: urc_hw_description/urdf/simplified_swerve/simplified_swerve_macro.xacro (robot description, xacro)
@@ -7,4 +7,12 @@
   <!-- Define the simplified swerve drive macro -->
   <xacro:macro name="simplified_swerve">
+  <!-- replacing package:// -->
+  <xacro:property name="package_path" value="$(find urc_hw_description)"/>
+  <!-- Wheel Cylinder Geometry -->
+  <xacro:property name="wheel_radius" value="0.119888" />
+  <xacro:property name="wheel_length" value="0.0762" />
+  <!-- remove wheel_origin_xyz if not needed -->
+  <xacro:property name="wheel_origin_xyz_left" value="0 0.0381 0" />
+  <xacro:property name="wheel_origin_xyz_right" value="0 -0.0381 0" />
     <link
       name="base_Link">
@@ -29,19 +37,19 @@
         <geometry>
           <mesh
-            filename="package://urc_hw_description/meshes/simplified_swerve/Base_Link.STL" />
-        </geometry>
-        <material
-          name="">
-          <color
-            rgba="0.792156862745098 0.819607843137255 0.933333333333333 1" />
-        </material>
-      </visual>
-      <collision>
-        <origin
-          xyz="0 0 0"
-          rpy="0 0 0" />
-        <geometry>
-          <mesh
-            filename="package://urc_hw_description/meshes/simplified_swerve/Base_Link.STL" />
+            filename="${package_path}/models/simplified_swerve/Base_Link.STL" />
+        </geometry>
+        <material
+          name="">
+          <color
+            rgba="0.792156862745098 0.819607843137255 0.933333333333333 1" />
+        </material>
+      </visual>
+      <collision>
+        <origin
+          xyz="0 0 0"
+          rpy="0 0 0" />
+        <geometry>
+          <mesh
+            filename="${package_path}/models/simplified_swerve/Base_Link.STL" />
         </geometry>
       </collision>
@@ -69,19 +77,19 @@
         <geometry>
           <mesh
-            filename="package://urc_hw_description/meshes/simplified_swerve/L_Rocker_Link.STL" />
-        </geometry>
-        <material
-          name="">
-          <color
-            rgba="0.792156862745098 0.819607843137255 0.933333333333333 1" />
-        </material>
-      </visual>
-      <collision>
-        <origin
-          xyz="0 0 0"
-          rpy="0 0 0" />
-        <geometry>
-          <mesh
-            filename="package://urc_hw_description/meshes/simplified_swerve/L_Rocker_Link.STL" />
+            filename="${package_path}/models/simplified_swerve/L_Rocker_Link.STL" />
+        </geometry>
+        <material
+          name="">
+          <color
+            rgba="0.792156862745098 0.819607843137255 0.933333333333333 1" />
+        </material>
+      </visual>
+      <collision>
+        <origin
+          xyz="0 0 0"
+          rpy="0 0 0" />
+        <geometry>
+          <mesh
+            filename="${package_path}/models/simplified_swerve/L_Rocker_Link.STL" />
         </geometry>
       </collision>
@@ -127,19 +135,19 @@
         <geometry>
           <mesh
-            filename="package://urc_hw_description/meshes/simplified_swerve/FL_Swivel_Link.STL" />
-        </geometry>
-        <material
-          name="">
-          <color
-            rgba="0.792156862745098 0.819607843137255 0.933333333333333 1" />
-        </material>
-      </visual>
-      <collision>
-        <origin
-          xyz="0 0 0"
-          rpy="0 0 0" />
-        <geometry>
-          <mesh
-            filename="package://urc_hw_description/meshes/simplified_swerve/FL_Swivel_Link.STL" />
+            filename="${package_path}/models/simplified_swerve/FL_Swivel_Link.STL" />
+        </geometry>
+        <material
+          name="">
+          <color
+            rgba="0.792156862745098 0.819607843137255 0.933333333333333 1" />
+        </material>
+      </visual>
+      <collision>
+        <origin
+          xyz="0 0 0"
+          rpy="0 0 0" />
+        <geometry>
+          <mesh
+            filename="${package_path}/models/simplified_swerve/FL_Swivel_Link.STL" />
         </geometry>
       </collision>
@@ -167,5 +175,5 @@
       <inertial>
         <origin
-          xyz="0 0.0381000000000001 1.38777878078145E-17"
+          xyz="${wheel_origin_xyz_left}"
           rpy="0 0 0" />
         <mass
@@ -181,23 +189,21 @@
       <visual>
         <origin
-          xyz="0 0 0"
-          rpy="0 0 0" />
-        <geometry>
-          <mesh
-            filename="package://urc_hw_description/meshes/simplified_swerve/FL_Wheel_Link.STL" />
-        </geometry>
-        <material
-          name="">
-          <color
-            rgba="0.792156862745098 0.819607843137255 0.933333333333333 1" />
-        </material>
-      </visual>
-      <collision>
-        <origin
-          xyz="0 0 0"
-          rpy="0 0 0" />
-        <geometry>
-          <mesh
-            filename="package://urc_hw_description/meshes/simplified_swerve/FL_Wheel_Link.STL" />
+          xyz="${wheel_origin_xyz_left}"
+          rpy="${pi/2} 0 0" />
+        <geometry>
+          <cylinder radius="${wheel_radius}"  length="${wheel_length}" />
+        </geometry>
+        <material
+          name="">
+          <color
+            rgba="0.792156862745098 0.819607843137255 0.933333333333333 1" />
+        </material>
+      </visual>
+      <collision>
+        <origin
+          xyz="${wheel_origin_xyz_left}"
+          rpy="${pi/2} 0 0" />
+        <geometry>
+          <cylinder radius="${wheel_radius}"  length="${wheel_length}" />
         </geometry>
       </collision>
@@ -238,19 +244,19 @@
         <geometry>
           <mesh
-            filename="package://urc_hw_description/meshes/simplified_swerve/BL_Swivel_Link.STL" />
-        </geometry>
-        <material
-          name="">
-          <color
-            rgba="0.792156862745098 0.819607843137255 0.933333333333333 1" />
-        </material>
-      </visual>
-      <collision>
-        <origin
-          xyz="0 0 0"
-          rpy="0 0 0" />
-        <geometry>
-          <mesh
-            filename="package://urc_hw_description/meshes/simplified_swerve/BL_Swivel_Link.STL" />
+            filename="${package_path}/models/simplified_swerve/BL_Swivel_Link.STL" />
+        </geometry>
+        <material
+          name="">
+          <color
+            rgba="0.792156862745098 0.819607843137255 0.933333333333333 1" />
+        </material>
+      </visual>
+      <collision>
+        <origin
+          xyz="0 0 0"
+          rpy="0 0 0" />
+        <geometry>
+          <mesh
+            filename="${package_path}/models/simplified_swerve/BL_Swivel_Link.STL" />
         </geometry>
       </collision>
@@ -278,5 +284,5 @@
       <inertial>
         <origin
-          xyz="0 0.0380999942740809 -2.08881547555939E-05"
+          xyz="${wheel_origin_xyz_left}"
           rpy="0 0 0" />
         <mass
@@ -292,23 +298,21 @@
       <visual>
         <origin
-          xyz="0 0 0"
-          rpy="0 0 0" />
-        <geometry>
-          <mesh
-            filename="package://urc_hw_description/meshes/simplified_swerve/BL_Wheel_Link.STL" />
-        </geometry>
-        <material
-          name="">
-          <color
-            rgba="0.792156862745098 0.819607843137255 0.933333333333333 1" />
-        </material>
-      </visual>
-      <collision>
-        <origin
-          xyz="0 0 0"
-          rpy="0 0 0" />
-        <geometry>
-          <mesh
-            filename="package://urc_hw_description/meshes/simplified_swerve/BL_Wheel_Link.STL" />
+          xyz="${wheel_origin_xyz_left}"
+          rpy="${pi/2} 0 0" />
+        <geometry>
+          <cylinder radius="${wheel_radius}"  length="${wheel_length}" />
+        </geometry>
+        <material
+          name="">
+          <color
+            rgba="0.792156862745098 0.819607843137255 0.933333333333333 1" />
+        </material>
+      </visual>
+      <collision>
+        <origin
+          xyz="${wheel_origin_xyz_left}"
+          rpy="${pi/2} 0 0" />
+        <geometry>
+          <cylinder radius="${wheel_radius}"  length="${wheel_length}" />
         </geometry>
       </collision>
@@ -349,19 +353,19 @@
         <geometry>
           <mesh
-            filename="package://urc_hw_description/meshes/simplified_swerve/R_Rocker_Link.STL" />
-        </geometry>
-        <material
-          name="">
-          <color
-            rgba="0.792156862745098 0.819607843137255 0.933333333333333 1" />
-        </material>
-      </visual>
-      <collision>
-        <origin
-          xyz="0 0 0"
-          rpy="0 0 0" />
-        <geometry>
-          <mesh
-            filename="package://urc_hw_description/meshes/simplified_swerve/R_Rocker_Link.STL" />
+            filename="${package_path}/models/simplified_swerve/R_Rocker_Link.STL" />
+        </geometry>
+        <material
+          name="">
+          <color
+            rgba="0.792156862745098 0.819607843137255 0.933333333333333 1" />
+        </material>
+      </visual>
+      <collision>
+        <origin
+          xyz="0 0 0"
+          rpy="0 0 0" />
+        <geometry>
+          <mesh
+            filename="${package_path}/models/simplified_swerve/R_Rocker_Link.STL" />
         </geometry>
       </collision>
@@ -407,19 +411,19 @@
         <geometry>
           <mesh
-            filename="package://urc_hw_description/meshes/simplified_swerve/FR_Swivel_Link.STL" />
-        </geometry>
-        <material
-          name="">
-          <color
-            rgba="0.792156862745098 0.819607843137255 0.933333333333333 1" />
-        </material>
-      </visual>
-      <collision>
-        <origin
-          xyz="0 0 0"
-          rpy="0 0 0" />
-        <geometry>
-          <mesh
-            filename="package://urc_hw_description/meshes/simplified_swerve/FR_Swivel_Link.STL" />
+            filename="${package_path}/models/simplified_swerve/FR_Swivel_Link.STL" />
+        </geometry>
+        <material
+          name="">
+          <color
+            rgba="0.792156862745098 0.819607843137255 0.933333333333333 1" />
+        </material>
+      </visual>
+      <collision>
+        <origin
+          xyz="0 0 0"
+          rpy="0 0 0" />
+        <geometry>
+          <mesh
+            filename="${package_path}/models/simplified_swerve/FR_Swivel_Link.STL" />
         </geometry>
       </collision>
@@ -447,5 +451,5 @@
       <inertial>
         <origin
-          xyz="0 -0.0381 6.93889390390723E-18"
+          xyz="${wheel_origin_xyz_right}"
           rpy="0 0 0" />
         <mass
@@ -461,23 +465,21 @@
       <visual>
         <origin
-          xyz="0 0 0"
-          rpy="0 0 0" />
-        <geometry>
-          <mesh
-            filename="package://urc_hw_description/meshes/simplified_swerve/FR_Wheel_Link.STL" />
-        </geometry>
-        <material
-          name="">
-          <color
-            rgba="0.792156862745098 0.819607843137255 0.933333333333333 1" />
-        </material>
-      </visual>
-      <collision>
-        <origin
-          xyz="0 0 0"
-          rpy="0 0 0" />
-        <geometry>
-          <mesh
-            filename="package://urc_hw_description/meshes/simplified_swerve/FR_Wheel_Link.STL" />
+          xyz="${wheel_origin_xyz_right}"
+          rpy="${pi/2} 0 0" />
+        <geometry>
+          <cylinder radius="${wheel_radius}"  length="${wheel_length}" />
+        </geometry>
+        <material
+          name="">
+          <color
+            rgba="0.792156862745098 0.819607843137255 0.933333333333333 1" />
+        </material>
+      </visual>
+      <collision>
+        <origin
+          xyz="${wheel_origin_xyz_right}"
+          rpy="${pi/2} 0 0" />
+        <geometry>
+          <cylinder radius="${wheel_radius}"  length="${wheel_length}" />
         </geometry>
       </collision>
@@ -518,19 +520,19 @@
         <geometry>
           <mesh
-            filename="package://urc_hw_description/meshes/simplified_swerve/BR_Swivel_Link.STL" />
-        </geometry>
-        <material
-          name="">
-          <color
-            rgba="0.792156862745098 0.819607843137255 0.933333333333333 1" />
-        </material>
-      </visual>
-      <collision>
-        <origin
-          xyz="0 0 0"
-          rpy="0 0 0" />
-        <geometry>
-          <mesh
-            filename="package://urc_hw_description/meshes/simplified_swerve/BR_Swivel_Link.STL" />
+            filename="${package_path}/models/simplified_swerve/BR_Swivel_Link.STL" />
+        </geometry>
+        <material
+          name="">
+          <color
+            rgba="0.792156862745098 0.819607843137255 0.933333333333333 1" />
+        </material>
+      </visual>
+      <collision>
+        <origin
+          xyz="0 0 0"
+          rpy="0 0 0" />
+        <geometry>
+          <mesh
+            filename="${package_path}/models/simplified_swerve/BR_Swivel_Link.STL" />
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
File: urc_hw_description/urdf/simplified_swerve/simplified_swerve_ros2_control.xacro (robot description, xacro)
@@ -12,5 +12,5 @@
       <hardware>
         <xacro:if value="${use_sim}">
-          <plugin>gz_ros2_control/GazeboSimSystem</plugin>
+          <plugin>ign_ros2_control/IgnitionSystem</plugin>
         </xacro:if>
         <xacro:unless value="${use_sim}">
@@ -78,4 +78,19 @@
     <!-- Gazebo specific elements for simulation -->
     <xacro:if value="${use_sim}">
+      <!-- ROS2 Control Plugin-->
+      <!-- <gazebo> -->
+      <!--   <plugin -->
+      <!--     filename = "libign_ros2_control-system.so" -->
+      <!--     name = "ign_ros2_control"> -->
+      <!--     <robot_param>robot_description</robot_param> -->
+      <!--     <robot_param_node>robot_state_publisher</robot_param_node> -->
+      <!--     <parameters>$(find urc_bringup)/config/test_controllers.yaml</parameters> -->
+      <!--   </plugin> -->
+      <!-- </gazebo> -->
+      <gazebo>
+        <plugin filename="ign_ros2_control-system" name="ign_ros2_control::IgnitionROS2ControlPlugin">
+          <parameters>$(find urc_bringup)/config/test_controllers.yaml</parameters>
+        </plugin>
+      </gazebo>
       <!-- Gazebo materials -->
       <gazebo reference="base_Link">
