Commit message: changed name of base link for debugging

File: urc_hw_description/urdf/simplified_swerve/simplified_swerve.urdf.xacro (robot description, xacro)
@@ -24,5 +24,5 @@
   <!--   <joint name="world_to_base" type="fixed"> -->
   <!--     <parent link="world" /> -->
-  <!--     <child link="base_Link" /> -->
+  <!--     <child link="base_link" /> -->
   <!--     <origin xyz="0 0 0" rpy="0 0 0" /> -->
   <!--   </joint> -->

File: urc_hw_description/urdf/simplified_swerve/simplified_swerve_macro.xacro (robot description, xacro)
@@ -43,19 +43,19 @@
         <geometry>
           <mesh
-            filename="${package_path}/models/simplified_swerve/Base_Link.STL" />
-        </geometry>
-        <material
-          name="">
-          <color
-            rgba="0.792156862745098 0.819607843137255 0.933333333333333 1" />
-        </material>
-      </visual>
-      <collision>
-        <origin
-          xyz="0 0 0"
-          rpy="0 0 0" />
-        <geometry>
-          <mesh
-            filename="${package_path}/models/simplified_swerve/Base_Link.STL" />
+            filename="${package_path}/models/simplified_swerve/base_link.STL" />
+        </geometry>
+        <material
+          name="">
+          <color
+            rgba="0.792156862745098 0.819607843137255 0.933333333333333 1" />
+        </material>
+      </visual>
+      <collision>
+        <origin
+          xyz="0 0 0"
+          rpy="0 0 0" />
+        <geometry>
+          <mesh
+            filename="${package_path}/models/simplified_swerve/base_link.STL" />
         </geometry>
       </collision>

File: urc_hw_description/urdf/simplified_swerve/simplified_swerve_ros2_control.xacro (robot description, xacro)
@@ -104,5 +104,5 @@
       </gazebo>
       <!-- Gazebo materials -->
-      <gazebo reference="base_Link">
+      <gazebo reference="base_link">
         <material>Gazebo/Grey</material>
       </gazebo>

File: urc_hw_description/urdf/simplified_swerve/simplified_swerve_sensors.xacro (robot description, xacro)
@@ -29,5 +29,5 @@
     <!-- Joint to attach lidar to base -->
     <joint name="lidar_joint" type="fixed">
-      <parent link="base_Link"/>
+      <parent link="base_link"/>
       <child link="lidar_link"/>
       <origin xyz="0 0 0.025" rpy="0 0 0"/>
@@ -93,5 +93,5 @@
     </link>
     <joint name="imu_joint" type="fixed">
-      <parent link="base_Link"/>
+      <parent link="base_link"/>
       <child link="imu_link"/>
       <origin xyz="0.1 0 0" rpy="0 0 0"/>
@@ -128,5 +128,5 @@
       </sensor>
     </gazebo>
-     <gazebo reference="base_Link">
+     <gazebo reference="base_link">
         <sensor name="gps" type="navsat">
             <always_on>1</always_on>
