Commit message: new ign names

File: urc_hw_description/urdf/simplified_swerve/simplified_swerve_ros2_control.xacro (robot description, xacro)
@@ -12,5 +12,5 @@
       <hardware>
         <xacro:if value="${use_sim}">
-          <plugin>ign_ros2_control/IgnitionSystem</plugin>
+          <plugin>gz_ros2_control/GazeboSimSystem</plugin>
         </xacro:if>
         <xacro:unless value="${use_sim}">
@@ -99,5 +99,5 @@
       <!-- </gazebo> -->
       <gazebo>
-        <plugin filename="ign_ros2_control-system" name="ign_ros2_control::IgnitionROS2ControlPlugin">
+        <plugin filename="gz_ros2_control-system" name="gz_ros2_control::GazeboSimROS2ControlPlugin">
           <parameters>$(find urc_bringup)/config/test_controllers.yaml</parameters>
         </plugin>

File: urc_hw_description/urdf/simplified_swerve/simplified_swerve_sensors.xacro (robot description, xacro)
@@ -79,7 +79,5 @@
       <collision name="imu_collision">
         <geometry>
-          <box>
-            <size>0.001 0.001 0.001</size>  <!-- tiny collision -->
-          </box>
+          <box size="0.001 0.001 0.001"/>  <!-- tiny collision -->
         </geometry>
       </collision>
@@ -87,7 +85,5 @@
         <origin xyz="0 0 0" rpy="0 0 0"/>
         <geometry>
-          <box>
-            <size>0.001 0.001 0.001</size>
-          </box>
+          <box size="0.001 0.001 0.001"/>
         </geometry>
       </visual>
