Commit message: remove unused param

File: urc_hw_description/urdf/simplified_swerve/simplified_swerve_macro.xacro (robot description, xacro)
@@ -6,5 +6,5 @@
 <robot xmlns:xacro="http://www.ros.org/wiki/xacro">
   <!-- Define the simplified swerve drive macro -->
-  <xacro:macro name="simplified_swerve" params="parent_link">
+  <xacro:macro name="simplified_swerve">
     <link
       name="base_Link">

Commit message: Integrate with swervedrive

File: urc_hw_description/urdf/simplified_swerve/simplified_swerve_macro.xacro (robot description, xacro)
@@ -29,19 +29,19 @@
         <geometry>
           <mesh
-            filename="package://urc_hw_description/meshes/simplified_swerve/Base_Link.STL" />
-        </geometry>
-        <material
-          name="">
-          <color
-            rgba="0.792156862745098 0.819607843137255 0.933333333333333 1" />
-        </material>
-      </visual>
-      <collision>
-        <origin
-          xyz="0 0 0"
-          rpy="0 0 0" />
-        <geometry>
-          <mesh
-            filename="package://urc_hw_description/meshes/simplified_swerve/Base_Link.STL" />
+            filename="package://urc_hw_description/models/simplified_swerve/Base_Link.STL" />
+        </geometry>
+        <material
+          name="">
+          <color
+            rgba="0.792156862745098 0.819607843137255 0.933333333333333 1" />
+        </material>
+      </visual>
+      <collision>
+        <origin
+          xyz="0 0 0"
+          rpy="0 0 0" />
+        <geometry>
+          <mesh
+            filename="package://urc_hw_description/models/simplified_swerve/Base_Link.STL" />
         </geometry>
       </collision>
@@ -69,19 +69,19 @@
         <geometry>
           <mesh
-            filename="package://urc_hw_description/meshes/simplified_swerve/L_Rocker_Link.STL" />
-        </geometry>
-        <material
-          name="">
-          <color
-            rgba="0.792156862745098 0.819607843137255 0.933333333333333 1" />
-        </material>
-      </visual>
-      <collision>
-        <origin
-          xyz="0 0 0"
-          rpy="0 0 0" />
-        <geometry>
-          <mesh
-            filename="package://urc_hw_description/meshes/simplified_swerve/L_Rocker_Link.STL" />
+            filename="package://urc_hw_description/models/simplified_swerve/L_Rocker_Link.STL" />
+        </geometry>
+        <material
+          name="">
+          <color
+            rgba="0.792156862745098 0.819607843137255 0.933333333333333 1" />
+        </material>
+      </visual>
+      <collision>
+        <origin
+          xyz="0 0 0"
+          rpy="0 0 0" />
+        <geometry>
+          <mesh
+            filename="package://urc_hw_description/models/simplified_swerve/L_Rocker_Link.STL" />
         </geometry>
       </collision>
@@ -127,19 +127,19 @@
         <geometry>
           <mesh
-            filename="package://urc_hw_description/meshes/simplified_swerve/FL_Swivel_Link.STL" />
-        </geometry>
-        <material
-          name="">
-          <color
-            rgba="0.792156862745098 0.819607843137255 0.933333333333333 1" />
-        </material>
-      </visual>
-      <collision>
-        <origin
-          xyz="0 0 0"
-          rpy="0 0 0" />
-        <geometry>
-          <mesh
-            filename="package://urc_hw_description/meshes/simplified_swerve/FL_Swivel_Link.STL" />
+            filename="package://urc_hw_description/models/simplified_swerve/FL_Swivel_Link.STL" />
+        </geometry>
+        <material
+          name="">
+          <color
+            rgba="0.792156862745098 0.819607843137255 0.933333333333333 1" />
+        </material>
+      </visual>
+      <collision>
+        <origin
+          xyz="0 0 0"
+          rpy="0 0 0" />
+        <geometry>
+          <mesh
+            filename="package://urc_hw_description/models/simplified_swerve/FL_Swivel_Link.STL" />
         </geometry>
       </collision>
@@ -185,19 +185,19 @@
         <geometry>
           <mesh
-            filename="package://urc_hw_description/meshes/simplified_swerve/FL_Wheel_Link.STL" />
-        </geometry>
-        <material
-          name="">
-          <color
-            rgba="0.792156862745098 0.819607843137255 0.933333333333333 1" />
-        </material>
-      </visual>
-      <collision>
-        <origin
-          xyz="0 0 0"
-          rpy="0 0 0" />
-        <geometry>
-          <mesh
-            filename="package://urc_hw_description/meshes/simplified_swerve/FL_Wheel_Link.STL" />
+            filename="package://urc_hw_description/models/simplified_swerve/FL_Wheel_Link.STL" />
+        </geometry>
+        <material
+          name="">
+          <color
+            rgba="0.792156862745098 0.819607843137255 0.933333333333333 1" />
+        </material>
+      </visual>
+      <collision>
+        <origin
+          xyz="0 0 0"
+          rpy="0 0 0" />
+        <geometry>
+          <mesh
+            filename="package://urc_hw_description/models/simplified_swerve/FL_Wheel_Link.STL" />
         </geometry>
       </collision>
@@ -238,19 +238,19 @@
         <geometry>
           <mesh
-            filename="package://urc_hw_description/meshes/simplified_swerve/BL_Swivel_Link.STL" />
-        </geometry>
-        <material
-          name="">
-          <color
-            rgba="0.792156862745098 0.819607843137255 0.933333333333333 1" />
-        </material>
-      </visual>
-      <collision>
-        <origin
-          xyz="0 0 0"
-          rpy="0 0 0" />
-        <geometry>
-          <mesh
-            filename="package://urc_hw_description/meshes/simplified_swerve/BL_Swivel_Link.STL" />
+            filename="package://urc_hw_description/models/simplified_swerve/BL_Swivel_Link.STL" />
+        </geometry>
+        <material
+          name="">
+          <color
+            rgba="0.792156862745098 0.819607843137255 0.933333333333333 1" />
+        </material>
+      </visual>
+      <collision>
+        <origin
+          xyz="0 0 0"
+          rpy="0 0 0" />
+        <geometry>
+          <mesh
+            filename="package://urc_hw_description/models/simplified_swerve/BL_Swivel_Link.STL" />
         </geometry>
       </collision>
@@ -296,19 +296,19 @@
         <geometry>
           <mesh
-            filename="package://urc_hw_description/meshes/simplified_swerve/BL_Wheel_Link.STL" />
-        </geometry>
-        <material
-          name="">
-          <color
-            rgba="0.792156862745098 0.819607843137255 0.933333333333333 1" />
-        </material>
-      </visual>
-      <collision>
-        <origin
-          xyz="0 0 0"
-          rpy="0 0 0" />
-        <geometry>
-          <mesh
-            filename="package://urc_hw_description/meshes/simplified_swerve/BL_Wheel_Link.STL" />
+            filename="package://urc_hw_description/models/simplified_swerve/BL_Wheel_Link.STL" />
+        </geometry>
+        <material
+          name="">
+          <color
+            rgba="0.792156862745098 0.819607843137255 0.933333333333333 1" />
+        </material>
+      </visual>
+      <collision>
+        <origin
+          xyz="0 0 0"
+          rpy="0 0 0" />
+        <geometry>
+          <mesh
+            filename="package://urc_hw_description/models/simplified_swerve/BL_Wheel_Link.STL" />
         </geometry>
       </collision>
@@ -349,19 +349,19 @@
         <geometry>
           <mesh
-            filename="package://urc_hw_description/meshes/simplified_swerve/R_Rocker_Link.STL" />
-        </geometry>
-        <material
-          name="">
-          <color
-            rgba="0.792156862745098 0.819607843137255 0.933333333333333 1" />
-        </material>
-      </visual>
-      <collision>
-        <origin
-          xyz="0 0 0"
-          rpy="0 0 0" />
-        <geometry>
-          <mesh
-            filename="package://urc_hw_description/meshes/simplified_swerve/R_Rocker_Link.STL" />
+            filename="package://urc_hw_description/models/simplified_swerve/R_Rocker_Link.STL" />
+        </geometry>
+        <material
+          name="">
+          <color
+            rgba="0.792156862745098 0.819607843137255 0.933333333333333 1" />
+        </material>
+      </visual>
+      <collision>
+        <origin
+          xyz="0 0 0"
+          rpy="0 0 0" />
+        <geometry>
+          <mesh
+            filename="package://urc_hw_description/models/simplified_swerve/R_Rocker_Link.STL" />
         </geometry>
       </collision>
@@ -407,19 +407,19 @@
         <geometry>
           <mesh
-            filename="package://urc_hw_description/meshes/simplified_swerve/FR_Swivel_Link.STL" />
-        </geometry>
-        <material
-          name="">
-          <color
-            rgba="0.792156862745098 0.819607843137255 0.933333333333333 1" />
-        </material>
-      </visual>
-      <collision>
-        <origin
-          xyz="0 0 0"
-          rpy="0 0 0" />
-        <geometry>
-          <mesh
-            filename="package://urc_hw_description/meshes/simplified_swerve/FR_Swivel_Link.STL" />
+            filename="package://urc_hw_description/models/simplified_swerve/FR_Swivel_Link.STL" />
+        </geometry>
+        <material
+          name="">
+          <color
+            rgba="0.792156862745098 0.819607843137255 0.933333333333333 1" />
+        </material>
+      </visual>
+      <collision>
+        <origin
+          xyz="0 0 0"
+          rpy="0 0 0" />
+        <geometry>
+          <mesh
+            filename="package://urc_hw_description/models/simplified_swerve/FR_Swivel_Link.STL" />
         </geometry>
       </collision>
@@ -465,19 +465,19 @@
         <geometry>
           <mesh
-            filename="package://urc_hw_description/meshes/simplified_swerve/FR_Wheel_Link.STL" />
-        </geometry>
-        <material
-          name="">
-          <color
-            rgba="0.792156862745098 0.819607843137255 0.933333333333333 1" />
-        </material>
-      </visual>
-      <collision>
-        <origin
-          xyz="0 0 0"
-          rpy="0 0 0" />
-        <geometry>
-          <mesh
-            filename="package://urc_hw_description/meshes/simplified_swerve/FR_Wheel_Link.STL" />
+            filename="package://urc_hw_description/models/simplified_swerve/FR_Wheel_Link.STL" />
+        </geometry>
+        <material
+          name="">
+          <color
+            rgba="0.792156862745098 0.819607843137255 0.933333333333333 1" />
+        </material>
+      </visual>
+      <collision>
+        <origin
+          xyz="0 0 0"
+          rpy="0 0 0" />
+        <geometry>
+          <mesh
+            filename="package://urc_hw_description/models/simplified_swerve/FR_Wheel_Link.STL" />
         </geometry>
       </collision>
@@ -518,19 +518,19 @@
         <geometry>
           <mesh
-            filename="package://urc_hw_description/meshes/simplified_swerve/BR_Swivel_Link.STL" />
-        </geometry>
-        <material
-          name="">
-          <color
-            rgba="0.792156862745098 0.819607843137255 0.933333333333333 1" />
-        </material>
-      </visual>
-      <collision>
-        <origin
-          xyz="0 0 0"
-          rpy="0 0 0" />
-        <geometry>
-          <mesh
-            filename="package://urc_hw_description/meshes/simplified_swerve/BR_Swivel_Link.STL" />
+            filename="package://urc_hw_description/models/simplified_swerve/BR_Swivel_Link.STL" />
+        </geometry>
+        <material
+          name="">
+          <color
+            rgba="0.792156862745098 0.819607843137255 0.933333333333333 1" />
+        </material>
+      </visual>
+      <collision>
+        <origin
+          xyz="0 0 0"
+          rpy="0 0 0" />
+        <geometry>
+          <mesh
+            filename="package://urc_hw_description/models/simplified_swerve/BR_Swivel_Link.STL" />
         </geometry>
       </collision>
@@ -576,19 +576,19 @@
         <geometry>
           <mesh
-            filename="package://urc_hw_description/meshes/simplified_swerve/BR_Wheel_Link.STL" />
-        </geometry>
-        <material
-          name="">
-          <color
-            rgba="0.792156862745098 0.819607843137255 0.933333333333333 1" />
-        </material>
-      </visual>
-      <collision>
-        <origin
-          xyz="0 0 0"
-          rpy="0 0 0" />
-        <geometry>
-          <mesh
-            filename="package://urc_hw_description/meshes/simplified_swerve/BR_Wheel_Link.STL" />
+            filename="package://urc_hw_description/models/simplified_swerve/BR_Wheel_Link.STL" />
+        </geometry>
+        <material
+          name="">
+          <color
+            rgba="0.792156862745098 0.819607843137255 0.933333333333333 1" />
+        </material>
+      </visual>
+      <collision>
+        <origin
+          xyz="0 0 0"
+          rpy="0 0 0" />
+        <geometry>
+          <mesh
+            filename="package://urc_hw_description/models/simplified_swerve/BR_Wheel_Link.STL" />
         </geometry>
       </collision>

Commit message: Add LiDAR sensor in Gazebo and bridge /scan topic to ROS

File: urc_hw_description/urdf/simplified_swerve/simplified_swerve_macro.xacro (robot description, xacro)
@@ -47,4 +47,59 @@
       </collision>
     </link>
+    <!-- Lidar Link -->
+    <link name="lidar_link">
+      <inertial>
+        <mass value="0.1"/>
+        <origin xyz="0 0 0" rpy="0 0 0"/>
+        <inertia ixx="0.001" ixy="0" ixz="0" iyy="0.001" iyz="0" izz="0.001"/>
+      </inertial>
+      <visual>
+        <origin xyz="0 0 0" rpy="0 0 0"/>
+        <geometry>
+          <cylinder radius="0.03" length="0.05"/>
+        </geometry>
+        <material name="black">
+          <color rgba="0 0 0 1"/>
+        </material>
+      </visual>
+    </link>
+    <!-- Joint to attach lidar to base -->
+    <joint name="lidar_joint" type="fixed">
+      <parent link="base_Link"/>
+      <child link="lidar_link"/>
+      <origin xyz="0 0 0.1" rpy="0 0 0"/>
+    </joint>
+    <!-- Gazebo plugin for lidar -->
+    <gazebo reference="lidar_link">
+      <sensor name="lidar" type="gpu_lidar">
+        <pose>0 0 0 0 0 0</pose>
+        <always_on>true</always_on>
+        <visualize>true</visualize>
+        <update_rate>10</update_rate>
+        <topic>scan</topic>
+        <gz_frame_id>lidar_link</gz_frame_id>
+        <lidar>
+          <scan>
+            <horizontal>
+              <samples>720</samples>
+              <resolution>1</resolution>
+              <min_angle>-3.14</min_angle>
+              <max_angle>3.14</max_angle>
+            </horizontal>
+          </scan>
+          <range>
+            <min>0.05</min>
+            <max>10.0</max>
+            <resolution>0.01</resolution>
+          </range>
+          <noise>
+            <type>gaussian</type>
+            <mean>0.0</mean>
+            <stddev>0.01</stddev>
+          </noise>
+          <frame_id>lidar_link</frame_id>
+        </lidar>
+      </sensor>
+    </gazebo>
     <link
       name="L_Rocker_Link">

Commit message: Add IMU sensor (no orientation calculation from plugin)

File: urc_hw_description/urdf/simplified_swerve/simplified_swerve_macro.xacro (robot description, xacro)
@@ -68,5 +68,5 @@
       <parent link="base_Link"/>
       <child link="lidar_link"/>
-      <origin xyz="0 0 0.1" rpy="0 0 0"/>
+      <origin xyz="0 0 0.025" rpy="0 0 0"/>
     </joint>
     <!-- Gazebo plugin for lidar -->
@@ -102,4 +102,61 @@
       </sensor>
     </gazebo>
+    <link name="imu_link">
+      <inertial>
+        <mass value="0.01"/>
+        <origin xyz="0 0 0" rpy="0 0 0"/>
+        <inertia ixx="0.001" ixy="0" ixz="0" iyy="0.001" iyz="0" izz="0.001"/>
+      </inertial>
+      <collision name="imu_collision">
+        <geometry>
+          <box>
+            <size>0.001 0.001 0.001</size>  <!-- tiny collision -->
+          </box>
+        </geometry>
+      </collision>
+      <visual name="imu_visual">
+        <geometry>
+          <box>
+            <size>0.001 0.001 0.001</size>
+          </box>
+        </geometry>
+      </visual>
+    </link>
+    <joint name="imu_joint" type="fixed">
+      <parent link="base_Link"/>
+      <child link="imu_link"/>
+      <origin xyz="0.1 0 0" rpy="0 0 0"/>
+    </joint>
+    <gazebo reference="imu_link">
+      <sensor name="imu_sensor" type="imu">
+        <always_on>1</always_on>
+        <update_rate>100</update_rate>
+        <visualize>true</visualize>
+        <topic>/imu/data_raw</topic>
+        <imu>
+          <orientation>
+            <noise>
+              <type>gaussian</type>
+              <mean>0.0</mean>
+              <stddev>0.0001</stddev>
+            </noise>
+          </orientation>
+          <angular_velocity>
+            <noise>
+              <type>gaussian</type>
+              <mean>0.0</mean>
+              <stddev>0.0005</stddev>
+            </noise>
+          </angular_velocity>
+          <linear_acceleration>
+            <noise>
+              <type>gaussian</type>
+              <mean>0.0</mean>
+              <stddev>0.01</stddev>
+            </noise>
+          </linear_acceleration>
+        </imu>
+      </sensor>
+    </gazebo>
     <link
       name="L_Rocker_Link">
