Commit message: marsyard2020 terrain works with walli

File: urc_hw_description/urdf/simplified_swerve/simplified_swerve_macro.xacro (robot description, xacro)
@@ -7,4 +7,11 @@
   <!-- Define the simplified swerve drive macro -->
   <xacro:macro name="simplified_swerve">
+  <!-- replacing package:// -->
+  <xacro:property name="package_path" value="$(find urc_hw_description)"/>
+  <!-- Wheel Cylinder Geometry -->
+  <xacro:property name="wheel_radius" value="0.15" />
+  <xacro:property name="wheel_length" value="0.1" />
+  <!-- remove wheel_origin_xyz if not needed -->
+  <xacro:property name="wheel_origin_xyz" value="0 0 0" />
     <link
       name="base_Link">
@@ -29,19 +36,19 @@
         <geometry>
           <mesh
-            filename="package://urc_hw_description/models/simplified_swerve/Base_Link.STL" />
-        </geometry>
-        <material
-          name="">
-          <color
-            rgba="0.792156862745098 0.819607843137255 0.933333333333333 1" />
-        </material>
-      </visual>
-      <collision>
-        <origin
-          xyz="0 0 0"
-          rpy="0 0 0" />
-        <geometry>
-          <mesh
-            filename="package://urc_hw_description/models/simplified_swerve/Base_Link.STL" />
+            filename="${package_path}/models/simplified_swerve/Base_Link.STL" />
+        </geometry>
+        <material
+          name="">
+          <color
+            rgba="0.792156862745098 0.819607843137255 0.933333333333333 1" />
+        </material>
+      </visual>
+      <collision>
+        <origin
+          xyz="0 0 0"
+          rpy="0 0 0" />
+        <geometry>
+          <mesh
+            filename="${package_path}/models/simplified_swerve/Base_Link.STL" />
         </geometry>
       </collision>
@@ -69,19 +76,19 @@
         <geometry>
           <mesh
-            filename="package://urc_hw_description/models/simplified_swerve/L_Rocker_Link.STL" />
-        </geometry>
-        <material
-          name="">
-          <color
-            rgba="0.792156862745098 0.819607843137255 0.933333333333333 1" />
-        </material>
-      </visual>
-      <collision>
-        <origin
-          xyz="0 0 0"
-          rpy="0 0 0" />
-        <geometry>
-          <mesh
-            filename="package://urc_hw_description/models/simplified_swerve/L_Rocker_Link.STL" />
+            filename="${package_path}/models/simplified_swerve/L_Rocker_Link.STL" />
+        </geometry>
+        <material
+          name="">
+          <color
+            rgba="0.792156862745098 0.819607843137255 0.933333333333333 1" />
+        </material>
+      </visual>
+      <collision>
+        <origin
+          xyz="0 0 0"
+          rpy="0 0 0" />
+        <geometry>
+          <mesh
+            filename="${package_path}/models/simplified_swerve/L_Rocker_Link.STL" />
         </geometry>
       </collision>
@@ -127,19 +134,19 @@
         <geometry>
           <mesh
-            filename="package://urc_hw_description/models/simplified_swerve/FL_Swivel_Link.STL" />
-        </geometry>
-        <material
-          name="">
-          <color
-            rgba="0.792156862745098 0.819607843137255 0.933333333333333 1" />
-        </material>
-      </visual>
-      <collision>
-        <origin
-          xyz="0 0 0"
-          rpy="0 0 0" />
-        <geometry>
-          <mesh
-            filename="package://urc_hw_description/models/simplified_swerve/FL_Swivel_Link.STL" />
+            filename="${package_path}/models/simplified_swerve/FL_Swivel_Link.STL" />
+        </geometry>
+        <material
+          name="">
+          <color
+            rgba="0.792156862745098 0.819607843137255 0.933333333333333 1" />
+        </material>
+      </visual>
+      <collision>
+        <origin
+          xyz="0 0 0"
+          rpy="0 0 0" />
+        <geometry>
+          <mesh
+            filename="${package_path}/models/simplified_swerve/FL_Swivel_Link.STL" />
         </geometry>
       </collision>
@@ -182,22 +189,20 @@
         <origin
           xyz="0 0 0"
-          rpy="0 0 0" />
-        <geometry>
-          <mesh
-            filename="package://urc_hw_description/models/simplified_swerve/FL_Wheel_Link.STL" />
-        </geometry>
-        <material
-          name="">
-          <color
-            rgba="0.792156862745098 0.819607843137255 0.933333333333333 1" />
-        </material>
-      </visual>
-      <collision>
-        <origin
-          xyz="0 0 0"
-          rpy="0 0 0" />
-        <geometry>
-          <mesh
-            filename="package://urc_hw_description/models/simplified_swerve/FL_Wheel_Link.STL" />
+          rpy="${pi/2} 0 0" />
+        <geometry>
+          <cylinder radius="${wheel_radius}"  length="${wheel_length}" />
+        </geometry>
+        <material
+          name="">
+          <color
+            rgba="0.792156862745098 0.819607843137255 0.933333333333333 1" />
+        </material>
+      </visual>
+      <collision>
+        <origin
+          xyz="0 0 0"
+          rpy="${pi/2} 0 0" />
+        <geometry>
+          <cylinder radius="${wheel_radius}"  length="${wheel_length}" />
         </geometry>
       </collision>
@@ -238,19 +243,19 @@
         <geometry>
           <mesh
-            filename="package://urc_hw_description/models/simplified_swerve/BL_Swivel_Link.STL" />
-        </geometry>
-        <material
-          name="">
-          <color
-            rgba="0.792156862745098 0.819607843137255 0.933333333333333 1" />
-        </material>
-      </visual>
-      <collision>
-        <origin
-          xyz="0 0 0"
-          rpy="0 0 0" />
-        <geometry>
-          <mesh
-            filename="package://urc_hw_description/models/simplified_swerve/BL_Swivel_Link.STL" />
+            filename="${package_path}/models/simplified_swerve/BL_Swivel_Link.STL" />
+        </geometry>
+        <material
+          name="">
+          <color
+            rgba="0.792156862745098 0.819607843137255 0.933333333333333 1" />
+        </material>
+      </visual>
+      <collision>
+        <origin
+          xyz="0 0 0"
+          rpy="0 0 0" />
+        <geometry>
+          <mesh
+            filename="${package_path}/models/simplified_swerve/BL_Swivel_Link.STL" />
         </geometry>
       </collision>
@@ -293,22 +298,20 @@
         <origin
           xyz="0 0 0"
-          rpy="0 0 0" />
-        <geometry>
-          <mesh
-            filename="package://urc_hw_description/models/simplified_swerve/BL_Wheel_Link.STL" />
-        </geometry>
-        <material
-          name="">
-          <color
-            rgba="0.792156862745098 0.819607843137255 0.933333333333333 1" />
-        </material>
-      </visual>
-      <collision>
-        <origin
-          xyz="0 0 0"
-          rpy="0 0 0" />
-        <geometry>
-          <mesh
-            filename="package://urc_hw_description/models/simplified_swerve/BL_Wheel_Link.STL" />
+          rpy="${pi/2} 0 0" />
+        <geometry>
+          <cylinder radius="${wheel_radius}"  length="${wheel_length}" />
+        </geometry>
+        <material
+          name="">
+          <color
+            rgba="0.792156862745098 0.819607843137255 0.933333333333333 1" />
+        </material>
+      </visual>
+      <collision>
+        <origin
+          xyz="0 0 0"
+          rpy="${pi/2} 0 0" />
+        <geometry>
+          <cylinder radius="${wheel_radius}"  length="${wheel_length}" />
         </geometry>
       </collision>
@@ -349,19 +352,19 @@
         <geometry>
           <mesh
-            filename="package://urc_hw_description/models/simplified_swerve/R_Rocker_Link.STL" />
-        </geometry>
-        <material
-          name="">
-          <color
-            rgba="0.792156862745098 0.819607843137255 0.933333333333333 1" />
-        </material>
-      </visual>
-      <collision>
-        <origin
-          xyz="0 0 0"
-          rpy="0 0 0" />
-        <geometry>
-          <mesh
-            filename="package://urc_hw_description/models/simplified_swerve/R_Rocker_Link.STL" />
+            filename="${package_path}/models/simplified_swerve/R_Rocker_Link.STL" />
+        </geometry>
+        <material
+          name="">
+          <color
+            rgba="0.792156862745098 0.819607843137255 0.933333333333333 1" />
+        </material>
+      </visual>
+      <collision>
+        <origin
+          xyz="0 0 0"
+          rpy="0 0 0" />
+        <geometry>
+          <mesh
+            filename="${package_path}/models/simplified_swerve/R_Rocker_Link.STL" />
         </geometry>
       </collision>
@@ -407,19 +410,19 @@
         <geometry>
           <mesh
-            filename="package://urc_hw_description/models/simplified_swerve/FR_Swivel_Link.STL" />
-        </geometry>
-        <material
-          name="">
-          <color
-            rgba="0.792156862745098 0.819607843137255 0.933333333333333 1" />
-        </material>
-      </visual>
-      <collision>
-        <origin
-          xyz="0 0 0"
-          rpy="0 0 0" />
-        <geometry>
-          <mesh
-            filename="package://urc_hw_description/models/simplified_swerve/FR_Swivel_Link.STL" />
+            filename="${package_path}/models/simplified_swerve/FR_Swivel_Link.STL" />
+        </geometry>
+        <material
+          name="">
+          <color
+            rgba="0.792156862745098 0.819607843137255 0.933333333333333 1" />
+        </material>
+      </visual>
+      <collision>
+        <origin
+          xyz="0 0 0"
+          rpy="0 0 0" />
+        <geometry>
+          <mesh
+            filename="${package_path}/models/simplified_swerve/FR_Swivel_Link.STL" />
         </geometry>
       </collision>
@@ -462,22 +465,20 @@
         <origin
           xyz="0 0 0"
-          rpy="0 0 0" />
-        <geometry>
-          <mesh
-            filename="package://urc_hw_description/models/simplified_swerve/FR_Wheel_Link.STL" />
-        </geometry>
-        <material
-          name="">
-          <color
-            rgba="0.792156862745098 0.819607843137255 0.933333333333333 1" />
-        </material>
-      </visual>
-      <collision>
-        <origin
-          xyz="0 0 0"
-          rpy="0 0 0" />
-        <geometry>
-          <mesh
-            filename="package://urc_hw_description/models/simplified_swerve/FR_Wheel_Link.STL" />
+          rpy="${pi/2} 0 0" />
+        <geometry>
+          <cylinder radius="${wheel_radius}"  length="${wheel_length}" />
+        </geometry>
+        <material
+          name="">
+          <color
+            rgba="0.792156862745098 0.819607843137255 0.933333333333333 1" />
+        </material>
+      </visual>
+      <collision>
+        <origin
+          xyz="0 0 0"
+          rpy="${pi/2} 0 0" />
+        <geometry>
+          <cylinder radius="${wheel_radius}"  length="${wheel_length}" />
         </geometry>
       </collision>
@@ -518,19 +519,19 @@
         <geometry>
           <mesh
-            filename="package://urc_hw_description/models/simplified_swerve/BR_Swivel_Link.STL" />
-        </geometry>
-        <material
-          name="">
-          <color
-            rgba="0.792156862745098 0.819607843137255 0.933333333333333 1" />
-        </material>
-      </visual>
-      <collision>
-        <origin
-          xyz="0 0 0"
-          rpy="0 0 0" />
-        <geometry>
-          <mesh
-            filename="package://urc_hw_description/models/simplified_swerve/BR_Swivel_Link.STL" />
+            filename="${package_path}/models/simplified_swerve/BR_Swivel_Link.STL" />
+        </geometry>
+        <material
+          name="">
+          <color
+            rgba="0.792156862745098 0.819607843137255 0.933333333333333 1" />
+        </material>
+      </visual>
+      <collision>
+        <origin
+          xyz="0 0 0"
+          rpy="0 0 0" />
+        <geometry>
+          <mesh
+            filename="${package_path}/models/simplified_swerve/BR_Swivel_Link.STL" />
         </geometry>
       </collision>
@@ -573,22 +574,20 @@
         <origin
           xyz="0 0 0"
-          rpy="0 0 0" />
-        <geometry>
-          <mesh
-            filename="package://urc_hw_description/models/simplified_swerve/BR_Wheel_Link.STL" />
-        </geometry>
-        <material
-          name="">
-          <color
-            rgba="0.792156862745098 0.819607843137255 0.933333333333333 1" />
-        </material>
-      </visual>
-      <collision>
-        <origin
-          xyz="0 0 0"
-          rpy="0 0 0" />
-        <geometry>
-          <mesh
-            filename="package://urc_hw_description/models/simplified_swerve/BR_Wheel_Link.STL" />
+          rpy="${pi/2} 0 0" />
+        <geometry>
+          <cylinder radius="${wheel_radius}"  length="${wheel_length}" />
+        </geometry>
+        <material
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
Commit message: fix wheel placement in urdf

File: urc_hw_description/urdf/simplified_swerve/simplified_swerve_macro.xacro (robot description, xacro)
@@ -10,8 +10,9 @@
   <xacro:property name="package_path" value="$(find urc_hw_description)"/>
   <!-- Wheel Cylinder Geometry -->
-  <xacro:property name="wheel_radius" value="0.15" />
-  <xacro:property name="wheel_length" value="0.1" />
+  <xacro:property name="wheel_radius" value="0.119888" />
+  <xacro:property name="wheel_length" value="0.0762" />
   <!-- remove wheel_origin_xyz if not needed -->
-  <xacro:property name="wheel_origin_xyz" value="0 0 0" />
+  <xacro:property name="wheel_origin_xyz_left" value="0 0.0381 0" />
+  <xacro:property name="wheel_origin_xyz_right" value="0 -0.0381 0" />
     <link
       name="base_Link">
@@ -174,5 +175,5 @@
       <inertial>
         <origin
-          xyz="0 0.0381000000000001 1.38777878078145E-17"
+          xyz="${wheel_origin_xyz_left}"
           rpy="0 0 0" />
         <mass
@@ -188,18 +189,18 @@
       <visual>
         <origin
-          xyz="0 0 0"
-          rpy="${pi/2} 0 0" />
-        <geometry>
-          <cylinder radius="${wheel_radius}"  length="${wheel_length}" />
-        </geometry>
-        <material
-          name="">
-          <color
-            rgba="0.792156862745098 0.819607843137255 0.933333333333333 1" />
-        </material>
-      </visual>
-      <collision>
-        <origin
-          xyz="0 0 0"
+          xyz="${wheel_origin_xyz_left}"
+          rpy="${pi/2} 0 0" />
+        <geometry>
+          <cylinder radius="${wheel_radius}"  length="${wheel_length}" />
+        </geometry>
+        <material
+          name="">
+          <color
+            rgba="0.792156862745098 0.819607843137255 0.933333333333333 1" />
+        </material>
+      </visual>
+      <collision>
+        <origin
+          xyz="${wheel_origin_xyz_left}"
           rpy="${pi/2} 0 0" />
         <geometry>
@@ -283,5 +284,5 @@
       <inertial>
         <origin
-          xyz="0 0.0380999942740809 -2.08881547555939E-05"
+          xyz="${wheel_origin_xyz_left}"
           rpy="0 0 0" />
         <mass
@@ -297,18 +298,18 @@
       <visual>
         <origin
-          xyz="0 0 0"
-          rpy="${pi/2} 0 0" />
-        <geometry>
-          <cylinder radius="${wheel_radius}"  length="${wheel_length}" />
-        </geometry>
-        <material
-          name="">
-          <color
-            rgba="0.792156862745098 0.819607843137255 0.933333333333333 1" />
-        </material>
-      </visual>
-      <collision>
-        <origin
-          xyz="0 0 0"
+          xyz="${wheel_origin_xyz_left}"
+          rpy="${pi/2} 0 0" />
+        <geometry>
+          <cylinder radius="${wheel_radius}"  length="${wheel_length}" />
+        </geometry>
+        <material
+          name="">
+          <color
+            rgba="0.792156862745098 0.819607843137255 0.933333333333333 1" />
+        </material>
+      </visual>
+      <collision>
+        <origin
+          xyz="${wheel_origin_xyz_left}"
           rpy="${pi/2} 0 0" />
         <geometry>
@@ -450,5 +451,5 @@
       <inertial>
         <origin
-          xyz="0 -0.0381 6.93889390390723E-18"
+          xyz="${wheel_origin_xyz_right}"
           rpy="0 0 0" />
         <mass
@@ -464,18 +465,18 @@
       <visual>
         <origin
-          xyz="0 0 0"
-          rpy="${pi/2} 0 0" />
-        <geometry>
-          <cylinder radius="${wheel_radius}"  length="${wheel_length}" />
-        </geometry>
-        <material
-          name="">
-          <color
-            rgba="0.792156862745098 0.819607843137255 0.933333333333333 1" />
-        </material>
-      </visual>
-      <collision>
-        <origin
-          xyz="0 0 0"
+          xyz="${wheel_origin_xyz_right}"
+          rpy="${pi/2} 0 0" />
+        <geometry>
+          <cylinder radius="${wheel_radius}"  length="${wheel_length}" />
+        </geometry>
+        <material
+          name="">
+          <color
+            rgba="0.792156862745098 0.819607843137255 0.933333333333333 1" />
+        </material>
+      </visual>
+      <collision>
+        <origin
+          xyz="${wheel_origin_xyz_right}"
           rpy="${pi/2} 0 0" />
         <geometry>
@@ -559,5 +560,5 @@
       <inertial>
         <origin
-          xyz="-6.93889390390723E-18 -0.0381 0"
+          xyz="${wheel_origin_xyz_right}"
           rpy="0 0 0" />
         <mass
@@ -573,18 +574,18 @@
       <visual>
         <origin
-          xyz="0 0 0"
-          rpy="${pi/2} 0 0" />
-        <geometry>
-          <cylinder radius="${wheel_radius}"  length="${wheel_length}" />
-        </geometry>
-        <material
-          name="">
-          <color
-            rgba="0.792156862745098 0.819607843137255 0.933333333333333 1" />
-        </material>
-      </visual>
-      <collision>
-        <origin
-          xyz="0 0 0"
+          xyz="${wheel_origin_xyz_right}"
+          rpy="${pi/2} 0 0" />
+        <geometry>
+          <cylinder radius="${wheel_radius}"  length="${wheel_length}" />
+        </geometry>
+        <material
+          name="">
+          <color
+            rgba="0.792156862745098 0.819607843137255 0.933333333333333 1" />
+        </material>
+      </visual>
+      <collision>
+        <origin
+          xyz="${wheel_origin_xyz_right}"
           rpy="${pi/2} 0 0" />
         <geometry>

Commit message: fix rviz and sim frame

File: urc_hw_description/urdf/simplified_swerve/simplified_swerve_macro.xacro (robot description, xacro)
@@ -8,5 +8,5 @@
   <xacro:macro name="simplified_swerve">
   <!-- replacing package:// -->
-  <xacro:property name="package_path" value="$(find urc_hw_description)"/>
+  <xacro:property name="package_path" value="file://$(find urc_hw_description)"/>
   <!-- Wheel Cylinder Geometry -->
   <xacro:property name="wheel_radius" value="0.119888" />
@@ -16,5 +16,5 @@
   <xacro:property name="wheel_origin_xyz_right" value="0 -0.0381 0" />
     <link
-      name="base_Link">
+      name="base_link">
       <inertial>
         <origin
@@ -102,5 +102,5 @@
         rpy="0 0.024048 0" />
       <parent
-        link="base_Link" />
+        link="base_link" />
       <child
         link="L_Rocker_Link" />
@@ -378,5 +378,5 @@
         rpy="0 0.069977 0" />
       <parent
-        link="base_Link" />
+        link="base_link" />
       <child
         link="R_Rocker_Link" />

File: urc_hw_description/urdf/simplified_swerve/simplified_swerve_ros2_control.xacro (robot description, xacro)
@@ -18,4 +18,10 @@
         </xacro:unless>
       </hardware>
+      <joint name="L_Rocker_Joint">
+        <state_interface name="position"/>
+      </joint>
+      <joint name="R_Rocker_Joint">
+        <state_interface name="position"/>
+      </joint>
       <!-- Joint State Interface -->
       <joint name="FL_Swivel_Joint">
@@ -32,4 +38,5 @@
         </command_interface>
         <state_interface name="velocity"/>
+        <state_interface name="position"/>
       </joint>
       <joint name="BL_Swivel_Joint">
@@ -46,4 +53,5 @@
         </command_interface>
         <state_interface name="velocity"/>
+        <state_interface name="position"/>
       </joint>
       <joint name="FR_Swivel_Joint">
@@ -60,4 +68,5 @@
         </command_interface>
         <state_interface name="velocity"/>
+        <state_interface name="position"/>
       </joint>
       <joint name="BR_Swivel_Joint">
@@ -74,4 +83,5 @@
         </command_interface>
         <state_interface name="velocity"/>
+        <state_interface name="position"/>
       </joint>
     </ros2_control>

Commit message: test for debugging

File: urc_hw_description/urdf/simplified_swerve/simplified_swerve_macro.xacro (robot description, xacro)
@@ -18,4 +18,5 @@
     <jointA>L_Rocker_Joint</jointA>
     <jointB>R_Rocker_Joint</jointB>
+    <barJoint>base_to_differential_bar</barJoint>
     <forceConstant>300.0</forceConstant>
   </plugin>
@@ -61,4 +62,24 @@
       </collision>
     </link>
+    <!-- Differential bar link fixed to base_link so its pose matches base_link.
+         Rockers will be reparented to this link and coupled by the
+         DifferentialSystem plugin to behave like a mechanical differential:
+         bar angle equals average of rocker angles. -->
+    <link name="differential_bar">
+      <inertial>
+        <origin xyz="0 0 0" rpy="0 0 0" />
+        <!-- Tiny mass/inertia; merged with base via fixed joint at runtime -->
+        <mass value="1e-6" />
+        <inertia ixx="1e-6" ixy="0" ixz="0" iyy="1e-6" iyz="0" izz="1e-6" />
+      </inertial>
+    </link>
+    <joint name="base_to_differential_bar" type="revolute">
+      <origin xyz="0 0 0" rpy="0 0 0" />
+      <parent link="base_link" />
+      <child link="differential_bar" />
+      <axis xyz="0 1 0" />
+      <limit lower="-1.57" upper="1.57" effort="1000" velocity="100" />
+      <dynamics damping="5.0" friction="0.0" />
+    </joint>
     <link
       name="L_Rocker_Link">
@@ -118,4 +139,5 @@
         effort="1000"
         velocity="100" />
+      <dynamics damping="3.0" friction="0.0" />
     </joint>
     <link
@@ -394,4 +416,5 @@
         effort="1000"
         velocity="100" />
+      <dynamics damping="3.0" friction="0.0" />
     </joint>
     <link

Commit message: swivel dampening and frcition to avoid tweaking

File: urc_hw_description/urdf/simplified_swerve/simplified_swerve_macro.xacro (robot description, xacro)
@@ -15,4 +15,6 @@
   <xacro:property name="wheel_origin_xyz_left" value="0 0.0381 0" />
   <xacro:property name="wheel_origin_xyz_right" value="0 -0.0381 0" />
+  <xacro:property name="swivel_damping_factor" value = "0.8" />
+  <xacro:property name="mu" value="0.8" />
     <link
       name="base_link">
@@ -170,4 +172,5 @@
         effort="10"
         velocity="100" />
+      <dynamics damping="${swivel_damping_factor}" friction="${mu}"/>
     </joint>
     <link
@@ -279,4 +282,5 @@
         effort="10"
         velocity="100" />
+      <dynamics damping="${swivel_damping_factor}" friction="${mu}"/>
     </joint>
     <link
@@ -446,4 +450,5 @@
         effort="10"
         velocity="100" />
+      <dynamics damping="${swivel_damping_factor}" friction="${mu}"/>
     </joint>
     <link
@@ -555,4 +560,5 @@
         effort="10"
         velocity="100" />
+      <dynamics damping="${swivel_damping_factor}" friction="${mu}"/>
     </joint>
     <link
