Commit message: Merge feat/pathplan (suspension + ekf) into master. (#314)
* removed bloat

* more testing needed

* Remove redundant launch files

* scan to point cloud

* Change point cloud topic in costmap

* added point cloud publisher to launch file

* added effort controller for rocker joints and fixed the having the click the button to start controllers

* 9 hours on this bro finally works

* swivel dampening and frcition to avoid tweaking

* Restoring realsense camera p launch files for aruco tag detectioion

* Fix point cloud processing and cost map subscriptions

* ekf exists in sim kinda buns

* push something

* thank goodness for EKF

* Delete rover_pose_bridge

* codex is cooking rn

* global ekf almost

* bro i think this is it fr

* added some covariances to /odom and also enabled altitute and make it smoother

* working ekf: currently 2d with potential for 3d, ground_truth odom for comparison, robot also now spawns in the middle of the world

---------

Signed-off-by: Hiptostee <99766909+Hiptostee@users.noreply.github.com>
Co-authored-by: shayaf84 <shayafmd@gmail.com>

File: urc_hw_description/urdf/simplified_swerve/simplified_swerve_macro.xacro (robot description, xacro)
@@ -15,4 +15,6 @@
   <xacro:property name="wheel_origin_xyz_left" value="0 0.0381 0" />
   <xacro:property name="wheel_origin_xyz_right" value="0 -0.0381 0" />
+  <xacro:property name="swivel_damping_factor" value = "0.8" />
+  <xacro:property name="mu" value="0.8" />
     <link
       name="base_link">
@@ -110,5 +112,5 @@
         lower="-0.523"
         upper="0.523"
-        effort="10"
+        effort="1000"
         velocity="100" />
     </joint>
@@ -170,4 +172,5 @@
         effort="10"
         velocity="100" />
+      <dynamics damping="${swivel_damping_factor}" friction="${mu}"/>
     </joint>
     <link
@@ -279,4 +282,5 @@
         effort="10"
         velocity="100" />
+      <dynamics damping="${swivel_damping_factor}" friction="${mu}"/>
     </joint>
     <link
@@ -386,5 +390,5 @@
         lower="-0.523"
         upper="0.523"
-        effort="10"
+        effort="1000"
         velocity="100" />
     </joint>
@@ -446,4 +450,5 @@
         effort="10"
         velocity="100" />
+      <dynamics damping="${swivel_damping_factor}" friction="${mu}"/>
     </joint>
     <link
@@ -555,4 +560,5 @@
         effort="10"
         velocity="100" />
+      <dynamics damping="${swivel_damping_factor}" friction="${mu}"/>
     </joint>
     <link
@@ -607,17 +613,4 @@
         xyz="-9.257E-05 1 0" />
     </joint>
-     <gazebo>
-      <plugin name="leo_gz::DifferentialSystem" filename="libleo_gz_differential_plugin.so">
-        <jointA>L_Rocker_Joint</jointA>
-        <jointB>R_Rocker_Joint</jointB>
-        <forceConstant>100.0</forceConstant>
-      </plugin>
-      <!-- Average Rocker Position: keeps base_link level at average of left/right rocker heights -->
-      <plugin name="leo_gz::AverageRockerPosition" filename="libleo_gz_average_rocker_plugin.so">
-        <rocker_left_joint>L_Rocker_Joint</rocker_left_joint>
-        <rocker_right_joint>R_Rocker_Joint</rocker_right_joint>
-        <base_link>base_link</base_link>
-      </plugin>
-    </gazebo>
   </xacro:macro>
 </robot>

File: urc_hw_description/urdf/simplified_swerve/simplified_swerve_sensors.xacro (robot description, xacro)
@@ -125,10 +125,62 @@
       </sensor>
     </gazebo>
-     <gazebo reference="base_link">
+    <!-- GPS Link -->
+    <link name="gps_link">
+      <inertial>
+        <mass value="0.01"/>
+        <origin xyz="0 0 0" rpy="0 0 0"/>
+        <inertia ixx="0.001" ixy="0" ixz="0" iyy="0.001" iyz="0" izz="0.001"/>
+      </inertial>
+      <!-- Tiny collision/visual just to have a frame in TF -->
+      <collision name="gps_collision">
+        <geometry>
+          <box size="0.001 0.001 0.001"/>
+        </geometry>
+      </collision>
+      <visual name="gps_visual">
+        <origin xyz="0 0 0" rpy="0 0 0"/>
+        <geometry>
+          <box size="0.001 0.001 0.001"/>
+        </geometry>
+      </visual>
+    </link>
+    <!-- Joint to attach GPS to base -->
+    <joint name="gps_joint" type="fixed">
+      <parent link="base_link"/>
+      <child link="gps_link"/>
+      <!-- Slightly above base so it's easy to visualize -->
+      <origin xyz="0 0 0.2" rpy="0 0 0"/>
+    </joint>
+     <gazebo reference="gps_link">
         <sensor name="gps" type="navsat">
             <always_on>1</always_on>
-            <update_rate>1</update_rate>
+            <update_rate>2</update_rate>
             <visualize>true</visualize>
             <topic>gps</topic>
+            <!-- Ensure downstream messages can use this frame name -->
+            <gz_frame_id>gps_link</gz_frame_id>
+            <navsat>
+                <latitude>
+                    <noise>
+                        <type>gaussian</type>
+                        <mean>0.0</mean>
+                        <stddev>0.15</stddev>
+                    </noise>
+                </latitude>
+                <longitude>
+                    <noise>
+                        <type>gaussian</type>
+                        <mean>0.0</mean>
+                        <stddev>0.15</stddev>
+                    </noise>
+                </longitude>
+                <altitude>
+                    <noise>
+                        <type>gaussian</type>
+                        <mean>0.0</mean>
+                        <stddev>0.15</stddev>
+                    </noise>
+                </altitude>
+            </navsat>
         </sensor>
     </gazebo>
