Commit message: robot appears now

File: urc_hw_description/urdf/simplified_swerve/simplified_swerve_sensors.xacro (robot description, xacro)
@@ -29,5 +29,5 @@
     <!-- Joint to attach lidar to base -->
     <joint name="lidar_joint" type="fixed">
-      <parent link="base_Link"/>
+      <parent link="base_link"/>
       <child link="lidar_link"/>
       <origin xyz="0 0 0.025" rpy="0 0 0"/>
@@ -85,4 +85,5 @@
       </collision>
       <visual name="imu_visual">
+        <origin xyz="0 0 0" rpy="0 0 0"/>
         <geometry>
           <box>
@@ -93,5 +94,5 @@
     </link>
     <joint name="imu_joint" type="fixed">
-      <parent link="base_Link"/>
+      <parent link="base_link"/>
       <child link="imu_link"/>
       <origin xyz="0.1 0 0" rpy="0 0 0"/>
@@ -128,5 +129,5 @@
       </sensor>
     </gazebo>
-     <gazebo reference="base_Link">
+     <gazebo reference="base_link">
         <sensor name="gps" type="navsat">
             <always_on>1</always_on>

Commit message: thank goodness for EKF

File: urc_hw_description/urdf/simplified_swerve/simplified_swerve_sensors.xacro (robot description, xacro)
@@ -125,5 +125,32 @@
       </sensor>
     </gazebo>
-     <gazebo reference="base_link">
+    <!-- GPS Link -->
+    <link name="gps_link">
+      <inertial>
+        <mass value="0.01"/>
+        <origin xyz="0 0 0" rpy="0 0 0"/>
+        <inertia ixx="0.001" ixy="0" ixz="0" iyy="0.001" iyz="0" izz="0.001"/>
+      </inertial>
+      <!-- Tiny collision/visual just to have a frame in TF -->
+      <collision name="gps_collision">
+        <geometry>
+          <box size="0.001 0.001 0.001"/>
+        </geometry>
+      </collision>
+      <visual name="gps_visual">
+        <origin xyz="0 0 0" rpy="0 0 0"/>
+        <geometry>
+          <box size="0.001 0.001 0.001"/>
+        </geometry>
+      </visual>
+    </link>
+    <!-- Joint to attach GPS to base -->
+    <joint name="gps_joint" type="fixed">
+      <parent link="base_link"/>
+      <child link="gps_link"/>
+      <!-- Slightly above base so it's easy to visualize -->
+      <origin xyz="0 0 0.2" rpy="0 0 0"/>
+    </joint>
+     <gazebo reference="gps_link">
         <sensor name="gps" type="navsat">
             <always_on>1</always_on>
@@ -131,4 +158,29 @@
             <visualize>true</visualize>
             <topic>gps</topic>
+            <!-- Ensure downstream messages can use this frame name -->
+            <gz_frame_id>gps_link</gz_frame_id>
+            <navsat>
+                <latitude>
+                    <noise>
+                        <type>gaussian</type>
+                        <mean>0.0</mean>
+                        <stddev>0.00001</stddev>
+                    </noise>
+                </latitude>
+                <longitude>
+                    <noise>
+                        <type>gaussian</type>
+                        <mean>0.0</mean>
+                        <stddev>0.00001</stddev>
+                    </noise>
+                </longitude>
+                <altitude>
+                    <noise>
+                        <type>gaussian</type>
+                        <mean>0.0</mean>
+                        <stddev>0.1</stddev>
+                    </noise>
+                </altitude>
+            </navsat>
         </sensor>
     </gazebo>

Commit message: added camera - does not detect aruco tags yet and the tags currently fall down in simulation

File: urc_hw_description/urdf/simplified_swerve/simplified_swerve_sensors.xacro (robot description, xacro)
@@ -185,3 +185,51 @@
         </sensor>
     </gazebo>
+    <!-- Camera Link -->
+    <link name="camera_link">
+      <inertial>
+        <mass value="0.01"/>
+        <origin xyz="0 0 0" rpy="0 0 0"/>
+        <inertia ixx="0.001" ixy="0" ixz="0" iyy="0.001" iyz="0" izz="0.001"/>
+      </inertial>
+      <!-- Tiny collision/visual just to have a frame in TF -->
+      <collision name="camera_collision">
+        <geometry>
+          <box size="0.05 0.05 0.05"/>
+        </geometry>
+      </collision>
+      <visual name="camera_visual">
+        <origin xyz="0 0 0" rpy="0 0 0"/>
+        <geometry>
+          <box size="0.05 0.05 0.05"/>
+        </geometry>
+      </visual>
+    </link>
+    <!-- Joint to attach camera to base -->
+    <joint name="camera_joint" type="fixed">
+      <parent link="base_link"/>
+      <child link="camera_link"/>
+      <!-- Slightly above base so it's easy to visualize -->
+    <origin xyz="0.2 0 0" rpy="0 0 0"/>
+    </joint>
+    <gazebo reference="camera_link">
+      <sensor name="camera" type="camera">
+        <always_on>1</always_on>
+        <update_rate>30</update_rate>
+        <visualize>true</visualize>
+        <topic>camera/image_raw</topic>
+        <gz_frame_id>camera_link</gz_frame_id>
+        <camera>
+          <horizontal_fov>1.047</horizontal_fov>
+          <image>
+            <width>640</width> <!-- 640 -->
+            <height>480</height> <!-- 480 -->
+            <format>R8G8B8</format>
+          </image>
+          <clip>
+            <near>0.1</near>
+            <far>100</far>
+          </clip>
+        </camera>
+      </sensor>
+    </gazebo>
 </robot>
