Commit message: camera position changed (needs to be changed back later)

File: urc_hw_description/urdf/simplified_swerve/simplified_swerve_sensors.xacro (robot description, xacro)
@@ -189,5 +189,5 @@
       <inertial>
         <mass value="0.01"/>
-        <origin xyz="0 0 0" rpy="0 0 0"/>
+        <origin xyz="0 0 0.4" rpy="0 0 0"/>
         <inertia ixx="0.001" ixy="0" ixz="0" iyy="0.001" iyz="0" izz="0.001"/>
       </inertial>
@@ -199,5 +199,5 @@
       </collision>
       <visual name="camera_visual">
-        <origin xyz="0 0 0" rpy="0 0 0"/>
+        <origin xyz="0 0 0.4" rpy="0 0 0"/>
         <geometry>
           <box size="0.05 0.05 0.05"/>
@@ -210,10 +210,10 @@
       <child link="camera_link"/>
       <!-- Slightly above base so it's easy to visualize -->
-    <origin xyz="0.2 0 0" rpy="0 0 0"/>
+    <origin xyz="0 0 0.4" rpy="0 0 0"/>
     </joint>
     <gazebo reference="camera_link">
       <sensor name="camera" type="camera">
         <!-- Face the camera toward negative X, where the test marker is spawned. -->
-        <pose>0 0 0 0 0 3.14159265359</pose>
+        <pose>1 0 0 0 0 0</pose>
         <always_on>1</always_on>
         <update_rate>30</update_rate>

Commit message: pose information

File: urc_hw_description/urdf/simplified_swerve/simplified_swerve_sensors.xacro (robot description, xacro)
@@ -4,8 +4,4 @@
  <plugin filename="libignition-gazebo-imu-system"
             name="ignition::gazebo::systems::Imu"/>
-<plugin filename="ignition-gazebo-sensors-system"
-            name="ignition::gazebo::systems::Sensors">
-      <render_engine>ogre2</render_engine>
-    </plugin>
      <plugin filename="ignition-gazebo-navsat-system" name="ignition::gazebo::systems::NavSat"/>
 </gazebo>
@@ -189,5 +185,5 @@
       <inertial>
         <mass value="0.01"/>
-        <origin xyz="0 0 0.4" rpy="0 0 0"/>
+        <origin xyz="0 0 0.3" rpy="0 0 0"/>
         <inertia ixx="0.001" ixy="0" ixz="0" iyy="0.001" iyz="0" izz="0.001"/>
       </inertial>
@@ -199,5 +195,5 @@
       </collision>
       <visual name="camera_visual">
-        <origin xyz="0 0 0.4" rpy="0 0 0"/>
+        <origin xyz="0 0 0.3" rpy="0 0 0"/>
         <geometry>
           <box size="0.05 0.05 0.05"/>
@@ -210,5 +206,5 @@
       <child link="camera_link"/>
       <!-- Slightly above base so it's easy to visualize -->
-    <origin xyz="0 0 0.4" rpy="0 0 0"/>
+    <origin xyz="0 0 0.3" rpy="0 0 0"/>
     </joint>
     <gazebo reference="camera_link">

Commit message: show distance from rover to aruco in /aruco/poses topic

File: urc_hw_description/urdf/simplified_swerve/simplified_swerve_sensors.xacro (robot description, xacro)
@@ -208,4 +208,10 @@
     <origin xyz="0 0 0.3" rpy="0 0 0"/>
     </joint>
+    <link name="camera_optical_frame"/>
+    <joint name="camera_optical_joint" type="fixed">
+      <parent link="camera_link"/>
+      <child link="camera_optical_frame"/>
+      <origin xyz="0 0 0" rpy="-1.57079632679 0 -1.57079632679"/>
+    </joint>
     <gazebo reference="camera_link">
       <sensor name="camera" type="camera">
@@ -216,5 +222,5 @@
         <visualize>true</visualize>
         <topic>camera/image_raw</topic>
-        <gz_frame_id>camera_link</gz_frame_id>
+        <gz_frame_id>camera_optical_frame</gz_frame_id>
         <camera>
           <horizontal_fov>1.047</horizontal_fov>

Commit message: pose information looks more accurate than earlier, but the z pose information is still off

File: urc_hw_description/urdf/simplified_swerve/simplified_swerve_sensors.xacro (robot description, xacro)
@@ -195,5 +195,5 @@
       </collision>
       <visual name="camera_visual">
-        <origin xyz="0 0 0.3" rpy="0 0 0"/>
+        <origin xyz="0.1 0 0.1" rpy="0 0 0"/>
         <geometry>
           <box size="0.05 0.05 0.05"/>
@@ -206,5 +206,5 @@
       <child link="camera_link"/>
       <!-- Slightly above base so it's easy to visualize -->
-    <origin xyz="0 0 0.3" rpy="0 0 0"/>
+    <origin xyz="0.1 0 0.1" rpy="0 0 0"/>
     </joint>
     <link name="camera_optical_frame"/>
@@ -216,6 +216,5 @@
     <gazebo reference="camera_link">
       <sensor name="camera" type="camera">
-        <!-- Face the camera toward negative X, where the test marker is spawned. -->
-        <pose>1 0 0 0 0 0</pose>
+        <pose>0 0 0 0 0 0</pose>
         <always_on>1</always_on>
         <update_rate>30</update_rate>
