Commit message: Set sim status light to teleop blue
Publish a solid blue status-light command at simulation startup, document the behavior, and adjust the light's URDF position.

File: urc_hw_description/urdf/simplified_swerve/simplified_swerve_status_light.xacro (robot description, xacro)
@@ -30,5 +30,5 @@
       <parent link="base_link" />
       <child link="status_light_link" />
-      <origin xyz="-0.28 0 ${status_light_size_z / 2}" rpy="0 0 0" />
+      <origin xyz="${-0.308 - status_light_size_x / 2} 0 -0.1" rpy="0 0 0" />
     </joint>
     <!-- Keep the light as its own link in Gazebo so its color can be changed by name -->
